File: cores/cps3/sch/memories.kicad_sch (KiCad schematic)
At the start: 2 parts, among them K12 29F016-90PFTN

Commit message: memories_gfx_main
Parts:
- removed K12, K?: 29F016-90PFTN, symbol arcade:29F016-90PFTN
- added SIMM1A? (x2), SIMM1B? (x2), SIMM2A? (x3), SIMM2B? (x3): Conn_01x36_Male, symbol Connector:Conn_01x36_Male
Connections:
- net VCC: now also SIMM1A?.1 (Pin_1), SIMM1A?.1 (Pin_1), SIMM1A?.2 (Pin_2), SIMM1A?.2 (Pin_2), SIMM2A?.1 (Pin_1), SIMM2A?.1 (Pin_1), SIMM2A?.1 (Pin_1), SIMM2A?.2 (Pin_2), SIMM2A?.2 (Pin_2), SIMM2A?.2 (Pin_2)
- net VSS: now also SIMM1A?.11 (Pin_11), SIMM1A?.11 (Pin_11), SIMM1A?.20 (Pin_20), SIMM1A?.20 (Pin_20), SIMM1A?.29 (Pin_29), SIMM1A?.29 (Pin_29), SIMM1B?.13 (Pin_13), SIMM1B?.13 (Pin_13), SIMM1B?.25 (Pin_25), SIMM1B?.25 (Pin_25), SIMM1B?.32 (Pin_32), SIMM1B?.32 (Pin_32), SIMM2A?.11 (Pin_11), SIMM2A?.11 (Pin_11), SIMM2A?.11 (Pin_11), SIMM2A?.20 (Pin_20), SIMM2A?.20 (Pin_20), SIMM2A?.20 (Pin_20), SIMM2A?.29 (Pin_29), SIMM2A?.29 (Pin_29), SIMM2A?.29 (Pin_29), SIMM2B?.13 (Pin_13), SIMM2B?.13 (Pin_13), SIMM2B?.13 (Pin_13), SIMM2B?.25 (Pin_25), SIMM2B?.25 (Pin_25), SIMM2B?.25 (Pin_25), SIMM2B?.27 (Pin_27), SIMM2B?.27 (Pin_27), SIMM2B?.27 (Pin_27), SIMM2B?.32 (Pin_32), SIMM2B?.32 (Pin_32), SIMM2B?.32 (Pin_32)
- new net GFXA_D0: SIMM1A?.10 (Pin_10), SIMM1A?.10 (Pin_10), SIMM2A?.10 (Pin_10), SIMM2A?.10 (Pin_10), SIMM2A?.10 (Pin_10)
- new net GFXA_D1: SIMM1A?.9 (Pin_9), SIMM1A?.9 (Pin_9), SIMM2A?.9 (Pin_9), SIMM2A?.9 (Pin_9), SIMM2A?.9 (Pin_9)
- new net GFXA_D2: SIMM1A?.8 (Pin_8), SIMM1A?.8 (Pin_8), SIMM2A?.8 (Pin_8), SIMM2A?.8 (Pin_8), SIMM2A?.8 (Pin_8)
- new net GFXA_D3: SIMM1A?.7 (Pin_7), SIMM1A?.7 (Pin_7), SIMM2A?.7 (Pin_7), SIMM2A?.7 (Pin_7), SIMM2A?.7 (Pin_7)
- new net GFXA_D4: SIMM1A?.6 (Pin_6), SIMM1A?.6 (Pin_6), SIMM2A?.6 (Pin_6), SIMM2A?.6 (Pin_6), SIMM2A?.6 (Pin_6)
- new net GFXA_D5: SIMM1A?.5 (Pin_5), SIMM1A?.5 (Pin_5), SIMM2A?.5 (Pin_5), SIMM2A?.5 (Pin_5), SIMM2A?.5 (Pin_5)
- new net GFXA_D6: SIMM1A?.4 (Pin_4), SIMM1A?.4 (Pin_4), SIMM2A?.4 (Pin_4), SIMM2A?.4 (Pin_4), SIMM2A?.4 (Pin_4)
- new net GFXA_D7: SIMM1A?.3 (Pin_3), SIMM1A?.3 (Pin_3), SIMM2A?.3 (Pin_3), SIMM2A?.3 (Pin_3), SIMM2A?.3 (Pin_3)
- new net ~{CE}: SIMM1B?.31 (Pin_31), SIMM1B?.31 (Pin_31), SIMM2B?.31 (Pin_31), SIMM2B?.31 (Pin_31), SIMM2B?.31 (Pin_31)
- new net ~{OE}: SIMM1B?.35 (Pin_35), SIMM1B?.35 (Pin_35), SIMM2B?.35 (Pin_35), SIMM2B?.35 (Pin_35), SIMM2B?.35 (Pin_35)
- new net ~{RESET}: SIMM1B?.26 (Pin_26), SIMM1B?.26 (Pin_26), SIMM2B?.26 (Pin_26), SIMM2B?.26 (Pin_26), SIMM2B?.26 (Pin_26)
- new net ~{WE}: SIMM1B?.34 (Pin_34), SIMM1B?.34 (Pin_34), SIMM2B?.34 (Pin_34), SIMM2B?.34 (Pin_34), SIMM2B?.34 (Pin_34)
Other:
- added sheet memories_gfx (memories_gfx.kicad_sch)
- added sheet memories_main (memories_main.kicad_sch)
- note added: "37"
- note added: "38"
- note added: "39 40"
- note added: "41 42"
- note added: "43 44"
- note added: "45 46"
- note added: "47 48"
- note added: "49 50"
- note added: "51 52"
- note added: "53 54"
- note added: "55 56"
- note added: "57 58"
- note added: "59 60"
- note added: "61 62"
- note added: "63 64"
- note added: "65 66"
- note added: "67 68"
- note added: "69 70"
- note added: "71 72"
- note added: "REVISAR"
- note added: "[37..72]"

Commit message: memories
Parts:
- removed SIMM1A?, SIMM1B? (x2), SIMM2B? (x2): Conn_01x36_Male, symbol Connector:Conn_01x36_Male
- added SIMM1A, SIMM1B, SIMM2A, SIMM2B, SIMM6B? (x3): Conn_01x36_Male, symbol Connector:Conn_01x36_Male
- gave numbers to parts that had none: 5
Connections:
- net GFXA_D0: now also SIMM1A.10 (Pin_10), SIMM2A.10 (Pin_10); no longer SIMM3A.10 (Pin_10), SIMM4A.10 (Pin_10), SIMM5A.10 (Pin_10), SIMM6A.10 (Pin_10)
- net GFXA_D1: now also SIMM1A.9 (Pin_9), SIMM2A.9 (Pin_9); no longer SIMM3A.9 (Pin_9), SIMM4A.9 (Pin_9), SIMM5A.9 (Pin_9), SIMM6A.9 (Pin_9)
- net GFXA_D2: now also SIMM1A.8 (Pin_8), SIMM2A.8 (Pin_8); no longer SIMM3A.8 (Pin_8), SIMM4A.8 (Pin_8), SIMM5A.8 (Pin_8), SIMM6A.8 (Pin_8)
- net GFXA_D3: now also SIMM1A.7 (Pin_7), SIMM2A.7 (Pin_7); no longer SIMM3A.7 (Pin_7), SIMM4A.7 (Pin_7), SIMM5A.7 (Pin_7), SIMM6A.7 (Pin_7)
- net GFXA_D4: now also SIMM1A.6 (Pin_6), SIMM2A.6 (Pin_6); no longer SIMM3A.6 (Pin_6), SIMM4A.6 (Pin_6), SIMM5A.6 (Pin_6), SIMM6A.6 (Pin_6)
- net GFXA_D5: now also SIMM1A.5 (Pin_5), SIMM2A.5 (Pin_5); no longer SIMM3A.5 (Pin_5), SIMM4A.5 (Pin_5), SIMM5A.5 (Pin_5), SIMM6A.5 (Pin_5)
- net GFXA_D6: now also SIMM1A.4 (Pin_4), SIMM2A.4 (Pin_4); no longer SIMM3A.4 (Pin_4), SIMM4A.4 (Pin_4), SIMM5A.4 (Pin_4), SIMM6A.4 (Pin_4)
- net GFXA_D7: now also SIMM1A.3 (Pin_3), SIMM2A.3 (Pin_3); no longer SIMM3A.3 (Pin_3), SIMM4A.3 (Pin_3), SIMM5A.3 (Pin_3), SIMM6A.3 (Pin_3)
- net VCC: now also SIMM1A.1 (Pin_1), SIMM1A.2 (Pin_2), SIMM2A.1 (Pin_1), SIMM2A.2 (Pin_2)
- net VSS: now also SIMM1A.11 (Pin_11), SIMM1A.20 (Pin_20), SIMM1A.29 (Pin_29), SIMM1B.13 (Pin_13), SIMM1B.25 (Pin_25), SIMM1B.32 (Pin_32), SIMM2A.11 (Pin_11), SIMM2A.20 (Pin_20), SIMM2A.29 (Pin_29), SIMM2B.13 (Pin_13), SIMM2B.25 (Pin_25), SIMM2B.27 (Pin_27), SIMM2B.32 (Pin_32), SIMM6B?.25 (Pin_25), SIMM6B?.25 (Pin_25), SIMM6B?.25 (Pin_25), SIMM6B?.27 (Pin_27), SIMM6B?.27 (Pin_27), SIMM6B?.27 (Pin_27), SIMM6B?.32 (Pin_32), SIMM6B?.32 (Pin_32), SIMM6B?.32 (Pin_32); no longer SIMM6B.13 (Pin_13)
- net ~{CE}: now also SIMM1B.31 (Pin_31), SIMM2B.31 (Pin_31), SIMM6B?.31 (Pin_31), SIMM6B?.31 (Pin_31), SIMM6B?.31 (Pin_31)
- net ~{OE}: now also SIMM1B.35 (Pin_35), SIMM2B.35 (Pin_35), SIMM6B?.35 (Pin_35), SIMM6B?.35 (Pin_35), SIMM6B?.35 (Pin_35)
- net ~{WE}: now also SIMM1B.34 (Pin_34), SIMM2B.34 (Pin_34), SIMM6B?.34 (Pin_34), SIMM6B?.34 (Pin_34), SIMM6B?.34 (Pin_34)
- net R_MAINA13: now reaches SIMM6B.10 (Pin_10)
- net R_MAINA13: now also SIMM6B?.10 (Pin_10), SIMM6B?.10 (Pin_10), SIMM6B?.10 (Pin_10)
- net R_MAINA12: now reaches SIMM6B.11 (Pin_11)
- net R_MAINA12: now also SIMM6B?.11 (Pin_11), SIMM6B?.11 (Pin_11), SIMM6B?.11 (Pin_11)
- net R_MAINA11: now reaches SIMM6B.12 (Pin_12)
- net R_MAINA11: now also SIMM6B?.12 (Pin_12), SIMM6B?.12 (Pin_12), SIMM6B?.12 (Pin_12)
- net R_MAINA10: now reaches SIMM6B.14 (Pin_14)
- net R_MAINA10: now also SIMM6B?.14 (Pin_14), SIMM6B?.14 (Pin_14), SIMM6B?.14 (Pin_14)
- net R_MAINA9: now reaches SIMM6B.15 (Pin_15)
- net R_MAINA9: now also SIMM6B?.15 (Pin_15), SIMM6B?.15 (Pin_15), SIMM6B?.15 (Pin_15)
- net R_MAINA8: now reaches SIMM6B.16 (Pin_16)
- net R_MAINA8: now also SIMM6B?.16 (Pin_16), SIMM6B?.16 (Pin_16), SIMM6B?.16 (Pin_16)
- net R_MAINA7: now reaches SIMM6B.17 (Pin_17)
- net R_MAINA7: now also SIMM6B?.17 (Pin_17), SIMM6B?.17 (Pin_17), SIMM6B?.17 (Pin_17)
- net R_MAINA6: now reaches SIMM6B.18 (Pin_18)
- net R_MAINA6: now also SIMM6B?.18 (Pin_18), SIMM6B?.18 (Pin_18), SIMM6B?.18 (Pin_18)
- net R_MAINA5: now reaches SIMM6B.19 (Pin_19)
- net R_MAINA5: now also SIMM6B?.19 (Pin_19), SIMM6B?.19 (Pin_19), SIMM6B?.19 (Pin_19)
- net R_MAINA4: now reaches SIMM6B.20 (Pin_20)
- net R_MAINA4: now also SIMM6B?.20 (Pin_20), SIMM6B?.20 (Pin_20), SIMM6B?.20 (Pin_20)
- net R_MAINA3: now reaches SIMM6B.21 (Pin_21)
- net R_MAINA3: now also SIMM6B?.21 (Pin_21), SIMM6B?.21 (Pin_21), SIMM6B?.21 (Pin_21)
- net R_MAINA2: now reaches SIMM6B.22 (Pin_22)
- net R_MAINA2: now also SIMM6B?.22 (Pin_22), SIMM6B?.22 (Pin_22), SIMM6B?.22 (Pin_22)
- net R_MAINA1: now reaches SIMM6B.23 (Pin_23)
- net R_MAINA1: now also SIMM6B?.23 (Pin_23), SIMM6B?.23 (Pin_23), SIMM6B?.23 (Pin_23)
- net R_MAINA0: now reaches SIMM6B.24 (Pin_24)
- net R_MAINA0: now also SIMM6B?.24 (Pin_24), SIMM6B?.24 (Pin_24), SIMM6B?.24 (Pin_24)
- net R_MAINA20: now reaches SIMM6B.3 (Pin_3)
- net R_MAINA20: now also SIMM6B?.3 (Pin_3), SIMM6B?.3 (Pin_3), SIMM6B?.3 (Pin_3)
- net R_MAINA19: now reaches SIMM6B.4 (Pin_4)
- net R_MAINA19: now also SIMM6B?.4 (Pin_4), SIMM6B?.4 (Pin_4), SIMM6B?.4 (Pin_4)
- net R_MAINA18: now reaches SIMM6B.5 (Pin_5)
- net R_MAINA18: now also SIMM6B?.5 (Pin_5), SIMM6B?.5 (Pin_5), SIMM6B?.5 (Pin_5)
- net R_MAINA17: now reaches SIMM6B.6 (Pin_6)
- net R_MAINA17: now also SIMM6B?.6 (Pin_6), SIMM6B?.6 (Pin_6), SIMM6B?.6 (Pin_6)
- net R_MAINA16: now reaches SIMM6B.7 (Pin_7)
- net R_MAINA16: now also SIMM6B?.7 (Pin_7), SIMM6B?.7 (Pin_7), SIMM6B?.7 (Pin_7)
- net R_MAINA15: now reaches SIMM6B.8 (Pin_8)
- net R_MAINA15: now also SIMM6B?.8 (Pin_8), SIMM6B?.8 (Pin_8), SIMM6B?.8 (Pin_8)
- net R_MAINA14: now reaches SIMM6B.9 (Pin_9)
- net R_MAINA14: now also SIMM6B?.9 (Pin_9), SIMM6B?.9 (Pin_9), SIMM6B?.9 (Pin_9)
- net ~{RESET} renamed ~{RESET2}
- net ~{RESET2}: now also SIMM6B?.26 (Pin_26), SIMM6B?.26 (Pin_26), SIMM6B?.26 (Pin_26)
- new net GFXB_D0: SIMM1A.19 (Pin_19), SIMM2A.19 (Pin_19)
- new net GFXB_D1: SIMM1A.18 (Pin_18), SIMM2A.18 (Pin_18)
- new net GFXB_D2: SIMM1A.17 (Pin_17), SIMM2A.17 (Pin_17)
- new net GFXB_D3: SIMM1A.16 (Pin_16), SIMM2A.16 (Pin_16)
- new net GFXB_D4: SIMM1A.15 (Pin_15), SIMM2A.15 (Pin_15)
- new net GFXB_D5: SIMM1A.14 (Pin_14), SIMM2A.14 (Pin_14)
- new net GFXB_D6: SIMM1A.13 (Pin_13), SIMM2A.13 (Pin_13)
- new net GFXB_D7: SIMM1A.12 (Pin_12), SIMM2A.12 (Pin_12)
- new net GFXC_D0: SIMM1A.28 (Pin_28), SIMM2A.28 (Pin_28)
- new net GFXC_D1: SIMM1A.27 (Pin_27), SIMM2A.27 (Pin_27)
- new net GFXC_D2: SIMM1A.26 (Pin_26), SIMM2A.26 (Pin_26)
- new net GFXC_D3: SIMM1A.25 (Pin_25), SIMM2A.25 (Pin_25)
- new net GFXC_D4: SIMM1A.24 (Pin_24), SIMM2A.24 (Pin_24)
- new net GFXC_D5: SIMM1A.23 (Pin_23), SIMM2A.23 (Pin_23)
- new net GFXC_D6: SIMM1A.22 (Pin_22), SIMM2A.22 (Pin_22)
- new net GFXC_D7: SIMM1A.21 (Pin_21), SIMM2A.21 (Pin_21)
- new net GFXD_D0: SIMM1B.1 (Pin_1), SIMM2B.1 (Pin_1)
- new net GFXD_D1: SIMM1A.36 (Pin_36), SIMM2A.36 (Pin_36)
- new net GFXD_D2: SIMM1A.35 (Pin_35), SIMM2A.35 (Pin_35)
- new net GFXD_D3: SIMM1A.34 (Pin_34), SIMM2A.34 (Pin_34)
- new net GFXD_D4: SIMM1A.33 (Pin_33), SIMM2A.33 (Pin_33)
- new net GFXD_D5: SIMM1A.32 (Pin_32), SIMM2A.32 (Pin_32)
- new net GFXD_D6: SIMM1A.31 (Pin_31), SIMM2A.31 (Pin_31)
- new net GFXD_D7: SIMM1A.30 (Pin_30), SIMM2A.30 (Pin_30)
- new net GFX_A0: SIMM1B.24 (Pin_24), SIMM2B.24 (Pin_24)
- new net GFX_A1: SIMM1B.23 (Pin_23), SIMM2B.23 (Pin_23)
- new net GFX_A10: SIMM1B.14 (Pin_14), SIMM2B.14 (Pin_14)
- new net GFX_A11: SIMM1B.12 (Pin_12), SIMM2B.12 (Pin_12)
- new net GFX_A12: SIMM1B.11 (Pin_11), SIMM2B.11 (Pin_11)
- new net GFX_A13: SIMM1B.10 (Pin_10), SIMM2B.10 (Pin_10)
- new net GFX_A14: SIMM1B.9 (Pin_9), SIMM2B.9 (Pin_9)
- new net GFX_A15: SIMM1B.8 (Pin_8), SIMM2B.8 (Pin_8)
- new net GFX_A16: SIMM1B.7 (Pin_7), SIMM2B.7 (Pin_7)
- new net GFX_A17: SIMM1B.6 (Pin_6), SIMM2B.6 (Pin_6)
- new net GFX_A18: SIMM1B.5 (Pin_5), SIMM2B.5 (Pin_5)
- new net GFX_A19: SIMM1B.4 (Pin_4), SIMM2B.4 (Pin_4)
- new net GFX_A2: SIMM1B.22 (Pin_22), SIMM2B.22 (Pin_22)
- new net GFX_A20: SIMM1B.3 (Pin_3), SIMM2B.3 (Pin_3)
- new net GFX_A3: SIMM1B.21 (Pin_21), SIMM2B.21 (Pin_21)
- new net GFX_A4: SIMM1B.20 (Pin_20), SIMM2B.20 (Pin_20)
- new net GFX_A5: SIMM1B.19 (Pin_19), SIMM2B.19 (Pin_19)
- new net GFX_A6: SIMM1B.18 (Pin_18), SIMM2B.18 (Pin_18)
- new net GFX_A7: SIMM1B.17 (Pin_17), SIMM2B.17 (Pin_17)
- new net GFX_A8: SIMM1B.16 (Pin_16), SIMM2B.16 (Pin_16)
- new net GFX_A9: SIMM1B.15 (Pin_15), SIMM2B.15 (Pin_15)
- new net RMAINA_D0: SIMM6A.3 (Pin_3)
- new net RMAINA_D1: SIMM6A.4 (Pin_4)
- new net RMAINA_D2: SIMM6A.5 (Pin_5)
- new net RMAINA_D3: SIMM6A.6 (Pin_6)
- new net RMAINA_D4: SIMM6A.7 (Pin_7)
- new net RMAINA_D5: SIMM6A.8 (Pin_8)
- new net RMAINA_D6: SIMM6A.9 (Pin_9)
- new net RMAINA_D7: SIMM6A.10 (Pin_10)
- new net RMAINB_D0: SIMM3A.3 (Pin_3), SIMM4A.3 (Pin_3), SIMM5A.3 (Pin_3)
- new net RMAINB_D1: SIMM3A.4 (Pin_4), SIMM4A.4 (Pin_4), SIMM5A.4 (Pin_4)
- new net RMAINB_D2: SIMM3A.5 (Pin_5), SIMM4A.5 (Pin_5), SIMM5A.5 (Pin_5)
- new net RMAINB_D3: SIMM3A.6 (Pin_6), SIMM4A.6 (Pin_6), SIMM5A.6 (Pin_6)
- new net RMAINB_D4: SIMM3A.7 (Pin_7), SIMM4A.7 (Pin_7), SIMM5A.7 (Pin_7)
- new net RMAINB_D5: SIMM3A.8 (Pin_8), SIMM4A.8 (Pin_8), SIMM5A.8 (Pin_8)
- new net RMAINB_D6: SIMM3A.9 (Pin_9), SIMM4A.9 (Pin_9), SIMM5A.9 (Pin_9)
- new net RMAINB_D7: SIMM3A.10 (Pin_10), SIMM4A.10 (Pin_10), SIMM5A.10 (Pin_10)
- new net UK: SIMM1B.33 (Pin_33), SIMM2B.33 (Pin_33)
- new net ~{RESET5}: SIMM1B.26 (Pin_26), SIMM2B.26 (Pin_26)
- no-connect marks 0 -> 11
Other:
- sheet memories_gfx ports: added GFXA_D[7..0], GFXB_D[7..0], GFXC_D[7..0], GFXD_D[7..0], GFX_A[20..0], UK, ~{CE}, ~{OE}, ~{RESET5}, ~{WE}; removed none
- sheet memories_main ports: added RMAINA_D[7..0], RMAINB_D[7..0], R_MAINA[20..0], R_MAINB[20..0], ~{CEA}, ~{CEB}, ~{CEC}, ~{CED}, ~{CEE}, ~{CEF}, ~{CEG}, ~{CEH}, ~{CEI}, ~{CEJ}, ~{CEK}, ~{CEL}, ~{CEM}, ~{CEN}, ~{CEO}, ~{CEP}, ~{OEB}, ~{OEC}, ~{OED}, ~{OEE}, ~{RESET1}, ~{RESET2}, ~{RESET3}, ~{RESET4}, ~{WEB}, ~{WEC}, ~{WED}, ~{WEE}; removed none
- note added: "REVISAR POSIBLE CORTO ENTRE VCC Y VSS"
- moved on the sheet: SIMM3A, SIMM4A, SIMM5A, SIMM6A, SIMM6B

Commit message: memories4
Parts:
- removed SIMM3A, SIMM4A: Conn_01x36_Male, symbol Connector:Conn_01x36_Male
- added SIMM3E, SIMM4D: Conn_01x36_Male, symbol Connector:Conn_01x36_Male
- gave numbers to parts that had none: 3
- renumbered SIMM1B to SIMM1E, SIMM1A to SIMM1E, SIMM2A to SIMM2D, SIMM2B to SIMM2D, SIMM5A to SIMM5C, SIMM6A to SIMM6B, SIMM6B to SIMM6BB
Connections:
- net RMAINA_D0: now also SIMM6B.18 (Pin_18); no longer SIMM6B.3 (Pin_3)
- net RMAINA_D1: now also SIMM6B.16 (Pin_16); no longer SIMM6B.4 (Pin_4)
- net RMAINA_D2: now also SIMM6B.14 (Pin_14); no longer SIMM6B.5 (Pin_5)
- net RMAINA_D3: now also SIMM6B.12 (Pin_12); no longer SIMM6B.6 (Pin_6)
- net RMAINA_D4: now also SIMM6B.9 (Pin_9); no longer SIMM6B.7 (Pin_7)
- net RMAINA_D5: now also SIMM6B.7 (Pin_7); no longer SIMM6B.8 (Pin_8)
- net RMAINA_D6: now also SIMM6B.5 (Pin_5); no longer SIMM6B.9 (Pin_9)
- net RMAINA_D7: now also SIMM6B.3 (Pin_3); no longer SIMM6B.10 (Pin_10)
- net RMAINB_D0: now also SIMM5C.18 (Pin_18), SIMM3E.18 (Pin_18), SIMM4D.18 (Pin_18); no longer SIMM5C.3 (Pin_3)
- net RMAINB_D1: now also SIMM5C.16 (Pin_16), SIMM3E.16 (Pin_16), SIMM4D.16 (Pin_16); no longer SIMM5C.4 (Pin_4)
- net RMAINB_D2: now also SIMM5C.14 (Pin_14), SIMM3E.14 (Pin_14), SIMM4D.14 (Pin_14); no longer SIMM5C.5 (Pin_5)
- net RMAINB_D3: now also SIMM5C.12 (Pin_12), SIMM3E.12 (Pin_12), SIMM4D.12 (Pin_12); no longer SIMM5C.6 (Pin_6)
- net RMAINB_D4: now also SIMM5C.9 (Pin_9), SIMM3E.9 (Pin_9), SIMM4D.9 (Pin_9); no longer SIMM5C.7 (Pin_7)
- net RMAINB_D5: now also SIMM5C.7 (Pin_7), SIMM3E.7 (Pin_7), SIMM4D.7 (Pin_7); no longer SIMM5C.8 (Pin_8)
- net RMAINB_D6: now also SIMM5C.5 (Pin_5), SIMM3E.5 (Pin_5), SIMM4D.5 (Pin_5); no longer SIMM5C.9 (Pin_9)
- net RMAINB_D7: now also SIMM5C.3 (Pin_3), SIMM3E.3 (Pin_3), SIMM4D.3 (Pin_3); no longer SIMM5C.10 (Pin_10)
- net R_MAINA0: no longer SIMM3EE.24 (Pin_24), SIMM4DD.24 (Pin_24), SIMM5CC.24 (Pin_24)
- net R_MAINA1: no longer SIMM3EE.23 (Pin_23), SIMM4DD.23 (Pin_23), SIMM5CC.23 (Pin_23)
- net R_MAINA10: no longer SIMM3EE.14 (Pin_14), SIMM4DD.14 (Pin_14), SIMM5CC.14 (Pin_14)
- net R_MAINA11: no longer SIMM3EE.12 (Pin_12), SIMM4DD.12 (Pin_12), SIMM5CC.12 (Pin_12)
- net R_MAINA12: no longer SIMM3EE.11 (Pin_11), SIMM4DD.11 (Pin_11), SIMM5CC.11 (Pin_11)
- net R_MAINA13: no longer SIMM3EE.10 (Pin_10), SIMM4DD.10 (Pin_10), SIMM5CC.10 (Pin_10)
- net R_MAINA14: no longer SIMM3EE.9 (Pin_9), SIMM4DD.9 (Pin_9), SIMM5CC.9 (Pin_9)
- net R_MAINA15: no longer SIMM3EE.8 (Pin_8), SIMM4DD.8 (Pin_8), SIMM5CC.8 (Pin_8)
- net R_MAINA16: no longer SIMM3EE.7 (Pin_7), SIMM4DD.7 (Pin_7), SIMM5CC.7 (Pin_7)
- net R_MAINA17: no longer SIMM3EE.6 (Pin_6), SIMM4DD.6 (Pin_6), SIMM5CC.6 (Pin_6)
- net R_MAINA18: no longer SIMM3EE.5 (Pin_5), SIMM4DD.5 (Pin_5), SIMM5CC.5 (Pin_5)
- net R_MAINA19: no longer SIMM3EE.4 (Pin_4), SIMM4DD.4 (Pin_4), SIMM5CC.4 (Pin_4)
- net R_MAINA2: no longer SIMM3EE.22 (Pin_22), SIMM4DD.22 (Pin_22), SIMM5CC.22 (Pin_22)
- net R_MAINA20: no longer SIMM3EE.3 (Pin_3), SIMM4DD.3 (Pin_3), SIMM5CC.3 (Pin_3)
- net R_MAINA3: no longer SIMM3EE.21 (Pin_21), SIMM4DD.21 (Pin_21), SIMM5CC.21 (Pin_21)
- net R_MAINA4: no longer SIMM3EE.20 (Pin_20), SIMM4DD.20 (Pin_20), SIMM5CC.20 (Pin_20)
- net R_MAINA5: no longer SIMM3EE.19 (Pin_19), SIMM4DD.19 (Pin_19), SIMM5CC.19 (Pin_19)
- net R_MAINA6: no longer SIMM3EE.18 (Pin_18), SIMM4DD.18 (Pin_18), SIMM5CC.18 (Pin_18)
- net R_MAINA7: no longer SIMM3EE.17 (Pin_17), SIMM4DD.17 (Pin_17), SIMM5CC.17 (Pin_17)
- net R_MAINA8: no longer SIMM3EE.16 (Pin_16), SIMM4DD.16 (Pin_16), SIMM5CC.16 (Pin_16)
- net R_MAINA9: no longer SIMM3EE.15 (Pin_15), SIMM4DD.15 (Pin_15), SIMM5CC.15 (Pin_15)
- net VCC: now also SIMM3E.1 (Pin_1), SIMM3E.2 (Pin_2), SIMM4D.1 (Pin_1), SIMM4D.2 (Pin_2)
- net VSS: now also SIMM3EE.13 (Pin_13), SIMM4DD.13 (Pin_13), SIMM5CC.13 (Pin_13), SIMM6BB.13 (Pin_13), SIMM3E.11 (Pin_11), SIMM3E.20 (Pin_20), SIMM3E.29 (Pin_29), SIMM4D.11 (Pin_11), SIMM4D.20 (Pin_20), SIMM4D.29 (Pin_29)
- net ~{CEA}: now also SIMM6BB.28 (Pin_28)
- net ~{CEB}: now also SIMM6BB.29 (Pin_29)
- net ~{CEC}: now also SIMM6BB.30 (Pin_30)
- net ~{CED}: now also SIMM6BB.31 (Pin_31)
- net ~{CEE}: now also SIMM5CC.28 (Pin_28)
- net ~{CEF}: now also SIMM5CC.29 (Pin_29)
- net ~{CEG}: now also SIMM5CC.30 (Pin_30)
- net ~{CEH}: now also SIMM5CC.31 (Pin_31)
- net ~{CEI}: now also SIMM4DD.28 (Pin_28)
- net ~{CEJ}: now also SIMM4DD.29 (Pin_29)
- net ~{CEK}: now also SIMM4DD.30 (Pin_30)
- net ~{CEL}: now also SIMM4DD.31 (Pin_31)
- net ~{CEM}: now also SIMM3EE.28 (Pin_28)
- net ~{CEN}: now also SIMM3EE.29 (Pin_29)
- net ~{CEO}: now also SIMM3EE.30 (Pin_30)
- net ~{CEP}: now also SIMM3EE.31 (Pin_31)
- net ~{CE}: no longer SIMM3EE.31 (Pin_31), SIMM4DD.31 (Pin_31), SIMM5CC.31 (Pin_31), SIMM6BB.31 (Pin_31)
- net ~{OEB}: now also SIMM6BB.35 (Pin_35)
- net ~{OEC}: now also SIMM5CC.35 (Pin_35)
- net ~{OED}: now also SIMM4DD.35 (Pin_35)
- net ~{OEE}: now also SIMM3EE.35 (Pin_35)
- net ~{OE}: no longer SIMM3EE.35 (Pin_35), SIMM4DD.35 (Pin_35), SIMM5CC.35 (Pin_35), SIMM6BB.35 (Pin_35)
- net ~{RESET1}: now also SIMM6BB.26 (Pin_26)
- net ~{RESET2}: no longer SIMM3EE.26 (Pin_26), SIMM4DD.26 (Pin_26), SIMM6BB.26 (Pin_26)
- net ~{RESET3}: now also SIMM4DD.26 (Pin_26)
- net ~{RESET4}: now also SIMM3EE.26 (Pin_26)
- net ~{WEB}: now also SIMM6BB.33 (Pin_33)
- net ~{WEC}: now also SIMM5CC.33 (Pin_33)
- net ~{WED}: now also SIMM4DD.33 (Pin_33)
- net ~{WEE}: now also SIMM3EE.33 (Pin_33)
- net ~{WE}: no longer SIMM3EE.34 (Pin_34), SIMM4DD.34 (Pin_34), SIMM5CC.34 (Pin_34), SIMM6BB.34 (Pin_34)
- net RMAINC_D7: now reaches SIMM6B.21 (Pin_21)
- net RMAINC_D6: now reaches SIMM6B.23 (Pin_23)
- net RMAINC_D5: now reaches SIMM6B.25 (Pin_25)
- net RMAINC_D4: now reaches SIMM6B.27 (Pin_27)
- net RMAINC_D3: now reaches SIMM6B.30 (Pin_30)
- net RMAINC_D2: now reaches SIMM6B.32 (Pin_32)
- net RMAINC_D1: now reaches SIMM6B.34 (Pin_34)
- net RMAINC_D0: now reaches SIMM6B.36 (Pin_36)
- net RMAIND_D7: now reaches SIMM5C.21 (Pin_21)
- net RMAIND_D7: now also SIMM3E.21 (Pin_21), SIMM4D.21 (Pin_21)
- net RMAIND_D6: now reaches SIMM5C.23 (Pin_23)
- net RMAIND_D6: now also SIMM3E.23 (Pin_23), SIMM4D.23 (Pin_23)
- net RMAIND_D5: now reaches SIMM5C.25 (Pin_25)
- net RMAIND_D5: now also SIMM3E.25 (Pin_25), SIMM4D.25 (Pin_25)
- net RMAIND_D4: now reaches SIMM5C.27 (Pin_27)
- net RMAIND_D4: now also SIMM3E.27 (Pin_27), SIMM4D.27 (Pin_27)
- net RMAIND_D3: now reaches SIMM5C.30 (Pin_30)
- net RMAIND_D3: now also SIMM3E.30 (Pin_30), SIMM4D.30 (Pin_30)
- net RMAIND_D2: now reaches SIMM5C.32 (Pin_32)
- net RMAIND_D2: now also SIMM3E.32 (Pin_32), SIMM4D.32 (Pin_32)
- net RMAIND_D1: now reaches SIMM5C.34 (Pin_34)
- net RMAIND_D1: now also SIMM3E.34 (Pin_34), SIMM4D.34 (Pin_34)
- net RMAIND_D0: now reaches SIMM5C.36 (Pin_36)
- net RMAIND_D0: now also SIMM3E.36 (Pin_36), SIMM4D.36 (Pin_36)
- new net R_MAINB0: SIMM3EE.24 (Pin_24), SIMM4DD.24 (Pin_24), SIMM5CC.24 (Pin_24)
- new net R_MAINB1: SIMM3EE.23 (Pin_23), SIMM4DD.23 (Pin_23), SIMM5CC.23 (Pin_23)
- new net R_MAINB10: SIMM3EE.14 (Pin_14), SIMM4DD.14 (Pin_14), SIMM5CC.14 (Pin_14)
- new net R_MAINB11: SIMM3EE.12 (Pin_12), SIMM4DD.12 (Pin_12), SIMM5CC.12 (Pin_12)
- new net R_MAINB12: SIMM3EE.11 (Pin_11), SIMM4DD.11 (Pin_11), SIMM5CC.11 (Pin_11)
- new net R_MAINB13: SIMM3EE.10 (Pin_10), SIMM4DD.10 (Pin_10), SIMM5CC.10 (Pin_10)
- new net R_MAINB14: SIMM3EE.9 (Pin_9), SIMM4DD.9 (Pin_9), SIMM5CC.9 (Pin_9)
- new net R_MAINB15: SIMM3EE.8 (Pin_8), SIMM4DD.8 (Pin_8), SIMM5CC.8 (Pin_8)
- new net R_MAINB16: SIMM3EE.7 (Pin_7), SIMM4DD.7 (Pin_7), SIMM5CC.7 (Pin_7)
- new net R_MAINB17: SIMM3EE.6 (Pin_6), SIMM4DD.6 (Pin_6), SIMM5CC.6 (Pin_6)
- new net R_MAINB18: SIMM3EE.5 (Pin_5), SIMM4DD.5 (Pin_5), SIMM5CC.5 (Pin_5)
- new net R_MAINB19: SIMM3EE.4 (Pin_4), SIMM4DD.4 (Pin_4), SIMM5CC.4 (Pin_4)
- new net R_MAINB2: SIMM3EE.22 (Pin_22), SIMM4DD.22 (Pin_22), SIMM5CC.22 (Pin_22)
- new net R_MAINB20: SIMM3EE.3 (Pin_3), SIMM4DD.3 (Pin_3), SIMM5CC.3 (Pin_3)
- new net R_MAINB3: SIMM3EE.21 (Pin_21), SIMM4DD.21 (Pin_21), SIMM5CC.21 (Pin_21)
- new net R_MAINB4: SIMM3EE.20 (Pin_20), SIMM4DD.20 (Pin_20), SIMM5CC.20 (Pin_20)
- new net R_MAINB5: SIMM3EE.19 (Pin_19), SIMM4DD.19 (Pin_19), SIMM5CC.19 (Pin_19)
- new net R_MAINB6: SIMM3EE.18 (Pin_18), SIMM4DD.18 (Pin_18), SIMM5CC.18 (Pin_18)
- new net R_MAINB7: SIMM3EE.17 (Pin_17), SIMM4DD.17 (Pin_17), SIMM5CC.17 (Pin_17)
- new net R_MAINB8: SIMM3EE.16 (Pin_16), SIMM4DD.16 (Pin_16), SIMM5CC.16 (Pin_16)
- new net R_MAINB9: SIMM3EE.15 (Pin_15), SIMM4DD.15 (Pin_15), SIMM5CC.15 (Pin_15)
- no-connect marks 11 -> 81
Other:
- sheet memories_main ports: added RMAINC_D[7..0], RMAIND_D[7..0]; removed none
- note removed: "REVISAR"
- moved on the sheet: SIMM5C, SIMM6B
