File: cores/cps3/sch/memories.kicad_sch (KiCad schematic)
At the start: 12 parts

Commit message: ppu
Other:
- note added: "MEMORIES DE GFX?"
- note added: "MEMORIES DE MAIN?"
Changed lines of the file:
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@@
     (effects (font (size 1.27 1.27)) (justify right bottom))
+  )
+  (text "MEMORIES DE MAIN?" (at 61.595 38.1 0)
+    (effects (font (size 3 3)) (justify left bottom))
   )
   (text "61\n62" (at 314.96 203.2 0)
@@
     (effects (font (size 1.27 1.27)) (justify left bottom))
   )
+  (text "MEMORIES DE GFX?" (at 59.055 69.215 0)
+    (effects (font (size 3 3)) (justify left bottom))
+  )
   (text "59\n60" (at 236.22 196.85 0)

Commit message: ppu_ research
Connections:
- net RMAINA_D0 renamed SPRITEA_D0
- net RMAINA_D1 renamed SPRITEA_D1
- net RMAINA_D2 renamed SPRITEA_D2
- net RMAINA_D3 renamed SPRITEA_D3
- net RMAINA_D4 renamed SPRITEA_D4
- net RMAINA_D5 renamed SPRITEA_D5
- net RMAINA_D6 renamed SPRITEA_D6
- net RMAINA_D7 renamed SPRITEA_D7
- net RMAINB_D0 renamed SPRITEB_D0
- net RMAINB_D1 renamed SPRITEB_D1
- net RMAINB_D2 renamed SPRITEB_D2
- net RMAINB_D3 renamed SPRITEB_D3
- net RMAINB_D4 renamed SPRITEB_D4
- net RMAINB_D5 renamed SPRITEB_D5
- net RMAINB_D6 renamed SPRITEB_D6
- net RMAINB_D7 renamed SPRITEB_D7
- net RMAINC_D0 renamed SPRITEC_D0
- net RMAINC_D1 renamed SPRITEC_D1
- net RMAINC_D2 renamed SPRITEC_D2
- net RMAINC_D3 renamed SPRITEC_D3
- net RMAINC_D4 renamed SPRITEC_D4
- net RMAINC_D5 renamed SPRITEC_D5
- net RMAINC_D6 renamed SPRITEC_D6
- net RMAINC_D7 renamed SPRITEC_D7
- net RMAIND_D0 renamed SPRITED_D0
- net RMAIND_D1 renamed SPRITED_D1
- net RMAIND_D2 renamed SPRITED_D2
- net RMAIND_D3 renamed SPRITED_D3
- net RMAIND_D4 renamed SPRITED_D4
- net RMAIND_D5 renamed SPRITED_D5
- net RMAIND_D6 renamed SPRITED_D6
- net RMAIND_D7 renamed SPRITED_D7
Other:
- sheet memories_gfx ports: added R_MAINA[20..0], R_MAINB[20..0], SPRITEA_D[7..0], SPRITEB_D[7..0], SPRITEC_D[7..0], SPRITED_D[7..0], ~{CEA}, ~{CEB}, ~{CEC}, ~{CED}, ~{CEE}, ~{CEF}, ~{CEG}, ~{CEH}, ~{CEI}, ~{CEJ}, ~{CEK}, ~{CEL}, ~{CEM}, ~{CEN}, ~{CEO}, ~{CEP}, ~{OEB}, ~{OEC}, ~{OED}, ~{OEE}, ~{RESET1}, ~{RESET2}, ~{RESET3}, ~{RESET4}, ~{WEB}, ~{WEC}, ~{WED}, ~{WEE}; removed GFXA_D[7..0], GFXB_D[7..0], GFXC_D[7..0], GFXD_D[7..0], GFX_A[20..0], UK, ~{CE}, ~{OE}, ~{RESET5}, ~{WE}
- sheet memories_main ports: added GFXA_D[7..0], GFXB_D[7..0], GFXC_D[7..0], GFXD_D[7..0], GFX_A[20..0], UK, ~{CE}, ~{OE}, ~{RESET5}, ~{WE}; removed RMAINA_D[7..0], RMAINB_D[7..0], RMAINC_D[7..0], RMAIND_D[7..0], R_MAINA[20..0], R_MAINB[20..0], ~{CEA}, ~{CEB}, ~{CEC}, ~{CED}, ~{CEE}, ~{CEF}, ~{CEG}, ~{CEH}, ~{CEI}, ~{CEJ}, ~{CEK}, ~{CEL}, ~{CEM}, ~{CEN}, ~{CEO}, ~{CEP}, ~{OEB}, ~{OEC}, ~{OED}, ~{OEE}, ~{RESET1}, ~{RESET2}, ~{RESET3}, ~{RESET4}, ~{WEB}, ~{WEC}, ~{WED}, ~{WEE}

Commit message: oam_sprite_ppu
Connections:
- net R_MAINA0 renamed OAMB_A0
- net R_MAINA1 renamed OAMB_A1
- net R_MAINA10 renamed OAMB_A10
- net R_MAINA11 renamed OAMB_A11
- net R_MAINA12 renamed OAMB_A12
- net R_MAINA13 renamed OAMB_A13
- net R_MAINA14 renamed OAMB_A14
- net R_MAINA15 renamed OAMB_A15
- net R_MAINA16 renamed OAMB_A16
- net R_MAINA17 renamed OAMB_A17
- net R_MAINA18 renamed OAMB_A18
- net R_MAINA19 renamed OAMB_A19
- net R_MAINA2 renamed OAMB_A2
- net R_MAINA20 renamed OAMB_A20
- net R_MAINA3 renamed OAMB_A3
- net R_MAINA4 renamed OAMB_A4
- net R_MAINA5 renamed OAMB_A5
- net R_MAINA6 renamed OAMB_A6
- net R_MAINA7 renamed OAMB_A7
- net R_MAINA8 renamed OAMB_A8
- net R_MAINA9 renamed OAMB_A9
- net R_MAINB0 renamed OAM_A0
- net R_MAINB1 renamed OAM_A1
- net R_MAINB10 renamed OAM_A10
- net R_MAINB11 renamed OAM_A11
- net R_MAINB12 renamed OAM_A12
- net R_MAINB13 renamed OAM_A13
- net R_MAINB14 renamed OAM_A14
- net R_MAINB15 renamed OAM_A15
- net R_MAINB16 renamed OAM_A16
- net R_MAINB17 renamed OAM_A17
- net R_MAINB18 renamed OAM_A18
- net R_MAINB19 renamed OAM_A19
- net R_MAINB2 renamed OAM_A2
- net R_MAINB20 renamed OAM_A20
- net R_MAINB3 renamed OAM_A3
- net R_MAINB4 renamed OAM_A4
- net R_MAINB5 renamed OAM_A5
- net R_MAINB6 renamed OAM_A6
- net R_MAINB7 renamed OAM_A7
- net R_MAINB8 renamed OAM_A8
- net R_MAINB9 renamed OAM_A9
Other:
- sheet memories_gfx ports: added OAMB_A[20..0], OAM_A[20..0]; removed R_MAINA[20..0], R_MAINB[20..0]
