File: cores/cps3/sch/memories.kicad_sch (KiCad schematic)
At the start: 12 parts

Commit message: ppu in process
Parts:
- removed SIMM1E (x2), SIMM2D (x2), SIMM3E, SIMM3EE, SIMM4D, SIMM4DD, SIMM5C, SIMM5CC, SIMM6B, SIMM6BB: Conn_01x36_Male, symbol Connector:Conn_01x36_Male
Connections:
- no-connect marks 81 -> 0
Other:
- removed sheet memories_gfx
- removed sheet memories_main
- note removed: "37"
- note removed: "38"
- note removed: "39 40"
- note removed: "41 42"
- note removed: "43 44"
- note removed: "45 46"
- note removed: "47 48"
- note removed: "49 50"
- note removed: "51 52"
- note removed: "53 54"
- note removed: "55 56"
- note removed: "57 58"
- note removed: "59 60"
- note removed: "61 62"
- note removed: "63 64"
- note removed: "65 66"
- note removed: "67 68"
- note removed: "69 70"
- note removed: "71 72"
- note removed: "MEMORIES DE GFX?"
- note removed: "MEMORIES DE MAIN?"
- note removed: "REVISAR POSIBLE CORTO ENTRE VCC Y VSS"
- note removed: "[37..72]"
