File: cores/cps3/sch/memories_gfx.kicad_sch (KiCad schematic)
At the start: 12 parts, among them K10 29F016-90PFTN, K11 29F016-90PFTN, K12 29F016-90PFTN, K13 29F016-90PFTN

Commit message: memories_main
Parts:
- renumbered K10 to KA10, K11 to KA11, K12 to KA12, K13 to KA13, KK10 to KB10, KK11 to KB11, KK12 to KB12, KK13 to KB13
Changed lines of the file:
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@@
   (symbol (lib_id "arcade:29F016-90PFTN") (at 355.6 66.04 0) (unit 1)
     (in_bom yes) (on_board yes)
-    (property "Reference" "K13" (id 0) (at 365.76 31.75 0))
+    (property "Reference" "KA13" (id 0) (at 365.76 31.75 0))
     (property "Value" "29F016-90PFTN" (id 1) (at 354.33 71.12 90))
     (property "Footprint" "" (id 2) (at 355.6 71.12 0)
@@
   (symbol (lib_id "arcade:29F016-90PFTN") (at 274.32 154.94 0) (unit 1)
     (in_bom yes) (on_board yes)
-    (property "Reference" "KK12" (id 0) (at 284.48 120.65 0))
+    (property "Reference" "KB12" (id 0) (at 284.48 120.65 0))
     (property "Value" "29F016-90PFTN" (id 1) (at 273.05 160.02 90))
     (property "Footprint" "" (id 2) (at 274.32 160.02 0)
@@
   (symbol (lib_id "arcade:29F016-90PFTN") (at 274.32 66.04 0) (unit 1)
     (in_bom yes) (on_board yes)
-    (property "Reference" "K12" (id 0) (at 284.48 31.75 0))
+    (property "Reference" "KA12" (id 0) (at 284.48 31.75 0))
     (property "Value" "29F016-90PFTN" (id 1) (at 273.05 71.12 90))
     (property "Footprint" "" (id 2) (at 274.32 71.12 0)
@@
   (symbol (lib_id "arcade:29F016-90PFTN") (at 355.6 154.94 0) (unit 1)
     (in_bom yes) (on_board yes)
-    (property "Reference" "KK13" (id 0) (at 365.76 120.65 0))
+    (property "Reference" "KB13" (id 0) (at 365.76 120.65 0))
     (property "Value" "29F016-90PFTN" (id 1) (at 354.33 160.02 90))
     (property "Footprint" "" (id 2) (at 355.6 160.02 0)
@@
   (symbol (lib_id "arcade:29F016-90PFTN") (at 196.85 154.94 0) (unit 1)
     (in_bom yes) (on_board yes)
-    (property "Reference" "KK11" (id 0) (at 207.01 120.65 0))
+    (property "Reference" "KB11" (id 0) (at 207.01 120.65 0))
     (property "Value" "29F016-90PFTN" (id 1) (at 195.58 160.02 90))
     (property "Footprint" "" (id 2) (at 196.85 160.02 0)
@@
   (symbol (lib_id "arcade:29F016-90PFTN") (at 120.65 154.94 0) (unit 1)
     (in_bom yes) (on_board yes)
-    (property "Reference" "KK10" (id 0) (at 130.81 120.65 0))
+    (property "Reference" "KB10" (id 0) (at 130.81 120.65 0))
     (property "Value" "29F016-90PFTN" (id 1) (at 119.38 160.02 90))
     (property "Footprint" "" (id 2) (at 120.65 160.02 0)
@@
   (symbol (lib_id "arcade:29F016-90PFTN") (at 196.85 66.04 0) (unit 1)
     (in_bom yes) (on_board yes)
-    (property "Reference" "K11" (id 0) (at 207.01 31.75 0))
+    (property "Reference" "KA11" (id 0) (at 207.01 31.75 0))
     (property "Value" "29F016-90PFTN" (id 1) (at 195.58 71.12 90))
     (property "Footprint" "" (id 2) (at 196.85 71.12 0)
@@
   (symbol (lib_id "arcade:29F016-90PFTN") (at 120.65 66.04 0) (unit 1)
     (in_bom yes) (on_board yes)
-    (property "Reference" "K10" (id 0) (at 130.81 31.75 0))
+    (property "Reference" "KA10" (id 0) (at 130.81 31.75 0))
     (property "Value" "29F016-90PFTN" (id 1) (at 119.38 71.12 90))
     (property "Footprint" "" (id 2) (at 120.65 71.12 0)

Commit message: memories
Parts:
- removed SIMM1A, SIMM1B, SIMM2A, SIMM2B: Conn_01x36_Male, symbol Connector:Conn_01x36_Male
Connections:
- net ~{OE}: now also KA10.1 (NC), KA11.1 (NC), KA11.2 (NC), KA12.1 (NC), KA12.2 (NC), KA13.1 (NC), KA13.2 (NC)
- net UK: now reaches KA10.2 (NC)
- net ~{RESET} renamed ~{RESET5}
Other:
- note removed: "37"
- note removed: "38"
- note removed: "39 40"
- note removed: "41 42"
- note removed: "43 44"
- note removed: "45 46"
- note removed: "47 48"
- note removed: "49 50"
- note removed: "51 52"
- note removed: "53 54"
- note removed: "55 56"
- note removed: "57 58"
- note removed: "59 60"
- note removed: "61 62"
- note removed: "63 64"
- note removed: "65 66"
- note removed: "67 68"
- note removed: "69 70"
- note removed: "71 72"
- note removed: "REVISAR"
- note removed: "[37..72]"
- moved on the sheet: KA10, KA11, KA12, KA13, KB10, KB11, KB12, KB13
