File: cores/cps3/sch/memories_gfx.kicad_sch (KiCad schematic)
At the start: 8 parts

Commit message: oam_sprite_ppu
Parts:
- removed KA10, KA11, KA12, KA13, KB10, KB11, KB12, KB13: 29F016-90PFTN, symbol arcade:29F016-90PFTN
- added JB1, JB2, JB3, JB4, JB5, JB6, JB7, JB8, JC1, JC2, JC3, JC4, JC5, JC6, JC7, JC8, JD1, JD2, JD3, JD4, JD5, JD6, JD7, JD8, JE1, JE2, JE3, JE4, JE5, JE6, JE7, JE8: 29F016-90PFTN, symbol arcade:29F016-90PFTN
Connections:
- net VCC: now also JB1.12 (VCC), JB1.37 (VCC), JB2.12 (VCC), JB2.37 (VCC), JB3.12 (VCC), JB3.37 (VCC), JB4.12 (VCC), JB4.37 (VCC), JB5.12 (VCC), JB5.37 (VCC), JB6.12 (VCC), JB6.37 (VCC), JB7.12 (VCC), JB7.37 (VCC), JB8.12 (VCC), JB8.37 (VCC), JC1.12 (VCC), JC1.37 (VCC), JC2.12 (VCC), JC2.37 (VCC), JC3.12 (VCC), JC3.37 (VCC), JC4.12 (VCC), JC4.37 (VCC), JC5.12 (VCC), JC5.37 (VCC), JC6.12 (VCC), JC6.37 (VCC), JC7.12 (VCC), JC7.37 (VCC), JC8.12 (VCC), JC8.37 (VCC), JD1.12 (VCC), JD1.37 (VCC), JD2.12 (VCC), JD2.37 (VCC), JD3.12 (VCC), JD3.37 (VCC), JD4.12 (VCC), JD4.37 (VCC), JD5.12 (VCC), JD5.37 (VCC), JD6.12 (VCC), JD6.37 (VCC), JD7.12 (VCC), JD7.37 (VCC), JD8.12 (VCC), JD8.37 (VCC), JE1.12 (VCC), JE1.37 (VCC), JE2.12 (VCC), JE2.37 (VCC), JE3.12 (VCC), JE3.37 (VCC), JE4.12 (VCC), JE4.37 (VCC), JE5.12 (VCC), JE5.37 (VCC), JE6.12 (VCC), JE6.37 (VCC), JE7.12 (VCC), JE7.37 (VCC), JE8.12 (VCC), JE8.37 (VCC)
- net VSS: now also JB1.35 (VSS), JB1.36 (VSS), JB1.42 (RY/~{BY}), JB2.35 (VSS), JB2.36 (VSS), JB2.42 (RY/~{BY}), JB3.35 (VSS), JB3.36 (VSS), JB3.42 (RY/~{BY}), JB4.35 (VSS), JB4.36 (VSS), JB4.42 (RY/~{BY}), JB5.35 (VSS), JB5.36 (VSS), JB5.42 (RY/~{BY}), JB6.35 (VSS), JB6.36 (VSS), JB6.42 (RY/~{BY}), JB7.35 (VSS), JB7.36 (VSS), JB7.42 (RY/~{BY}), JB8.35 (VSS), JB8.36 (VSS), JB8.42 (RY/~{BY}), JC1.35 (VSS), JC1.36 (VSS), JC1.42 (RY/~{BY}), JC2.35 (VSS), JC2.36 (VSS), JC2.42 (RY/~{BY}), JC3.35 (VSS), JC3.36 (VSS), JC3.42 (RY/~{BY}), JC4.35 (VSS), JC4.36 (VSS), JC4.42 (RY/~{BY}), JC5.35 (VSS), JC5.36 (VSS), JC5.42 (RY/~{BY}), JC6.35 (VSS), JC6.36 (VSS), JC6.42 (RY/~{BY}), JC7.35 (VSS), JC7.36 (VSS), JC7.42 (RY/~{BY}), JC8.35 (VSS), JC8.36 (VSS), JC8.42 (RY/~{BY}), JD1.35 (VSS), JD1.36 (VSS), JD1.42 (RY/~{BY}), JD2.35 (VSS), JD2.36 (VSS), JD2.42 (RY/~{BY}), JD3.35 (VSS), JD3.36 (VSS), JD3.42 (RY/~{BY}), JD4.35 (VSS), JD4.36 (VSS), JD4.42 (RY/~{BY}), JD5.35 (VSS), JD5.36 (VSS), JD5.42 (RY/~{BY}), JD6.35 (VSS), JD6.36 (VSS), JD6.42 (RY/~{BY}), JD7.35 (VSS), JD7.36 (VSS), JD7.42 (RY/~{BY}), JD8.35 (VSS), JD8.36 (VSS), JD8.42 (RY/~{BY}), JE1.35 (VSS), JE1.36 (VSS), JE1.42 (RY/~{BY}), JE2.35 (VSS), JE2.36 (VSS), JE2.42 (RY/~{BY}), JE3.35 (VSS), JE3.36 (VSS), JE3.42 (RY/~{BY}), JE4.35 (VSS), JE4.36 (VSS), JE4.42 (RY/~{BY}), JE5.35 (VSS), JE5.36 (VSS), JE5.42 (RY/~{BY}), JE6.35 (VSS), JE6.36 (VSS), JE6.42 (RY/~{BY}), JE7.35 (VSS), JE7.36 (VSS), JE7.42 (RY/~{BY}), JE8.35 (VSS), JE8.36 (VSS), JE8.42 (RY/~{BY})
- new net: JB5., JB5.23 (NC)
- new net: JE7., JE7.23 (NC)
- new net: JD2., JD2.23 (NC)
- new net: JB7., JB7.23 (NC)
- new net: JD7., JD7.23 (NC)
- new net: JC5., JC5.23 (NC)
- new net: JE4., JE4.23 (NC)
- new net: JC4., JC4.23 (NC)
- new net: JD3., JD3.23 (NC)
- new net: JC6., JC6.23 (NC)
- new net: JB4., JB4.23 (NC)
- new net: JE6., JE6.23 (NC)
- new net: JB2., JB2.23 (NC)
- new net: JE8., JE8.23 (NC)
- new net: JE5., JE5.23 (NC)
- new net: JB6., JB6.23 (NC)
- new net: JC1., JC1.23 (NC)
- new net: JD8., JD8.23 (NC)
- new net: JE3., JE3.23 (NC)
- new net: JC8., JC8.23 (NC)
- new net: JD4., JD4.23 (NC)
- new net: JC2., JC2.23 (NC)
- new net: JE2., JE2.23 (NC)
- new net: JB8., JB8.23 (NC)
- new net: JD6., JD6.23 (NC)
- new net: JB1., JB1.23 (NC)
- new net: JB3., JB3.23 (NC)
- new net: JD1., JD1.23 (NC)
- new net: JD5., JD5.23 (NC)
- new net: JC7., JC7.23 (NC)
- new net: JC3., JC3.23 (NC)
- new net: JE1., JE1.23 (NC)
- new net OAMB_A0: JB1.30 (A0), JB2.30 (A0), JB3.30 (A0), JB4.30 (A0), JB5.30 (A0), JB6.30 (A0), JB7.30 (A0), JB8.30 (A0)
- new net OAMB_A1: JB1.29 (A1), JB2.29 (A1), JB3.29 (A1), JB4.29 (A1), JB5.29 (A1), JB6.29 (A1), JB7.29 (A1), JB8.29 (A1)
- new net OAMB_A10: JB1.16 (A10), JB2.16 (A10), JB3.16 (A10), JB4.16 (A10), JB5.16 (A10), JB6.16 (A10), JB7.16 (A10), JB8.16 (A10)
- new net OAMB_A11: JB1.15 (A11), JB2.15 (A11), JB3.15 (A11), JB4.15 (A11), JB5.15 (A11), JB6.15 (A11), JB7.15 (A11), JB8.15 (A11)
- new net OAMB_A12: JB1.10 (A12), JB2.10 (A12), JB3.10 (A12), JB4.10 (A12), JB5.10 (A12), JB6.10 (A12), JB7.10 (A12), JB8.10 (A12)
- new net OAMB_A13: JB1.9 (A13), JB2.9 (A13), JB3.9 (A13), JB4.9 (A13), JB5.9 (A13), JB6.9 (A13), JB7.9 (A13), JB8.9 (A13)
- new net OAMB_A14: JB1.8 (A14), JB2.8 (A14), JB3.8 (A14), JB4.8 (A14), JB5.8 (A14), JB6.8 (A14), JB7.8 (A14), JB8.8 (A14)
- new net OAMB_A15: JB1.7 (A15), JB2.7 (A15), JB3.7 (A15), JB4.7 (A15), JB5.7 (A15), JB6.7 (A15), JB7.7 (A15), JB8.7 (A15)
- new net OAMB_A16: JB1.6 (A16), JB2.6 (A16), JB3.6 (A16), JB4.6 (A16), JB5.6 (A16), JB6.6 (A16), JB7.6 (A16), JB8.6 (A16)
- new net OAMB_A17: JB1.5 (A17), JB2.5 (A17), JB3.5 (A17), JB4.5 (A17), JB5.5 (A17), JB6.5 (A17), JB7.5 (A17), JB8.5 (A17)
- new net OAMB_A18: JB1.4 (A18), JB2.4 (A18), JB3.4 (A18), JB4.4 (A18), JB5.4 (A18), JB6.4 (A18), JB7.4 (A18), JB8.4 (A18)
- new net OAMB_A19: JB1.3 (A19), JB2.3 (A19), JB3.3 (A19), JB4.3 (A19), JB5.3 (A19), JB6.3 (A19), JB7.3 (A19), JB8.3 (A19)
- new net OAMB_A2: JB1.28 (A2), JB2.28 (A2), JB3.28 (A2), JB4.28 (A2), JB5.28 (A2), JB6.28 (A2), JB7.28 (A2), JB8.28 (A2)
- new net OAMB_A20: JB1.46 (A20), JB2.46 (A20), JB3.46 (A20), JB4.46 (A20), JB5.46 (A20), JB6.46 (A20), JB7.46 (A20), JB8.46 (A20)
- new net OAMB_A3: JB1.27 (A3), JB2.27 (A3), JB3.27 (A3), JB4.27 (A3), JB5.27 (A3), JB6.27 (A3), JB7.27 (A3), JB8.27 (A3)
- new net OAMB_A4: JB1.22 (A4), JB2.22 (A4), JB3.22 (A4), JB4.22 (A4), JB5.22 (A4), JB6.22 (A4), JB7.22 (A4), JB8.22 (A4)
- new net OAMB_A5: JB1.21 (A5), JB2.21 (A5), JB3.21 (A5), JB4.21 (A5), JB5.21 (A5), JB6.21 (A5), JB7.21 (A5), JB8.21 (A5)
- new net OAMB_A6: JB1.20 (A6), JB2.20 (A6), JB3.20 (A6), JB4.20 (A6), JB5.20 (A6), JB6.20 (A6), JB7.20 (A6), JB8.20 (A6)
- new net OAMB_A7: JB1.19 (A7), JB2.19 (A7), JB3.19 (A7), JB4.19 (A7), JB5.19 (A7), JB6.19 (A7), JB7.19 (A7), JB8.19 (A7)
- new net OAMB_A8: JB1.18 (A8), JB2.18 (A8), JB3.18 (A8), JB4.18 (A8), JB5.18 (A8), JB6.18 (A8), JB7.18 (A8), JB8.18 (A8)
- new net OAMB_A9: JB1.17 (A9), JB2.17 (A9), JB3.17 (A9), JB4.17 (A9), JB5.17 (A9), JB6.17 (A9), JB7.17 (A9), JB8.17 (A9)
- new net OAM_A0: JC1.30 (A0), JC2.30 (A0), JC3.30 (A0), JC4.30 (A0), JC5.30 (A0), JC6.30 (A0), JC7.30 (A0), JC8.30 (A0), JD1.30 (A0), JD2.30 (A0), JD3.30 (A0), JD4.30 (A0), JD5.30 (A0), JD6.30 (A0), JD7.30 (A0), JD8.30 (A0), JE1.30 (A0), JE2.30 (A0), JE3.30 (A0), JE4.30 (A0), JE5.30 (A0), JE6.30 (A0), JE7.30 (A0), JE8.30 (A0)
- new net OAM_A1: JC1.29 (A1), JC2.29 (A1), JC3.29 (A1), JC4.29 (A1), JC5.29 (A1), JC6.29 (A1), JC7.29 (A1), JC8.29 (A1), JD1.29 (A1), JD2.29 (A1), JD3.29 (A1), JD4.29 (A1), JD5.29 (A1), JD6.29 (A1), JD7.29 (A1), JD8.29 (A1), JE1.29 (A1), JE2.29 (A1), JE3.29 (A1), JE4.29 (A1), JE5.29 (A1), JE6.29 (A1), JE7.29 (A1), JE8.29 (A1)
- new net OAM_A10: JC1.16 (A10), JC2.16 (A10), JC3.16 (A10), JC4.16 (A10), JC5.16 (A10), JC6.16 (A10), JC7.16 (A10), JC8.16 (A10), JD1.16 (A10), JD2.16 (A10), JD3.16 (A10), JD4.16 (A10), JD5.16 (A10), JD6.16 (A10), JD7.16 (A10), JD8.16 (A10), JE1.16 (A10), JE2.16 (A10), JE3.16 (A10), JE4.16 (A10), JE5.16 (A10), JE6.16 (A10), JE7.16 (A10), JE8.16 (A10)
- new net OAM_A11: JC1.15 (A11), JC2.15 (A11), JC3.15 (A11), JC4.15 (A11), JC5.15 (A11), JC6.15 (A11), JC7.15 (A11), JC8.15 (A11), JD1.15 (A11), JD2.15 (A11), JD3.15 (A11), JD4.15 (A11), JD5.15 (A11), JD6.15 (A11), JD7.15 (A11), JD8.15 (A11), JE1.15 (A11), JE2.15 (A11), JE3.15 (A11), JE4.15 (A11), JE5.15 (A11), JE6.15 (A11), JE7.15 (A11), JE8.15 (A11)
- new net OAM_A12: JC1.10 (A12), JC2.10 (A12), JC3.10 (A12), JC4.10 (A12), JC5.10 (A12), JC6.10 (A12), JC7.10 (A12), JC8.10 (A12), JD1.10 (A12), JD2.10 (A12), JD3.10 (A12), JD4.10 (A12), JD5.10 (A12), JD6.10 (A12), JD7.10 (A12), JD8.10 (A12), JE1.10 (A12), JE2.10 (A12), JE3.10 (A12), JE4.10 (A12), JE5.10 (A12), JE6.10 (A12), JE7.10 (A12), JE8.10 (A12)
- new net OAM_A13: JC1.9 (A13), JC2.9 (A13), JC3.9 (A13), JC4.9 (A13), JC5.9 (A13), JC6.9 (A13), JC7.9 (A13), JC8.9 (A13), JD1.9 (A13), JD2.9 (A13), JD3.9 (A13), JD4.9 (A13), JD5.9 (A13), JD6.9 (A13), JD7.9 (A13), JD8.9 (A13), JE1.9 (A13), JE2.9 (A13), JE3.9 (A13), JE4.9 (A13), JE5.9 (A13), JE6.9 (A13), JE7.9 (A13), JE8.9 (A13)
- new net OAM_A14: JC1.8 (A14), JC2.8 (A14), JC3.8 (A14), JC4.8 (A14), JC5.8 (A14), JC6.8 (A14), JC7.8 (A14), JC8.8 (A14), JD1.8 (A14), JD2.8 (A14), JD3.8 (A14), JD4.8 (A14), JD5.8 (A14), JD6.8 (A14), JD7.8 (A14), JD8.8 (A14), JE1.8 (A14), JE2.8 (A14), JE3.8 (A14), JE4.8 (A14), JE5.8 (A14), JE6.8 (A14), JE7.8 (A14), JE8.8 (A14)
- new net OAM_A15: JC1.7 (A15), JC2.7 (A15), JC3.7 (A15), JC4.7 (A15), JC5.7 (A15), JC6.7 (A15), JC7.7 (A15), JC8.7 (A15), JD1.7 (A15), JD2.7 (A15), JD3.7 (A15), JD4.7 (A15), JD5.7 (A15), JD6.7 (A15), JD7.7 (A15), JD8.7 (A15), JE1.7 (A15), JE2.7 (A15), JE3.7 (A15), JE4.7 (A15), JE5.7 (A15), JE6.7 (A15), JE7.7 (A15), JE8.7 (A15)
- new net OAM_A16: JC1.6 (A16), JC2.6 (A16), JC3.6 (A16), JC4.6 (A16), JC5.6 (A16), JC6.6 (A16), JC7.6 (A16), JC8.6 (A16), JD1.6 (A16), JD2.6 (A16), JD3.6 (A16), JD4.6 (A16), JD5.6 (A16), JD6.6 (A16), JD7.6 (A16), JD8.6 (A16), JE1.6 (A16), JE2.6 (A16), JE3.6 (A16), JE4.6 (A16), JE5.6 (A16), JE6.6 (A16), JE7.6 (A16), JE8.6 (A16)
- new net OAM_A17: JC1.5 (A17), JC2.5 (A17), JC3.5 (A17), JC4.5 (A17), JC5.5 (A17), JC6.5 (A17), JC7.5 (A17), JC8.5 (A17), JD1.5 (A17), JD2.5 (A17), JD3.5 (A17), JD4.5 (A17), JD5.5 (A17), JD6.5 (A17), JD7.5 (A17), JD8.5 (A17), JE1.5 (A17), JE2.5 (A17), JE3.5 (A17), JE4.5 (A17), JE5.5 (A17), JE6.5 (A17), JE7.5 (A17), JE8.5 (A17)
- new net OAM_A18: JC1.4 (A18), JC2.4 (A18), JC3.4 (A18), JC4.4 (A18), JC5.4 (A18), JC6.4 (A18), JC7.4 (A18), JC8.4 (A18), JD1.4 (A18), JD2.4 (A18), JD3.4 (A18), JD4.4 (A18), JD5.4 (A18), JD6.4 (A18), JD7.4 (A18), JD8.4 (A18), JE1.4 (A18), JE2.4 (A18), JE3.4 (A18), JE4.4 (A18), JE5.4 (A18), JE6.4 (A18), JE7.4 (A18), JE8.4 (A18)
- new net OAM_A19: JC1.3 (A19), JC2.3 (A19), JC3.3 (A19), JC4.3 (A19), JC5.3 (A19), JC6.3 (A19), JC7.3 (A19), JC8.3 (A19), JD1.3 (A19), JD2.3 (A19), JD3.3 (A19), JD4.3 (A19), JD5.3 (A19), JD6.3 (A19), JD7.3 (A19), JD8.3 (A19), JE1.3 (A19), JE2.3 (A19), JE3.3 (A19), JE4.3 (A19), JE5.3 (A19), JE6.3 (A19), JE7.3 (A19), JE8.3 (A19)
- new net OAM_A2: JC1.28 (A2), JC2.28 (A2), JC3.28 (A2), JC4.28 (A2), JC5.28 (A2), JC6.28 (A2), JC7.28 (A2), JC8.28 (A2), JD1.28 (A2), JD2.28 (A2), JD3.28 (A2), JD4.28 (A2), JD5.28 (A2), JD6.28 (A2), JD7.28 (A2), JD8.28 (A2), JE1.28 (A2), JE2.28 (A2), JE3.28 (A2), JE4.28 (A2), JE5.28 (A2), JE6.28 (A2), JE7.28 (A2), JE8.28 (A2)
- new net OAM_A20: JC1.46 (A20), JC2.46 (A20), JC3.46 (A20), JC4.46 (A20), JC5.46 (A20), JC6.46 (A20), JC7.46 (A20), JC8.46 (A20), JD1.46 (A20), JD2.46 (A20), JD3.46 (A20), JD4.46 (A20), JD5.46 (A20), JD6.46 (A20), JD7.46 (A20), JD8.46 (A20), JE1.46 (A20), JE2.46 (A20), JE3.46 (A20), JE4.46 (A20), JE5.46 (A20), JE6.46 (A20), JE7.46 (A20), JE8.46 (A20)
- new net OAM_A3: JC1.27 (A3), JC2.27 (A3), JC3.27 (A3), JC4.27 (A3), JC5.27 (A3), JC6.27 (A3), JC7.27 (A3), JC8.27 (A3), JD1.27 (A3), JD2.27 (A3), JD3.27 (A3), JD4.27 (A3), JD5.27 (A3), JD6.27 (A3), JD7.27 (A3), JD8.27 (A3), JE1.27 (A3), JE2.27 (A3), JE3.27 (A3), JE4.27 (A3), JE5.27 (A3), JE6.27 (A3), JE7.27 (A3), JE8.27 (A3)
- new net OAM_A4: JC1.22 (A4), JC2.22 (A4), JC3.22 (A4), JC4.22 (A4), JC5.22 (A4), JC6.22 (A4), JC7.22 (A4), JC8.22 (A4), JD1.22 (A4), JD2.22 (A4), JD3.22 (A4), JD4.22 (A4), JD5.22 (A4), JD6.22 (A4), JD7.22 (A4), JD8.22 (A4), JE1.22 (A4), JE2.22 (A4), JE3.22 (A4), JE4.22 (A4), JE5.22 (A4), JE6.22 (A4), JE7.22 (A4), JE8.22 (A4)
- new net OAM_A5: JC1.21 (A5), JC2.21 (A5), JC3.21 (A5), JC4.21 (A5), JC5.21 (A5), JC6.21 (A5), JC7.21 (A5), JC8.21 (A5), JD1.21 (A5), JD2.21 (A5), JD3.21 (A5), JD4.21 (A5), JD5.21 (A5), JD6.21 (A5), JD7.21 (A5), JD8.21 (A5), JE1.21 (A5), JE2.21 (A5), JE3.21 (A5), JE4.21 (A5), JE5.21 (A5), JE6.21 (A5), JE7.21 (A5), JE8.21 (A5)
- new net OAM_A6: JC1.20 (A6), JC2.20 (A6), JC3.20 (A6), JC4.20 (A6), JC5.20 (A6), JC6.20 (A6), JC7.20 (A6), JC8.20 (A6), JD1.20 (A6), JD2.20 (A6), JD3.20 (A6), JD4.20 (A6), JD5.20 (A6), JD6.20 (A6), JD7.20 (A6), JD8.20 (A6), JE1.20 (A6), JE2.20 (A6), JE3.20 (A6), JE4.20 (A6), JE5.20 (A6), JE6.20 (A6), JE7.20 (A6), JE8.20 (A6)
- new net OAM_A7: JC1.19 (A7), JC2.19 (A7), JC3.19 (A7), JC4.19 (A7), JC5.19 (A7), JC6.19 (A7), JC7.19 (A7), JC8.19 (A7), JD1.19 (A7), JD2.19 (A7), JD3.19 (A7), JD4.19 (A7), JD5.19 (A7), JD6.19 (A7), JD7.19 (A7), JD8.19 (A7), JE1.19 (A7), JE2.19 (A7), JE3.19 (A7), JE4.19 (A7), JE5.19 (A7), JE6.19 (A7), JE7.19 (A7), JE8.19 (A7)
- new net OAM_A8: JC1.18 (A8), JC2.18 (A8), JC3.18 (A8), JC4.18 (A8), JC5.18 (A8), JC6.18 (A8), JC7.18 (A8), JC8.18 (A8), JD1.18 (A8), JD2.18 (A8), JD3.18 (A8), JD4.18 (A8), JD5.18 (A8), JD6.18 (A8), JD7.18 (A8), JD8.18 (A8), JE1.18 (A8), JE2.18 (A8), JE3.18 (A8), JE4.18 (A8), JE5.18 (A8), JE6.18 (A8), JE7.18 (A8), JE8.18 (A8)
- new net OAM_A9: JC1.17 (A9), JC2.17 (A9), JC3.17 (A9), JC4.17 (A9), JC5.17 (A9), JC6.17 (A9), JC7.17 (A9), JC8.17 (A9), JD1.17 (A9), JD2.17 (A9), JD3.17 (A9), JD4.17 (A9), JD5.17 (A9), JD6.17 (A9), JD7.17 (A9), JD8.17 (A9), JE1.17 (A9), JE2.17 (A9), JE3.17 (A9), JE4.17 (A9), JE5.17 (A9), JE6.17 (A9), JE7.17 (A9), JE8.17 (A9)
- new net SPRITEA_D0: JB1.31 (D0), JB3.31 (D0), JB5.31 (D0), JB7.31 (D0)
- new net SPRITEA_D1: JB1.32 (D1), JB3.32 (D1), JB5.32 (D1), JB7.32 (D1)
- new net SPRITEA_D2: JB1.33 (D2), JB3.33 (D2), JB5.33 (D2), JB7.33 (D2)
- new net SPRITEA_D3: JB1.34 (D3), JB3.34 (D3), JB5.34 (D3), JB7.34 (D3)
- new net SPRITEA_D4: JB1.38 (D4), JB3.38 (D4), JB5.38 (D4), JB7.38 (D4)
- new net SPRITEA_D5: JB1.39 (D5), JB3.39 (D5), JB5.39 (D5), JB7.39 (D5)
- new net SPRITEA_D6: JB1.40 (D6), JB3.40 (D6), JB5.40 (D6), JB7.40 (D6)
- new net SPRITEA_D7: JB1.41 (D7), JB3.41 (D7), JB5.41 (D7), JB7.41 (D7)
- new net SPRITEB_D0: JC1.31 (D0), JC3.31 (D0), JC5.31 (D0), JC7.31 (D0), JD1.31 (D0), JD3.31 (D0), JD5.31 (D0), JD7.31 (D0), JE1.31 (D0), JE3.31 (D0), JE5.31 (D0), JE7.31 (D0)
- new net SPRITEB_D1: JC1.32 (D1), JC3.32 (D1), JC5.32 (D1), JC7.32 (D1), JD1.32 (D1), JD3.32 (D1), JD5.32 (D1), JD7.32 (D1), JE1.32 (D1), JE3.32 (D1), JE5.32 (D1), JE7.32 (D1)
- new net SPRITEB_D2: JC1.33 (D2), JC3.33 (D2), JC5.33 (D2), JC7.33 (D2), JD1.33 (D2), JD3.33 (D2), JD5.33 (D2), JD7.33 (D2), JE1.33 (D2), JE3.33 (D2), JE5.33 (D2), JE7.33 (D2)
- new net SPRITEB_D3: JC1.34 (D3), JC3.34 (D3), JC5.34 (D3), JC7.34 (D3), JD1.34 (D3), JD3.34 (D3), JD5.34 (D3), JD7.34 (D3), JE1.34 (D3), JE3.34 (D3), JE5.34 (D3), JE7.34 (D3)
- new net SPRITEB_D4: JC1.38 (D4), JC3.38 (D4), JC5.38 (D4), JC7.38 (D4), JD1.38 (D4), JD3.38 (D4), JD5.38 (D4), JD7.38 (D4), JE1.38 (D4), JE3.38 (D4), JE5.38 (D4), JE7.38 (D4)
- new net SPRITEB_D5: JC1.39 (D5), JC3.39 (D5), JC5.39 (D5), JC7.39 (D5), JD1.39 (D5), JD3.39 (D5), JD5.39 (D5), JD7.39 (D5), JE1.39 (D5), JE3.39 (D5), JE5.39 (D5), JE7.39 (D5)
- new net SPRITEB_D6: JC1.40 (D6), JC3.40 (D6), JC5.40 (D6), JC7.40 (D6), JD1.40 (D6), JD3.40 (D6), JD5.40 (D6), JD7.40 (D6), JE1.40 (D6), JE3.40 (D6), JE5.40 (D6), JE7.40 (D6)
- new net SPRITEB_D7: JC1.41 (D7), JC3.41 (D7), JC5.41 (D7), JC7.41 (D7), JD1.41 (D7), JD3.41 (D7), JD5.41 (D7), JD7.41 (D7), JE1.41 (D7), JE3.41 (D7), JE5.41 (D7), JE7.41 (D7)
- new net SPRITEC_D0: JB2.31 (D0), JB4.31 (D0), JB6.31 (D0), JB8.31 (D0)
- new net SPRITEC_D1: JB2.32 (D1), JB4.32 (D1), JB6.32 (D1), JB8.32 (D1)
- new net SPRITEC_D2: JB2.33 (D2), JB4.33 (D2), JB6.33 (D2), JB8.33 (D2)
- new net SPRITEC_D3: JB2.34 (D3), JB4.34 (D3), JB6.34 (D3), JB8.34 (D3)
- new net SPRITEC_D4: JB2.38 (D4), JB4.38 (D4), JB6.38 (D4), JB8.38 (D4)
- new net SPRITEC_D5: JB2.39 (D5), JB4.39 (D5), JB6.39 (D5), JB8.39 (D5)
- new net SPRITEC_D6: JB2.40 (D6), JB4.40 (D6), JB6.40 (D6), JB8.40 (D6)
- new net SPRITEC_D7: JB2.41 (D7), JB4.41 (D7), JB6.41 (D7), JB8.41 (D7)
- new net SPRITED_D0: JC2.31 (D0), JC4.31 (D0), JC6.31 (D0), JC8.31 (D0), JD2.31 (D0), JD4.31 (D0), JD6.31 (D0), JD8.31 (D0), JE2.31 (D0), JE4.31 (D0), JE6.31 (D0), JE8.31 (D0)
- new net SPRITED_D1: JC2.32 (D1), JC4.32 (D1), JC6.32 (D1), JC8.32 (D1), JD2.32 (D1), JD4.32 (D1), JD6.32 (D1), JD8.32 (D1), JE2.32 (D1), JE4.32 (D1), JE6.32 (D1), JE8.32 (D1)
- new net SPRITED_D2: JC2.33 (D2), JC4.33 (D2), JC6.33 (D2), JC8.33 (D2), JD2.33 (D2), JD4.33 (D2), JD6.33 (D2), JD8.33 (D2), JE2.33 (D2), JE4.33 (D2), JE6.33 (D2), JE8.33 (D2)
- new net SPRITED_D3: JC2.34 (D3), JC4.34 (D3), JC6.34 (D3), JC8.34 (D3), JD2.34 (D3), JD4.34 (D3), JD6.34 (D3), JD8.34 (D3), JE2.34 (D3), JE4.34 (D3), JE6.34 (D3), JE8.34 (D3)
- new net SPRITED_D4: JC2.38 (D4), JC4.38 (D4), JC6.38 (D4), JC8.38 (D4), JD2.38 (D4), JD4.38 (D4), JD6.38 (D4), JD8.38 (D4), JE2.38 (D4), JE4.38 (D4), JE6.38 (D4), JE8.38 (D4)
- new net SPRITED_D5: JC2.39 (D5), JC4.39 (D5), JC6.39 (D5), JC8.39 (D5), JD2.39 (D5), JD4.39 (D5), JD6.39 (D5), JD8.39 (D5), JE2.39 (D5), JE4.39 (D5), JE6.39 (D5), JE8.39 (D5)
- new net SPRITED_D6: JC2.40 (D6), JC4.40 (D6), JC6.40 (D6), JC8.40 (D6), JD2.40 (D6), JD4.40 (D6), JD6.40 (D6), JD8.40 (D6), JE2.40 (D6), JE4.40 (D6), JE6.40 (D6), JE8.40 (D6)
- new net SPRITED_D7: JC2.41 (D7), JC4.41 (D7), JC6.41 (D7), JC8.41 (D7), JD2.41 (D7), JD4.41 (D7), JD6.41 (D7), JD8.41 (D7), JE2.41 (D7), JE4.41 (D7), JE6.41 (D7), JE8.41 (D7)
- new net ~{CEA}: JB1.11 (~{CE}), JB4.11 (~{CE})
- new net ~{CEB}: JB2.11 (~{CE}), JB3.11 (~{CE})
- new net ~{CEC}: JB5.11 (~{CE}), JB8.11 (~{CE})
- new net ~{CED}: JB6.11 (~{CE}), JB7.11 (~{CE})
- new net ~{CEE}: JC1.11 (~{CE}), JC4.11 (~{CE})
- new net ~{CEF}: JC2.11 (~{CE}), JC3.11 (~{CE})
- new net ~{CEG}: JC5.11 (~{CE}), JC8.11 (~{CE})
- new net ~{CEH}: JC6.11 (~{CE}), JC7.11 (~{CE})
- new net ~{CEI}: JD1.11 (~{CE}), JD4.11 (~{CE})
- new net ~{CEJ}: JD2.11 (~{CE}), JD3.11 (~{CE})
- new net ~{CEK}: JD5.11 (~{CE}), JD8.11 (~{CE})
- new net ~{CEL}: JD6.11 (~{CE}), JD7.11 (~{CE})
- new net ~{CEM}: JE1.11 (~{CE}), JE4.11 (~{CE})
- new net ~{CEN}: JE2.11 (~{CE}), JE3.11 (~{CE})
- new net ~{CEO}: JE5.11 (~{CE}), JE8.11 (~{CE})
- new net ~{CEP}: JE6.11 (~{CE}), JE7.11 (~{CE})
- new net ~{OEB}: JB1.43 (~{OE}), JB2.43 (~{OE}), JB3.43 (~{OE}), JB4.43 (~{OE}), JB5.43 (~{OE}), JB6.43 (~{OE}), JB7.43 (~{OE}), JB8.43 (~{OE})
- new net ~{OEC}: JC1.43 (~{OE}), JC2.43 (~{OE}), JC3.43 (~{OE}), JC4.43 (~{OE}), JC5.43 (~{OE}), JC6.43 (~{OE}), JC7.43 (~{OE}), JC8.43 (~{OE}), JD4.43 (~{OE}), JD6.43 (~{OE}), JD8.43 (~{OE})
- new net ~{OED}: JD1.43 (~{OE}), JD2.43 (~{OE}), JD3.43 (~{OE}), JD5.43 (~{OE}), JD7.43 (~{OE})
- new net ~{OEE}: JE1.43 (~{OE}), JE2.43 (~{OE}), JE3.43 (~{OE}), JE4.43 (~{OE}), JE5.43 (~{OE}), JE6.43 (~{OE}), JE7.43 (~{OE}), JE8.43 (~{OE})
- new net ~{RESET1}: JB1.14 (~{RESET}), JB2.14 (~{RESET}), JB3.14 (~{RESET}), JB4.14 (~{RESET}), JB5.14 (~{RESET}), JB6.14 (~{RESET}), JB7.14 (~{RESET}), JB8.14 (~{RESET})
- new net ~{RESET2}: JC1.14 (~{RESET}), JC2.14 (~{RESET}), JC3.14 (~{RESET}), JC4.14 (~{RESET}), JC5.14 (~{RESET}), JC6.14 (~{RESET}), JC7.14 (~{RESET}), JC8.14 (~{RESET})
- new net ~{RESET3}: JD1.14 (~{RESET}), JD2.14 (~{RESET}), JD3.14 (~{RESET}), JD4.14 (~{RESET}), JD5.14 (~{RESET}), JD6.14 (~{RESET}), JD7.14 (~{RESET}), JD8.14 (~{RESET})
- new net ~{RESET4}: JE1.14 (~{RESET}), JE2.14 (~{RESET}), JE3.14 (~{RESET}), JE4.14 (~{RESET}), JE5.14 (~{RESET}), JE6.14 (~{RESET}), JE7.14 (~{RESET}), JE8.14 (~{RESET})
- new net ~{WEB}: JB1.44 (~{WE}), JB2.44 (~{WE}), JB3.44 (~{WE}), JB4.44 (~{WE}), JB5.44 (~{WE}), JB6.44 (~{WE}), JB7.44 (~{WE}), JB8.44 (~{WE})
- new net ~{WEC}: JC1.44 (~{WE}), JC2.44 (~{WE}), JC3.44 (~{WE}), JC4.44 (~{WE}), JC5.44 (~{WE}), JC6.44 (~{WE}), JC7.44 (~{WE}), JC8.44 (~{WE}), JD4.44 (~{WE}), JD6.44 (~{WE}), JD8.44 (~{WE})
- new net ~{WED}: JD1.44 (~{WE}), JD2.44 (~{WE}), JD3.44 (~{WE}), JD5.44 (~{WE}), JD7.44 (~{WE})
- new net ~{WEE}: JE1.44 (~{WE}), JE2.44 (~{WE}), JE3.44 (~{WE}), JE4.44 (~{WE}), JE5.44 (~{WE}), JE6.44 (~{WE}), JE7.44 (~{WE}), JE8.44 (~{WE})
Other:
- added sheet plane_color (plane_color.kicad_sch)
- note added: "SIMM3E"
- note added: "SIMM4D"
- note added: "SIMM5C"
- note added: "SIMM6B"
- note added: "first plane controls bit 0 of the color"
