File: cores/cps3/sch/untitled.kicad_sch (KiCad schematic)
At the start: 0 parts

Commit message: memories4
Parts:
- added CAP: C_P, symbol Device:C_Polarized_Small_US
Other:
- note added: "79 CAPACITORS"
Changed lines of the file:
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@@
     )
   )
+  (text "79 CAPACITORS\n" (at 24.13 82.55 0)
+    (effects (font (size 1.27 1.27)) (justify left bottom))
+  )
+  (symbol (lib_id "Device:C_Polarized_Small_US") (at 25.4 21.59 0) (unit 1)
+    (in_bom yes) (on_board yes)
+    (property "Reference" "CAP" (id 0) (at 25.654 19.812 0)
+      (effects (font (size 1.27 1.27)) (justify left))
+    )
+    (property "Value" "C_P" (id 1) (at 25.654 23.622 0)
+      (effects (font (size 1.27 1.27)) (justify left))
+    )
+    (property "Footprint" "" (id 2) (at 25.4 21.59 0)
+      (effects (font (size 1.27 1.27)) hide)
+    )
+    (property "Datasheet" "~" (id 3) (at 25.4 21.59 0)
+      (effects (font (size 1.27 1.27)) hide)
+    )
+    (pin "1")
+    (pin "2")
+  )
 )
