File: cores/cps3/sch/untitled.kicad_sch (KiCad schematic)
At the start: 0 parts

Commit message: update_cps3
Parts:
- added U1: 74LS08, symbol jt74:74LS08
Connections:
- new net VCC: U1.14 (VCC)
- new net VSS: U1.7 (VSS)
Changed lines of the file:
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@@
     (comment 1 "E.Triana")
   )
+  (symbol (lib_id "jt74:74LS08") (at 27.94 182.88 0) (unit 5)
+    (in_bom yes) (on_board yes)
+    (property "Reference" "U1" (id 0) (at 27.94 181.61 0))
+    (property "Value" "74LS08" (id 1) (at 27.94 184.15 0))
+    (property "Footprint" "" (id 2) (at 27.94 182.88 0)
+      (effects (font (size 1.27 1.27)) hide)
+    )
+    (property "Datasheet" "http://www.ti.com/lit/gpn/sn74LS08" (id 3) (at 27.94 182.88 0)
+      (effects (font (size 1.27 1.27)) hide)
+    )
+    (pin "1")
+    (pin "2")
+    (pin "3")
+    (pin "4")
+    (pin "5")
+    (pin "6")
+    (pin "10")
+    (pin "8")
+    (pin "9")
+    (pin "11")
+    (pin "12")
+    (pin "13")
+    (pin "14")
+    (pin "7")
+  )
 )
