File: cores/cps3/sch/untitled.kicad_sch (KiCad schematic)
At the start: 1 part, among them U1 74LS08

Commit message: update6_cps
Parts:
- added CP10, CP11, CP12, CP13, CP14, CP15, CP16, CP17, CP18, CP19, CP2, CP20, CP21, CP22, CP23, CP24, CP25, CP26, CP27, CP28, CP29, CP3, CP30, CP31, CP32, CP33, CP34, CP35, CP36, CP37, CP38, CP39, CP4, CP40, CP41, CP42, CP43, CP44, CP45, CP46, CP47, CP48, CP49, CP5, CP50, CP51, CP52, CP53, CP54, CP55, CP56, CP57, CP58, CP59, CP6, CP60, CP61, CP62, CP63, CP64, CP65, CP66, CP67, CP68, CP69, CP7, CP70, CP71, CP72, CP73, CP74, CP75, CP76, CP8, CP9: μ, symbol Device:C_Polarized_US
- renumbered U1 to U2
Connections:
- net VCC: now also CP10.1, CP11.1, CP12.1, CP13.1, CP14.1, CP15.1, CP16.1, CP17.1, CP18.1, CP19.1, CP2.1, CP20.1, CP21.1, CP22.1, CP23.1, CP24.1, CP25.1, CP26.1, CP27.1, CP28.1, CP29.1, CP3.1, CP30.1, CP31.1, CP32.1, CP33.1, CP34.1, CP35.1, CP36.1, CP37.1, CP38.1, CP39.1, CP4.1, CP40.1, CP41.1, CP42.1, CP43.1, CP44.1, CP45.1, CP46.1, CP47.1, CP48.1, CP49.1, CP5.1, CP50.1, CP51.1, CP52.1, CP53.1, CP54.1, CP55.1, CP56.1, CP57.1, CP58.1, CP59.1, CP6.1, CP60.1, CP61.1, CP62.1, CP63.1, CP64.1, CP65.1, CP66.1, CP67.1, CP68.1, CP69.1, CP7.1, CP70.1, CP71.1, CP72.1, CP73.1, CP74.1, CP75.1, CP76.1, CP8.1, CP9.1
- net VSS: now also CP10.2, CP11.2, CP12.2, CP13.2, CP14.2, CP15.2, CP16.2, CP17.2, CP18.2, CP19.2, CP2.2, CP20.2, CP21.2, CP22.2, CP23.2, CP24.2, CP25.2, CP26.2, CP27.2, CP28.2, CP29.2, CP3.2, CP30.2, CP31.2, CP32.2, CP33.2, CP34.2, CP35.2, CP36.2, CP37.2, CP38.2, CP39.2, CP4.2, CP40.2, CP41.2, CP42.2, CP43.2, CP44.2, CP45.2, CP46.2, CP47.2, CP48.2, CP49.2, CP5.2, CP50.2, CP51.2, CP52.2, CP53.2, CP54.2, CP55.2, CP56.2, CP57.2, CP58.2, CP59.2, CP6.2, CP60.2, CP61.2, CP62.2, CP63.2, CP64.2, CP65.2, CP66.2, CP67.2, CP68.2, CP69.2, CP7.2, CP70.2, CP71.2, CP72.2, CP73.2, CP74.2, CP75.2, CP76.2, CP8.2, CP9.2
