File: cores/cps3/sch/main.kicad_sch (KiCad schematic)
At the start: 8 parts

Commit message: ppu
Parts:
- removed G3: DL-2729_PPU, symbol capcom:DL-2729_PPU
- removed H1, H2, H3, H4: CU383-69K, symbol arcade:CU383-69K
- removed U? (x3): 74FCT-16244ATPV, symbol arcade:74FCT-16244ATPV
