File: cores/cps3/sch/plane_color.kicad_sch (KiCad schematic)
At the start: 0 parts

Commit message: oam_sprite_ppu
Other:
- company: (none) -> JOTEGO
- title: (none) -> CP SYSTEM III
Changed lines of the file:
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@@
 (kicad_sch (version 20211123) (generator eeschema)
   (paper "A4")
+  (title_block
+    (title "CP SYSTEM III")
+    (date "14/10/22")
+    (rev "José Tejada G.")
+    (company "JOTEGO")
+    (comment 1 "E.Triana")
+  )
 )
