File: cores/cps3/sch/gfx.kicad_sch (KiCad schematic)
At the start: 0 parts

Commit message: ppu
Parts:
- added G2: DL-2729_PPU, symbol capcom:DL-2729_PPU
- added H1, H2, H3, H4: CU383-69K, symbol arcade:CU383-69K
- added U?: 74FCT-16244ATPV, symbol arcade:74FCT-16244ATPV
Connections:
- new net A0: H2.3 (A1-1)
- new net A1: H2.7 (A2-1)
- new net A10: H4.11 (A3-1)
- new net A11: H4.17 (A4-1)
- new net A12: H3.3 (A1-1)
- new net A13: H3.7 (A2-1)
- new net A14: H3.11 (A3-1)
- new net A15: H3.17 (A4-1)
- new net A2: H2.11 (A3-1)
- new net A3: H2.17 (A4-1)
- new net A4: H1.3 (A1-1)
- new net A5: H1.7 (A2-1)
- new net A6: H1.11 (A3-1)
- new net A7: H1.17 (A4-1)
- new net A8: H4.3 (A1-1)
- new net A9: H4.7 (A2-1)
- new net PIN110: U?.47 (A1-1)
- new net RMAINA_D0: H1.5 (B1-2)
- new net RMAINA_D1: H1.9 (B2-2)
- new net RMAINA_D2: H1.15 (B3-2)
- new net RMAINA_D3: H1.19 (B4-2)
- new net RMAINA_D4: H2.5 (B1-2)
- new net RMAINA_D5: H2.9 (B2-2)
- new net RMAINA_D6: H2.15 (B3-2)
- new net RMAINA_D7: H2.19 (B4-2)
- new net RMAINB_D0: H1.2 (B1-1)
- new net RMAINB_D1: H1.6 (B2-1)
- new net RMAINB_D2: H1.10 (B3-1)
- new net RMAINB_D3: H1.16 (B4-1)
- new net RMAINB_D4: H2.2 (B1-1)
- new net RMAINB_D5: H2.6 (B2-1)
- new net RMAINB_D6: H2.10 (B3-1)
- new net RMAINB_D7: H2.16 (B4-1)
- new net RMAINC_D0: H4.5 (B1-2)
- new net RMAINC_D1: H4.9 (B2-2)
- new net RMAINC_D2: H4.15 (B3-2)
- new net RMAINC_D3: H4.19 (B4-2)
- new net RMAINC_D4: H3.5 (B1-2)
- new net RMAINC_D5: H3.9 (B2-2)
- new net RMAINC_D6: H3.15 (B3-2)
- new net RMAINC_D7: H3.19 (B4-2)
- new net RMAIND_D0: H4.2 (B1-1)
- new net RMAIND_D1: H4.6 (B2-1)
- new net RMAIND_D2: H4.10 (B3-1)
- new net RMAIND_D3: H4.16 (B4-1)
- new net RMAIND_D4: H3.2 (B1-1)
- new net RMAIND_D5: H3.6 (B2-1)
- new net RMAIND_D6: H3.10 (B3-1)
- new net RMAIND_D7: H3.16 (B4-1)
- new net VCC: H1.24 (VCC), H2.24 (VCC), H3.24 (VCC), H4.24 (VCC)
- new net VRAM0: G2.124 (VRAM0)
- new net VRAM1: G2.125 (VRAM1)
- new net VRAM10: G2.135 (VRAM10)
- new net VRAM11: G2.136 (VRAM11)
- new net VRAM12: G2.137 (VRAM12)
- new net VRAM13: G2.138 (VRAM13)
- new net VRAM14: G2.139 (VRAM14)
- new net VRAM15: G2.140 (VRAM15)
- new net VRAM2: G2.126 (VRAM2)
- new net VRAM3: G2.127 (VRAM3)
- new net VRAM4: G2.128 (VRAM4)
- new net VRAM5: G2.129 (VRAM5)
- new net VRAM6: G2.130 (VRAM6)
- new net VRAM7: G2.131 (VRAM7)
- new net VRAM8: G2.132 (VRAM8)
- new net VRAM9: G2.134 (VRAM9)
- new net VSS: G2.1 (VSS), G2.114 (VSS), G2.115 (VSS), G2.133 (VSS), G2.172 (VSS), G2.190 (VSS), G2.191 (VSS), G2.209 (VSS), G2.210 (VSS), G2.231 (VSS), G2.234 (VSS), G2.237 (VSS), G2.257 (VSS), G2.276 (VSS), G2.296 (VSS), G2.299 (VSS), G2.3 (VSS), G2.302 (VSS), G2.304 (VSS), G2.38 (VSS), G2.68 (VSS), G2.71 (VSS), G2.74 (VSS), G2.76 (VSS), G2.77 (VSS), G2.79 (VSS), G2.82 (VSS), G2.85 (VSS), H1.1 (~{BE}), H1.12 (VSS), H2.1 (~{BE}), H2.12 (VSS), H3.1 (~{BE}), H3.12 (VSS), H4.1 (~{BE}), H4.12 (VSS)
- no-connect marks 0 -> 2
Other:
- note added: "?"
- note added: "Picture Processing Unit"

Commit message: ppu_ research
Parts:
- removed G2: DL-2729_PPU, symbol capcom:DL-2729_PPU
- added U?: DL-2729_PPU, symbol capcom:DL-2729_PPU
- gave numbers to parts that had none: 1
Connections:
- net PIN110 is gone; now on net PIN109: H5.47 (A1-1)
- net VCC: now also H5.18 (VCC), H5.31 (VCC), H5.42 (VCC), H5.7 (VCC), U?.152 (VCC)
- net VSS: now also H5.1 (~{OE}-1), H5.10 (VSS), H5.15 (VSS), H5.21 (VSS), H5.24 (~{OE}-4), H5.25 (~{OE}-3), H5.26 (A4-4), H5.27 (A4-3), H5.28 (VSS), H5.29 (A4-2), H5.30 (A4-1), H5.34 (VSS), H5.39 (VSS), H5.4 (VSS), H5.45 (VSS), H5.48 (~{OE}-2)
- net 114: now reaches H5.32 (A3-4)
- net 114: now also H5.33 (A3-3)
- net 113: now reaches H5.35 (A3-2)
- net 113: now also H5.36 (A3-1)
- net 112: now reaches H5.37 (A2-4)
- net 112: now also H5.38 (A2-3)
- net 111: now reaches H5.40 (A2-2)
- net 111: now also H5.41 (A2-1)
- net 110: now reaches H5.43 (A1-4)
- net 110: now also H5.44 (A1-3)
- net PIN109: now reaches H5.46 (A1-2)
- net A0 renamed SPRITE0
- net SPRITE0: now also U?.124 (SPRITE0)
- net A1 renamed SPRITE1
- net SPRITE1: now also U?.125 (SPRITE1)
- net A10 renamed SPRITE10
- net SPRITE10: now also U?.135 (SPRITE10)
- net A11 renamed SPRITE11
- net SPRITE11: now also U?.136 (SPRITE11)
- net A12 renamed SPRITE12
- net SPRITE12: now also U?.137 (SPRITE12)
- net A13 renamed SPRITE13
- net SPRITE13: now also U?.138 (SPRITE13)
- net A14 renamed SPRITE14
- net SPRITE14: now also U?.139 (SPRITE14)
- net A15 renamed SPRITE15
- net SPRITE15: now also U?.140 (SPRITE15)
- net A2 renamed SPRITE2
- net SPRITE2: now also U?.126 (SPRITE2)
- net A3 renamed SPRITE3
- net SPRITE3: now also U?.127 (SPRITE3)
- net A4 renamed SPRITE4
- net SPRITE4: now also U?.128 (SPRITE4)
- net A5 renamed SPRITE5
- net SPRITE5: now also U?.129 (SPRITE5)
- net A6 renamed SPRITE6
- net SPRITE6: now also U?.130 (SPRITE6)
- net A7 renamed SPRITE7
- net SPRITE7: now also U?.131 (SPRITE7)
- net A8 renamed SPRITE8
- net SPRITE8: now also U?.132 (SPRITE8)
- net A9 renamed SPRITE9
- net SPRITE9: now also U?.134 (SPRITE9)
- net RMAINA_D0 renamed SPRITEA_D0
- net RMAINA_D1 renamed SPRITEA_D1
- net RMAINA_D2 renamed SPRITEA_D2
- net RMAINA_D3 renamed SPRITEA_D3
- net RMAINA_D4 renamed SPRITEA_D4
- net RMAINA_D5 renamed SPRITEA_D5
- net RMAINA_D6 renamed SPRITEA_D6
- net RMAINA_D7 renamed SPRITEA_D7
- net RMAINB_D0 renamed SPRITEB_D0
- net RMAINB_D1 renamed SPRITEB_D1
- net RMAINB_D2 renamed SPRITEB_D2
- net RMAINB_D3 renamed SPRITEB_D3
- net RMAINB_D4 renamed SPRITEB_D4
- net RMAINB_D5 renamed SPRITEB_D5
- net RMAINB_D6 renamed SPRITEB_D6
- net RMAINB_D7 renamed SPRITEB_D7
- net RMAINC_D0 renamed SPRITEC_D0
- net RMAINC_D1 renamed SPRITEC_D1
- net RMAINC_D2 renamed SPRITEC_D2
- net RMAINC_D3 renamed SPRITEC_D3
- net RMAINC_D4 renamed SPRITEC_D4
- net RMAINC_D5 renamed SPRITEC_D5
- net RMAINC_D6 renamed SPRITEC_D6
- net RMAINC_D7 renamed SPRITEC_D7
- net RMAIND_D0 renamed SPRITED_D0
- net RMAIND_D1 renamed SPRITED_D1
- net RMAIND_D2 renamed SPRITED_D2
- net RMAIND_D3 renamed SPRITED_D3
- net RMAIND_D4 renamed SPRITED_D4
- net RMAIND_D5 renamed SPRITED_D5
- net RMAIND_D6 renamed SPRITED_D6
- net RMAIND_D7 renamed SPRITED_D7
Other:
- note added: "PRIORITY SPRITES"
- moved on the sheet: H1, H2, H3, H4, H5

Commit message: oam_sprite_ppu
Parts:
- removed U?: DL-2729_PPU, symbol capcom:DL-2729_PPU
- added H6, H9: 74FCT-16244ATPV, symbol arcade:74FCT-16244ATPV
- added U?: DL-2729_PPU, symbol capcom:DL-2729_PPU
Connections:
- net 114 is gone; now on net VSS: H5.32 (A3-4), H5.33 (A3-3)
- net SPRITE0: now also U?.124 (SPRITE0)
- net SPRITE1: now also U?.125 (SPRITE1)
- net SPRITE10: now also U?.135 (SPRITE10)
- net SPRITE11: now also U?.136 (SPRITE11)
- net SPRITE12: now also U?.137 (SPRITE12)
- net SPRITE13: now also U?.138 (SPRITE13)
- net SPRITE14: now also U?.139 (SPRITE14)
- net SPRITE15: now also U?.140 (SPRITE15)
- net SPRITE2: now also U?.126 (SPRITE2)
- net SPRITE3: now also U?.127 (SPRITE3)
- net SPRITE4: now also U?.128 (SPRITE4)
- net SPRITE5: now also U?.129 (SPRITE5)
- net SPRITE6: now also U?.130 (SPRITE6)
- net SPRITE7: now also U?.131 (SPRITE7)
- net SPRITE8: now also U?.132 (SPRITE8)
- net SPRITE9: now also U?.134 (SPRITE9)
- net VCC: now also H6.18 (VCC), H6.31 (VCC), H6.42 (VCC), H6.7 (VCC), H9.18 (VCC), H9.31 (VCC), H9.42 (VCC), H9.7 (VCC), U?.12 (VCC), U?.123 (VCC), U?.13 (VCC), U?.144 (VCC), U?.147 (VCC), U?.150 (VCC), U?.152 (VCC), U?.153 (VCC), U?.155 (VCC), U?.158 (VCC), U?.161 (VCC), U?.17 (VCC), U?.181 (VCC), U?.20 (VCC), U?.201 (VCC), U?.220 (VCC), U?.221 (VCC), U?.226 (VCC), U?.229 (VCC), U?.24 (VCC), U?.248 (VCC), U?.26 (VCC), U?.266 (VCC), U?.267 (VCC), U?.285 (VCC), U?.57 (VCC), U?.9 (VCC), U?.96 (VCC)
- net VSS: now also H6.10 (VSS), H6.15 (VSS), H6.21 (VSS), H6.28 (VSS), H6.34 (VSS), H6.39 (VSS), H6.4 (VSS), H6.45 (VSS), H9.10 (VSS), H9.15 (VSS), H9.21 (VSS), H9.28 (VSS), H9.34 (VSS), H9.39 (VSS), H9.4 (VSS), H9.45 (VSS), U?.1 (VSS), U?.114 (VSS), U?.115 (VSS), U?.133 (VSS), U?.172 (VSS), U?.190 (VSS), U?.191 (VSS), U?.209 (VSS), U?.210 (VSS), U?.231 (VSS), U?.234 (VSS), U?.237 (VSS), U?.257 (VSS), U?.276 (VSS), U?.296 (VSS), U?.299 (VSS), U?.3 (VSS), U?.302 (VSS), U?.304 (VSS), U?.38 (VSS), U?.68 (VSS), U?.71 (VSS), U?.74 (VSS), U?.76 (VSS), U?.77 (VSS), U?.79 (VSS), U?.82 (VSS), U?.85 (VSS)
- net OAM_A19: now reaches H5.11 (Y2-3)
- net OAMB_A19: now reaches H5.12 (Y2-4)
- net OAM_A20: now reaches H5.13 (Y3-1)
- net OAMB_A20: now reaches H5.14 (Y3-2)
- net OAM_A16: now reaches H5.2 (Y1-1)
- net OAMB_A16: now reaches H5.3 (Y1-2)
- net OAM_A17: now reaches H5.5 (Y1-3)
- net OAMB_A17: now reaches H5.6 (Y1-4)
- net OAM_A18: now reaches H5.8 (Y2-1)
- net OAMB_A18: now reaches H5.9 (Y2-2)
- net 110 renamed PPU17
- net PPU17: now also U?.110 (PPU17)
- net 111 renamed PPU18
- net PPU18: now also U?.111 (PPU18)
- net 112 renamed PPU19
- net PPU19: now also U?.112 (PPU19)
- net 113 renamed PPU20
- net PPU20: now also U?.113 (PPU20)
- net PIN109 renamed PPU16
- net PPU16: now also U?.109 (PPU16)
- new net OAMB_A0: H9.3 (Y1-2)
- new net OAMB_A1: H9.6 (Y1-4)
- new net OAMB_A10: H6.9 (Y2-2)
- new net OAMB_A11: H6.12 (Y2-4)
- new net OAMB_A12: H6.14 (Y3-2)
- new net OAMB_A13: H6.17 (Y3-4)
- new net OAMB_A14: H6.20 (Y4-2)
- new net OAMB_A15: H6.23 (Y4-4)
- new net OAMB_A2: H9.9 (Y2-2)
- new net OAMB_A3: H9.12 (Y2-4)
- new net OAMB_A4: H9.14 (Y3-2)
- new net OAMB_A5: H9.17 (Y3-4)
- new net OAMB_A6: H9.20 (Y4-2)
- new net OAMB_A7: H9.23 (Y4-4)
- new net OAMB_A8: H6.3 (Y1-2)
- new net OAMB_A9: H6.6 (Y1-4)
- new net OAM_A0: H9.2 (Y1-1)
- new net OAM_A1: H9.5 (Y1-3)
- new net OAM_A10: H6.8 (Y2-1)
- new net OAM_A11: H6.11 (Y2-3)
- new net OAM_A12: H6.13 (Y3-1)
- new net OAM_A13: H6.16 (Y3-3)
- new net OAM_A14: H6.19 (Y4-1)
- new net OAM_A15: H6.22 (Y4-3)
- new net OAM_A2: H9.8 (Y2-1)
- new net OAM_A3: H9.11 (Y2-3)
- new net OAM_A4: H9.13 (Y3-1)
- new net OAM_A5: H9.16 (Y3-3)
- new net OAM_A6: H9.19 (Y4-1)
- new net OAM_A7: H9.22 (Y4-3)
- new net OAM_A8: H6.2 (Y1-1)
- new net OAM_A9: H6.5 (Y1-3)
- new net PPU0: H9.46 (A1-2), H9.47 (A1-1), U?.92 (PPU0)
- new net PPU1: H9.43 (A1-4), H9.44 (A1-3), U?.93 (PPU1)
- new net PPU10: H6.40 (A2-2), H6.41 (A2-1), U?.103 (PPU10)
- new net PPU11: H6.37 (A2-4), H6.38 (A2-3), U?.104 (PPU11)
- new net PPU12: H6.35 (A3-2), H6.36 (A3-1), U?.105 (PPU12)
- new net PPU13: H6.32 (A3-4), H6.33 (A3-3), U?.106 (PPU13)
- new net PPU14: H6.29 (A4-2), H6.30 (A4-1), U?.107 (PPU14)
- new net PPU15: H6.26 (A4-4), H6.27 (A4-3), U?.108 (PPU15)
- new net PPU2: H9.40 (A2-2), H9.41 (A2-1), U?.94 (PPU2)
- new net PPU3: H9.37 (A2-4), H9.38 (A2-3), U?.95 (PPU3)
- new net PPU4: H9.35 (A3-2), H9.36 (A3-1), U?.97 (PPU4)
- new net PPU5: H9.32 (A3-4), H9.33 (A3-3), U?.98 (PPU5)
- new net PPU6: H9.29 (A4-2), H9.30 (A4-1), U?.99 (PPU6)
- new net PPU7: H9.26 (A4-4), H9.27 (A4-3), U?.100 (PPU7)
- new net PPU8: H6.46 (A1-2), H6.47 (A1-1), U?.101 (PPU8)
- new net PPU9: H6.43 (A1-4), H6.44 (A1-3), U?.102 (PPU9)
- no-connect marks 2 -> 8
Other:
- note added: "Object Attribute Memory?"
- note added: "counters and shift registers.?"
- moved on the sheet: H1, H2, H3, H4, H5

Commit message: modification in progress_ppu
Parts:
- removed U?: DL-2729_PPU, symbol capcom:DL-2729_PPU
- added R63, R74, R75: 110Ω, symbol Device:R_US
- added U?: DL-2729_PPU, symbol capcom:DL-2729_PPU
- added X1, X2: 7100A OSC 9640, Oscillator:Oscillator_SMD_Abracon_ASDMB-4Pin_2.5x2.0mm, symbol Oscillator:ASDMB-xxxMHz
Connections:
- net PPU0: now also U?.92 (PPU0)
- net PPU1: now also U?.93 (PPU1)
- net PPU10: now also U?.103 (PPU10)
- net PPU11: now also U?.104 (PPU11)
- net PPU12: now also U?.105 (PPU12)
- net PPU13: now also U?.106 (PPU13)
- net PPU14: now also U?.107 (PPU14)
- net PPU15: now also U?.108 (PPU15)
- net PPU16: now also U?.109 (PPU16)
- net PPU17: now also U?.110 (PPU17)
- net PPU18: now also U?.111 (PPU18)
- net PPU19: now also U?.112 (PPU19)
- net PPU2: now also U?.94 (PPU2)
- net PPU20: now also U?.113 (PPU20)
- net PPU3: now also U?.95 (PPU3)
- net PPU4: now also U?.97 (PPU4)
- net PPU5: now also U?.98 (PPU5)
- net PPU6: now also U?.99 (PPU6)
- net PPU7: now also U?.100 (PPU7)
- net PPU8: now also U?.101 (PPU8)
- net PPU9: now also U?.102 (PPU9)
- net SPRITE0: now also U?.124 (SPRITE0)
- net SPRITE1: now also U?.125 (SPRITE1)
- net SPRITE10: now also U?.135 (SPRITE10)
- net SPRITE11: now also U?.136 (SPRITE11)
- net SPRITE12: now also U?.137 (SPRITE12)
- net SPRITE13: now also U?.138 (SPRITE13)
- net SPRITE14: now also U?.139 (SPRITE14)
- net SPRITE15: now also U?.140 (SPRITE15)
- net SPRITE2: now also U?.126 (SPRITE2)
- net SPRITE3: now also U?.127 (SPRITE3)
- net SPRITE4: now also U?.128 (SPRITE4)
- net SPRITE5: now also U?.129 (SPRITE5)
- net SPRITE6: now also U?.130 (SPRITE6)
- net SPRITE7: now also U?.131 (SPRITE7)
- net SPRITE8: now also U?.132 (SPRITE8)
- net SPRITE9: now also U?.134 (SPRITE9)
- net VCC: now also U?.12 (VCC), U?.123 (VCC), U?.13 (VCC), U?.144 (VCC), U?.147 (VCC), U?.150 (VCC), U?.152 (VCC), U?.153 (VCC), U?.155 (VCC), U?.158 (VCC), U?.161 (VCC), U?.17 (VCC), U?.181 (VCC), U?.20 (VCC), U?.201 (VCC), U?.220 (VCC), U?.221 (VCC), U?.226 (VCC), U?.229 (VCC), U?.24 (VCC), U?.248 (VCC), U?.26 (VCC), U?.266 (VCC), U?.267 (VCC), U?.285 (VCC), U?.57 (VCC), U?.9 (VCC), U?.96 (VCC), X1.4 (VDD), X2.4 (VDD)
- net VSS: now also H6.1 (~{OE}-1), H6.24 (~{OE}-4), H6.25 (~{OE}-3), H6.48 (~{OE}-2), H9.1 (~{OE}-1), H9.24 (~{OE}-4), H9.25 (~{OE}-3), H9.48 (~{OE}-2), U?.1 (VSS), U?.114 (VSS), U?.115 (VSS), U?.133 (VSS), U?.172 (VSS), U?.190 (VSS), U?.191 (VSS), U?.209 (VSS), U?.210 (VSS), U?.231 (VSS), U?.234 (VSS), U?.237 (VSS), U?.257 (VSS), U?.276 (VSS), U?.296 (VSS), U?.299 (VSS), U?.3 (VSS), U?.302 (VSS), U?.304 (VSS), U?.38 (VSS), U?.68 (VSS), U?.71 (VSS), U?.74 (VSS), U?.76 (VSS), U?.77 (VSS), U?.79 (VSS), U?.82 (VSS), U?.85 (VSS), X1.2 (GND), X2.2 (GND)
- new net: R74.2, R75.2, X2.3 (Out)
- new net: R63.1, U?.18 (CLK)
- new net: R63.2, X1.3 (Out)
- new net: R74.1, U?.19 (CLK)
- new net 128 DL 3329: R75.1
- no-connect marks 8 -> 10
Other:
- note added: "42.9545MHz"
- note added: "60.000MHz"

Commit message: ppu_d0-a0
Parts:
- removed U?: DL-2729_PPU, symbol capcom:DL-2729_PPU
- added U? (x4): HM5118160AJ, symbol oki:HM5118160AJ
- added U?: DL-2729_PPU, symbol capcom:DL-2729_PPU
Connections:
- net PPU0: now also U?.92 (PPU0)
- net PPU1: now also U?.93 (PPU1)
- net PPU10: now also U?.103 (PPU10)
- net PPU11: now also U?.104 (PPU11)
- net PPU12: now also U?.105 (PPU12)
- net PPU13: now also U?.106 (PPU13)
- net PPU14: now also U?.107 (PPU14)
- net PPU15: now also U?.108 (PPU15)
- net PPU16: now also U?.109 (PPU16)
- net PPU17: now also U?.110 (PPU17)
- net PPU18: now also U?.111 (PPU18)
- net PPU19: now also U?.112 (PPU19)
- net PPU2: now also U?.94 (PPU2)
- net PPU20: now also U?.113 (PPU20)
- net PPU3: now also U?.95 (PPU3)
- net PPU4: now also U?.97 (PPU4)
- net PPU5: now also U?.98 (PPU5)
- net PPU6: now also U?.99 (PPU6)
- net PPU7: now also U?.100 (PPU7)
- net PPU8: now also U?.101 (PPU8)
- net PPU9: now also U?.102 (PPU9)
- net SPRITE0: now also U?.124 (SPRITE0)
- net SPRITE1: now also U?.125 (SPRITE1)
- net SPRITE10: now also U?.135 (SPRITE10)
- net SPRITE11: now also U?.136 (SPRITE11)
- net SPRITE12: now also U?.137 (SPRITE12)
- net SPRITE13: now also U?.138 (SPRITE13)
- net SPRITE14: now also U?.139 (SPRITE14)
- net SPRITE15: now also U?.140 (SPRITE15)
- net SPRITE2: now also U?.126 (SPRITE2)
- net SPRITE3: now also U?.127 (SPRITE3)
- net SPRITE4: now also U?.128 (SPRITE4)
- net SPRITE5: now also U?.129 (SPRITE5)
- net SPRITE6: now also U?.130 (SPRITE6)
- net SPRITE7: now also U?.131 (SPRITE7)
- net SPRITE8: now also U?.132 (SPRITE8)
- net SPRITE9: now also U?.134 (SPRITE9)
- net VCC: now also U?.12 (VCC), U?.123 (VCC), U?.13 (VCC), U?.144 (VCC), U?.147 (VCC), U?.150 (VCC), U?.152 (VCC), U?.153 (VCC), U?.155 (VCC), U?.158 (VCC), U?.161 (VCC), U?.17 (VCC), U?.181 (VCC), U?.20 (VCC), U?.201 (VCC), U?.220 (VCC), U?.221 (VCC), U?.226 (VCC), U?.229 (VCC), U?.24 (VCC), U?.248 (VCC), U?.26 (VCC), U?.266 (VCC), U?.267 (VCC), U?.285 (VCC), U?.57 (VCC), U?.9 (VCC), U?.96 (VCC)
- net VSS: now also U?.1 (VSS), U?.114 (VSS), U?.115 (VSS), U?.133 (VSS), U?.16 (UK), U?.172 (VSS), U?.190 (VSS), U?.191 (VSS), U?.209 (VSS), U?.210 (VSS), U?.231 (VSS), U?.234 (VSS), U?.237 (VSS), U?.257 (VSS), U?.276 (VSS), U?.296 (VSS), U?.299 (VSS), U?.3 (VSS), U?.302 (VSS), U?.38 (VSS), U?.6 (VSS), U?.68 (VSS), U?.71 (VSS), U?.74 (VSS), U?.76 (VSS), U?.77 (VSS), U?.79 (VSS), U?.82 (VSS), U?.85 (VSS)
- net at R63.1: now also U?.28 (UK)
- net at R74.1: now also U?.29 (UK)
- new net PPU_A0: U?.17 (A0), U?.17 (A0), U?.17 (A0), U?.17 (A0), U?.260 (A0)
- new net PPU_A1: U?.18 (A1), U?.18 (A1), U?.18 (A1), U?.18 (A1), U?.261 (A1)
- new net PPU_A2: U?.19 (A2), U?.19 (A2), U?.19 (A2), U?.19 (A2), U?.262 (A2)
- new net PPU_A3: U?.20 (A3), U?.20 (A3), U?.20 (A3), U?.20 (A3), U?.263 (A3)
- new net PPU_A4: U?.23 (A4), U?.23 (A4), U?.23 (A4), U?.23 (A4), U?.264 (A4)
- new net PPU_A5: U?.24 (A5), U?.24 (A5), U?.24 (A5), U?.24 (A5), U?.265 (A5)
- new net PPU_A6: U?.25 (A6), U?.25 (A6), U?.25 (A6), U?.25 (A6), U?.268 (A6)
- new net PPU_A7: U?.26 (A7), U?.26 (A7), U?.26 (A7), U?.26 (A7), U?.269 (A7)
- new net PPU_A8: U?.27 (A8), U?.27 (A8), U?.27 (A8), U?.27 (A8), U?.270 (A8)
- new net PPU_A9: U?.271 (A9), U?.28 (A9), U?.28 (A9), U?.28 (A9), U?.28 (A9)
- new net PPU_D0: U?.2 (D0), U?.2 (D0), U?.274 (D0)
- new net PPU_D1: U?.275 (D1), U?.3 (D1), U?.3 (D1)
- new net PPU_D10: U?.286 (D10), U?.35 (D10), U?.35 (D10)
- new net PPU_D11: U?.287 (D11), U?.36 (D11), U?.36 (D11)
- new net PPU_D12: U?.288 (D12), U?.38 (D12), U?.38 (D12)
- new net PPU_D13: U?.289 (D13), U?.39 (D13), U?.39 (D13)
- new net PPU_D14: U?.290 (D14), U?.40 (D14), U?.40 (D14)
- new net PPU_D15: U?.291 (D15), U?.41 (D15), U?.41 (D15)
- new net PPU_D16: U?.2 (D0), U?.2 (D0), U?.292 (D16)
- new net PPU_D17: U?.293 (D17), U?.3 (D1), U?.3 (D1)
- new net PPU_D18: U?.294 (D18), U?.4 (D2), U?.4 (D2)
- new net PPU_D19: U?.295 (D19), U?.5 (D3), U?.5 (D3)
- new net PPU_D2: U?.277 (D2), U?.4 (D2), U?.4 (D2)
- new net PPU_D20: U?.297 (D20), U?.7 (D4), U?.7 (D4)
- new net PPU_D21: U?.298 (D21), U?.8 (D5), U?.8 (D5)
- new net PPU_D22: U?.300 (D22), U?.9 (D6), U?.9 (D6)
- new net PPU_D23: U?.10 (D7), U?.10 (D7), U?.301 (D23)
- new net PPU_D24: U?.303 (D24), U?.33 (D8), U?.33 (D8)
- new net PPU_D25: U?.2 (D25), U?.34 (D9), U?.34 (D9)
- new net PPU_D26: U?.35 (D10), U?.35 (D10), U?.4 (D26)
- new net PPU_D27: U?.36 (D11), U?.36 (D11), U?.5 (D27)
- new net PPU_D28: U?.38 (D12), U?.38 (D12), U?.7 (D28)
- new net PPU_D29: U?.39 (D13), U?.39 (D13), U?.8 (D29)
- new net PPU_D3: U?.278 (D3), U?.5 (D3), U?.5 (D3)
- new net PPU_D30: U?.10 (D30), U?.40 (D14), U?.40 (D14)
- new net PPU_D31: U?.11 (D31), U?.41 (D15), U?.41 (D15)
- new net PPU_D4: U?.279 (D4), U?.7 (D4), U?.7 (D4)
- new net PPU_D5: U?.280 (D5), U?.8 (D5), U?.8 (D5)
- new net PPU_D6: U?.281 (D6), U?.9 (D6), U?.9 (D6)
- new net PPU_D7: U?.10 (D7), U?.10 (D7), U?.282 (D7)
- new net PPU_D8: U?.283 (D8), U?.33 (D8), U?.33 (D8)
- new net PPU_D9: U?.284 (D9), U?.34 (D9), U?.34 (D9)
Other:
- note added: "291...274"
- moved on the sheet: H1, H2, H3, H4, H5, H6, H9, R63, R74, R75, X1, X2
