File: cores/cps3/sch/gfx.kicad_sch (KiCad schematic)
At the start: 26 parts, among them X1 7100A OSC 9640, X2 7100A OSC 9640

Commit message: main_obj
Parts:
- removed 2D, 3D, 4D, 5D: HM5118160AJ, symbol oki:HM5118160AJ
- added U?: PS6406B_9808OAFB, symbol arcade:PS6406B_9808OAFB
- gave numbers to parts that had none: 1
- renumbered RN9 to RN8, RN8 to RN9
Connections:
- net OE_A: now also RN14.8 (R1.2)
- net OE_B: now also RN14.7 (R2.2)
- net PPU_A0: now also RN12.5 (R4.2); no longer U?.260 (A0)
- net PPU_A1: now also RN12.6 (R3.2); no longer U?.261 (A1)
- net PPU_A2: now also RN12.7 (R2.2); no longer U?.262 (A2)
- net PPU_A3: now also RN12.8 (R1.2); no longer U?.263 (A3)
- net PPU_A4: now also RN13.5 (R4.2); no longer U?.264 (A4)
- net PPU_A5: now also RN13.6 (R3.2); no longer U?.265 (A5)
- net PPU_A6: now also RN13.7 (R2.2); no longer U?.268 (A6)
- net PPU_A7: now also RN13.8 (R1.2); no longer U?.269 (A7)
- net VCC: now also D1.1 (VCC), D1.20 (VCC), D1.6 (VCC)
- net VSS: now also D1.21 (VSS), D1.35 (VSS), D1.40 (VSS)
- net ~{LCAS}_A: now also RN11.5 (R4.2); no longer RN11.1 (R1.1)
- net ~{LCAS}_B: now also RN10.5 (R4.2); no longer RN10.1 (R1.1)
- net ~{LCAS}_C: now also RN11.7 (R2.2); no longer RN11.3 (R3.1)
- net ~{LCAS}_D: now also RN10.7 (R2.2); no longer RN10.3 (R3.1)
- net ~{UCAS}_A: now also RN11.6 (R3.2); no longer RN11.2 (R2.1)
- net ~{UCAS}_B: now also RN10.6 (R3.2); no longer RN10.2 (R2.1)
- net ~{UCAS}_C: now also RN11.8 (R1.2); no longer RN11.4 (R4.1)
- net ~{UCAS}_D: now also RN10.8 (R1.2); no longer RN10.4 (R4.1)
- net ~{WE}_A: now also RN14.6 (R3.2)
- net ~{WE}_B: now also RN14.5 (R4.2)
- net at RN12.1 (R1.1): now also U?.263 (A3)
- net at RN12.2 (R2.1): now also U?.262 (A2)
- net at RN12.3 (R3.1): now also U?.261 (A1)
- net at RN12.4 (R4.1): now also U?.260 (A0)
- net at RN13.1 (R1.1): now also U?.269 (A7)
- net at RN13.2 (R2.1): now also U?.268 (A6)
- net at RN13.3 (R3.1): now also U?.265 (A5)
- net at RN13.4 (R4.1): now also U?.264 (A4)
- net at RN8.1 (R1.1): now also U?.197 (RAMA4); no longer D1.22 (A4)
- net at RN8.2 (R2.1): now also U?.198 (RAMA5); no longer D1.23 (A5)
- net at RN8.3 (R3.1): now also U?.199 (RAMA6); no longer D1.24 (A6)
- net at RN8.4 (R4.1): now also U?.200 (RAMA7); no longer D1.25 (A7)
- net at RN8.5 (R4.2): now also D1.25 (A7)
- net at RN8.6 (R3.2): now also D1.24 (A6)
- net at RN8.7 (R2.2): now also D1.23 (A5)
- net at RN8.8 (R1.2): now also D1.22 (A4)
- net at RN9.1 (R1.1): now also U?.193 (RAMA0); no longer D1.16 (A0)
- net at RN9.2 (R2.1): now also U?.194 (RAMA1); no longer D1.17 (A1)
- net at RN9.3 (R3.1): now also U?.195 (RAMA2); no longer D1.18 (A2)
- net at RN9.4 (R4.1): now also U?.196 (RAMA3); no longer D1.19 (A3)
- net at RN9.5 (R4.2): now also D1.19 (A3)
- net at RN9.6 (R3.2): now also D1.18 (A2)
- net at RN9.7 (R2.2): now also D1.17 (A1)
- net at RN9.8 (R1.2): now also D1.16 (A0)
- net RAMD0: now reaches U?.207 (RAMD0)
- net RAMD0: now also D1.2 (D0)
- net RAMD1: now reaches U?.208 (RAMD1)
- net RAMD1: now also D1.3 (D1)
- net RAMD2: now reaches U?.211 (RAMD2)
- net RAMD2: now also D1.4 (D2)
- net RAMD3: now reaches U?.212 (RAMD3)
- net RAMD3: now also D1.5 (D3)
- net RAMD4: now reaches U?.213 (RAMD4)
- net RAMD4: now also D1.7 (D4)
- net RAMD5: now reaches U?.214 (RAMD5)
- net RAMD5: now also D1.8 (D5)
- net RAMD6: now reaches U?.215 (RAMD6)
- net RAMD6: now also D1.9 (D6)
- net RAMD7: now reaches U?.216 (RAMD7)
- net RAMD7: now also D1.10 (D7)
- net RAMD8: now reaches U?.217 (RAMD8)
- net RAMD8: now also D1.31 (D8)
- net RAMD9: now reaches U?.218 (RAMD9)
- net RAMD9: now also D1.32 (D9)
- net RAMD10: now reaches U?.219 (RAMD10)
- net RAMD10: now also D1.33 (D10)
- net RAMD11: now reaches U?.222 (RAMD11)
- net RAMD11: now also D1.34 (D11)
- net RAMD12: now reaches U?.223 (RAMD12)
- net RAMD12: now also D1.36 (D12)
- net RAMD13: now reaches U?.224 (RAMD13)
- net RAMD13: now also D1.37 (D13)
- net RAMD14: now reaches U?.225 (RAMD14)
- net RAMD14: now also D1.38 (D14)
- net RAMD15: now reaches U?.227 (RAMD15)
- net RAMD15: now also D1.39 (D15)
- net at U?.232 (~{LCAS}_B): now also RN10.4 (R4.1); no longer RN10.8 (R1.2)
- net at U?.233 (~{UCAS}_B): now also RN10.3 (R3.1); no longer RN10.7 (R2.2)
- net at U?.235 (~{LCAS}_D): now also RN10.2 (R2.1); no longer RN10.6 (R3.2)
- net at U?.236 (~{UCAS}_D): now also RN10.1 (R1.1); no longer RN10.5 (R4.2)
- net at U?.238 (~{WE}_B): now also RN14.4 (R4.1)
- net at U?.239 (OE_B): now also RN14.2 (R2.1)
- net at U?.240 (~{LCAS}_A): now also RN11.3 (R3.1); no longer RN11.8 (R1.2)
- net at U?.241 (~{UCAS}_A): now also RN11.4 (R4.1); no longer RN11.7 (R2.2)
- net at U?.242 (~{LCAS}_C): now also RN11.2 (R2.1); no longer RN11.6 (R3.2)
- net at U?.243 (~{UCAS}_C): now also RN11.1 (R1.1); no longer RN11.5 (R4.2)
- net at U?.244 (~{WE}_A): now also RN14.3 (R3.1)
- net at U?.245 (OE_A): now also RN14.1 (R1.1)
- no-connect marks 10 -> 11
Other:
- sheet memories renamed memories_main
- sheet memories_main: file memories.kicad_sch -> memories_main.kicad_sch
- sheet memories_main ports: added OE_A, OE_B, PPU_A[9..0], PPU_D[0..31], ~{LCAS}_A, ~{LCAS}_B, ~{LCAS}_C, ~{LCAS}_D, ~{RAS}, ~{UCAS}_A, ~{UCAS}_B, ~{UCAS}_C, ~{UCAS}_D, ~{WE}_A, ~{WE}_B; removed none
- note added: "RAM DE VIDEO D0?"
- moved on the sheet: D1, H1, H2, H3, H4, H5, H6, H9, R63, R74, R75, RN10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

Commit message: ppu in process
Connections:
- net VSS: now also D1.27 (~{OE})
- net 36: now reaches U?.148 (UK)
- net 35: now reaches U?.149 (UK)
- net 34: now reaches U?.151 (UK)
- net 33: now reaches U?.154 (UK)
- net 32: now reaches U?.156 (UK)
- net 31: now reaches U?.157 (UK)
- net 29: now reaches U?.160 (UK)
- net 28: now reaches U?.162 (UK)
- net 27: now reaches U?.163 (UK)
- net 26: now reaches U?.164 (UK)
- net 25: now reaches U?.165 (UK)
- net 24: now reaches U?.166 (UK)
- net 23: now reaches U?.167 (UK)
- net 22: now reaches U?.168 (UK)
- net 21: now reaches U?.169 (UK)
- net 20: now reaches U?.170 (UK)
- net ~{RAS}: now reaches U?.203 (UK)
- net ~{RAS}: now also D1.14 (~{RAS})
- net ~{LCAS}: now reaches U?.204 (UK)
- net ~{LCAS}: now also D1.29 (~{LCAS})
- net ~{UCAS}: now reaches U?.205 (UK)
- net ~{UCAS}: now also D1.28 (~{UCAS})
- net ~{WE}: now reaches U?.206 (UK)
- net ~{WE}: now also D1.13 (~{WE})
- net ~{RAS}_MAIN: now reaches U?.230 (UK)

Commit message: ppu_in-process
Parts:
- added H? (x4): CU383-69K, symbol arcade:CU383-69K
- added U1, U? (x4): 74LS08, symbol jt74:74LS08
Connections:
- net VCC: now also U?.14 (VCC)
- net VSS: now also U?.228 (UK), U?.304 (VSS), H?.13 (BX), U?.7 (VSS)
- net BX_SPR: now reaches H4.13 (BX)
- net BX_SPR: now also H1.13 (BX), H2.13 (BX), H3.13 (BX)
- net at R63.1: now also U?.18 (CLK); no longer U?.28 (UK)
- net 70_GLL2: now reaches U?.116 (UK)
- net 69: now reaches U?.117 (UK)
- net 68: now reaches U?.118 (UK)
- net 67: now reaches U?.119 (UK)
- net 66: now reaches U?.120 (UK)
- net 71: now reaches U?.121 (UK)
- net B1-2: now reaches U?.14 (UK)
- net B1-2: now also H?.5 (B1-2)
- net A1-2: now reaches U?.15 (UK)
- net A1-2: now also H?.4 (A1-2)
- net at U?.19 (CLK): now also R74.1
- net BX_SND: now reaches U?.21 (UK)
- net BX_SND: now also H?.13 (BX), H?.13 (BX), H?.13 (BX)
- net 133_GLL: now reaches U?.23 (UK)
- net at U?.29 (UK): now also U1.1; no longer R74.1
- net 131_GLL: now reaches U?.31 (UK)
- net 132_GLL: now reaches U?.32 (UK)
- net 137_GLL: now reaches U?.33 (UK)
- net 32_GLL: now reaches U?.34 (UK)
- net 67_GLL: now reaches U?.35 (UK)
- net 30_GLL: now reaches U?.36 (UK)
- net 29_GLL: now reaches U?.37 (UK)
- net 3_SSU: now reaches U?.42 (UK)
- net 2_SSU: now reaches U?.43 (UK)
- net 1_SSU: now reaches U?.44 (UK)
- net 144_SSU: now reaches U?.45 (UK)
- net 143_SSU: now reaches U?.46 (UK)
- net 142_SSU: now reaches U?.47 (UK)
- net 141_SSU: now reaches U?.48 (UK)
- net 140_SSU: now reaches U?.49 (UK)
- net 139_SSU: now reaches U?.50 (UK)
- net 138_SSU: now reaches U?.51 (UK)
- net 137_SSU: now reaches U?.52 (UK)
- net 136_SSU: now reaches U?.53 (UK)
- net 135_SSU: now reaches U?.54 (UK)
- net 134_SSU: now reaches U?.55 (UK)
- net 133_SSU: now reaches U?.56 (UK)
- net 132_SSU: now reaches U?.58 (UK)
- net 131_SSU: now reaches U?.59 (UK)
- net 7_GLL: now reaches U?.60 (UK)
- net 6: now reaches U?.61 (UK)
- net 43: now reaches U?.64 (UK)
- net 42: now reaches U?.65 (UK)
- net 10_SSU: now reaches U?.66 (UK)
- net 9_SSU: now reaches U?.67 (UK)
- net 8_SSU: now reaches U?.69 (UK)
- net 7_SSU: now reaches U?.70 (UK)
- net 6_SSU: now reaches U?.72 (UK)
- net 20_33c93: now reaches U?.73 (UK)
- net 43_GLL: now reaches U?.75 (UK)
- net 27_33c93: now reaches U?.78 (UK)
- net 36_GLL: now reaches U?.86 (UK)
- net 35_GLL: now reaches U?.87 (UK)
- new net: U1.2, U?.28 (UK)
- new net 34_GLL: U?.39 (UK)
- no-connect marks 11 -> 66
Other:
- note added: "SSU"
- moved on the sheet: R63, R74, R75, X1, X2
