File: cores/cps3/sch/memories_main.kicad_sch (KiCad schematic)
At the start: 32 parts

Commit message: ppu_ research
Parts:
- renumbered JA8 to JA?, JB5 to JB?, JB3 to JB?, JB4 to JB?, JB2 to JB?, JB7 to JB?, JB6 to JB?, JB1 to JB?, JC5 to JC?, JC8 to JC?, JC7 to JC?, JC2 to JC?, JC1 to JC?, JC4 to JC?, JC3 to JC?, JC6 to JC?, JD7 to JD?, JD8 to JD?, JD3 to JD?, JD1 to JD?, JD4 to JD?, JD6 to JD?, JD5 to JD?, JD2 to JD?, JE1 to JE?, JE2 to JE?, JE8 to JE?, JE5 to JE?, JE3 to JE?, JE7 to JE?, JE6 to JE?, JE4 to JE?
Other:
- added sheet plane_color (plane_color.kicad_sch)
- note added: "The pattern table"
- note added: "first plane controls bit 0 of the color"

Commit message: oam_sprite_ppu
Parts:
- removed JA?, JB? (x7), JC? (x8), JD? (x8), JE? (x8): 29F016-90PFTN, symbol arcade:29F016-90PFTN
- added KA10, KA12, KA13, KA14, KB10, KB12, KB13, KB14: 29F016-90PFTN, symbol arcade:29F016-90PFTN
Connections:
- net VCC: now also KA10.12 (VCC), KA10.37 (VCC), KA12.12 (VCC), KA12.37 (VCC), KA13.12 (VCC), KA13.37 (VCC), KA14.12 (VCC), KA14.37 (VCC), KB10.12 (VCC), KB10.37 (VCC), KB12.12 (VCC), KB12.37 (VCC), KB13.12 (VCC), KB13.37 (VCC), KB14.12 (VCC), KB14.37 (VCC)
- net VSS: now also KA10.35 (VSS), KA10.36 (VSS), KA10.42 (RY/~{BY}), KA12.35 (VSS), KA12.36 (VSS), KA12.42 (RY/~{BY}), KA13.35 (VSS), KA13.36 (VSS), KA13.42 (RY/~{BY}), KA14.35 (VSS), KA14.36 (VSS), KA14.42 (RY/~{BY}), KB10.35 (VSS), KB10.36 (VSS), KB10.42 (RY/~{BY}), KB12.35 (VSS), KB12.36 (VSS), KB12.42 (RY/~{BY}), KB13.35 (VSS), KB13.36 (VSS), KB13.42 (RY/~{BY}), KB14.35 (VSS), KB14.36 (VSS), KB14.42 (RY/~{BY})
- new net: KA12., KA12.23 (NC)
- new net: KA10., KA10.23 (NC)
- new net: KB12., KB12.23 (NC)
- new net: KB14., KB14.23 (NC)
- new net: KB10., KB10.23 (NC)
- new net: KA13., KA13.23 (NC)
- new net: KB13., KB13.23 (NC)
- new net: KA14., KA14.23 (NC)
- new net GFXA_D0: KA10.31 (D0), KB10.31 (D0)
- new net GFXA_D1: KA10.32 (D1), KB10.32 (D1)
- new net GFXA_D2: KA10.33 (D2), KB10.33 (D2)
- new net GFXA_D3: KA10.34 (D3), KB10.34 (D3)
- new net GFXA_D4: KA10.38 (D4), KB10.38 (D4)
- new net GFXA_D5: KA10.39 (D5), KB10.39 (D5)
- new net GFXA_D6: KA10.40 (D6), KB10.40 (D6)
- new net GFXA_D7: KA10.41 (D7), KB10.41 (D7)
- new net GFXB_D0: KA12.31 (D0), KB12.31 (D0)
- new net GFXB_D1: KA12.32 (D1), KB12.32 (D1)
- new net GFXB_D2: KA12.33 (D2), KB12.33 (D2)
- new net GFXB_D3: KA12.34 (D3), KB12.34 (D3)
- new net GFXB_D4: KA12.38 (D4), KB12.38 (D4)
- new net GFXB_D5: KA12.39 (D5), KB12.39 (D5)
- new net GFXB_D6: KA12.40 (D6), KB12.40 (D6)
- new net GFXB_D7: KA12.41 (D7), KB12.41 (D7)
- new net GFXC_D0: KA13.31 (D0), KB13.31 (D0)
- new net GFXC_D1: KA13.32 (D1), KB13.32 (D1)
- new net GFXC_D2: KA13.33 (D2), KB13.33 (D2)
- new net GFXC_D3: KA13.34 (D3), KB13.34 (D3)
- new net GFXC_D4: KA13.38 (D4), KB13.38 (D4)
- new net GFXC_D5: KA13.39 (D5), KB13.39 (D5)
- new net GFXC_D6: KA13.40 (D6), KB13.40 (D6)
- new net GFXC_D7: KA13.41 (D7), KB13.41 (D7)
- new net GFXD_D0: KA14.31 (D0), KB14.31 (D0)
- new net GFXD_D1: KA14.32 (D1), KB14.32 (D1)
- new net GFXD_D2: KA14.33 (D2), KB14.33 (D2)
- new net GFXD_D3: KA14.34 (D3), KB14.34 (D3)
- new net GFXD_D4: KA14.38 (D4), KB14.38 (D4)
- new net GFXD_D5: KA14.39 (D5), KB14.39 (D5)
- new net GFXD_D6: KA14.40 (D6), KB14.40 (D6)
- new net GFXD_D7: KA14.41 (D7), KB14.41 (D7)
- new net GFX_A0: KA10.30 (A0), KA12.30 (A0), KA13.30 (A0), KA14.30 (A0), KB10.30 (A0), KB12.30 (A0), KB13.30 (A0), KB14.30 (A0)
- new net GFX_A1: KA10.29 (A1), KA12.29 (A1), KA13.29 (A1), KA14.29 (A1), KB10.29 (A1), KB12.29 (A1), KB13.29 (A1), KB14.29 (A1)
- new net GFX_A10: KA10.16 (A10), KA12.16 (A10), KA13.16 (A10), KA14.16 (A10), KB10.16 (A10), KB12.16 (A10), KB13.16 (A10), KB14.16 (A10)
- new net GFX_A11: KA10.15 (A11), KA12.15 (A11), KA13.15 (A11), KA14.15 (A11), KB10.15 (A11), KB12.15 (A11), KB13.15 (A11), KB14.15 (A11)
- new net GFX_A12: KA10.10 (A12), KA12.10 (A12), KA13.10 (A12), KA14.10 (A12), KB10.10 (A12), KB12.10 (A12), KB13.10 (A12), KB14.10 (A12)
- new net GFX_A13: KA10.9 (A13), KA12.9 (A13), KA13.9 (A13), KA14.9 (A13), KB10.9 (A13), KB12.9 (A13), KB13.9 (A13), KB14.9 (A13)
- new net GFX_A14: KA10.8 (A14), KA12.8 (A14), KA13.8 (A14), KA14.8 (A14), KB10.8 (A14), KB12.8 (A14), KB13.8 (A14), KB14.8 (A14)
- new net GFX_A15: KA10.7 (A15), KA12.7 (A15), KA13.7 (A15), KA14.7 (A15), KB10.7 (A15), KB12.7 (A15), KB13.7 (A15), KB14.7 (A15)
- new net GFX_A16: KA10.6 (A16), KA12.6 (A16), KA13.6 (A16), KA14.6 (A16), KB10.6 (A16), KB12.6 (A16), KB13.6 (A16), KB14.6 (A16)
- new net GFX_A17: KA10.5 (A17), KA12.5 (A17), KA13.5 (A17), KA14.5 (A17), KB10.5 (A17), KB12.5 (A17), KB13.5 (A17), KB14.5 (A17)
- new net GFX_A18: KA10.4 (A18), KA12.4 (A18), KA13.4 (A18), KA14.4 (A18), KB10.4 (A18), KB12.4 (A18), KB13.4 (A18), KB14.4 (A18)
- new net GFX_A19: KA10.3 (A19), KA12.3 (A19), KA13.3 (A19), KA14.3 (A19), KB10.3 (A19), KB12.3 (A19), KB13.3 (A19), KB14.3 (A19)
- new net GFX_A2: KA10.28 (A2), KA12.28 (A2), KA13.28 (A2), KA14.28 (A2), KB10.28 (A2), KB12.28 (A2), KB13.28 (A2), KB14.28 (A2)
- new net GFX_A20: KA10.46 (A20), KA12.46 (A20), KA13.46 (A20), KA14.46 (A20), KB10.46 (A20), KB12.46 (A20), KB13.46 (A20), KB14.46 (A20)
- new net GFX_A3: KA10.27 (A3), KA12.27 (A3), KA13.27 (A3), KA14.27 (A3), KB10.27 (A3), KB12.27 (A3), KB13.27 (A3), KB14.27 (A3)
- new net GFX_A4: KA10.22 (A4), KA12.22 (A4), KA13.22 (A4), KA14.22 (A4), KB10.22 (A4), KB12.22 (A4), KB13.22 (A4), KB14.22 (A4)
- new net GFX_A5: KA10.21 (A5), KA12.21 (A5), KA13.21 (A5), KA14.21 (A5), KB10.21 (A5), KB12.21 (A5), KB13.21 (A5), KB14.21 (A5)
- new net GFX_A6: KA10.20 (A6), KA12.20 (A6), KA13.20 (A6), KA14.20 (A6), KB10.20 (A6), KB12.20 (A6), KB13.20 (A6), KB14.20 (A6)
- new net GFX_A7: KA10.19 (A7), KA12.19 (A7), KA13.19 (A7), KA14.19 (A7), KB10.19 (A7), KB12.19 (A7), KB13.19 (A7), KB14.19 (A7)
- new net GFX_A8: KA10.18 (A8), KA12.18 (A8), KA13.18 (A8), KA14.18 (A8), KB10.18 (A8), KB12.18 (A8), KB13.18 (A8), KB14.18 (A8)
- new net GFX_A9: KA10.17 (A9), KA12.17 (A9), KA13.17 (A9), KA14.17 (A9), KB10.17 (A9), KB12.17 (A9), KB13.17 (A9), KB14.17 (A9)
- new net UK: KA10.2 (NC)
- new net ~{CE}: KA10.11 (~{CE}), KA12.11 (~{CE}), KA13.11 (~{CE}), KA14.11 (~{CE}), KB10.11 (~{CE}), KB12.11 (~{CE}), KB13.11 (~{CE}), KB14.11 (~{CE})
- new net ~{OE}: KA10.1 (NC), KA10.43 (~{OE}), KA12.1 (NC), KA12.2 (NC), KA12.43 (~{OE}), KA13.1 (NC), KA13.2 (NC), KA13.43 (~{OE}), KA14.1 (NC), KA14.2 (NC), KA14.43 (~{OE}), KB10.43 (~{OE}), KB12.43 (~{OE}), KB13.43 (~{OE}), KB14.43 (~{OE})
- new net ~{RESET5}: KA10.14 (~{RESET}), KA12.14 (~{RESET}), KA13.14 (~{RESET}), KA14.14 (~{RESET}), KB10.14 (~{RESET}), KB12.14 (~{RESET}), KB13.14 (~{RESET}), KB14.14 (~{RESET})
- new net ~{WE}: KA10.44 (~{WE}), KA12.44 (~{WE}), KA13.44 (~{WE}), KA14.44 (~{WE}), KB10.44 (~{WE}), KB12.44 (~{WE}), KB13.44 (~{WE}), KB14.44 (~{WE})
Other:
- removed sheet plane_color
- note removed: "SIMM3E"
- note removed: "SIMM4D"
- note removed: "SIMM5C"
- note removed: "SIMM6B"
- note removed: "first plane controls bit 0 of the color"
