File: cores/cps3/sch/_autosave-memories_gfx.kicad_sch (KiCad schematic)
At the start: 32 parts

Commit message: ppu in process
Connections:
- net OAMB_A0: no longer JB1.30 (A0), JB2.30 (A0), JB3.30 (A0), JB4.30 (A0), JB5.30 (A0), JB6.30 (A0), JB7.30 (A0), JB8.30 (A0)
- net OAMB_A1: no longer JB1.29 (A1), JB2.29 (A1), JB3.29 (A1), JB4.29 (A1), JB5.29 (A1), JB6.29 (A1), JB7.29 (A1), JB8.29 (A1)
- net OAMB_A10: no longer JB1.16 (A10), JB2.16 (A10), JB3.16 (A10), JB4.16 (A10), JB5.16 (A10), JB6.16 (A10), JB7.16 (A10), JB8.16 (A10)
- net OAMB_A11: no longer JB1.15 (A11), JB2.15 (A11), JB3.15 (A11), JB4.15 (A11), JB5.15 (A11), JB6.15 (A11), JB7.15 (A11), JB8.15 (A11)
- net OAMB_A12: no longer JB1.10 (A12), JB2.10 (A12), JB3.10 (A12), JB4.10 (A12), JB5.10 (A12), JB6.10 (A12), JB7.10 (A12), JB8.10 (A12)
- net OAMB_A13: no longer JB1.9 (A13), JB2.9 (A13), JB3.9 (A13), JB4.9 (A13), JB5.9 (A13), JB6.9 (A13), JB7.9 (A13), JB8.9 (A13)
- net OAMB_A14: no longer JB1.8 (A14), JB2.8 (A14), JB3.8 (A14), JB4.8 (A14), JB5.8 (A14), JB6.8 (A14), JB7.8 (A14), JB8.8 (A14)
- net OAMB_A15: no longer JB1.7 (A15), JB2.7 (A15), JB3.7 (A15), JB4.7 (A15), JB5.7 (A15), JB6.7 (A15), JB7.7 (A15), JB8.7 (A15)
- net OAMB_A16: no longer JB1.6 (A16), JB2.6 (A16), JB3.6 (A16), JB4.6 (A16), JB5.6 (A16), JB6.6 (A16), JB7.6 (A16), JB8.6 (A16)
- net OAMB_A17: no longer JB1.5 (A17), JB2.5 (A17), JB3.5 (A17), JB4.5 (A17), JB5.5 (A17), JB6.5 (A17), JB7.5 (A17), JB8.5 (A17)
- net OAMB_A18: no longer JB1.4 (A18), JB2.4 (A18), JB3.4 (A18), JB4.4 (A18), JB5.4 (A18), JB6.4 (A18), JB7.4 (A18), JB8.4 (A18)
- net OAMB_A19: no longer JB1.3 (A19), JB2.3 (A19), JB3.3 (A19), JB4.3 (A19), JB5.3 (A19), JB6.3 (A19), JB7.3 (A19), JB8.3 (A19)
- net OAMB_A2: no longer JB1.28 (A2), JB2.28 (A2), JB3.28 (A2), JB4.28 (A2), JB5.28 (A2), JB6.28 (A2), JB7.28 (A2), JB8.28 (A2)
- net OAMB_A20: no longer JB1.46 (A20), JB2.46 (A20), JB3.46 (A20), JB4.46 (A20), JB5.46 (A20), JB6.46 (A20), JB7.46 (A20), JB8.46 (A20)
- net OAMB_A3: no longer JB1.27 (A3), JB2.27 (A3), JB3.27 (A3), JB4.27 (A3), JB5.27 (A3), JB6.27 (A3), JB7.27 (A3), JB8.27 (A3)
- net OAMB_A4: no longer JB1.22 (A4), JB2.22 (A4), JB3.22 (A4), JB4.22 (A4), JB5.22 (A4), JB6.22 (A4), JB7.22 (A4), JB8.22 (A4)
- net OAMB_A5: no longer JB1.21 (A5), JB2.21 (A5), JB3.21 (A5), JB4.21 (A5), JB5.21 (A5), JB6.21 (A5), JB7.21 (A5), JB8.21 (A5)
- net OAMB_A6: no longer JB1.20 (A6), JB2.20 (A6), JB3.20 (A6), JB4.20 (A6), JB5.20 (A6), JB6.20 (A6), JB7.20 (A6), JB8.20 (A6)
- net OAMB_A7: no longer JB1.19 (A7), JB2.19 (A7), JB3.19 (A7), JB4.19 (A7), JB5.19 (A7), JB6.19 (A7), JB7.19 (A7), JB8.19 (A7)
- net OAMB_A8: no longer JB1.18 (A8), JB2.18 (A8), JB3.18 (A8), JB4.18 (A8), JB5.18 (A8), JB6.18 (A8), JB7.18 (A8), JB8.18 (A8)
- net OAMB_A9: no longer JB1.17 (A9), JB2.17 (A9), JB3.17 (A9), JB4.17 (A9), JB5.17 (A9), JB6.17 (A9), JB7.17 (A9), JB8.17 (A9)
- net OAM_A0: no longer JC1.30 (A0), JC2.30 (A0), JC3.30 (A0), JC4.30 (A0), JC5.30 (A0), JC6.30 (A0), JC7.30 (A0), JC8.30 (A0), JD1.30 (A0), JD2.30 (A0), JD3.30 (A0), JD4.30 (A0), JD5.30 (A0), JD6.30 (A0), JD7.30 (A0), JD8.30 (A0), JE1.30 (A0), JE2.30 (A0), JE3.30 (A0), JE4.30 (A0), JE5.30 (A0), JE6.30 (A0), JE7.30 (A0), JE8.30 (A0)
- net OAM_A1: no longer JC1.29 (A1), JC2.29 (A1), JC3.29 (A1), JC4.29 (A1), JC5.29 (A1), JC6.29 (A1), JC7.29 (A1), JC8.29 (A1), JD1.29 (A1), JD2.29 (A1), JD3.29 (A1), JD4.29 (A1), JD5.29 (A1), JD6.29 (A1), JD7.29 (A1), JD8.29 (A1), JE1.29 (A1), JE2.29 (A1), JE3.29 (A1), JE4.29 (A1), JE5.29 (A1), JE6.29 (A1), JE7.29 (A1), JE8.29 (A1)
- net OAM_A10: no longer JC1.16 (A10), JC2.16 (A10), JC3.16 (A10), JC4.16 (A10), JC5.16 (A10), JC6.16 (A10), JC7.16 (A10), JC8.16 (A10), JD1.16 (A10), JD2.16 (A10), JD3.16 (A10), JD4.16 (A10), JD5.16 (A10), JD6.16 (A10), JD7.16 (A10), JD8.16 (A10), JE1.16 (A10), JE2.16 (A10), JE3.16 (A10), JE4.16 (A10), JE5.16 (A10), JE6.16 (A10), JE7.16 (A10), JE8.16 (A10)
- net OAM_A11: no longer JC1.15 (A11), JC2.15 (A11), JC3.15 (A11), JC4.15 (A11), JC5.15 (A11), JC6.15 (A11), JC7.15 (A11), JC8.15 (A11), JD1.15 (A11), JD2.15 (A11), JD3.15 (A11), JD4.15 (A11), JD5.15 (A11), JD6.15 (A11), JD7.15 (A11), JD8.15 (A11), JE1.15 (A11), JE2.15 (A11), JE3.15 (A11), JE4.15 (A11), JE5.15 (A11), JE6.15 (A11), JE7.15 (A11), JE8.15 (A11)
- net OAM_A12: no longer JC1.10 (A12), JC2.10 (A12), JC3.10 (A12), JC4.10 (A12), JC5.10 (A12), JC6.10 (A12), JC7.10 (A12), JC8.10 (A12), JD1.10 (A12), JD2.10 (A12), JD3.10 (A12), JD4.10 (A12), JD5.10 (A12), JD6.10 (A12), JD7.10 (A12), JD8.10 (A12), JE1.10 (A12), JE2.10 (A12), JE3.10 (A12), JE4.10 (A12), JE5.10 (A12), JE6.10 (A12), JE7.10 (A12), JE8.10 (A12)
- net OAM_A13: no longer JC1.9 (A13), JC2.9 (A13), JC3.9 (A13), JC4.9 (A13), JC5.9 (A13), JC6.9 (A13), JC7.9 (A13), JC8.9 (A13), JD1.9 (A13), JD2.9 (A13), JD3.9 (A13), JD4.9 (A13), JD5.9 (A13), JD6.9 (A13), JD7.9 (A13), JD8.9 (A13), JE1.9 (A13), JE2.9 (A13), JE3.9 (A13), JE4.9 (A13), JE5.9 (A13), JE6.9 (A13), JE7.9 (A13), JE8.9 (A13)
- net OAM_A14: no longer JC1.8 (A14), JC2.8 (A14), JC3.8 (A14), JC4.8 (A14), JC5.8 (A14), JC6.8 (A14), JC7.8 (A14), JC8.8 (A14), JD1.8 (A14), JD2.8 (A14), JD3.8 (A14), JD4.8 (A14), JD5.8 (A14), JD6.8 (A14), JD7.8 (A14), JD8.8 (A14), JE1.8 (A14), JE2.8 (A14), JE3.8 (A14), JE4.8 (A14), JE5.8 (A14), JE6.8 (A14), JE7.8 (A14), JE8.8 (A14)
- net OAM_A15: no longer JC1.7 (A15), JC2.7 (A15), JC3.7 (A15), JC4.7 (A15), JC5.7 (A15), JC6.7 (A15), JC7.7 (A15), JC8.7 (A15), JD1.7 (A15), JD2.7 (A15), JD3.7 (A15), JD4.7 (A15), JD5.7 (A15), JD6.7 (A15), JD7.7 (A15), JD8.7 (A15), JE1.7 (A15), JE2.7 (A15), JE3.7 (A15), JE4.7 (A15), JE5.7 (A15), JE6.7 (A15), JE7.7 (A15), JE8.7 (A15)
- net OAM_A16: no longer JC1.6 (A16), JC2.6 (A16), JC3.6 (A16), JC4.6 (A16), JC5.6 (A16), JC6.6 (A16), JC7.6 (A16), JC8.6 (A16), JD1.6 (A16), JD2.6 (A16), JD3.6 (A16), JD4.6 (A16), JD5.6 (A16), JD6.6 (A16), JD7.6 (A16), JD8.6 (A16), JE1.6 (A16), JE2.6 (A16), JE3.6 (A16), JE4.6 (A16), JE5.6 (A16), JE6.6 (A16), JE7.6 (A16), JE8.6 (A16)
- net OAM_A17: no longer JC1.5 (A17), JC2.5 (A17), JC3.5 (A17), JC4.5 (A17), JC5.5 (A17), JC6.5 (A17), JC7.5 (A17), JC8.5 (A17), JD1.5 (A17), JD2.5 (A17), JD3.5 (A17), JD4.5 (A17), JD5.5 (A17), JD6.5 (A17), JD7.5 (A17), JD8.5 (A17), JE1.5 (A17), JE2.5 (A17), JE3.5 (A17), JE4.5 (A17), JE5.5 (A17), JE6.5 (A17), JE7.5 (A17), JE8.5 (A17)
- net OAM_A18: no longer JC1.4 (A18), JC2.4 (A18), JC3.4 (A18), JC4.4 (A18), JC5.4 (A18), JC6.4 (A18), JC7.4 (A18), JC8.4 (A18), JD1.4 (A18), JD2.4 (A18), JD3.4 (A18), JD4.4 (A18), JD5.4 (A18), JD6.4 (A18), JD7.4 (A18), JD8.4 (A18), JE1.4 (A18), JE2.4 (A18), JE3.4 (A18), JE4.4 (A18), JE5.4 (A18), JE6.4 (A18), JE7.4 (A18), JE8.4 (A18)
- net OAM_A19: no longer JC1.3 (A19), JC2.3 (A19), JC3.3 (A19), JC4.3 (A19), JC5.3 (A19), JC6.3 (A19), JC7.3 (A19), JC8.3 (A19), JD1.3 (A19), JD2.3 (A19), JD3.3 (A19), JD4.3 (A19), JD5.3 (A19), JD6.3 (A19), JD7.3 (A19), JD8.3 (A19), JE1.3 (A19), JE2.3 (A19), JE3.3 (A19), JE4.3 (A19), JE5.3 (A19), JE6.3 (A19), JE7.3 (A19), JE8.3 (A19)
- net OAM_A2: no longer JC1.28 (A2), JC2.28 (A2), JC3.28 (A2), JC4.28 (A2), JC5.28 (A2), JC6.28 (A2), JC7.28 (A2), JC8.28 (A2), JD1.28 (A2), JD2.28 (A2), JD3.28 (A2), JD4.28 (A2), JD5.28 (A2), JD6.28 (A2), JD7.28 (A2), JD8.28 (A2), JE1.28 (A2), JE2.28 (A2), JE3.28 (A2), JE4.28 (A2), JE5.28 (A2), JE6.28 (A2), JE7.28 (A2), JE8.28 (A2)
- net OAM_A20: no longer JC1.46 (A20), JC2.46 (A20), JC3.46 (A20), JC4.46 (A20), JC5.46 (A20), JC6.46 (A20), JC7.46 (A20), JC8.46 (A20), JD1.46 (A20), JD2.46 (A20), JD3.46 (A20), JD4.46 (A20), JD5.46 (A20), JD6.46 (A20), JD7.46 (A20), JD8.46 (A20), JE1.46 (A20), JE2.46 (A20), JE3.46 (A20), JE4.46 (A20), JE5.46 (A20), JE6.46 (A20), JE7.46 (A20), JE8.46 (A20)
- net OAM_A3: no longer JC1.27 (A3), JC2.27 (A3), JC3.27 (A3), JC4.27 (A3), JC5.27 (A3), JC6.27 (A3), JC7.27 (A3), JC8.27 (A3), JD1.27 (A3), JD2.27 (A3), JD3.27 (A3), JD4.27 (A3), JD5.27 (A3), JD6.27 (A3), JD7.27 (A3), JD8.27 (A3), JE1.27 (A3), JE2.27 (A3), JE3.27 (A3), JE4.27 (A3), JE5.27 (A3), JE6.27 (A3), JE7.27 (A3), JE8.27 (A3)
- net OAM_A4: no longer JC1.22 (A4), JC2.22 (A4), JC3.22 (A4), JC4.22 (A4), JC5.22 (A4), JC6.22 (A4), JC7.22 (A4), JC8.22 (A4), JD1.22 (A4), JD2.22 (A4), JD3.22 (A4), JD4.22 (A4), JD5.22 (A4), JD6.22 (A4), JD7.22 (A4), JD8.22 (A4), JE1.22 (A4), JE2.22 (A4), JE3.22 (A4), JE4.22 (A4), JE5.22 (A4), JE6.22 (A4), JE7.22 (A4), JE8.22 (A4)
- net OAM_A5: no longer JC1.21 (A5), JC2.21 (A5), JC3.21 (A5), JC4.21 (A5), JC5.21 (A5), JC6.21 (A5), JC7.21 (A5), JC8.21 (A5), JD1.21 (A5), JD2.21 (A5), JD3.21 (A5), JD4.21 (A5), JD5.21 (A5), JD6.21 (A5), JD7.21 (A5), JD8.21 (A5), JE1.21 (A5), JE2.21 (A5), JE3.21 (A5), JE4.21 (A5), JE5.21 (A5), JE6.21 (A5), JE7.21 (A5), JE8.21 (A5)
- net OAM_A6: no longer JC1.20 (A6), JC2.20 (A6), JC3.20 (A6), JC4.20 (A6), JC5.20 (A6), JC6.20 (A6), JC7.20 (A6), JC8.20 (A6), JD1.20 (A6), JD2.20 (A6), JD3.20 (A6), JD4.20 (A6), JD5.20 (A6), JD6.20 (A6), JD7.20 (A6), JD8.20 (A6), JE1.20 (A6), JE2.20 (A6), JE3.20 (A6), JE4.20 (A6), JE5.20 (A6), JE6.20 (A6), JE7.20 (A6), JE8.20 (A6)
- net OAM_A7: no longer JC1.19 (A7), JC2.19 (A7), JC3.19 (A7), JC4.19 (A7), JC5.19 (A7), JC6.19 (A7), JC7.19 (A7), JC8.19 (A7), JD1.19 (A7), JD2.19 (A7), JD3.19 (A7), JD4.19 (A7), JD5.19 (A7), JD6.19 (A7), JD7.19 (A7), JD8.19 (A7), JE1.19 (A7), JE2.19 (A7), JE3.19 (A7), JE4.19 (A7), JE5.19 (A7), JE6.19 (A7), JE7.19 (A7), JE8.19 (A7)
- net OAM_A8: no longer JC1.18 (A8), JC2.18 (A8), JC3.18 (A8), JC4.18 (A8), JC5.18 (A8), JC6.18 (A8), JC7.18 (A8), JC8.18 (A8), JD1.18 (A8), JD2.18 (A8), JD3.18 (A8), JD4.18 (A8), JD5.18 (A8), JD6.18 (A8), JD7.18 (A8), JD8.18 (A8), JE1.18 (A8), JE2.18 (A8), JE3.18 (A8), JE4.18 (A8), JE5.18 (A8), JE6.18 (A8), JE7.18 (A8), JE8.18 (A8)
- net OAM_A9: no longer JC1.17 (A9), JC2.17 (A9), JC3.17 (A9), JC4.17 (A9), JC5.17 (A9), JC6.17 (A9), JC7.17 (A9), JC8.17 (A9), JD1.17 (A9), JD2.17 (A9), JD3.17 (A9), JD4.17 (A9), JD5.17 (A9), JD6.17 (A9), JD7.17 (A9), JD8.17 (A9), JE1.17 (A9), JE2.17 (A9), JE3.17 (A9), JE4.17 (A9), JE5.17 (A9), JE6.17 (A9), JE7.17 (A9), JE8.17 (A9)
- net ~{CEA}: no longer JB1.11 (~{CE}), JB4.11 (~{CE})
- net ~{CEB}: no longer JB2.11 (~{CE}), JB3.11 (~{CE})
- net ~{CEC}: no longer JB5.11 (~{CE}), JB8.11 (~{CE})
- net ~{CED}: no longer JB6.11 (~{CE}), JB7.11 (~{CE})
- net ~{CEE}: no longer JC1.11 (~{CE}), JC4.11 (~{CE})
- net ~{CEF}: no longer JC2.11 (~{CE}), JC3.11 (~{CE})
- net ~{CEG}: no longer JC5.11 (~{CE}), JC8.11 (~{CE})
- net ~{CEH}: no longer JC6.11 (~{CE}), JC7.11 (~{CE})
- net ~{CEI}: no longer JD1.11 (~{CE}), JD4.11 (~{CE})
- net ~{CEJ}: no longer JD2.11 (~{CE}), JD3.11 (~{CE})
- net ~{CEK}: no longer JD5.11 (~{CE}), JD8.11 (~{CE})
- net ~{CEL}: no longer JD6.11 (~{CE}), JD7.11 (~{CE})
- net ~{CEM}: no longer JE1.11 (~{CE}), JE4.11 (~{CE})
- net ~{CEN}: no longer JE2.11 (~{CE}), JE3.11 (~{CE})
- net ~{CEO}: no longer JE5.11 (~{CE}), JE8.11 (~{CE})
- net ~{CEP}: no longer JE6.11 (~{CE}), JE7.11 (~{CE})
- net ~{OEB}: no longer JB1.43 (~{OE}), JB2.43 (~{OE}), JB3.43 (~{OE}), JB4.43 (~{OE}), JB5.43 (~{OE}), JB6.43 (~{OE}), JB7.43 (~{OE}), JB8.43 (~{OE})
- net ~{OEC}: no longer JC1.43 (~{OE}), JC2.43 (~{OE}), JC3.43 (~{OE}), JC4.43 (~{OE}), JC5.43 (~{OE}), JC6.43 (~{OE}), JC7.43 (~{OE}), JC8.43 (~{OE}), JD4.43 (~{OE}), JD6.43 (~{OE}), JD8.43 (~{OE})
- net ~{OED}: no longer JD1.43 (~{OE}), JD2.43 (~{OE}), JD3.43 (~{OE}), JD5.43 (~{OE}), JD7.43 (~{OE})
- net ~{OEE}: no longer JE1.43 (~{OE}), JE2.43 (~{OE}), JE3.43 (~{OE}), JE4.43 (~{OE}), JE5.43 (~{OE}), JE6.43 (~{OE}), JE7.43 (~{OE}), JE8.43 (~{OE})
- net ~{RESET1}: no longer JB1.14 (~{RESET}), JB2.14 (~{RESET}), JB3.14 (~{RESET}), JB4.14 (~{RESET}), JB5.14 (~{RESET}), JB6.14 (~{RESET}), JB7.14 (~{RESET}), JB8.14 (~{RESET})
- net ~{RESET2}: no longer JC1.14 (~{RESET}), JC2.14 (~{RESET}), JC3.14 (~{RESET}), JC4.14 (~{RESET}), JC5.14 (~{RESET}), JC6.14 (~{RESET}), JC7.14 (~{RESET}), JC8.14 (~{RESET})
- net ~{RESET3}: no longer JD1.14 (~{RESET}), JD2.14 (~{RESET}), JD3.14 (~{RESET}), JD4.14 (~{RESET}), JD5.14 (~{RESET}), JD6.14 (~{RESET}), JD7.14 (~{RESET}), JD8.14 (~{RESET})
- net ~{RESET4}: no longer JE1.14 (~{RESET}), JE2.14 (~{RESET}), JE3.14 (~{RESET}), JE4.14 (~{RESET}), JE5.14 (~{RESET}), JE6.14 (~{RESET}), JE7.14 (~{RESET}), JE8.14 (~{RESET})
- net ~{WEB}: no longer JB1.44 (~{WE}), JB2.44 (~{WE}), JB3.44 (~{WE}), JB4.44 (~{WE}), JB5.44 (~{WE}), JB6.44 (~{WE}), JB7.44 (~{WE}), JB8.44 (~{WE})
- net ~{WEC}: no longer JC1.44 (~{WE}), JC2.44 (~{WE}), JC3.44 (~{WE}), JC4.44 (~{WE}), JC5.44 (~{WE}), JC6.44 (~{WE}), JC7.44 (~{WE}), JC8.44 (~{WE}), JD4.44 (~{WE}), JD6.44 (~{WE}), JD8.44 (~{WE})
- net ~{WED}: no longer JD1.44 (~{WE}), JD2.44 (~{WE}), JD3.44 (~{WE}), JD5.44 (~{WE}), JD7.44 (~{WE})
- net ~{WEE}: no longer JE1.44 (~{WE}), JE2.44 (~{WE}), JE3.44 (~{WE}), JE4.44 (~{WE}), JE5.44 (~{WE}), JE6.44 (~{WE}), JE7.44 (~{WE}), JE8.44 (~{WE})
- net at JB5.23 (N.C): no longer JB5.
- net at JE7.23 (N.C): no longer JE7.
- net at JD2.23 (N.C): no longer JD2.
- net at JB7.23 (N.C): no longer JB7.
- net at JD7.23 (N.C): no longer JD7.
- net at JC5.23 (N.C): no longer JC5.
- net at JE4.23 (N.C): no longer JE4.
- net at JC4.23 (N.C): no longer JC4.
- net at JD3.23 (N.C): no longer JD3.
- net at JC6.23 (N.C): no longer JC6.
- net at JB4.23 (N.C): no longer JB4.
- net at JE6.23 (N.C): no longer JE6.
- net at JB2.23 (N.C): no longer JB2.
- net at JE8.23 (N.C): no longer JE8.
- net at JE5.23 (N.C): no longer JE5.
- net at JB6.23 (N.C): no longer JB6.
- net at JC1.23 (N.C): no longer JC1.
- net at JD8.23 (N.C): no longer JD8.
- net at JE3.23 (N.C): no longer JE3.
- net at JC8.23 (N.C): no longer JC8.
- net at JD4.23 (N.C): no longer JD4.
- net at JC2.23 (N.C): no longer JC2.
- net at JE2.23 (N.C): no longer JE2.
- net at JB8.23 (N.C): no longer JB8.
- net at JD6.23 (N.C): no longer JD6.
- net at JB1.23 (N.C): no longer JB1.
- net at JB3.23 (N.C): no longer JB3.
- net at JD1.23 (N.C): no longer JD1.
- net at JD5.23 (N.C): no longer JD5.
- net at JC7.23 (N.C): no longer JC7.
- net at JC3.23 (N.C): no longer JC3.
- net at JE1.23 (N.C): no longer JE1.
