File: cores/cps3/sch/bic.kicad_sch (KiCad schematic)
At the start: 1 part, among them K14 Am33C93A

Commit message: ssu_gll
Connections:
- net CDI_D0: now reaches K14.13 (D0)
- net CDI_D1: now reaches K14.14 (D1)
- net CDI_D2: now reaches K14.15 (D2)
- net CDI_D3: now reaches K14.16 (D3)
- net CDI_D4: now reaches K14.17 (D4)
- net CDI_D5: now reaches K14.18 (D5)
- net CDI_D6: now reaches K14.19 (D6)
- net CDI_D7: now reaches K14.20 (D7)
- net VSS: now reaches K14.23 (VSS)
- net VSS: now also K14.31 (VSS), K14.39 (VSS), K14.44 (VCC)
- net ALE: now reaches K14.27 (ALE)
- net VCC: now reaches K14.4 (VSS)
Changed lines of the file:
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@@
 (kicad_sch (version 20211123) (generator eeschema)
   (paper "A4")
+  (junction (at 137.16 125.73) (diameter 0) (color 0 0 0 0)
+  )
+  (junction (at 139.7 125.73) (diameter 0) (color 0 0 0 0)
+  )
+  (junction (at 138.43 125.73) (diameter 0) (color 0 0 0 0)
+  )
+  (bus_entry (at 165.1 87.63) (size 2.54 -2.54)
+    (stroke (width 0) (type default) (color 0 0 0 0))
+  )
+  (bus_entry (at 165.1 74.93) (size 2.54 -2.54)
+    (stroke (width 0) (type default) (color 0 0 0 0))
+  )
+  (bus_entry (at 165.1 85.09) (size 2.54 -2.54)
+    (stroke (width 0) (type default) (color 0 0 0 0))
+  )
+  (bus_entry (at 165.1 77.47) (size 2.54 -2.54)
+    (stroke (width 0) (type default) (color 0 0 0 0))
+  )
+  (bus_entry (at 165.1 90.17) (size 2.54 -2.54)
+    (stroke (width 0) (type default) (color 0 0 0 0))
+  )
+  (bus_entry (at 165.1 82.55) (size 2.54 -2.54)
+    (stroke (width 0) (type default) (color 0 0 0 0))
+  )
+  (bus_entry (at 165.1 72.39) (size 2.54 -2.54)
+    (stroke (width 0) (type default) (color 0 0 0 0))
+  )
+  (bus_entry (at 165.1 80.01) (size 2.54 -2.54)
+    (stroke (width 0) (type default) (color 0 0 0 0))
+  )
+  (wire (pts (xy 165.1 82.55) (xy 152.4 82.55))
+    (stroke (width 0) (type default) (color 0 0 0 0))
+  )
+  (bus (pts (xy 167.64 77.47) (xy 167.64 80.01))
+    (stroke (width 0) (type default) (color 0 0 0 0))
+  )
+  (wire (pts (xy 139.7 125.73) (xy 142.24 125.73))
+    (stroke (width 0) (type default) (color 0 0 0 0))
+  )
+  (bus (pts (xy 167.64 72.39) (xy 167.64 74.93))
+    (stroke (width 0) (type default) (color 0 0 0 0))
+  )
+  (wire (pts (xy 165.1 72.39) (xy 152.4 72.39))
+    (stroke (width 0) (type default) (color 0 0 0 0))
+  )
+  (wire (pts (xy 165.1 77.47) (xy 152.4 77.47))
+    (stroke (width 0) (type default) (color 0 0 0 0))
+  )
+  (wire (pts (xy 137.16 125.73) (xy 138.43 125.73))
+    (stroke (width 0) (type default) (color 0 0 0 0))
+  )
+  (wire (pts (xy 134.62 125.73) (xy 137.16 125.73))
+    (stroke (width 0) (type default) (color 0 0 0 0))
+  )
+  (wire (pts (xy 165.1 80.01) (xy 152.4 80.01))
+    (stroke (width 0) (type default) (color 0 0 0 0))
+  )
+  (wire (pts (xy 138.43 125.73) (xy 139.7 125.73))
+    (stroke (width 0) (type default) (color 0 0 0 0))
+  )
+  (wire (pts (xy 138.43 64.77) (xy 138.43 67.31))
+    (stroke (width 0) (type default) (color 0 0 0 0))
+  )
+  (bus (pts (xy 167.64 80.01) (xy 167.64 82.55))
+    (stroke (width 0) (type default) (color 0 0 0 0))
+  )
+  (wire (pts (xy 165.1 74.93) (xy 152.4 74.93))
+    (stroke (width 0) (type default) (color 0 0 0 0))
+  )
+  (wire (pts (xy 138.43 125.73) (xy 138.43 128.27))
+    (stroke (width 0) (type default) (color 0 0 0 0))
+  )
+  (wire (pts (xy 165.1 90.17) (xy 152.4 90.17))
+    (stroke (width 0) (type default) (color 0 0 0 0))
+  )
+  (bus (pts (xy 167.64 85.09) (xy 167.64 87.63))
+    (stroke (width 0) (type default) (color 0 0 0 0))
+  )
+  (bus (pts (xy 167.64 69.85) (xy 172.72 69.85))
+    (stroke (width 0) (type default) (color 0 0 0 0))
+  )
+  (bus (pts (xy 167.64 74.93) (xy 167.64 77.47))
+    (stroke (width 0) (type default) (color 0 0 0 0))
+  )
+  (wire (pts (xy 165.1 87.63) (xy 152.4 87.63))
+    (stroke (width 0) (type default) (color 0 0 0 0))
+  )
+  (bus (pts (xy 167.64 82.55) (xy 167.64 85.09))
+    (stroke (width 0) (type default) (color 0 0 0 0))
+  )
+  (wire (pts (xy 119.38 85.09) (xy 124.46 85.09))
+    (stroke (width 0) (type default) (color 0 0 0 0))
+  )
+  (bus (pts (xy 167.64 69.85) (xy 167.64 72.39))
+    (stroke (width 0) (type default) (color 0 0 0 0))
+  )
+  (wire (pts (xy 165.1 85.09) (xy 152.4 85.09))
+    (stroke (width 0) (type default) (color 0 0 0 0))
+  )
   (image (at 275.59 173.99) (scale 0.294008)
     (data
@@
     (effects (font (size 1.27 1.27)) (justify left bottom))
   )
+  (label "CDI_D2" (at 165.1 77.47 180)
+    (effects (font (size 1.27 1.27)) (justify right bottom))
+  )
+  (label "CDI_D5" (at 165.1 85.09 180)
+    (effects (font (size 1.27 1.27)) (justify right bottom))
+  )
+  (label "CDI_D6" (at 165.1 87.63 180)
+    (effects (font (size 1.27 1.27)) (justify right bottom))
+  )
+  (label "CDI_D0" (at 165.1 72.39 180)
+    (effects (font (size 1.27 1.27)) (justify right bottom))
+  )
+  (label "CDI_D4" (at 165.1 82.55 180)
+    (effects (font (size 1.27 1.27)) (justify right bottom))
+  )
+  (label "CDI_D1" (at 165.1 74.93 180)
+    (effects (font (size 1.27 1.27)) (justify right bottom))
+  )
+  (label "CDI_D7" (at 165.1 90.17 180)
+    (effects (font (size 1.27 1.27)) (justify right bottom))
+  )
+  (label "CDI_D3" (at 165.1 80.01 180)
+    (effects (font (size 1.27 1.27)) (justify right bottom))
+  )
+  (hierarchical_label "ALE" (shape input) (at 119.38 85.09 180)
+    (effects (font (size 1.27 1.27)) (justify right))
+  )
+  (hierarchical_label "CDI_D[7..0]" (shape bidirectional) (at 172.72 69.85 0)
+    (effects (font (size 1.27 1.27)) (justify left))
+  )
   (symbol (lib_id "arcade:Am33C93A") (at 138.43 96.52 0) (unit 1)
     (in_bom yes) (on_board yes)
@@
     (pin "9")
   )
+  (symbol (lib_id "power:VCC") (at 138.43 64.77 0) (unit 1)
+    (in_bom yes) (on_board yes)
+    (property "Reference" "#PWR?" (id 0) (at 138.43 68.58 0)
+      (effects (font (size 1.27 1.27)) hide)
+    )
+    (property "Value" "VCC" (id 1) (at 138.43 60.96 0))
+    (property "Footprint" "" (id 2) (at 138.43 64.77 0)
+      (effects (font (size 1.27 1.27)) hide)
+    )
+    (property "Datasheet" "" (id 3) (at 138.43 64.77 0)
+      (effects (font (size 1.27 1.27)) hide)
+    )
+    (pin "1")
+  )
+  (symbol (lib_id "power:VSS") (at 138.43 128.27 180) (unit 1)
+    (in_bom yes) (on_board yes)
+    (property "Reference" "#PWR?" (id 0) (at 138.43 124.46 0)
+      (effects (font (size 1.27 1.27)) hide)
+    )
+    (property "Value" "VSS" (id 1) (at 138.43 132.08 0))
+    (property "Footprint" "" (id 2) (at 138.43 128.27 0)
+      (effects (font (size 1.27 1.27)) hide)
+    )
+    (property "Datasheet" "" (id 3) (at 138.43 128.27 0)
+      (effects (font (size 1.27 1.27)) hide)
+    )
+    (pin "1")
+  )
 )

Commit message: update_symbols_capcom
Connections:
- net BIC_CLK: now reaches K14.8 (CLK)
Changed lines of the file:
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@@
+    (stroke (width 0) (type default) (color 0 0 0 0))
+  )
+  (wire (pts (xy 116.84 77.47) (xy 124.46 77.47))
     (stroke (width 0) (type default) (color 0 0 0 0))
   )
@@
     )
   )
-  (text "8-20MHz square wave clk" (at 96.52 77.47 0)
+  (text "8-20MHz square wave clk" (at 78.74 77.47 0)
     (effects (font (size 1.27 1.27)) (justify left bottom))
   )
@@
     (effects (font (size 1.27 1.27)) (justify right bottom))
   )
+  (hierarchical_label "BIC_CLK" (shape input) (at 116.84 77.47 180)
+    (effects (font (size 1.27 1.27)) (justify right))
+  )
   (hierarchical_label "ALE" (shape input) (at 119.38 85.09 180)
