File: cores/cps3/sch/cps3.kicad_sch (KiCad schematic)
At the start: 13 parts

Commit message: ssu_gll
Other:
- sheet ppu ports: added CLK_SSU, SSU_A[16..0], SSU_D[16..0]; removed SSU[17..0], SSU_Z[16..0]
- sheet ssu ports: added CLK_SSU, SSU_A[16..0], SSU_D[16..0]; removed none
Changed lines of the file:
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@@
     (stroke (width 0) (type default) (color 0 0 0 0))
   )
+  (bus (pts (xy 279.4 93.98) (xy 292.1 93.98))
+    (stroke (width 0) (type default) (color 0 0 0 0))
+  )
   (wire (pts (xy 33.02 80.01) (xy 45.72 80.01))
     (stroke (width 0) (type default) (color 0 0 0 0))
@@
     (stroke (width 0) (type default) (color 0 0 0 0))
   )
+  (bus (pts (xy 279.4 91.44) (xy 292.1 91.44))
+    (stroke (width 0) (type default) (color 0 0 0 0))
+  )
   (wire (pts (xy 219.71 271.78) (xy 208.28 271.78))
     (stroke (width 0) (type default) (color 0 0 0 0))
@@
     (stroke (width 0) (type default) (color 0 0 0 0))
   )
+  (wire (pts (xy 381 62.23) (xy 394.97 62.23))
+    (stroke (width 0) (type default) (color 0 0 0 0))
+  )
   (wire (pts (xy 219.71 238.76) (xy 208.28 238.76))
     (stroke (width 0) (type default) (color 0 0 0 0))
@@
     (stroke (width 0) (type default) (color 0 0 0 0))
   )
+  (wire (pts (xy 231.14 91.44) (xy 241.3 91.44))
+    (stroke (width 0) (type default) (color 0 0 0 0))
+  )
   (wire (pts (xy 189.23 113.03) (xy 179.07 113.03))
     (stroke (width 0) (type default) (color 0 0 0 0))
@@
     (effects (font (size 1.27 1.27)) (justify left bottom))
   )
+  (label "CLK_SSU" (at 394.97 62.23 180)
+    (effects (font (size 1.27 1.27)) (justify right bottom))
+  )
   (label "VSS" (at 35.56 220.98 0)
     (effects (font (size 1.27 1.27)) (justify left bottom))
@@
     (effects (font (size 1.27 1.27)) (justify left bottom))
   )
-  (label "SSU_Z[16..0]" (at 394.97 44.45 180)
+  (label "SSU_A[16..0]" (at 394.97 44.45 180)
     (effects (font (size 1.27 1.27)) (justify right bottom))
   )
@@
     (effects (font (size 1.27 1.27)) (justify left bottom))
   )
+  (label "CLK_SSU" (at 231.14 91.44 0)
+    (effects (font (size 1.27 1.27)) (justify left bottom))
+  )
   (label "OAM_A8" (at 146.05 228.6 0)
     (effects (font (size 1.27 1.27)) (justify left bottom))
@@
     (effects (font (size 1.27 1.27)) (justify right bottom))
   )
+  (label "SSU_D[16..0]" (at 292.1 91.44 180)
+    (effects (font (size 1.27 1.27)) (justify right bottom))
+  )
   (label "VSS" (at 179.07 166.37 0)
     (effects (font (size 1.27 1.27)) (justify left bottom))
@@
     (effects (font (size 1.27 1.27)) (justify left bottom))
   )
+  (label "SSU_A[16..0]" (at 292.1 93.98 180)
+    (effects (font (size 1.27 1.27)) (justify right bottom))
+  )
   (label "VSS" (at 146.05 256.54 0)
     (effects (font (size 1.27 1.27)) (justify left bottom))
@@
     (effects (font (size 1.27 1.27)) (justify left bottom))
   )
-  (label "SSU[17..0]" (at 394.97 46.99 180)
+  (label "SSU_D[16..0]" (at 394.97 46.99 180)
     (effects (font (size 1.27 1.27)) (justify right bottom))
   )
@@
       (effects (font (size 1.27 1.27)) (justify right))
     )
-    (pin "SSU_Z[16..0]" bidirectional (at 381 44.45 0)
+    (pin "SSU_A[16..0]" bidirectional (at 381 44.45 0)
       (effects (font (size 1.27 1.27)) (justify right))
     )
-    (pin "SSU[17..0]" bidirectional (at 381 46.99 0)
+    (pin "SSU_D[16..0]" bidirectional (at 381 46.99 0)
       (effects (font (size 1.27 1.27)) (justify right))
     )
@@
       (effects (font (size 1.27 1.27)) (justify right))
     )
+    (pin "CLK_SSU" output (at 381 62.23 0)
+      (effects (font (size 1.27 1.27)) (justify right))
+    )
   )
   (sheet (at 241.3 254) (size 38.1 12.7) (fields_autoplaced)
@@
       (effects (font (size 1.27 1.27)) (justify left top))
     )
+    (pin "SSU_D[16..0]" tri_state (at 279.4 91.44 0)
+      (effects (font (size 1.27 1.27)) (justify right))
+    )
+    (pin "SSU_A[16..0]" bidirectional (at 279.4 93.98 0)
+      (effects (font (size 1.27 1.27)) (justify right))
+    )
+    (pin "CLK_SSU" input (at 241.3 91.44 180)
+      (effects (font (size 1.27 1.27)) (justify left))
+    )
   )
   (sheet_instances
@@
       (reference "#PWR?") (unit 1) (value "VCC") (footprint "")
     )
+    (path "/faff34ab-5a16-490e-bc64-379c4a71ae98/55eeadef-a19e-4e23-849f-565ebbd7b241"
+      (reference "#PWR?") (unit 1) (value "VCC") (footprint "")
+    )
     (path "/108e58e9-06a6-483d-aa3f-469d137462b0/ecabe3b9-3cbd-418e-8efb-2cc94bb41ede/59052694-7a8c-473e-98dd-dc69652279db"
       (reference "#PWR?") (unit 1) (value "VSS") (footprint "")
@@
       (reference "#PWR?") (unit 1) (value "VSS") (footprint "")
     )
+    (path "/a1185fe8-0f30-42b6-aa0b-c4c1c57c93fb/501c2507-2861-4aa2-836f-6876a697c5dd/90f5f986-cba9-4de9-8fa5-1a4014ee5dc6"
+      (reference "#PWR?") (unit 1) (value "VCC") (footprint "")
+    )
+    (path "/a1185fe8-0f30-42b6-aa0b-c4c1c57c93fb/501c2507-2861-4aa2-836f-6876a697c5dd/aa00f025-3860-4a62-bf4e-748bf075fc50"
+      (reference "#PWR?") (unit 1) (value "VSS") (footprint "")
+    )
     (path "/108e58e9-06a6-483d-aa3f-469d137462b0/ecabe3b9-3cbd-418e-8efb-2cc94bb41ede/aca08efb-edfc-48a0-92ca-55c0782cb626"
       (reference "#PWR?") (unit 1) (value "VCC") (footprint "")
@@
       (reference "#PWR?") (unit 1) (value "VSS") (footprint "")
     )
+    (path "/faff34ab-5a16-490e-bc64-379c4a71ae98/dba9ecae-cdb7-492a-a811-07084a983473"
+      (reference "#PWR?") (unit 1) (value "VSS") (footprint "")
+    )
     (path "/108e58e9-06a6-483d-aa3f-469d137462b0/ecabe3b9-3cbd-418e-8efb-2cc94bb41ede/e5a8efe9-f8a2-4814-9080-59875dcf173e"
       (reference "#PWR?") (unit 1) (value "VCC") (footprint "")
@@
       (reference "G2") (unit 1) (value "DL-2729_PPU") (footprint "")
     )
+    (path "/faff34ab-5a16-490e-bc64-379c4a71ae98/ca660643-0945-46fe-9d04-aa2bf85944b7"
+      (reference "G6") (unit 1) (value "DL-3329-SSU") (footprint "")
+    )
     (path "/a1185fe8-0f30-42b6-aa0b-c4c1c57c93fb/8c3d90cf-6cdd-4533-acff-b9b3bd32c492"
       (reference "H1") (unit 1) (value "CU383-69K") (footprint "")
@@
       (reference "H9") (unit 1) (value "74FCT-16244ATPV") (footprint "")
     )
+    (path "/7609a0d1-d1f1-41e0-a233-39fd327a66c8/cca0a59c-941f-4e30-a904-3346440fa12b/ac5482b0-aeb5-429f-bac3-996b50f97c3a"
+      (reference "J11") (unit 1) (value "DL-3429-GLL1") (footprint "")
+    )
     (path "/108e58e9-06a6-483d-aa3f-469d137462b0/77bbff4f-2c87-4530-b594-97c3e9a50aa8/afca0431-7c84-439b-8da5-427b127abbc3"
       (reference "JB1") (unit 1) (value "29F016-90PFTN") (footprint "")
@@
       (reference "U?") (unit 1) (value "DL-2829-CCU") (footprint "")
     )
-    (path "/7609a0d1-d1f1-41e0-a233-39fd327a66c8/cca0a59c-941f-4e30-a904-3346440fa12b/ac5482b0-aeb5-429f-bac3-996b50f97c3a"
-      (reference "U?") (unit 1) (value "DL-3429-GLL1") (footprint "")
-    )
-    (path "/faff34ab-5a16-490e-bc64-379c4a71ae98/ca660643-0945-46fe-9d04-aa2bf85944b7"
-      (reference "U?") (unit 1) (value "DL-3329-SSU") (footprint "")
+    (path "/faff34ab-5a16-490e-bc64-379c4a71ae98/c20b2701-4012-4ce3-9758-9714bde36c02"
+      (reference "U?") (unit 1) (value "HD6417604F28_SH2") (footprint "")
     )
     (path "/1b942bf0-f209-4faa-8423-ee254f4f1637/e90cc38c-a92b-4991-a90f-f2489df2b299"

Commit message: update_symbols_capcom
Other:
- sheet ppu ports: added GLL_A[6..0]; removed GLL[7..0]
Changed lines of the file:
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@@
     (effects (font (size 1.27 1.27)) (justify left bottom))
   )
-  (label "GLL[7..0]" (at 394.97 26.67 180)
+  (label "GLL_A[6..0]" (at 394.97 26.67 180)
     (effects (font (size 1.27 1.27)) (justify right bottom))
   )
@@
       (effects (font (size 1.27 1.27)) (justify right))
     )
-    (pin "GLL[7..0]" bidirectional (at 381 26.67 0)
+    (pin "GLL_A[6..0]" bidirectional (at 381 26.67 0)
       (effects (font (size 1.27 1.27)) (justify right))
     )
@@
       (reference "#PWR?") (unit 1) (value "VSS") (footprint "")
     )
+    (path "/7609a0d1-d1f1-41e0-a233-39fd327a66c8/cca0a59c-941f-4e30-a904-3346440fa12b/646ab279-6641-444e-8c1b-38ac187e5b28"
+      (reference "#PWR?") (unit 1) (value "VSS") (footprint "")
+    )
     (path "/108e58e9-06a6-483d-aa3f-469d137462b0/ecabe3b9-3cbd-418e-8efb-2cc94bb41ede/7641990b-3c80-473b-bc92-2a675daa7226"
       (reference "#PWR?") (unit 1) (value "VCC") (footprint "")
@@
       (reference "#PWR?") (unit 1) (value "VSS") (footprint "")
     )
+    (path "/7609a0d1-d1f1-41e0-a233-39fd327a66c8/cca0a59c-941f-4e30-a904-3346440fa12b/e0334253-a77d-443a-ace9-d50e47622a0e"
+      (reference "#PWR?") (unit 1) (value "VCC") (footprint "")
+    )
     (path "/108e58e9-06a6-483d-aa3f-469d137462b0/ecabe3b9-3cbd-418e-8efb-2cc94bb41ede/e5a8efe9-f8a2-4814-9080-59875dcf173e"
       (reference "#PWR?") (unit 1) (value "VCC") (footprint "")
@@
       (reference "U1") (unit 4) (value "74LS08") (footprint "")
     )
+    (path "/a1185fe8-0f30-42b6-aa0b-c4c1c57c93fb/ef8b54cb-f742-4d73-8bd2-0679363ce61e"
+      (reference "U1") (unit 5) (value "74LS08") (footprint "")
+    )
     (path "/7609a0d1-d1f1-41e0-a233-39fd327a66c8/8353ddb9-f5ea-4a41-b04d-8c48f9582ff0/1579195c-802f-442a-9bd1-dfc1a459e19c"
       (reference "U?") (unit 1) (value "DL-3529-GLL2") (footprint "")
@@
       (reference "U?") (unit 1) (value "DL-2829-CCU") (footprint "")
     )
-    (path "/faff34ab-5a16-490e-bc64-379c4a71ae98/c20b2701-4012-4ce3-9758-9714bde36c02"
-      (reference "U?") (unit 1) (value "HD6417604F28_SH2") (footprint "")
-    )
     (path "/1b942bf0-f209-4faa-8423-ee254f4f1637/e90cc38c-a92b-4991-a90f-f2489df2b299"
       (reference "U?") (unit 1) (value "DL-2929-IOU") (footprint "")
     )
-    (path "/a1185fe8-0f30-42b6-aa0b-c4c1c57c93fb/ef8b54cb-f742-4d73-8bd2-0679363ce61e"
-      (reference "U?") (unit 5) (value "74LS08") (footprint "")
-    )
     (path "/a1185fe8-0f30-42b6-aa0b-c4c1c57c93fb/cdc8fbe6-64bf-4c2f-a581-d3e9076ec1c5"

Commit message: iou
Other:
- sheet objects ports: added 2GLL_A[5..0], CBI_CLK, CBI_D[7..0], GLL_A[14..0], SSU_D[16..0]; removed none
- sheet ppu ports: added 2GLL_A[5..0], CBI_D[7..0], GLL_A[14..0]; removed 2GLL[5..0], CDI_D[7..0], GLL_A[6..0], GLL_DRV0, GLL_DRV1, GLL_DRV2, GLL_DRV3, GLL_DRV4, GLL_DRV5

Commit message: uptate_ns
Other:
- sheet iou ports: added CBI_D[7..0], MAIN_A[13..0], MAIN_D[15..0]; removed none
- sheet ssu ports: added CBI_D[7..0]; removed none
Changed lines of the file:
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@@
     (stroke (width 0) (type default) (color 0 0 0 0))
   )
+  (bus (pts (xy 279.4 96.52) (xy 292.1 96.52))
+    (stroke (width 0) (type default) (color 0 0 0 0))
+  )
   (wire (pts (xy 77.47 252.73) (xy 69.85 252.73))
     (stroke (width 0) (type default) (color 0 0 0 0))
@@
     (stroke (width 0) (type default) (color 0 0 0 0))
   )
+  (bus (pts (xy 279.4 154.94) (xy 293.37 154.94))
+    (stroke (width 0) (type default) (color 0 0 0 0))
+  )
   (bus (pts (xy 64.77 240.03) (xy 64.77 242.57))
     (stroke (width 0) (type default) (color 0 0 0 0))
@@
     (stroke (width 0) (type default) (color 0 0 0 0))
   )
+  (bus (pts (xy 279.4 157.48) (xy 293.37 157.48))
+    (stroke (width 0) (type default) (color 0 0 0 0))
+  )
   (wire (pts (xy 189.23 146.05) (xy 177.8 146.05))
     (stroke (width 0) (type default) (color 0 0 0 0))
@@
     (stroke (width 0) (type default) (color 0 0 0 0))
   )
+  (bus (pts (xy 279.4 160.02) (xy 293.37 160.02))
+    (stroke (width 0) (type default) (color 0 0 0 0))
+  )
   (wire (pts (xy 77.47 137.16) (xy 67.31 137.16))
     (stroke (width 0) (type default) (color 0 0 0 0))
@@
     (effects (font (size 1.27 1.27)) (justify left bottom))
   )
+  (label "SSU_D[16..0]" (at 293.37 154.94 180)
+    (effects (font (size 1.27 1.27)) (justify right bottom))
+  )
   (label "~{CED}" (at 332.74 171.45 0)
     (effects (font (size 1.27 1.27)) (justify left bottom))
@@
     (effects (font (size 1.27 1.27)) (justify left bottom))
   )
+  (label "CBI_D[7..0]" (at 293.37 160.02 180)
+    (effects (font (size 1.27 1.27)) (justify right bottom))
+  )
   (label "2P_UP" (at 93.98 57.15 180)
     (effects (font (size 1.27 1.27)) (justify right bottom))
@@
     (effects (font (size 1.27 1.27)) (justify right bottom))
   )
-  (label "CDI_D[7..0]" (at 394.97 34.29 180)
+  (label "CBI_D[7..0]" (at 394.97 34.29 180)
     (effects (font (size 1.27 1.27)) (justify right bottom))
   )
@@
     (effects (font (size 1.27 1.27)) (justify left bottom))
   )
+  (label "GLL_A[14..0]" (at 293.37 157.48 180)
+    (effects (font (size 1.27 1.27)) (justify right bottom))
+  )
   (label "A1-2" (at 129.54 16.51 0)
     (effects (font (size 1.27 1.27)) (justify left bottom))
@@
     (effects (font (size 1.27 1.27)) (justify left bottom))
   )
+  (label "CBI_D[7..0]" (at 292.1 96.52 180)
+    (effects (font (size 1.27 1.27)) (justify right bottom))
+  )
   (label "2P_SELECT" (at 93.98 77.47 180)
     (effects (font (size 1.27 1.27)) (justify right bottom))
@@
       (effects (font (size 1.27 1.27)) (justify left top))
     )
+    (pin "MAIN_D[15..0]" bidirectional (at 279.4 154.94 0)
+      (effects (font (size 1.27 1.27)) (justify right))
+    )
+    (pin "MAIN_A[13..0]" bidirectional (at 279.4 157.48 0)
+      (effects (font (size 1.27 1.27)) (justify right))
+    )
+    (pin "CBI_D[7..0]" bidirectional (at 279.4 160.02 0)
+      (effects (font (size 1.27 1.27)) (justify right))
+    )
   )
   (sheet (at 139.7 15.24) (size 38.1 62.23) (fields_autoplaced)
@@
       (effects (font (size 1.27 1.27)) (justify left))
     )
+    (pin "CBI_D[7..0]" bidirectional (at 279.4 96.52 0)
+      (effects (font (size 1.27 1.27)) (justify right))
+    )
   )
   (sheet_instances
@@
       (reference "#PWR?") (unit 1) (value "VCC") (footprint "")
     )
+    (path "/1b942bf0-f209-4faa-8423-ee254f4f1637/1463f4f0-a3ba-45eb-9040-3533a728a045"
+      (reference "#PWR?") (unit 1) (value "VSS") (footprint "")
+    )
     (path "/a1185fe8-0f30-42b6-aa0b-c4c1c57c93fb/17ee9ce7-9ba5-44e8-a230-49dc7ead613b"
       (reference "#PWR?") (unit 1) (value "VSS") (footprint "")
@@
       (reference "#PWR?") (unit 1) (value "VCC") (footprint "")
     )
+    (path "/1b942bf0-f209-4faa-8423-ee254f4f1637/509ab7ae-2d97-4d21-9981-89d9f6a0753c"
+      (reference "#PWR?") (unit 1) (value "VCC") (footprint "")
+    )
     (path "/faff34ab-5a16-490e-bc64-379c4a71ae98/55eeadef-a19e-4e23-849f-565ebbd7b241"
       (reference "#PWR?") (unit 1) (value "VCC") (footprint "")
@@
       (reference "J11") (unit 1) (value "DL-3429-GLL1") (footprint "")
     )
+    (path "/3d8f6216-acf8-42c6-a729-9aab2d99566f/476cd7eb-7172-4140-b277-c795ec45f8fb"
+      (reference "J13") (unit 1) (value "DL-2829-CCU") (footprint "")
+    )
     (path "/108e58e9-06a6-483d-aa3f-469d137462b0/77bbff4f-2c87-4530-b594-97c3e9a50aa8/afca0431-7c84-439b-8da5-427b127abbc3"
       (reference "JB1") (unit 1) (value "29F016-90PFTN") (footprint "")
@@
       (reference "U1") (unit 5) (value "74LS08") (footprint "")
     )
-    (path "/3d8f6216-acf8-42c6-a729-9aab2d99566f/476cd7eb-7172-4140-b277-c795ec45f8fb"
-      (reference "U?") (unit 1) (value "DL-2829-CCU") (footprint "")
-    )
     (path "/a1185fe8-0f30-42b6-aa0b-c4c1c57c93fb/cdc8fbe6-64bf-4c2f-a581-d3e9076ec1c5"

Commit message: update_cps3
Other:
- sheet iou ports: added ALE, IO_SND31, IO_SND32, IO_SND41, MAIN_A[26..0], MAIN_D[14..0]; removed CBI_D[7..0], MAIN_A[13..0], MAIN_D[15..0]
- sheet objects ports: added ALE, MAIN_A[28..0], MAIN_D[14..0]; removed CBI_D[7..0], GLL_A[14..0], SSU_D[16..0]
- sheet ppu ports: added MAIN_A[28..0], MAIN_D[0..14], PPU2CCU0, PPU2CCU1; removed CBI_D[7..0], GLL_A[14..0], SSU_D[16..0]
- sheet sound ports: added IO_SND31, IO_SND32, IO_SND41; removed none
- note added: "CHECK POSSIBLE SHORT COME IN VSS AND VCC"
- note removed: "REVISAR POSIBLE CORTO ENTRE VSS Y VCC"

Commit message: cps_saved
Parts:
- added U? (x2): 74LS00, symbol jt74:74LS00
Changed lines of the file:
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@@
     (pin "1")
+  )
+  (symbol (lib_id "jt74:74LS00") (at 210.82 33.02 0) (unit 2)
+    (in_bom yes) (on_board yes)
+    (property "Reference" "U?" (id 0) (at 210.82 31.75 0))
+    (property "Value" "74LS00" (id 1) (at 210.82 34.29 0))
+    (property "Footprint" "" (id 2) (at 210.82 33.02 0)
+      (effects (font (size 1.27 1.27)) hide)
+    )
+    (property "Datasheet" "http://www.ti.com/lit/gpn/sn74ls00" (id 3) (at 210.82 33.02 0)
+      (effects (font (size 1.27 1.27)) hide)
+    )
+    (pin "1")
+    (pin "2")
+    (pin "3")
+    (pin "4")
+    (pin "5")
+    (pin "6")
+    (pin "10")
+    (pin "8")
+    (pin "9")
+    (pin "11")
+    (pin "12")
+    (pin "13")
+    (pin "14")
+    (pin "7")
   )
   (symbol (lib_id "Connector:Conn_01x36_Female") (at 132.08 233.68 0) (unit 1)
@@
     (pin "8")
     (pin "9")
+  )
+  (symbol (lib_id "jt74:74LS00") (at 201.93 43.18 0) (unit 1)
+    (in_bom yes) (on_board yes)
+    (property "Reference" "U?" (id 0) (at 201.93 41.91 0))
+    (property "Value" "74LS00" (id 1) (at 201.93 44.45 0))
+    (property "Footprint" "" (id 2) (at 201.93 43.18 0)
+      (effects (font (size 1.27 1.27)) hide)
+    )
+    (property "Datasheet" "http://www.ti.com/lit/gpn/sn74ls00" (id 3) (at 201.93 43.18 0)
+      (effects (font (size 1.27 1.27)) hide)
+    )
+    (pin "1")
+    (pin "2")
+    (pin "3")
+    (pin "4")
+    (pin "5")
+    (pin "6")
+    (pin "10")
+    (pin "8")
+    (pin "9")
+    (pin "11")
+    (pin "12")
+    (pin "13")
+    (pin "14")
+    (pin "7")
   )
   (symbol (lib_id "Connector:Conn_01x36_Female") (at 224.79 138.43 0) (unit 1)
@@
       (reference "U1") (unit 5) (value "74LS08") (footprint "")
     )
+    (path "/626c83eb-2f0f-455c-8914-3764d1d749fb"
+      (reference "U?") (unit 1) (value "74LS00") (footprint "")
+    )
+    (path "/34a8ab43-b6a7-41a1-a89f-c4fefdbe3eed"
+      (reference "U?") (unit 2) (value "74LS00") (footprint "")
+    )
     (path "/a1185fe8-0f30-42b6-aa0b-c4c1c57c93fb/cdc8fbe6-64bf-4c2f-a581-d3e9076ec1c5"

Commit message: update5
Parts:
- removed U? (x2): 74LS00, symbol jt74:74LS00
Other:
- sheet iou ports: added MAIN_D[13..0], MAIN_D[23..0]; removed MAIN_A[26..0], MAIN_D[14..0]
- sheet objects ports: added MAIN_A[20..0], MAIN_D[23..0]; removed MAIN_A[28..0], MAIN_D[14..0]
- sheet ppu ports: added MAIN_A[20..0], MAIN_D[23..0]; removed MAIN_A[28..0], MAIN_D[0..14]
Changed lines of the file:
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@@
     (effects (font (size 1.27 1.27)) (justify left bottom))
   )
-  (label "MAIN_D[14..0]" (at 293.37 154.94 180)
+  (label "MAIN_D[23..0]" (at 293.37 154.94 180)
     (effects (font (size 1.27 1.27)) (justify right bottom))
   )
@@
     (effects (font (size 1.27 1.27)) (justify left bottom))
   )
-  (label "MAIN_D[14..0]" (at 293.37 19.05 180)
+  (label "MAIN_D[23..0]" (at 293.37 19.05 180)
     (effects (font (size 1.27 1.27)) (justify right bottom))
   )
@@
     (effects (font (size 1.27 1.27)) (justify left bottom))
   )
-  (label "MAIN_A[28..0]" (at 293.37 21.59 180)
+  (label "MAIN_A[20..0]" (at 293.37 21.59 180)
     (effects (font (size 1.27 1.27)) (justify right bottom))
   )
@@
     (effects (font (size 1.27 1.27)) (justify left bottom))
   )
-  (label "MAIN_D[0..14]" (at 394.97 31.75 180)
+  (label "MAIN_D[23..0]" (at 394.97 31.75 180)
     (effects (font (size 1.27 1.27)) (justify right bottom))
   )
@@
     (effects (font (size 1.27 1.27)) (justify left bottom))
   )
-  (label "MAIN_A[28..0]" (at 293.37 157.48 180)
+  (label "MAIN_A[20..0]" (at 293.37 157.48 180)
     (effects (font (size 1.27 1.27)) (justify right bottom))
   )
@@
     (effects (font (size 1.27 1.27)) (justify left bottom))
   )
-  (label "MAIN_A[28..0]" (at 394.97 26.67 180)
+  (label "MAIN_A[20..0]" (at 394.97 26.67 180)
     (effects (font (size 1.27 1.27)) (justify right bottom))
   )
@@
     (pin "1")
   )
-  (symbol (lib_id "jt74:74LS00") (at 210.82 33.02 0) (unit 2)
-    (in_bom yes) (on_board yes)
-    (property "Reference" "U?" (id 0) (at 210.82 31.75 0))
-    (property "Value" "74LS00" (id 1) (at 210.82 34.29 0))
-    (property "Footprint" "" (id 2) (at 210.82 33.02 0)
-      (effects (font (size 1.27 1.27)) hide)
-    )
-    (property "Datasheet" "http://www.ti.com/lit/gpn/sn74ls00" (id 3) (at 210.82 33.02 0)
-      (effects (font (size 1.27 1.27)) hide)
-    )
-    (pin "1")
-    (pin "2")
-    (pin "3")
-    (pin "4")
-    (pin "5")
-    (pin "6")
-    (pin "10")
-    (pin "8")
-    (pin "9")
-    (pin "11")
-    (pin "12")
-    (pin "13")
-    (pin "14")
-    (pin "7")
-  )
   (symbol (lib_id "Connector:Conn_01x36_Female") (at 132.08 233.68 0) (unit 1)
     (in_bom yes) (on_board yes)
@@
     (pin "8")
     (pin "9")
-  )
-  (symbol (lib_id "jt74:74LS00") (at 201.93 43.18 0) (unit 1)
-    (in_bom yes) (on_board yes)
-    (property "Reference" "U?" (id 0) (at 201.93 41.91 0))
-    (property "Value" "74LS00" (id 1) (at 201.93 44.45 0))
-    (property "Footprint" "" (id 2) (at 201.93 43.18 0)
-      (effects (font (size 1.27 1.27)) hide)
-    )
-    (property "Datasheet" "http://www.ti.com/lit/gpn/sn74ls00" (id 3) (at 201.93 43.18 0)
-      (effects (font (size 1.27 1.27)) hide)
-    )
-    (pin "1")
-    (pin "2")
-    (pin "3")
-    (pin "4")
-    (pin "5")
-    (pin "6")
-    (pin "10")
-    (pin "8")
-    (pin "9")
-    (pin "11")
-    (pin "12")
-    (pin "13")
-    (pin "14")
-    (pin "7")
   )
   (symbol (lib_id "Connector:Conn_01x36_Female") (at 224.79 138.43 0) (unit 1)
@@
       (effects (font (size 1.27 1.27)) (justify left))
     )
-    (pin "MAIN_D[14..0]" bidirectional (at 279.4 154.94 0)
-      (effects (font (size 1.27 1.27)) (justify right))
-    )
-    (pin "MAIN_A[26..0]" bidirectional (at 279.4 157.48 0)
+    (pin "MAIN_D[23..0]" bidirectional (at 279.4 154.94 0)
+      (effects (font (size 1.27 1.27)) (justify right))
+    )
+    (pin "MAIN_D[13..0]" bidirectional (at 279.4 157.48 0)
       (effects (font (size 1.27 1.27)) (justify right))
     )
@@
       (effects (font (size 1.27 1.27)) (justify right))
     )
-    (pin "MAIN_D[14..0]" bidirectional (at 279.4 19.05 0)
-      (effects (font (size 1.27 1.27)) (justify right))
-    )
-    (pin "MAIN_A[28..0]" tri_state (at 279.4 21.59 0)
+    (pin "MAIN_D[23..0]" bidirectional (at 279.4 19.05 0)
+      (effects (font (size 1.27 1.27)) (justify right))
+    )
+    (pin "MAIN_A[20..0]" tri_state (at 279.4 21.59 0)
       (effects (font (size 1.27 1.27)) (justify right))
     )
@@
       (effects (font (size 1.27 1.27)) (justify right))
     )
-    (pin "MAIN_D[0..14]" bidirectional (at 381 31.75 0)
+    (pin "MAIN_D[23..0]" bidirectional (at 381 31.75 0)
       (effects (font (size 1.27 1.27)) (justify right))
     )
@@
       (effects (font (size 1.27 1.27)) (justify right))
     )
-    (pin "MAIN_A[28..0]" bidirectional (at 381 26.67 0)
+    (pin "MAIN_A[20..0]" bidirectional (at 381 26.67 0)
       (effects (font (size 1.27 1.27)) (justify right))
     )
@@
       (reference "U1") (unit 5) (value "74LS08") (footprint "")
     )
-    (path "/626c83eb-2f0f-455c-8914-3764d1d749fb"
-      (reference "U?") (unit 1) (value "74LS00") (footprint "")
-    )
-    (path "/34a8ab43-b6a7-41a1-a89f-c4fefdbe3eed"
-      (reference "U?") (unit 2) (value "74LS00") (footprint "")
-    )
     (path "/a1185fe8-0f30-42b6-aa0b-c4c1c57c93fb/cdc8fbe6-64bf-4c2f-a581-d3e9076ec1c5"
