File: cores/cps3/sch/cps3.kicad_sch (KiCad schematic)
At the start: 13 parts

Commit message: update6_cps
Connections:
- net VSS is gone; now on net GNDPWR: JM1.1 (GND), JM1.14 (VIDEO_GND), JM1.2 (VSSA), JM1.27 (GND), JM1.28 (GND), JM1.A (GND), JM1.B (GND), JM1.e (GND), JM1.f (GND), JSIMM1E.11 (Pin_11), JSIMM1E.20 (Pin_20), JSIMM1E.29 (Pin_29), JSIMM1EE.13 (Pin_13), JSIMM1EE.25 (Pin_25), JSIMM1EE.32 (Pin_32), JSIMM2D.11 (Pin_11), JSIMM2D.20 (Pin_20), JSIMM2D.29 (Pin_29), JSIMM2DD.13 (Pin_13), JSIMM2DD.25 (Pin_25), JSIMM2DD.27 (Pin_27), JSIMM2DD.32 (Pin_32), JSIMM3E.11 (Pin_11), JSIMM3E.20 (Pin_20), JSIMM3E.29 (Pin_29), JSIMM3EE.13 (Pin_13), JSIMM3EE.25 (Pin_25), JSIMM3EE.27 (Pin_27), JSIMM3EE.32 (Pin_32), JSIMM4D.11 (Pin_11), JSIMM4D.20 (Pin_20), JSIMM4D.29 (Pin_29), JSIMM4DD.13 (Pin_13), JSIMM4DD.25 (Pin_25), JSIMM4DD.27 (Pin_27), JSIMM4DD.32 (Pin_32), JSIMM5C.11 (Pin_11), JSIMM5C.20 (Pin_20), JSIMM5C.29 (Pin_29), JSIMM5CC.13 (Pin_13), JSIMM5CC.25 (Pin_25), JSIMM5CC.27 (Pin_27), JSIMM5CC.32 (Pin_32), JSIMM6B.11 (Pin_11), JSIMM6B.20 (Pin_20), JSIMM6B.29 (Pin_29), JSIMM6BB.13 (Pin_13), JSIMM6BB.25 (Pin_25), JSIMM6BB.27 (Pin_27), JSIMM6BB.32 (Pin_32)
- net -5V renamed GNDPWR
Other:
- sheet ccu ports: added PPU2CCU[1..0]; removed none
- sheet iou ports: added GLL2IO0, RESET?, SU2IO0; removed ALE
- sheet objects ports: added GLL2IO0, GLL2IO1, RESET?; removed ALE
- sheet ppu ports: added PPU2CCU[1..0]; removed PPU2CCU0, PPU2CCU1
- sheet ssu ports: added MAIN_A[3..1], MAIN_D[23..0], SU2IO0; removed SSU_D[16..0]
- note added: "OK"
