File: cores/cps3/sch/cps3.kicad_sch (KiCad schematic)
At the start: 12 parts, among them CN5 Conn_02x60_Female, CN6 Conn_02x27_Odd_Even, Q15 ZR, U1 74LS08

Commit message: wip_ccu
Connections:
- net ~{STBY_WD}: now reaches CN5.58 (Pin_58)
Other:
- added sheet trans (trans.kicad_sch)

Commit message: wip_ccu_gll2_cassette
Parts:
- removed U1: 74LS08, symbol jt74:74LS08
- R67: value 202Ω -> 202
- R86: value 472Ω -> 472
Other:
- removed sheet slots_female
- removed sheet trans
- sheet cbi ports: added PPU2CCU1; removed PPU_A0
- sheet ccu ports: added +12V, GLL2CCU[4..0], VBAT_S1-2, VBAT_S6~3; removed none
- sheet iou ports: added 2GLL2IOU0, GLL2CCU5, ~{RESET5}; removed none
- sheet objects ports: added 2GLL2IOU0, ~{STBY_WD}; removed none
- sheet ppu ports: added SYNCA, SYNCB; removed none
- sheet simms_flash ports: added VBAT_S1-2, VBAT_S6~3; removed none
- moved on the sheet: CP165, Q15, R67, R73

Commit message: wip_ccu_cassette
Other:
- sheet simms_flash ports: added ~{RESET[4..0]}; removed UK, ~{RESET1}, ~{RESET2}, ~{RESET3}, ~{RESET4}
Changed lines of the file:
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@@
     (stroke (width 0) (type default) (color 0 0 0 0))
   )
-  (wire (pts (xy 170.18 179.07) (xy 184.15 179.07))
-    (stroke (width 0) (type default) (color 0 0 0 0))
-  )
   (wire (pts (xy 222.25 44.45) (xy 237.49 44.45))
     (stroke (width 0) (type default) (color 0 0 0 0))
@@
     (stroke (width 0) (type default) (color 0 0 0 0))
   )
-  (wire (pts (xy 170.18 173.99) (xy 184.15 173.99))
-    (stroke (width 0) (type default) (color 0 0 0 0))
-  )
   (bus (pts (xy 222.25 200.66) (xy 237.49 200.66))
     (stroke (width 0) (type default) (color 0 0 0 0))
@@
     (stroke (width 0) (type default) (color 0 0 0 0))
   )
-  (wire (pts (xy 222.25 135.89) (xy 237.49 135.89))
-    (stroke (width 0) (type default) (color 0 0 0 0))
-  )
   (bus (pts (xy 304.8 35.56) (xy 322.58 35.56))
     (stroke (width 0) (type default) (color 0 0 0 0))
@@
     (stroke (width 0) (type default) (color 0 0 0 0))
   )
-  (wire (pts (xy 170.18 176.53) (xy 184.15 176.53))
-    (stroke (width 0) (type default) (color 0 0 0 0))
-  )
   (bus (pts (xy 304.8 55.88) (xy 322.58 55.88))
     (stroke (width 0) (type default) (color 0 0 0 0))
@@
     (stroke (width 0) (type default) (color 0 0 0 0))
   )
+  (bus (pts (xy 170.18 173.99) (xy 184.15 173.99))
+    (stroke (width 0) (type default) (color 0 0 0 0))
+  )
   (wire (pts (xy 48.26 118.11) (xy 53.34 118.11))
     (stroke (width 0) (type default) (color 0 0 0 0))
@@
     (stroke (width 0) (type default) (color 0 0 0 0))
   )
-  (wire (pts (xy 170.18 181.61) (xy 184.15 181.61))
-    (stroke (width 0) (type default) (color 0 0 0 0))
-  )
   (bus (pts (xy 184.15 34.29) (xy 168.91 34.29))
     (stroke (width 0) (type default) (color 0 0 0 0))
@@
     (effects (font (size 1.27 1.27)) (justify left bottom))
   )
-  (label "UK" (at 237.49 135.89 180)
-    (effects (font (size 1.27 1.27)) (justify right bottom))
-  )
   (label "SPRITEC_D[7..0]" (at 168.91 31.75 0)
     (effects (font (size 1.27 1.27)) (justify left bottom))
@@
     (effects (font (size 1.27 1.27)) (justify right bottom))
   )
-  (label "~{RESET3}" (at 170.18 179.07 0)
-    (effects (font (size 1.27 1.27)) (justify left bottom))
-  )
   (label "RED" (at 403.86 171.45 180)
     (effects (font (size 1.27 1.27)) (justify right bottom))
@@
     (effects (font (size 1.27 1.27)) (justify right bottom))
   )
-  (label "~{RESET1}" (at 170.18 173.99 0)
-    (effects (font (size 1.27 1.27)) (justify left bottom))
-  )
   (label "1P_BTN_1" (at 251.46 193.04 0)
     (effects (font (size 1.27 1.27)) (justify left bottom))
@@
     (effects (font (size 1.27 1.27)) (justify right bottom))
   )
-  (label "~{RESET2}" (at 170.18 176.53 0)
-    (effects (font (size 1.27 1.27)) (justify left bottom))
-  )
   (label "VCC" (at 71.12 123.19 180)
     (effects (font (size 1.27 1.27)) (justify right bottom))
@@
     (effects (font (size 1.27 1.27)) (justify right bottom))
   )
-  (label "~{RESET4}" (at 170.18 181.61 0)
+  (label "~{RESET[4..0]}" (at 170.18 173.99 0)
     (effects (font (size 1.27 1.27)) (justify left bottom))
   )
@@
       (effects (font (size 1.27 1.27)) (justify left))
     )
-    (pin "UK" output (at 222.25 135.89 0)
-      (effects (font (size 1.27 1.27)) (justify right))
-    )
     (pin "~{OE}" input (at 184.15 148.59 180)
       (effects (font (size 1.27 1.27)) (justify left))
@@
       (effects (font (size 1.27 1.27)) (justify left))
     )
-    (pin "~{RESET1}" input (at 184.15 173.99 180)
-      (effects (font (size 1.27 1.27)) (justify left))
-    )
-    (pin "~{RESET4}" input (at 184.15 181.61 180)
-      (effects (font (size 1.27 1.27)) (justify left))
-    )
-    (pin "~{RESET2}" input (at 184.15 176.53 180)
-      (effects (font (size 1.27 1.27)) (justify left))
-    )
-    (pin "~{RESET3}" input (at 184.15 179.07 180)
-      (effects (font (size 1.27 1.27)) (justify left))
-    )
     (pin "~{CEK}" input (at 184.15 133.35 180)
       (effects (font (size 1.27 1.27)) (justify left))
@@
       (effects (font (size 1.27 1.27)) (justify left))
     )
+    (pin "~{RESET[4..0]}" input (at 184.15 173.99 180)
+      (effects (font (size 1.27 1.27)) (justify left))
+    )
   )
   (sheet (at 266.7 167.64) (size 38.1 63.5) (fields_autoplaced)
@@
       (reference "J13") (unit 1) (value "DL-2829-CCU") (footprint "")
     )
+    (path "/3d8f6216-acf8-42c6-a729-9aab2d99566f/0c269afb-4436-427e-b162-5783df5bf96d"
+      (reference "J15") (unit 1) (value "MB814260-70PJ") (footprint "")
+    )
     (path "/108e58e9-06a6-483d-aa3f-469d137462b0/77bbff4f-2c87-4530-b594-97c3e9a50aa8/afca0431-7c84-439b-8da5-427b127abbc3"
       (reference "JB1") (unit 1) (value "29F016-90PFTN") (footprint "")
@@
       (reference "RN19") (unit 1) (value "620") (footprint "")
     )
+    (path "/3d8f6216-acf8-42c6-a729-9aab2d99566f/aa4cd00d-ea90-45db-b865-009fe18ca168"
+      (reference "RN20") (unit 1) (value "330") (footprint "")
+    )
+    (path "/3d8f6216-acf8-42c6-a729-9aab2d99566f/f955f39e-a746-4bf8-bae9-46d3982565f8"
+      (reference "RN21") (unit 1) (value "330") (footprint "")
+    )
     (path "/73e97af8-8757-47bc-9106-1c8a44eb3cd5/a0a5c18c-f4ec-4364-8e5e-2a536ee6337f"
       (reference "RN22") (unit 1) (value "221") (footprint "")
@@
       (reference "SIMM3E") (unit 1) (value "Conn_01x36_Male") (footprint "")
     )
-    (path "/108e58e9-06a6-483d-aa3f-469d137462b0/f1a6563b-7cdb-4252-889d-dd4a49e136cc/ac75238d-b3fe-48af-a967-0160e0c03855"
+    (path "/108e58e9-06a6-483d-aa3f-469d137462b0/f1a6563b-7cdb-4252-889d-dd4a49e136cc/2e3dacc8-f8e7-43cd-bc44-5fb968216df7"
       (reference "SIMM3EE") (unit 1) (value "Conn_01x36_Male") (footprint "")
     )
@@
       (reference "SIMM4D") (unit 1) (value "Conn_01x36_Male") (footprint "")
     )
-    (path "/108e58e9-06a6-483d-aa3f-469d137462b0/f1a6563b-7cdb-4252-889d-dd4a49e136cc/3be5e64c-0175-4d33-aaa5-7137e328d0b2"
+    (path "/108e58e9-06a6-483d-aa3f-469d137462b0/f1a6563b-7cdb-4252-889d-dd4a49e136cc/fec6b5b8-0817-417d-8cf7-862b9e3e2c8f"
       (reference "SIMM4DD") (unit 1) (value "Conn_01x36_Male") (footprint "")
     )

Commit message: wip_cassette
Parts:
- removed CN5: Conn_02x60_Female, symbol arcade:Conn_02x60_Female
- added CN5: Conn_02x60_Male, symbol arcade:Conn_02x60_Male
Connections:
- net 35CCU: now also CN5.116 (Pin_116)
- net GLL_A0: now also CN5.76 (Pin_76)
- net GLL_A1: now also CN5.89 (Pin_89)
- net GLL_A10: now also CN5.100 (Pin_100)
- net GLL_A11: now also CN5.101 (Pin_101)
- net GLL_A12: now also CN5.102 (Pin_102)
- net GLL_A13: now also CN5.103 (Pin_103)
- net GLL_A14: now also CN5.104 (Pin_104)
- net GLL_A15: now also CN5.105 (Pin_105)
- net GLL_A16: now also CN5.106 (Pin_106)
- net GLL_A17: now also CN5.109 (Pin_109)
- net GLL_A18: now also CN5.110 (Pin_110)
- net GLL_A19: now also CN5.111 (Pin_111)
- net GLL_A2: now also CN5.90 (Pin_90)
- net GLL_A20: now also CN5.112 (Pin_112)
- net GLL_A3: now also CN5.91 (Pin_91)
- net GLL_A4: now also CN5.92 (Pin_92)
- net GLL_A5: now also CN5.93 (Pin_93)
- net GLL_A6: now also CN5.94 (Pin_94)
- net GLL_A7: now also CN5.95 (Pin_95)
- net GLL_A8: now also CN5.96 (Pin_96)
- net GLL_A9: now also CN5.99 (Pin_99)
- net GLL_D0: now also CN5.113 (Pin_113)
- net GLL_D1: now also CN5.114 (Pin_114)
- net GLL_D2: now also CN5.115 (Pin_115)
- net GLL_D3: now also CN5.49 (Pin_49)
- net GLL_D4: now also CN5.50 (Pin_50)
- net GLL_D5: now also CN5.47 (Pin_47)
- net GLL_D6: now also CN5.48 (Pin_48)
- net GLL_D7: now also CN5.56 (Pin_56)
- net PULL_UP1: now also CN5.1
- net VCC: now also CN5.10 (Pin_10), CN5.108 (Pin_108), CN5.118 (Pin_118), CN5.120 (Pin_120), CN5.2, CN5.26 (Pin_26), CN5.36 (Pin_36), CN5.46 (Pin_46), CN5.54 (Pin_54), CN5.6, CN5.60 (Pin_60), CN5.68 (Pin_68), CN5.74 (Pin_74), CN5.78 (Pin_78), CN5.80 (Pin_80), CN5.88 (Pin_88), CN5.98 (Pin_98)
- net VSS: now also CN5.107 (Pin_107), CN5.117 (Pin_117), CN5.119 (Pin_119), CN5.15 (Pin_15), CN5.25 (Pin_25), CN5.35 (Pin_35), CN5.45 (Pin_45), CN5.5 (Pin_5), CN5.51 (Pin_51), CN5.55 (Pin_55), CN5.57 (Pin_57), CN5.61 (Pin_61), CN5.69 (Pin_69), CN5.75 (Pin_75), CN5.79 (Pin_79), CN5.87 (Pin_87), CN5.97 (Pin_97)
- net ~{RST_WD}: now also CN5.53 (Pin_53)
- net ~{STBY_WD}: now also CN5.58 (Pin_58)
- new net ~{CE}R_CST: CN5.3
Other:
- sheet objects ports: added BX_SPR, ~{CEA}, ~{CEB}, ~{CEC}, ~{CED}, ~{CEE}, ~{CEF}, ~{CEG}, ~{CEH}, ~{CEI}, ~{CEJ}, ~{CEK}, ~{CEL}, ~{CEM}, ~{CEN}, ~{CEO}, ~{CEP}, ~{OEB}, ~{OEC}, ~{OED}, ~{OEE}, ~{RESET[4..0]}, ~{WEB}, ~{WEC}, ~{WED}, ~{WEE}; removed none
- sheet ppu ports: added none; removed GFX_A[20..0]
- sheet simms_flash ports: added GFX_A21, UK_CCU, ~{CE_}S1, ~{CE_}S2, ~{OE}_CCU, ~{WE}_CCU; removed ~{CE}, ~{OE}, ~{WE}
- moved on the sheet: CN6, CP151, CP152, D1, JM1, R86

Commit message: wip_cassette
Connections:
- net ~{RST_WD}: no longer CN5.53 (Pin_53), R73.1
- new net ~{RST}_WD: CN5.53 (Pin_53), R73.1
Other:
- sheet objects ports: added ~{RST}_WD; removed ~{RST_WD}
Changed lines of the file:
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@@
     (effects (font (size 1.27 1.27)) (justify left))
   )
-  (hierarchical_label "~{RST_WD}" (shape input) (at 76.2 180.34 0)
+  (hierarchical_label "~{RST}_WD" (shape input) (at 76.2 180.34 0)
     (effects (font (size 1.27 1.27)) (justify left))
   )
@@
       (effects (font (size 1.27 1.27)) (justify right))
     )
-    (pin "~{RST_WD}" output (at 304.8 36.83 0)
+    (pin "~{RST}_WD" output (at 304.8 36.83 0)
       (effects (font (size 1.27 1.27)) (justify right))
     )
@@
       (reference "B3") (unit 1) (value "TA8201AK") (footprint "")
     )
+    (path "/7609a0d1-d1f1-41e0-a233-39fd327a66c8/a3eaa016-f145-419c-a632-73f45a370a93/bf3ffa95-1b11-4477-a87e-972ca55fc4ec"
+      (reference "BT1") (unit 1) (value "Battery-95682B-3") (footprint "")
+    )
     (path "/39349e27-3581-43b0-a2a9-76c521c74f3d/f15d360c-8cbf-40e3-9256-cc14cc8f4b1a"
       (reference "C5") (unit 1) (value "TDA1306T") (footprint "")
@@
       (reference "CP176") (unit 1) (value "10μF") (footprint "")
     )
+    (path "/7609a0d1-d1f1-41e0-a233-39fd327a66c8/a3eaa016-f145-419c-a632-73f45a370a93/a2ab4cb3-538a-4460-b86e-127bd3d646a6"
+      (reference "CP177") (unit 1) (value "10μF") (footprint "")
+    )
+    (path "/7609a0d1-d1f1-41e0-a233-39fd327a66c8/a3eaa016-f145-419c-a632-73f45a370a93/8873ebc7-90ee-47b2-afba-10386fede4bc"
+      (reference "CP178") (unit 1) (value "10μF") (footprint "")
+    )
+    (path "/7609a0d1-d1f1-41e0-a233-39fd327a66c8/a3eaa016-f145-419c-a632-73f45a370a93/74d29f50-64dd-490e-b9bf-f070f9704057"
+      (reference "CP179") (unit 1) (value "10μF") (footprint "")
+    )
+    (path "/7609a0d1-d1f1-41e0-a233-39fd327a66c8/a3eaa016-f145-419c-a632-73f45a370a93/0e67ee65-ecf8-4593-8a94-a00a4c610063"
+      (reference "CP180") (unit 1) (value "10μF") (footprint "")
+    )
+    (path "/a8c99e2c-a143-4c69-9194-e7df3ea5db5d/96342f1c-5f29-4a8c-9aa1-e66e2a01d525"
+      (reference "CP180") (unit 1) (value "1nF") (footprint "")
+    )
+    (path "/a8c99e2c-a143-4c69-9194-e7df3ea5db5d/956ca1b1-ee92-4b8a-8ff8-5553eef48d7e"
+      (reference "CP181") (unit 1) (value "1nF") (footprint "")
+    )
+    (path "/a8c99e2c-a143-4c69-9194-e7df3ea5db5d/59b70842-14a0-4b8f-915c-c89362e8bf57"
+      (reference "CP182") (unit 1) (value "1nF") (footprint "")
+    )
+    (path "/a8c99e2c-a143-4c69-9194-e7df3ea5db5d/d5641cff-f309-45d2-8286-409f3e649142"
+      (reference "CP183") (unit 1) (value "1nF") (footprint "")
+    )
+    (path "/a8c99e2c-a143-4c69-9194-e7df3ea5db5d/591b5d43-2a82-4d31-9fea-30cd53b1e256"
+      (reference "CP184") (unit 1) (value "47μF") (footprint "")
+    )
+    (path "/7609a0d1-d1f1-41e0-a233-39fd327a66c8/a3eaa016-f145-419c-a632-73f45a370a93/0ddb4e18-b93f-467f-ba2d-1cbee3a7cbbf"
+      (reference "CP185") (unit 1) (value "47μF") (footprint "")
+    )
+    (path "/7609a0d1-d1f1-41e0-a233-39fd327a66c8/a3eaa016-f145-419c-a632-73f45a370a93/26274de2-5e27-4490-a9bb-b4ee01af3d60"
+      (reference "CP186") (unit 1) (value "101") (footprint "")
+    )
+    (path "/7609a0d1-d1f1-41e0-a233-39fd327a66c8/a3eaa016-f145-419c-a632-73f45a370a93/3596df93-745c-4995-a1fa-baee9c0b992a"
+      (reference "CP186") (unit 1) (value "1nF") (footprint "")
+    )
+    (path "/7609a0d1-d1f1-41e0-a233-39fd327a66c8/a3eaa016-f145-419c-a632-73f45a370a93/a76d0fe9-e814-4285-8099-16d94e0e3d3b"
+      (reference "CP187") (unit 1) (value "47μF") (footprint "")
+    )
+    (path "/7609a0d1-d1f1-41e0-a233-39fd327a66c8/a3eaa016-f145-419c-a632-73f45a370a93/38f6a11d-5668-4734-af52-ec80206a8e9f"
+      (reference "CP188") (unit 1) (value "1nF") (footprint "")
+    )
+    (path "/7609a0d1-d1f1-41e0-a233-39fd327a66c8/a3eaa016-f145-419c-a632-73f45a370a93/162937ed-e9cc-4879-a421-8e4cefaea861"
+      (reference "CP189") (unit 1) (value "47μF") (footprint "")
+    )
     (path "/1b942bf0-f209-4faa-8423-ee254f4f1637/85558694-7a3f-454d-aaeb-5c2cbe23fce8"
       (reference "CR1") (unit 1) (value "CRE438-60") (footprint "")
@@
       (reference "R1") (unit 1) (value "103Ω") (footprint "Resistor_THT:R_Array_SIP5")
     )
-    (path "/7609a0d1-d1f1-41e0-a233-39fd327a66c8/a3eaa016-f145-419c-a632-73f45a370a93/5be6cbf3-c241-471f-9074-804eae105192"
-      (reference "R2") (unit 1) (value "105") (footprint "")
-    )
     (path "/39349e27-3581-43b0-a2a9-76c521c74f3d/e7b653f9-8e32-46dc-952f-3ec87fbd7597"
       (reference "R2") (unit 1) (value "100kΩ") (footprint "")
@@
       (reference "R20") (unit 1) (value "1.8kΩ") (footprint "")
     )
-    (path "/7609a0d1-d1f1-41e0-a233-39fd327a66c8/a3eaa016-f145-419c-a632-73f45a370a93/ab40ae4e-8f88-43ff-97df-4c9532b2ea7a"
-      (reference "R20") (unit 1) (value "103") (footprint "")
-    )
     (path "/39349e27-3581-43b0-a2a9-76c521c74f3d/f1404f90-84cc-46fd-8901-11cca612e31e"
       (reference "R21") (unit 1) (value "1kΩ") (footprint "")
@@
       (reference "RN29") (unit 1) (value "331") (footprint "")
     )
+    (path "/7609a0d1-d1f1-41e0-a233-39fd327a66c8/a3eaa016-f145-419c-a632-73f45a370a93/5be6cbf3-c241-471f-9074-804eae105192"
+      (reference "RR2") (unit 1) (value "105") (footprint "")
+    )
+    (path "/7609a0d1-d1f1-41e0-a233-39fd327a66c8/a3eaa016-f145-419c-a632-73f45a370a93/e64c987b-171d-44a3-9561-8b223320e521"
+      (reference "RR3") (unit 1) (value "103") (footprint "")
+    )
+    (path "/7609a0d1-d1f1-41e0-a233-39fd327a66c8/a3eaa016-f145-419c-a632-73f45a370a93/aeea68a4-ce56-473b-993d-63b890f919a3"
+      (reference "RR4") (unit 1) (value "103") (footprint "")
+    )
+    (path "/7609a0d1-d1f1-41e0-a233-39fd327a66c8/a3eaa016-f145-419c-a632-73f45a370a93/fb96323e-cc51-4733-88e0-78175974dac5"
+      (reference "RR19") (unit 1) (value "103") (footprint "")
+    )
+    (path "/7609a0d1-d1f1-41e0-a233-39fd327a66c8/a3eaa016-f145-419c-a632-73f45a370a93/ab40ae4e-8f88-43ff-97df-4c9532b2ea7a"
+      (reference "RR20") (unit 1) (value "103") (footprint "")
+    )
     (path "/39349e27-3581-43b0-a2a9-76c521c74f3d/c89e518b-4da1-4105-bd3d-77c26149f4cb"
       (reference "RV1") (unit 1) (value "R_POT_5PINS") (footprint "")
@@
       (reference "U1") (unit 4) (value "7400") (footprint "")
     )
-    (path "/7609a0d1-d1f1-41e0-a233-39fd327a66c8/a3eaa016-f145-419c-a632-73f45a370a93/760753b0-6b34-4da2-90b5-05f40a002b14"
+    (path "/a8c99e2c-a143-4c69-9194-e7df3ea5db5d/7b9a49a3-3970-47fb-b44b-bd6c6d77c96c"
       (reference "U1") (unit 5) (value "7400") (footprint "")
+    )
+    (path "/7609a0d1-d1f1-41e0-a233-39fd327a66c8/a3eaa016-f145-419c-a632-73f45a370a93/c49da8be-88dd-4c93-a42e-52a529930885"
+      (reference "U2") (unit 1) (value "29F400TA-90PF") (footprint "")
     )
     (path "/a8c99e2c-a143-4c69-9194-e7df3ea5db5d/732cc323-9204-491d-a9f7-f245bcc6b607"
@@
       (reference "U3-SCU") (unit 1) (value "HD6417604F28_SH2") (footprint "")
     )
-    (path "/7609a0d1-d1f1-41e0-a233-39fd327a66c8/a3eaa016-f145-419c-a632-73f45a370a93/32ae4a24-246a-4b00-975f-cd34a0e84ea1"
-      (reference "U4") (unit 1) (value "7400") (footprint "")
-    )
     (path "/7609a0d1-d1f1-41e0-a233-39fd327a66c8/a3eaa016-f145-419c-a632-73f45a370a93/ffd344e8-ebc8-4958-b312-b78fd57c0250"
       (reference "U4") (unit 2) (value "7400") (footprint "")
@@
       (reference "U4") (unit 4) (value "7400") (footprint "")
     )
-    (path "/7609a0d1-d1f1-41e0-a233-39fd327a66c8/a3eaa016-f145-419c-a632-73f45a370a93/bebcf3ba-694f-43a4-959e-3bb6087ea390"
+    (path "/a8c99e2c-a143-4c69-9194-e7df3ea5db5d/c2b99580-ef96-406d-bab7-257583ce834f"
       (reference "U4") (unit 5) (value "7400") (footprint "")
+    )
+    (path "/7609a0d1-d1f1-41e0-a233-39fd327a66c8/a3eaa016-f145-419c-a632-73f45a370a93/3bc5710f-80fb-4997-b862-d8cb3b79c88d"
+      (reference "U6") (unit 1) (value "FM1208S-250SC") (footprint "")
     )
     (path "/7609a0d1-d1f1-41e0-a233-39fd327a66c8/a3eaa016-f145-419c-a632-73f45a370a93/8e2fe8e0-4369-467b-9f6e-3e18372b1c20"
       (reference "U?") (unit 1) (value "Conn_02x60_Male") (footprint "")
     )
-    (path "/7609a0d1-d1f1-41e0-a233-39fd327a66c8/a3eaa016-f145-419c-a632-73f45a370a93/c49da8be-88dd-4c93-a42e-52a529930885"
-      (reference "U?") (unit 1) (value "29F400TA-90PF") (footprint "")
-    )
-    (path "/47f33d46-1dcf-406e-b526-e95dcccc85cf/8cc2b494-2485-496e-8999-a31de4c00fca"
-      (reference "VD2") (unit 1) (value "BAV99") (footprint "")
+    (path "/7609a0d1-d1f1-41e0-a233-39fd327a66c8/a3eaa016-f145-419c-a632-73f45a370a93/c876bd98-be3b-4292-8d1f-4a2648b7cabf"
+      (reference "VD1") (unit 1) (value "VD-ESDAxxSCx") (footprint "")
+    )
+    (path "/47f33d46-1dcf-406e-b526-e95dcccc85cf/2fb0cabf-2955-4c8b-85fd-fcc789b1ba45"
+      (reference "VD2") (unit 1) (value "VD-BAV99") (footprint "")
     )
     (path "/39349e27-3581-43b0-a2a9-76c521c74f3d/e3c0198b-3fa3-487a-9d23-0dc3f22513d4"
       (reference "VD3") (unit 1) (value "BAV99") (footprint "")
     )
+    (path "/7609a0d1-d1f1-41e0-a233-39fd327a66c8/a3eaa016-f145-419c-a632-73f45a370a93/4e49ee4c-6b88-4686-9464-3b8223bca96e"
+      (reference "VDD2") (unit 1) (value "VD-ESDAxxSCx") (footprint "")
+    )
     (path "/7609a0d1-d1f1-41e0-a233-39fd327a66c8/a3eaa016-f145-419c-a632-73f45a370a93/32e1aa2c-9da3-44ba-956e-779bb7b7b900"

Commit message: wip_cassette_rg
Parts:
- removed CN5: Conn_02x60_Male, symbol arcade:Conn_02x60_Male
- added U?: Conn_02x60_Female, symbol arcade:Conn_02x60_Female
Connections:
- net 35CCU: now also U?.116 (Pin_116)
- net GLL_A0: now also U?.76 (Pin_76)
- net GLL_A1: now also U?.89 (Pin_89)
- net GLL_A10: now also U?.100 (Pin_100)
- net GLL_A11: now also U?.101 (Pin_101)
- net GLL_A12: now also U?.102 (Pin_102)
- net GLL_A13: now also U?.103 (Pin_103)
- net GLL_A14: now also U?.104 (Pin_104)
- net GLL_A15: now also U?.105 (Pin_105)
- net GLL_A16: now also U?.106 (Pin_106)
- net GLL_A17: now also U?.109 (Pin_109)
- net GLL_A18: now also U?.110 (Pin_110)
- net GLL_A19: now also U?.111 (Pin_111)
- net GLL_A2: now also U?.90 (Pin_90)
- net GLL_A20: now also U?.112 (Pin_112)
- net GLL_A3: now also U?.91 (Pin_91)
- net GLL_A4: now also U?.92 (Pin_92)
- net GLL_A5: now also U?.93 (Pin_93)
- net GLL_A6: now also U?.94 (Pin_94)
- net GLL_A7: now also U?.95 (Pin_95)
- net GLL_A8: now also U?.96 (Pin_96)
- net GLL_A9: now also U?.99 (Pin_99)
- net GLL_D0: now also U?.113 (Pin_113)
- net GLL_D1: now also U?.114 (Pin_114)
- net GLL_D2: now also U?.115 (Pin_115)
- net GLL_D3: now also U?.49 (Pin_49)
- net GLL_D4: now also U?.50 (Pin_50)
- net GLL_D5: now also U?.47 (Pin_47)
- net GLL_D6: now also U?.48 (Pin_48)
- net PULL_UP1: now also U?.1
- net VCC: now also U?.117 (Pin_117), U?.118 (Pin_118), U?.119 (Pin_119), U?.120 (Pin_120), U?.5 (Pin_5), U?.54 (Pin_54)
- net VSS: now also U?.107 (Pin_107), U?.108 (Pin_108), U?.15 (Pin_15), U?.16 (Pin_16), U?.2, U?.25 (Pin_25), U?.26 (Pin_26), U?.35 (Pin_35), U?.36 (Pin_36), U?.45 (Pin_45), U?.46 (Pin_46), U?.51 (Pin_51), U?.57 (Pin_57), U?.6, U?.60 (Pin_60), U?.61 (Pin_61), U?.68 (Pin_68), U?.69 (Pin_69), U?.74 (Pin_74), U?.75 (Pin_75), U?.78 (Pin_78), U?.79 (Pin_79), U?.87 (Pin_87), U?.88 (Pin_88), U?.97 (Pin_97), U?.98 (Pin_98)
- net ~{CE}R_CST: now also U?.3
- net ~{RST}_WD: now also U?.53 (Pin_53)
- net ~{STBY_WD}: now also U?.58 (Pin_58)
- new net P66: U?.66 (Pin_66)
- new net SCU_A24: U?.86 (Pin_86)
- new net ~{CS1}: U?.82 (Pin_82)
- new net ~{RST}_SCU: U?.56 (Pin_56)
Other:
- moved on the sheet: CP165, Q15, R67, R73, R86

Commit message: wip_cassette_scu
Other:
- added sheet cassette (cassette.kicad_sch)

Commit message: 74ls157#11
Parts:
- added U?: 74LS157, symbol jt74:74LS157
Changed lines of the file:
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@@
     (pin "1")
   )
+  (symbol (lib_id "jt74:74LS157") (at -33.02 132.08 0) (unit 1)
+    (in_bom yes) (on_board yes)
+    (property "Reference" "U?" (id 0) (at -27.94 119.38 0))
+    (property "Value" "74LS157" (id 1) (at -33.02 148.59 0))
+    (property "Footprint" "" (id 2) (at -33.02 132.08 0)
+      (effects (font (size 1.27 1.27)) hide)
+    )
+    (property "Datasheet" "http://www.ti.com/lit/gpn/sn74LS157" (id 3) (at -33.02 132.08 0)
+      (effects (font (size 1.27 1.27)) hide)
+    )
+    (pin "1")
+    (pin "10")
+    (pin "11")
+    (pin "12")
+    (pin "13")
+    (pin "14")
+    (pin "15")
+    (pin "2")
+    (pin "3")
+    (pin "4")
+    (pin "5")
+    (pin "6")
+    (pin "7")
+    (pin "9")
+  )
   (symbol (lib_id "Device:R_US") (at 93.98 181.61 90) (unit 1)
     (in_bom yes) (on_board yes)
@@
       (reference "U6") (unit 1) (value "FM1208S-250SC") (footprint "")
     )
+    (path "/3a38ea7a-7e6a-491f-ae4e-2c2342500859"
+      (reference "U?") (unit 1) (value "74LS157") (footprint "")
+    )
     (path "/665cca94-22a1-4cbd-b590-03ed84e6712d"
