File: cores/cps3/sch/simm_gfx.kicad_sch (KiCad schematic)
At the start: 32 parts

Commit message: update6_cps
Other:
- removed sheet plane_color
Changed lines of the file:
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@@
     (pin "9")
   )
-  (sheet (at 16.51 378.46) (size 59.69 24.13) (fields_autoplaced)
-    (stroke (width 0.1524) (type solid) (color 0 0 0 0))
-    (fill (color 0 0 0 0.0000))
-    (property "Sheet name" "plane_color" (id 0) (at 16.51 377.7484 0)
-      (effects (font (size 1.27 1.27)) (justify left bottom))
-    )
-    (property "Sheet file" "plane_color.kicad_sch" (id 1) (at 16.51 403.1746 0)
-      (effects (font (size 1.27 1.27)) (justify left top))
-    )
-  )
 )
