File: cores/cps3/sch/_autosave-simm_main.kicad_sch (KiCad schematic)
At the start: 8 parts

Commit message: clear_sch_hk_cr
Other:
- note added: "Warzard / Red Earth 64MBit 128MBit 128MBit 32MBit o 128MBit"
Changed lines of the file:
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@@
     )
+  )
+  (text "Warzard / Red Earth 	64MBit 		128MBit 	128MBit 	32MBit o 128MBit "
+    (at -53.34 62.23 0)
+    (effects (font (size 1.27 1.27) bold) (justify left bottom))
   )
   (text "The pattern table ?\n" (at 148.59 26.67 0)
