File: cores/cps3/sch/iou.kicad_sch (KiCad schematic)
At the start: 1 part

Commit message: iou
Parts:
- gave numbers to parts that had none: 1
Changed lines of the file:
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@@
   (symbol (lib_id "capcom:DL-2929-IOU") (at 209.55 137.16 0) (unit 1)
     (in_bom yes) (on_board yes)
-    (property "Reference" "U?" (id 0) (at 208.915 132.08 0)
+    (property "Reference" "F11" (id 0) (at 208.915 132.08 0)
       (effects (font (size 3.81 3.81)))
     )

Commit message: update_006
Changed lines of the file:
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@@
     (pin "125")
+    (pin "126")
     (pin "126")
     (pin "127")
@@
     (pin "205")
     (pin "206")
-    (pin "207")
     (pin "208")
     (pin "21")

Commit message: uptate_ns
Connections:
- net VSS: now reaches F11.10 (VSS)
- net VSS: now also F11.2 (VSS), F11.28 (VSS), F11.38 (VSS), F11.43 (VSS), F11.47 (VSS), F11.53 (VSS), F11.56 (VSS), F11.6 (VSS), F11.60 (VSS), F11.61 (VSS), F11.62 (VSS), F11.70 (VSS), F11.75 (VSS), F11.81 (VSS), F11.82 (VSS), F11.83 (VSS), F11.85 (VSS), F11.86 (VSS), F11.96 (VSS), F11.97 (VSS)
- net VCC: now reaches F11.109 (VCC)
- net VCC: now also F11.112 (VCC), F11.114 (VCC), F11.119 (VCC), F11.130 (VCC), F11.142 (VCC), F11.147 (VCC), F11.160 (VCC), F11.161 (VCC), F11.164 (VCC), F11.165 (VCC), F11.166 (VCC), F11.169 (VC2), F11.170 (VCC), F11.179 (VCC), F11.188 (VCC), F11.200 (VCC), F11.201 (VCC)
- net MAIN_D6: now reaches F11.11 (MAIN_D6)
- net MAIN_D7: now reaches F11.12 (MAIN_D7)
- net MAIN_D8: now reaches F11.13 (MAIN_D8)
- net MAIN_D9: now reaches F11.14 (MAIN_D9)
- net MAIN_D10: now reaches F11.16 (MAIN_D10)
- net MAIN_D11: now reaches F11.17 (MAIN_D11)
- net MAIN_D12: now reaches F11.18 (MAIN_D12)
- net MAIN_D13: now reaches F11.19 (MAIN_D13)
- net MAIN_D14: now reaches F11.20 (MAIN_D14)
- net MAIN_D15: now reaches F11.21 (MAIN_D15)
- net MAIN_A0: now reaches F11.22 (MAIN_A0)
- net MAIN_A1: now reaches F11.23 (MAIN_A1)
- net MAIN_A2: now reaches F11.24 (MAIN_A2)
- net MAIN_A3: now reaches F11.25 (MAIN_A3)
- net MAIN_A4: now reaches F11.26 (MAIN_A4)
- net MAIN_A5: now reaches F11.27 (MAIN_A5)
- net MAIN_A6: now reaches F11.29 (MAIN_A6)
- net MAIN_D0: now reaches F11.3 (MAIN_D0)
- net MAIN_A7: now reaches F11.30 (MAIN_A7)
- net MAIN_A8: now reaches F11.31 (MAIN_A8)
- net MAIN_A9: now reaches F11.32 (MAIN_A9)
- net MAIN_A10: now reaches F11.33 (MAIN_A10)
- net MAIN_A11: now reaches F11.34 (MAIN_A11)
- net MAIN_A12: now reaches F11.35 (MAIN_A12)
- net MAIN_A13: now reaches F11.36 (MAIN_A13)
- net CBI_D0: now reaches F11.37 (CBI_D0)
- net CBI_D1: now reaches F11.39 (CBI_D1)
- net MAIN_D1: now reaches F11.4 (MAIN_D1)
- net CBI_D2: now reaches F11.40 (CBI_D2)
- net CBI_D3: now reaches F11.41 (CBI_D3)
- net CBI_D4: now reaches F11.42 (CBI_D4)
- net CBI_D5: now reaches F11.44 (CBI_D5)
- net CBI_D6: now reaches F11.45 (CBI_D6)
- net CBI_D7: now reaches F11.46 (CBI_D7)
- net MAIN_D2: now reaches F11.5 (MAIN_D2)
- net MAIN_D3: now reaches F11.7 (MAIN_D3)
- net MAIN_D4: now reaches F11.8 (MAIN_D4)
- net MAIN_D5: now reaches F11.9 (MAIN_D5)
Other:
- note added: "CON SALIDA"
- note added: "SIN SALIDA"

Commit message: update_cps3
Parts:
- added A13, A14: 2501, symbol Nec:2501
- added R1: 103Ω, Resistor_THT:R_Array_SIP5, symbol Device:R_Network_Dividers_x03_SIP
- added R2: R_Network08, Resistor_THT:R_Array_SIP9, symbol Device:R_Network08
Connections:
- net CBI_D0 is gone; now on net MAIN_D7: F11.37 (MAIN_D7)
- net CBI_D1 is gone; now on net MAIN_D6: F11.39 (MAIN_D6)
- net CBI_D2 is gone; now on net MAIN_D5: F11.40 (MAIN_D5)
- net CBI_D3 is gone; now on net MAIN_D4: F11.41 (MAIN_D4)
- net CBI_D4 is gone; now on net MAIN_D3: F11.42 (MAIN_D3)
- net CBI_D5 is gone; now on net MAIN_D2: F11.44 (MAIN_D2)
- net CBI_D6 is gone; now on net MAIN_D1: F11.45 (MAIN_D1)
- net CBI_D7 is gone; now on net MAIN_D0: F11.46 (MAIN_D0)
- net MAIN_A0 is gone; now on net MAIN_A13: F11.22 (MAIN_A13)
- net MAIN_A1 is gone; now on net MAIN_A12: F11.23 (MAIN_A12)
- net MAIN_A2 is gone; now on net MAIN_A11: F11.24 (MAIN_A11)
- net MAIN_A3 is gone; now on net MAIN_A10: F11.25 (MAIN_A10)
- net MAIN_A5 is gone; now on net MAIN_A8: F11.27 (MAIN_A8)
- net MAIN_A10: no longer F11.33 (MAIN_A10)
- net MAIN_A11: no longer F11.34 (MAIN_A11)
- net MAIN_A12: no longer F11.35 (MAIN_A12)
- net MAIN_A13: no longer F11.36 (MAIN_A13)
- net MAIN_A4: now also F11.3 (MAIN_A4); no longer F11.26 (MAIN_A4)
- net MAIN_A6: now also F11.4 (MAIN_A6); no longer F11.29 (MAIN_A6)
- net MAIN_A7: now also F11.5 (MAIN_A7); no longer F11.30 (MAIN_A7)
- net MAIN_A8: no longer F11.31 (MAIN_A8)
- net MAIN_A9: now also F11.26 (MAIN_A9); no longer F11.32 (MAIN_A9)
- net MAIN_D0: no longer F11.3 (MAIN_D0)
- net MAIN_D1: no longer F11.4 (MAIN_D1)
- net MAIN_D10: now also F11.33 (MAIN_D10); no longer F11.16 (MAIN_D10)
- net MAIN_D11: now also F11.32 (MAIN_D11); no longer F11.17 (MAIN_D11)
- net MAIN_D12: now also F11.31 (MAIN_D12); no longer F11.18 (MAIN_D12)
- net MAIN_D13: now also F11.30 (MAIN_D13); no longer F11.19 (MAIN_D13)
- net MAIN_D14: now also F11.29 (MAIN_D14); no longer F11.20 (MAIN_D14)
- net MAIN_D2: no longer F11.5 (MAIN_D2)
- net MAIN_D3: no longer F11.7 (MAIN_D3)
- net MAIN_D4: no longer F11.8 (MAIN_D4)
- net MAIN_D5: no longer F11.9 (MAIN_D5)
- net MAIN_D6: no longer F11.11 (MAIN_D6)
- net MAIN_D7: no longer F11.12 (MAIN_D7)
- net MAIN_D8: now also F11.35 (MAIN_D8); no longer F11.13 (MAIN_D8)
- net MAIN_D9: now also F11.34 (MAIN_D9); no longer F11.14 (MAIN_D9)
- net VCC: now also F11.50 (A3), R1.2 (R1), R2.1 (common); no longer F11.169 (VC2)
- net VSS: now also F11.104 (VSS), F11.106 (VSS), F11.108 (VSS), A13.11, A13.13, A13.15, A13.9, A14.11, A14.13, A14.15, A14.2, A14.4, A14.6, A14.8, A14.9
- net IO_SND41: now reaches F11.100 (BES_A4-1)
- net IO_SND32: now reaches F11.101 (BES_A3-2)
- net IOU116: now reaches F11.116 (~{WEH})
- net IOU116: now also A13.16, R1.1 (COM1)
- net IOU117: now reaches F11.117 (RAMD15)
- net IOU117: now also A13.12, R1.5 (COM2)
- net IO_SND31: now reaches F11.99 (BES_A3-1)
- net MAIN_D15 renamed MAIN_A14
- new net: A13.1, R2.2 (R1)
- new net: A13.10, R1.4 (R3)
- new net: A13.14, R1.3 (R2)
- new net: A13.2, A14.16
- new net: A13.3, R2.4 (R3)
- new net: A13.4, A14.14
- new net: A13.5, R2.6 (R5)
- new net: A13.6, A14.12
- new net: A13.7, R2.8 (R7)
- new net: A13.8, A14.10
- new net ALE: F11.36 (ALE)
- new net MAIN_A15: F11.20 (MAIN_A15)
- new net MAIN_A16: F11.19 (MAIN_A16)
- new net MAIN_A17: F11.18 (MAIN_A17)
- new net MAIN_A18: F11.17 (MAIN_A18)
- new net MAIN_A19: F11.16 (MAIN_A19)
- new net MAIN_A20: F11.14 (MAIN_A20)
- new net MAIN_A21: F11.13 (MAIN_A21)
- new net MAIN_A22: F11.12 (MAIN_A22)
- new net MAIN_A23: F11.11 (MAIN_A23)
- new net MAIN_A24: F11.9 (MAIN_A24)
- new net MAIN_A25: F11.8 (MAIN_A25)
- new net MAIN_A26: F11.7 (MAIN_A26)
- no-connect marks 0 -> 4

Commit message: update5
Connections:
- net ALE is gone; now on net MAIN_A6: F11.36 (MAIN_D6)
- net MAIN_A14 is gone; now on net MAIN_D14: F11.21 (MAIN_D14)
- net MAIN_A25 is gone; now on net MAIN_A4: F11.8 (MAIN_A4)
- net MAIN_A26 is gone; now on net MAIN_A4: F11.7 (MAIN_A5)
- net MAIN_A10: now also F11.32 (MAIN_D10); no longer F11.25 (MAIN_A10)
- net MAIN_A11: now also F11.31 (MAIN_D11); no longer F11.24 (MAIN_A11)
- net MAIN_A12: now also F11.30 (MAIN_D12); no longer F11.23 (MAIN_A12)
- net MAIN_A13: now also F11.29 (MAIN_D13); no longer F11.22 (MAIN_A13)
- net MAIN_A4: no longer F11.3 (MAIN_A4)
- net MAIN_A6: no longer F11.4 (MAIN_A6)
- net MAIN_A7: now also F11.35 (MAIN_D7); no longer F11.5 (MAIN_A7)
- net MAIN_A8: now also F11.34 (MAIN_D8); no longer F11.27 (MAIN_A8)
- net MAIN_A9: now also F11.33 (MAIN_D9); no longer F11.26 (MAIN_A9)
- net MAIN_D10: now also F11.25 (MAIN_D10); no longer F11.33 (MAIN_D10)
- net MAIN_D11: now also F11.24 (MAIN_D11); no longer F11.32 (MAIN_D11)
- net MAIN_D12: now also F11.23 (MAIN_D12); no longer F11.31 (MAIN_D12)
- net MAIN_D13: now also F11.22 (MAIN_D13); no longer F11.30 (MAIN_D13)
- net MAIN_D14: no longer F11.29 (MAIN_D14)
- net MAIN_D8: now also F11.27 (MAIN_D8); no longer F11.35 (MAIN_D8)
- net MAIN_D9: now also F11.26 (MAIN_D9); no longer F11.34 (MAIN_D9)
- net MAIN_A15 renamed MAIN_D15
- net MAIN_A16 renamed MAIN_D16
- net MAIN_A17 renamed MAIN_D17
- net MAIN_A18 renamed MAIN_D18
- net MAIN_A19 renamed MAIN_D19
- net MAIN_A20 renamed MAIN_D20
- net MAIN_A21 renamed MAIN_D21
- net MAIN_A22 renamed MAIN_D22
- net MAIN_A23 renamed MAIN_D23
- net MAIN_A24 renamed MAIN_A3
- new net MAIN_A0: F11.3 (MAIN_A0)
- new net MAIN_A1: F11.4 (MAIN_A1)
- new net MAIN_A2: F11.5 (MAIN_A2)

Commit message: update6_cps
Parts:
- added CP0, CP1: CP, symbol Device:C_Polarized_Small_US
- added R76: 105Ω, symbol Device:R_US
- added R77: 330Ω, symbol Device:R_US
- added R84: 101Ω, symbol Device:R_US
- added XTAL3: 3.6864MHz, symbol Device:Crystal_Small
Connections:
- net VCC: no longer F11.50 (A3)
- net VSS: now also F11.207 (VSS), CP0.2, CP1.2
- net RESET?: now reaches F11.1 (RESET?)
- net RESET?: now also R84.1, R84.2
- net GLL2IO0: now reaches F11.208 (GLL2IO0)
- net GLL2IO1: now reaches F11.48 (GLL2IO1)
- net SU2IO0: now reaches F11.49 (SSU2IO0)
- net at F11.54 (XTAL_3.6864MHz): now also CP1.1, R76.1, XTAL3.2
- net IOU116 renamed COLL0
- net IOU117 renamed COLL1
- new net: CP0.1, R77.1, XTAL3.1
- new net: R76.2, R77.2
Other:
- note added: "1. Anode 2. Cathode 15. Emitter 16. Collector"
- note added: "PHOTOCOUPLER"
- moved on the sheet: A13, A14, R1, R2

Commit message: clear_sch_hk_cr
Parts:
- added B11, B12: TD62064, symbol toshiba:TD62064
- added CN1: Conn_01x34_Male, symbol Connector:Conn_01x34_Male
- added FB13, FB14, FB16, FB17, FB18 (x2): FB, symbol Device:FerriteBead_Small
Connections:
- net COLL0: no longer F11.116 (COLLECTOR0)
- net COLL1: now also A13.14, R1.3 (R2); no longer A13.12, F11.117 (COLLECTOR1), R1.5 (COM2)
- net VCC: now also F11.176 (D12), F11.177 (D11), F11.178 (D10), F11.181 (D7), F11.182 (D6), F11.183 (D5), F11.184 (D4), F11.186 (D3), F11.82 (VCC), F11.83 (VCC), F11.85 (VCC), F11.86 (VCC), CN1.3 (Pin_3), CN1.4 (Pin_4)
- net VSS: now also B12.12 (GND), B12.13 (GND), B12.4 (GND), B12.5 (GND), CN1.1 (Pin_1), CN1.2 (Pin_2), CN1.31 (Pin_31), CN1.32 (Pin_32), CN1.33 (Pin_33), CN1.34 (Pin_34); no longer F11.82 (VCC), F11.83 (VCC), F11.85 (VCC), F11.86 (VCC)
- net BA: now reaches CP0.1, R77.1, XTAL3.1
- net BA: now also F11.55 (BUFFER_A)
- net COLL3: now reaches A13.10, R1.4 (R3)
- net CLL2_0: now reaches A13.2, A14.16
- net CLL2_0: now also CN1.28 (Pin_28), FB18.2
- net CLL2_1: now reaches A13.4, A14.14
- net CLL2_1: now also CN1.27 (Pin_27), FB16.2
- net CLL2_2: now reaches A13.6, A14.12
- net CLL2_2: now also CN1.26 (Pin_26), FB17.1
- net CLL2_3: now reaches A13.8, A14.10
- net CLL2_3: now also CN1.25 (Pin_25), FB18.1
- net MAIN_A0 renamed GFX_A0
- net MAIN_A1 renamed GFX_A1
- net MAIN_A10 renamed GFX_A10
- net MAIN_A11 renamed GFX_A11
- net MAIN_A12 renamed GFX_A12
- net MAIN_A13 renamed GFX_A13
- net MAIN_A2 renamed GFX_A2
- net MAIN_A3 renamed GFX_A3
- net MAIN_A4 renamed GFX_A4
- net MAIN_A6 renamed GFX_A6
- net MAIN_A7 renamed GFX_A7
- net MAIN_A8 renamed GFX_A8
- net MAIN_A9 renamed GFX_A9
- new net: B12.7 (O2), FB14.1
- new net: CN1.7 (Pin_7), FB14.2
- new net: CN1.8 (Pin_8), FB13.1
- new net: B12.2 (O1), FB13.2
- new net +12V: CN1.5 (Pin_5), CN1.6 (Pin_6)
- new net 1P_BTN4: CN1.19 (Pin_19)
- new net 1P_BTN5: CN1.17 (Pin_17)
- new net 1P_BTN6: CN1.15 (Pin_15)
- new net 2P_BTN4: CN1.21 (Pin_21)
- new net 2P_BTN5: CN1.23 (Pin_23)
- new net 2P_BTN6: CN1.9 (Pin_9)
- new net COLL2: A13.12, R1.5 (COM2)
- new net CR10_P8: CN1.13 (Pin_13)
- new net CR11_P2: CN1.29 (Pin_29)
- new net CR11_P4: CN1.30 (Pin_30)
- new net CR5_P2: CN1.12 (Pin_12)
- new net CR5_P4: CN1.11 (Pin_11)
- new net CR6_P2: CN1.10 (Pin_10)
- new net CR8_P2: CN1.24 (Pin_24)
- new net CR8_P4: CN1.22 (Pin_22)
- new net CR9_P2: CN1.20 (Pin_20)
- new net CR9_P4: CN1.18 (Pin_18)
- new net CR9_P6: CN1.16 (Pin_16)
- new net CR9_P8: CN1.14 (Pin_14)
Other:
- note added: "Ferrite Bead"
- note added: "Kick Harness"
- moved on the sheet: A13, A14, CP0, CP1, R1, R2, R76, R77, XTAL3
