File: cores/cps3/sch/iou.kicad_sch (KiCad schematic)
At the start: 20 parts, among them CN1 Conn_01x34_Male

Commit message: iou_jm_kh
Parts:
- added CR1, CR10, CR11, CR2, CR3, CR4, CR5, CR6, CR7, CR8, CR9: CRE438-60, symbol arcade:CRE438-60
Connections:
- net 2P_BTN6: now also CR6.4 (R1)
- net CR10_P8: now also CR10.8 (R3)
- net CR11_P2: now also CR11.2 (R0)
- net CR11_P4: now also CR11.4 (R1)
- net CR5_P2: now also CR5.2 (R0)
- net CR5_P4: now also CR5.4 (R1)
- net CR6_P2: now also CR6.2 (R0)
- net CR8_P2: now also CR8.2 (R0)
- net CR8_P4: now also CR8.4 (R1)
- net CR9_P2: now also CR9.2 (R0)
- net CR9_P4: now also CR9.4 (R1)
- net CR9_P6: now also CR9.6 (R2)
- net CR9_P8: now also CR9.8 (R3)
- net VCC: now also CR1.1 (VCC), CR10.1 (VCC), CR11.1 (VCC), CR2.1 (VCC), CR3.1 (VCC), CR4.1 (VCC), CR5.1 (VCC), CR6.1 (VCC), CR7.1 (VCC), CR8.1 (VCC), CR9.1 (VCC)
- net VSS: now also B11.12 (GND), B11.13 (GND), B11.4 (GND), B11.5 (GND), CR1.10 (VSS), CR10.10 (VSS), CR11.10 (VSS), CR2.10 (VSS), CR3.10 (VSS), CR4.10 (VSS), CR5.10 (VSS), CR6.10 (VSS), CR7.10 (VSS), CR8.10 (VSS), CR9.10 (VSS)
- new net 1P_BNT_1: CR3.8 (R3)
- new net 1P_BNT_2: CR3.6 (R2)
- new net 1P_BNT_3: CR3.4 (R1)
- new net 1P_BNT_4: CR10.2 (R0), CR3.2 (R0)
- new net 1P_BNT_5: CR10.4 (R1)
- new net 1P_BNT_6: CR10.6 (R2)
- new net 1P_DOWN: CR4.6 (R2)
- new net 1P_LEFT: CR4.4 (R1)
- new net 1P_RIGHT: CR4.2 (R0)
- new net 1P_START: CR5.6 (R2)
- new net 1P_UP: CR4.8 (R3)
- new net 2P_BNT_1: CR1.8 (R3)
- new net 2P_BNT_2: CR1.6 (R2)
- new net 2P_BNT_3: CR1.4 (R1)
- new net 2P_BNT_4: CR1.2 (R0), CR8.8 (R3)
- new net 2P_BNT_5: CR8.6 (R2)
- new net 2P_DOWN: CR2.6 (R2)
- new net 2P_LEFT: CR2.4 (R1)
- new net 2P_RIGHT: CR2.2 (R0)
- new net 2P_START: CR5.8 (R3)
- new net 2P_UP: CR2.8 (R3)
- new net COIN_1: CR6.8 (R3)
- new net COIN_2: CR6.6 (R2)
- new net IOU127: CR8.7 (C2)
- new net IOU128: CR8.9 (C3)
- new net IOU129: CR10.3 (C0)
- new net IOU131: CR10.5 (C1)
- new net IOU132: CR10.7 (C2)
- new net IOU133: CR10.9 (C3)
- new net IOU157: CR6.5 (C1)
- new net N.C: CR7.2 (R0)
- new net N.C1: CR7.4 (R1)
- new net SERVICE: CR7.6 (R2)
- no-connect marks 4 -> 10
Other:
- moved on the sheet: A13, A14, B11, B12, CN1, CP0, CP1, F11, FB13, FB14, FB16, FB17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

Commit message: update7
Parts:
- added RN1: R_Pack04, symbol Device:R_Pack04
Connections:
- net COLL0 is gone; now on net P_C0: A13.16, R1.1 (COM1)
- net COLL1 is gone; now on net P_C2: A13.14, R1.3 (R2)
- net COLL2 is gone; now on net P_C1: A13.12, R1.5 (COM2)
- net COLL3 is gone; now on net P_C3: A13.10, R1.4 (R3)
- net IOU127 is gone; now on an unnamed net: CR8.7 (C2)
- net IOU128 is gone; now on an unnamed net: CR8.9 (C3)
- net IOU129 is gone; now on an unnamed net: CR10.3 (C0)
- net IOU131 is gone; now on an unnamed net: CR10.5 (C1)
- net IOU132 is gone; now on an unnamed net: CR10.7 (C2)
- net IOU133 is gone; now on an unnamed net: CR10.9 (C3)
- net IOU157 is gone; now on an unnamed net: CR6.5 (C1)
- net 1P_BNT_4: no longer CR10.2 (R0)
- net 2P_BNT_4: no longer CR8.8 (R3)
- net CLL2_0: now also FB18.1
- net CLL2_1: now also FB16.1
- net CLL2_2: now also FB17.2
- net CLL2_3: now also FB18.2
- net GLL2IO0: now also F11.49 (SSU2IO0); no longer F11.208 (GLL2IO0)
- net RESET?: no longer F11.1 (RESET?), R84.2
- net SU2IO0: now also F11.208 (GLL2IO0); no longer F11.49 (SSU2IO0)
- net VCC: now also F11.10 (VCC), F11.104 (VCC), F11.106 (VCC), F11.108 (VCC), F11.15 (VCC), F11.2 (VCC), F11.28 (VCC), F11.38 (VCC), F11.43 (VCC), F11.47 (VCC), F11.53 (VCC), F11.56 (VCC), F11.6 (VCC), F11.60 (VCC), F11.61 (VCC), F11.62 (VCC), F11.70 (VCC), F11.75 (VCC), F11.81 (VCC), F11.96 (VCC), F11.97 (VCC); no longer F11.109 (VCC), F11.112 (VCC), F11.114 (VCC), F11.119 (VCC), F11.130 (VCC), F11.142 (VCC), F11.147 (VCC), F11.160 (VCC), F11.161 (VCC), F11.164 (VCC), F11.165 (VCC), F11.166 (VCC), F11.170 (VCC), F11.176 (D12), F11.177 (D11), F11.178 (D10), F11.179 (VCC), F11.181 (D7), F11.182 (D6), F11.183 (D5), F11.184 (D4), F11.186 (D3), F11.188 (VCC), F11.200 (VCC), F11.201 (VCC), F11.82 (VCC), F11.83 (VCC), F11.85 (VCC), F11.86 (VCC)
- net VSS: now also F11.109 (VSS), F11.112 (VSS), F11.114 (VSS), F11.119 (VSS), F11.130 (VSS), F11.142 (VSS), F11.147 (VSS), F11.160 (VSS), F11.161 (VSS), F11.164 (VSS), F11.165 (VSS), F11.166 (VSS), F11.170 (VSS), F11.179 (VSS), F11.188 (VSS), F11.200 (VSS), F11.201 (VSS), F11.82 (VSS), F11.83 (VSS), F11.85 (VSS), F11.86 (VSS); no longer F11.10 (VSS), F11.104 (VSS), F11.106 (VSS), F11.108 (VSS), F11.2 (VSS), F11.28 (VSS), F11.38 (VSS), F11.43 (VSS), F11.47 (VSS), F11.53 (VSS), F11.56 (VSS), F11.6 (VSS), F11.60 (VSS), F11.61 (VSS), F11.62 (VSS), F11.70 (VSS), F11.75 (VSS), F11.81 (VSS), F11.96 (VSS), F11.97 (VSS)
- net at CR4.3 (C0): now also F11.148 (1P_RIGHT)
- net at CR4.5 (C1): now also F11.149 (1P_LEFT)
- net at CR4.7 (C2): now also F11.150 (1P_DOWN)
- net at CR4.9 (C3): now also F11.151 (1P_UP)
- net at CR2.3 (C0): now also F11.138 (2P_RIGHT)
- net at CR2.5 (C1): now also F11.139 (2P_LEFT)
- net at CR2.7 (C2): now also F11.140 (2P_DOWN)
- net at CR2.9 (C3): now also F11.141 (2P_UP)
- net at CR7.3 (C0): now also F11.167 (N.C_JAMMA)
- net at CR7.5 (C1): now also F11.168 (N.C1_JAMMA)
- net at CR7.7 (C2): now also F11.169 (SERVICE)
- net at CR11.3 (C0): now also F11.162 (K_H29)
- net at CR11.5 (C1): now also F11.163 (K_H30)
- net at CR1.3 (C0): now also F11.134 (2P_BTN4)
- net at CR1.5 (C1): now also F11.135 (2P_BTN3)
- net at CR1.7 (C2): now also F11.136 (2P_BTN2)
- net at CR1.9 (C3): now also F11.137 (2P_BTN1)
- net at CR5.3 (C0): now also F11.152 (K_H12)
- net at CR5.5 (C1): now also F11.153 (K_H11)
- net at CR5.7 (C2): now also F11.154 (1P_STAR)
- net at CR5.9 (C3): now also F11.155 (2P_STAR)
- net at CR8.3 (C0): now also F11.123 (K_H16)
- net at CR8.5 (C1): now also F11.124 (K_H14)
- net P_C0: now reaches F11.116 (P_COUPLER0)
- net P_C1: now reaches F11.117 (P_COUPLER1)
- net at F11.118 (K_H24): now also CR9.3 (C0)
- net at F11.120 (K_H22): now also CR9.5 (C1)
- net at F11.121 (K_H20): now also CR9.7 (C2)
- net at F11.122 (K_H18): now also CR9.9 (C3)
- net P_C2: now reaches F11.125 (P_COUPLER2)
- net P_C3: now reaches F11.126 (P_COUPLER3)
- net at F11.143 (1P_BTN4): now also CR3.3 (C0)
- net at F11.144 (1P_BTN3): now also CR3.5 (C1)
- net at F11.145 (1P_BTN2): now also CR3.7 (C2)
- net at F11.146 (1P_BTN1): now also CR3.9 (C3)
- net at F11.156 (K_H10): now also CR6.3 (C0)
- net at F11.158 (COIN_2): now also CR6.7 (C2)
- net at F11.159 (COIN_1): now also CR6.9 (C3)
- net at F11.193 (P_COUPLER4): now also RN1.1 (R1.1)
- net at F11.194 (P_COUPLER5): now also RN1.2 (R2.1)
- net at F11.195 (P_COUPLER6): now also RN1.3 (R3.1)
- net at F11.196 (P_COUPLER7): now also RN1.4 (R4.1)
- net at A14.1: now also RN1.8 (R1.2)
- net at A14.3: now also RN1.7 (R2.2)
- net at A14.5: now also RN1.6 (R3.2)
- net at A14.7: now also RN1.5 (R4.2)
- net 1P_BTN4 renamed KH_2P_BTN4
- net KH_2P_BTN4: now also CR8.8 (R3)
- net 2P_BTN4 renamed KH_1P_BTN4
- net KH_1P_BTN4: now also CR10.2 (R0)
- net CR10_P8 renamed K_H13
- net CR11_P2 renamed K_H29
- net K_H29: now also CR11.4 (R1); no longer CR11.2 (R0)
- net CR11_P4 renamed K_H30
- net K_H30: now also CR11.2 (R0); no longer CR11.4 (R1)
- net CR5_P2 renamed K_H12
- net CR5_P4 renamed K_H11
- net CR6_P2 renamed K_H10
- net CR8_P2 renamed K_H16
- net K_H16: now also CN1.16 (Pin_16); no longer CN1.24 (Pin_24)
- net CR8_P4 renamed K_H14
- net K_H14: now also CN1.14 (Pin_14); no longer CN1.22 (Pin_22)
- net CR9_P2 renamed K_H20
- net K_H20: now also CR9.6 (R2); no longer CR9.2 (R0)
- net CR9_P4 renamed K_H18
- net K_H18: now also CR9.8 (R3); no longer CR9.4 (R1)
- removed net CR9_P6: CN1.16 (Pin_16), CR9.6 (R2)
- removed net CR9_P8: CN1.14 (Pin_14), CR9.8 (R3)
- net GFX_A0 renamed MAIN_A0
- net GFX_A1 renamed MAIN_A1
- net GFX_A10 renamed MAIN_A10
- net GFX_A11 renamed MAIN_A11
- net GFX_A12 renamed MAIN_A12
- net GFX_A13 renamed MAIN_A13
- net GFX_A2 renamed MAIN_A2
- net GFX_A3 renamed MAIN_A3
- net GFX_A4 renamed MAIN_A4
- net MAIN_A4: no longer F11.7 (MAIN_A5)
- net GFX_A6 renamed MAIN_A6
- net GFX_A7 renamed MAIN_A7
- net GFX_A8 renamed MAIN_A8
- net GFX_A9 renamed MAIN_A9
- new net: F11.1 (RESET?), R84.2
- new net K_H22: CN1.22 (Pin_22), CR9.4 (R1)
- new net K_H24: CN1.24 (Pin_24), CR9.2 (R0)
- new net MAIN_A5: F11.7 (MAIN_A5)
Other:
- note added: "NO OUTPUT OBSERVED PHYSICAL SIGNAL. PENDING TO VERIFY"
- note removed: "CON SALIDA"
- note removed: "SIN SALIDA"
- moved on the sheet: A13, A14, B11, B12, CN1, CP0, CP1, CR1, CR10, CR11, CR2, CR3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

Commit message: snd_colmix
Parts:
- added CP124: 10μF, symbol Device:C_Polarized_US
- added CP125: 47μF, symbol Device:C_Polarized_US
- added FB? (x4): F_Small, symbol Device:L_Ferrite_Small
Connections:
- new net: CP124.1, CP125.1, FB?.2, FB?.2, FB?.2, FB?.2
- new net: CP124.2, CP125.2, FB?.1, FB?.1, FB?.1, FB?.1

Commit message: wip_colmix_snd
Parts:
- added SW1: SW_MEC_5G, symbol Switch:SW_MEC_5G
- gave numbers to parts that had none: 4
Connections:
- net N.C1: now also SW1.3 (B), SW1.4 (B)
- net VCC: now also CP124.1, CP125.1, FB10.2, FB7.2, FB8.2, FB9.2
- net VSS: now also CP124.2, CP125.2, FB10.1, FB7.1, FB8.1, FB9.1, SW1.1 (A), SW1.2 (A)
Other:
- note added: "GP1"
- note added: "TEST"
- moved on the sheet: CP124, CP125, FB10, FB7, FB8, FB9

Commit message: wip_cps3_vdac
Connections:
- net IO_SND31 renamed APP0
- net IO_SND32 renamed APP1
- net IO_SND41 renamed APP2
Changed lines of the file:
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@@
     (effects (font (size 1.27 1.27)) (justify left bottom))
   )
-  (hierarchical_label "IO_SND32" (shape output) (at 293.37 57.15 0)
+  (hierarchical_label "APP1" (shape output) (at 293.37 54.61 0)
     (effects (font (size 1.27 1.27)) (justify left))
   )
@@
     (effects (font (size 1.27 1.27)) (justify right))
   )
-  (hierarchical_label "IO_SND31" (shape output) (at 293.37 52.07 0)
+  (hierarchical_label "APP0" (shape output) (at 293.37 52.07 0)
     (effects (font (size 1.27 1.27)) (justify left))
   )
@@
     (effects (font (size 1.27 1.27)) (justify right))
   )
-  (hierarchical_label "IO_SND41" (shape output) (at 293.37 54.61 0)
+  (hierarchical_label "APP2" (shape output) (at 293.37 57.15 0)
     (effects (font (size 1.27 1.27)) (justify left))
   )

Commit message: wip_gfx_gll
Connections:
- net GLL2IO0 is gone; now on net SU2IO0: F11.49 (SSU2IO0)
- net MAIN_A0: now also F11.29 (MAIN_D13); no longer F11.3 (MAIN_A0)
- net MAIN_A1: now also F11.30 (MAIN_D12); no longer F11.4 (MAIN_A1)
- net MAIN_A10: now also F11.9 (MAIN_A3); no longer F11.32 (MAIN_D10)
- net MAIN_A11: now also F11.5 (MAIN_A2); no longer F11.31 (MAIN_D11)
- net MAIN_A12: now also F11.4 (MAIN_A1); no longer F11.30 (MAIN_D12)
- net MAIN_A13: now also F11.3 (MAIN_A0); no longer F11.29 (MAIN_D13)
- net MAIN_A2: now also F11.31 (MAIN_D11); no longer F11.5 (MAIN_A2)
- net MAIN_A3: now also F11.32 (MAIN_D10); no longer F11.9 (MAIN_A3)
- net MAIN_A4: now also F11.33 (MAIN_D9); no longer F11.8 (MAIN_A4)
- net MAIN_A5: now also F11.34 (MAIN_D8); no longer F11.7 (MAIN_A5)
- net MAIN_A6: now also F11.35 (MAIN_D7); no longer F11.36 (MAIN_D6)
- net MAIN_A7: now also F11.36 (MAIN_D6); no longer F11.35 (MAIN_D7)
- net MAIN_A8: now also F11.7 (MAIN_A5); no longer F11.34 (MAIN_D8)
- net MAIN_A9: now also F11.8 (MAIN_A4); no longer F11.33 (MAIN_D9)
- net SU2IO0: no longer F11.208 (GLL2IO0)
- net GLL2IO1 renamed GLL_DRIVER3
- new net GLL_DRIVER1: F11.208 (GLL2IO0)

Commit message: wip_gll_cassette
Connections:
- net RESET? renamed GLL2IOU0
Changed lines of the file:
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@@
     (effects (font (size 1.27 1.27)) (justify right))
   )
-  (hierarchical_label "RESET?" (shape input) (at 114.3 31.75 180)
+  (hierarchical_label "GLL2IOU0" (shape input) (at 114.3 31.75 180)
     (effects (font (size 1.27 1.27)) (justify right))
   )

Commit message: wip_iou_wd
Parts:
- removed B11: TD62064, symbol toshiba:TD62064
- added C11: TD62064, symbol toshiba:TD62064
- added E13: AT93C46-10SC, symbol arcade:AT93C46-10SC
- added R64, R78: 472Ω, symbol Device:R_US
- added R71, R80: 103Ω, symbol Device:R_US
- added R79: 102Ω, symbol Device:R_US
- renumbered B12 to C12
Connections:
- net +12V: now also C12.1 (COM), C12.8 (COM), C11.1 (COM), C11.8 (COM)
- net VCC: now also F11.171 (UK), E13.6 (ORG), E13.8 (VCC), R64.2, R71.2, R78.2, R79.2, R80.2; no longer F11.70 (VCC)
- net VSS: now also F11.70 (VSS), C11.12 (GND), C11.13 (GND), C11.3 (I1), C11.4 (GND), C11.5 (GND), C11.6 (I2), E13.5 (VSS)
- net at RN1.1 (R1.1): now also F11.194 (P_COUPLER5); no longer F11.193 (P_COUPLER4)
- net at RN1.2 (R2.1): now also F11.195 (P_COUPLER6); no longer F11.194 (P_COUPLER5)
- net at RN1.3 (R3.1): now also F11.196 (P_COUPLER7); no longer F11.195 (P_COUPLER6)
- net at RN1.4 (R4.1): now also F11.103 (VSS); no longer F11.196 (P_COUPLER7)
- net 1DSD_I3: now reaches C12.11 (I3)
- net 1DSD_I3: now also F11.205 (XI3)
- net 1DSD_I4: now reaches C12.14 (I4)
- net 1DSD_I4: now also F11.206 (XI4)
- net 1DSD_I1: now reaches C12.3 (I1)
- net 1DSD_I1: now also F11.203 (XI1)
- net 1DSD_I2: now reaches C12.6 (I2)
- net 1DSD_I2: now also F11.204 (XI2)
- net GLL2CCU5: now reaches F11.111 (GLL2CCU5)
- net at F11.115 (PULL_UP): now also R64.1
- net ~{RESET5}: now reaches F11.189 (~{RESET5})
- net 2GLL2IOU0: now reaches F11.190 (2GLL2IOU0)
- net DSD_I3: now reaches F11.199 (I3)
- net DSD_I4: now reaches F11.202 (I4)
- net at F11.63 (PULL_UP): now also R80.1
- net at F11.64 (PULL_UP): now also R78.1
- net at F11.65 (PULL_UP): now also R79.1
- net at F11.71 (D0): now also E13.4 (DO)
- net at F11.72 (DI): now also E13.3 (DI)
- net at F11.73 (SCLK): now also E13.2 (SCLK)
- net at F11.74 (CS): now also E13.1 (CS)
- net at F11.76 (PULL_UP): now also R71.1
- net GLL_DRIVER1 renamed DRIVER_GLL1
- net GLL_DRIVER3 renamed DRIVER_GLL3
- net MAIN_A13 renamed DRIVER_GLL4
- new net 2DSD_I3: C11.11 (I3)
- new net 2DSD_I4: C11.14 (I4)
- new net P_C4: F11.193 (P_COUPLER4)
- no-connect marks 10 -> 17
Other:
- note added: "4CH HIGH−CURRENT DARLINGTON SINK DRIVER"
- note added: "64/128/256 words of 16 bits each. According to programming"
- note removed: "NO OUTPUT OBSERVED PHYSICAL SIGNAL. PENDING TO VERIFY"
- moved on the sheet: A13, A14, CN1, CP0, CP1, CP124, CP125, CR1, CR10, CR11, CR2, CR3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
