File: cores/cps3/sch/ppu.kicad_sch (KiCad schematic)
At the start: 22 parts, among them U1 74LS08, X1 7100A OSC 9640, X2 7100A OSC 9640

Commit message: iou
Connections:
- net 2GLL0 renamed 2GLL_A0
- net 2GLL1 renamed 2GLL_A1
- net 2GLL2 renamed 2GLL_A2
- net 2GLL3 renamed 2GLL_A3
- net 2GLL4 renamed 2GLL_A4
- net 2GLL5 renamed 2GLL_A5
- net ALE: no longer names the net of G2.78 (ALE)
- net CDI_D0 renamed CBI_D0
- net CDI_D1 renamed CBI_D1
- net CDI_D2 renamed CBI_D2
- net CDI_D3 renamed CBI_D3
- net CDI_D4 renamed CBI_D4
- net CDI_D5 renamed CBI_D5
- net CDI_D6 renamed CBI_D6
- net CDI_D7 renamed CBI_D7
- no-connect marks 63 -> 65
Other:
- sheet bic renamed cbi
- sheet cbi: file bic.kicad_sch -> cbi.kicad_sch
- sheet cbi ports: added CBI_D[7..0]; removed ALE, CDI_D[7..0]
Changed lines of the file:
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@@
   (no_connect (at 269.24 322.58))
   (no_connect (at 269.24 327.66))
+  (no_connect (at 195.58 347.98))
+  (no_connect (at 198.12 347.98))
   (no_connect (at 269.24 330.2))
   (no_connect (at 269.24 309.88))
@@
     (stroke (width 0) (type default) (color 0 0 0 0))
   )
-  (wire (pts (xy 510.54 27.94) (xy 520.7 27.94))
-    (stroke (width 0) (type default) (color 0 0 0 0))
-  )
   (wire (pts (xy 248.92 88.9) (xy 248.92 109.22))
     (stroke (width 0) (type default) (color 0 0 0 0))
@@
     (stroke (width 0) (type default) (color 0 0 0 0))
   )
-  (wire (pts (xy 187.96 99.06) (xy 187.96 109.22))
-    (stroke (width 0) (type default) (color 0 0 0 0))
-  )
   (wire (pts (xy 392.43 245.11) (xy 392.43 246.38))
     (stroke (width 0) (type default) (color 0 0 0 0))
@@
     (effects (font (size 1.27 1.27)) (justify left bottom))
   )
-  (label "CDI_D7" (at 185.42 96.52 270)
+  (label "CBI_D7" (at 185.42 96.52 270)
     (effects (font (size 1.27 1.27)) (justify right bottom))
   )
@@
     (effects (font (size 1.27 1.27)) (justify right bottom))
   )
-  (label "CDI_D4" (at 177.8 96.52 270)
+  (label "CBI_D4" (at 177.8 96.52 270)
     (effects (font (size 1.27 1.27)) (justify right bottom))
   )
@@
     (effects (font (size 1.27 1.27)) (justify right bottom))
   )
-  (label "2GLL3" (at 218.44 92.71 270)
+  (label "2GLL_A3" (at 218.44 92.71 270)
     (effects (font (size 1.27 1.27)) (justify right bottom))
   )
@@
     (effects (font (size 1.27 1.27)) (justify right bottom))
   )
-  (label "CDI_D3" (at 175.26 96.52 270)
+  (label "CBI_D3" (at 175.26 96.52 270)
     (effects (font (size 1.27 1.27)) (justify right bottom))
   )
@@
     (effects (font (size 1.27 1.27)) (justify right bottom))
   )
-  (label "2GLL4" (at 220.98 92.71 270)
+  (label "2GLL_A4" (at 220.98 92.71 270)
     (effects (font (size 1.27 1.27)) (justify right bottom))
   )
@@
     (effects (font (size 1.27 1.27)) (justify right bottom))
   )
-  (label "CDI_D2" (at 172.72 96.52 270)
+  (label "CBI_D2" (at 172.72 96.52 270)
     (effects (font (size 1.27 1.27)) (justify right bottom))
   )
@@
     (effects (font (size 1.27 1.27)) (justify left bottom))
   )
-  (label "CDI_D[7..0]" (at 562.61 27.94 180)
+  (label "CBI_D[7..0]" (at 562.61 27.94 180)
     (effects (font (size 1.27 1.27)) (justify right bottom))
   )
@@
     (effects (font (size 1.27 1.27)) (justify right bottom))
   )
-  (label "CDI_D5" (at 180.34 96.52 270)
+  (label "CBI_D5" (at 180.34 96.52 270)
     (effects (font (size 1.27 1.27)) (justify right bottom))
   )
@@
     (effects (font (size 1.27 1.27)) (justify left bottom))
   )
-  (label "ALE" (at 510.54 27.94 0)
-    (effects (font (size 1.27 1.27)) (justify left bottom))
-  )
   (label "PPU18" (at 283.21 162.56 180)
     (effects (font (size 1.27 1.27)) (justify right bottom))
@@
     (effects (font (size 1.27 1.27)) (justify left bottom))
   )
-  (label "2GLL1" (at 213.36 92.71 270)
+  (label "2GLL_A1" (at 213.36 92.71 270)
     (effects (font (size 1.27 1.27)) (justify right bottom))
   )
@@
     (effects (font (size 1.27 1.27)) (justify left bottom))
   )
-  (label "2GLL5" (at 223.52 92.71 270)
+  (label "2GLL_A5" (at 223.52 92.71 270)
     (effects (font (size 1.27 1.27)) (justify right bottom))
   )
-  (label "CDI_D6" (at 182.88 96.52 270)
+  (label "CBI_D6" (at 182.88 96.52 270)
     (effects (font (size 1.27 1.27)) (justify right bottom))
   )
@@
     (effects (font (size 1.27 1.27)) (justify left bottom))
   )
-  (label "2GLL0" (at 210.82 92.71 270)
+  (label "2GLL_A0" (at 210.82 92.71 270)
     (effects (font (size 1.27 1.27)) (justify right bottom))
   )
@@
     (effects (font (size 1.27 1.27)) (justify left bottom))
   )
-  (label "2GLL2" (at 215.9 92.71 270)
+  (label "2GLL_A2" (at 215.9 92.71 270)
     (effects (font (size 1.27 1.27)) (justify right bottom))
   )
@@
     (effects (font (size 1.27 1.27)) (justify right bottom))
   )
-  (label "CDI_D1" (at 170.18 96.52 270)
+  (label "CBI_D1" (at 170.18 96.52 270)
     (effects (font (size 1.27 1.27)) (justify right bottom))
   )
-  (label "CDI_D0" (at 167.64 96.52 270)
+  (label "CBI_D0" (at 167.64 96.52 270)
     (effects (font (size 1.27 1.27)) (justify right bottom))
   )
@@
     (effects (font (size 1.27 1.27)) (justify left))
   )
-  (hierarchical_label "CDI_D[7..0]" (shape bidirectional) (at 157.48 93.98 180)
+  (hierarchical_label "CBI_D[7..0]" (shape bidirectional) (at 157.48 93.98 180)
     (effects (font (size 1.27 1.27)) (justify right))
   )
@@
     (effects (font (size 1.27 1.27)) (justify left))
   )
-  (hierarchical_label "2GLL[5..0]" (shape bidirectional) (at 203.2 90.17 180)
+  (hierarchical_label "2GLL_A[5..0]" (shape bidirectional) (at 203.2 90.17 180)
     (effects (font (size 1.27 1.27)) (justify right))
   )
@@
     (effects (font (size 1.27 1.27)) (justify right))
   )
-  (hierarchical_label "ALE" (shape output) (at 187.96 99.06 90)
-    (effects (font (size 1.27 1.27)) (justify left))
-  )
   (hierarchical_label "GLL_A[14..0]" (shape bidirectional) (at 222.25 86.36 180)
     (effects (font (size 1.27 1.27)) (justify right))
@@
     (stroke (width 0.1524) (type solid) (color 0 0 0 0))
     (fill (color 0 0 0 0.0000))
-    (property "Sheet name" "bic" (id 0) (at 520.7 24.6884 0)
+    (property "Sheet name" "cbi" (id 0) (at 520.7 24.6884 0)
       (effects (font (size 1.27 1.27)) (justify left bottom))
     )
-    (property "Sheet file" "bic.kicad_sch" (id 1) (at 520.7 62.8146 0)
+    (property "Sheet file" "cbi.kicad_sch" (id 1) (at 520.7 62.8146 0)
       (effects (font (size 1.27 1.27)) (justify left top))
     )
-    (pin "ALE" input (at 520.7 27.94 180)
-      (effects (font (size 1.27 1.27)) (justify left))
-    )
-    (pin "CDI_D[7..0]" bidirectional (at 548.64 27.94 0)
+    (pin "CBI_D[7..0]" bidirectional (at 548.64 27.94 0)
       (effects (font (size 1.27 1.27)) (justify right))
     )

Commit message: update_006
Connections:
- net at U1.1: no longer G2.29 (AND1)
- net at U1.2: no longer G2.28 (AND2)
Other:
- moved on the sheet: U1A, U1B, U1C, U1D, U1E
Changed lines of the file:
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@@
     (stroke (width 0) (type default) (color 0 0 0 0))
   )
-  (wire (pts (xy 292.1 340.36) (xy 297.18 340.36))
+  (wire (pts (xy 299.72 82.55) (xy 304.8 82.55))
     (stroke (width 0) (type default) (color 0 0 0 0))
   )
@@
     (stroke (width 0) (type default) (color 0 0 0 0))
   )
-  (wire (pts (xy 276.86 340.36) (xy 276.86 342.9))
+  (wire (pts (xy 284.48 82.55) (xy 284.48 85.09))
     (stroke (width 0) (type default) (color 0 0 0 0))
   )
@@
     (stroke (width 0) (type default) (color 0 0 0 0))
   )
-  (wire (pts (xy 269.24 337.82) (xy 276.86 337.82))
+  (wire (pts (xy 276.86 80.01) (xy 284.48 80.01))
     (stroke (width 0) (type default) (color 0 0 0 0))
   )
@@
     (stroke (width 0) (type default) (color 0 0 0 0))
   )
-  (wire (pts (xy 269.24 340.36) (xy 276.86 340.36))
+  (wire (pts (xy 276.86 82.55) (xy 284.48 82.55))
     (stroke (width 0) (type default) (color 0 0 0 0))
   )
@@
     (pin "9")
   )
-  (symbol (lib_id "jt74:74LS08") (at 297.18 353.06 0) (unit 3)
+  (symbol (lib_id "jt74:74LS08") (at 304.8 95.25 0) (unit 3)
     (in_bom yes) (on_board yes)
-    (property "Reference" "U1" (id 0) (at 297.18 351.79 0))
-    (property "Value" "74LS08" (id 1) (at 297.18 354.33 0))
-    (property "Footprint" "" (id 2) (at 297.18 353.06 0)
+    (property "Reference" "U1" (id 0) (at 304.8 93.98 0))
+    (property "Value" "74LS08" (id 1) (at 304.8 96.52 0))
+    (property "Footprint" "" (id 2) (at 304.8 95.25 0)
       (effects (font (size 1.27 1.27)) hide)
     )
-    (property "Datasheet" "http://www.ti.com/lit/gpn/sn74LS08" (id 3) (at 297.18 353.06 0)
+    (property "Datasheet" "http://www.ti.com/lit/gpn/sn74LS08" (id 3) (at 304.8 95.25 0)
       (effects (font (size 1.27 1.27)) hide)
     )
@@
     (pin "9")
   )
-  (symbol (lib_id "jt74:74LS08") (at 276.86 353.06 0) (unit 2)
+  (symbol (lib_id "jt74:74LS08") (at 284.48 95.25 0) (unit 2)
     (in_bom yes) (on_board yes)
-    (property "Reference" "U1" (id 0) (at 276.86 351.79 0))
-    (property "Value" "74LS08" (id 1) (at 276.86 354.33 0))
-    (property "Footprint" "" (id 2) (at 276.86 353.06 0)
+    (property "Reference" "U1" (id 0) (at 284.48 93.98 0))
+    (property "Value" "74LS08" (id 1) (at 284.48 96.52 0))
+    (property "Footprint" "" (id 2) (at 284.48 95.25 0)
       (effects (font (size 1.27 1.27)) hide)
     )
-    (property "Datasheet" "http://www.ti.com/lit/gpn/sn74LS08" (id 3) (at 276.86 353.06 0)
+    (property "Datasheet" "http://www.ti.com/lit/gpn/sn74LS08" (id 3) (at 284.48 95.25 0)
       (effects (font (size 1.27 1.27)) hide)
     )
@@
     (pin "9")
   )
-  (symbol (lib_id "jt74:74LS08") (at 314.96 353.06 0) (unit 4)
+  (symbol (lib_id "jt74:74LS08") (at 322.58 95.25 0) (unit 4)
     (in_bom yes) (on_board yes)
-    (property "Reference" "U1" (id 0) (at 314.96 351.79 0))
-    (property "Value" "74LS08" (id 1) (at 314.96 354.33 0))
-    (property "Footprint" "" (id 2) (at 314.96 353.06 0)
+    (property "Reference" "U1" (id 0) (at 322.58 93.98 0))
+    (property "Value" "74LS08" (id 1) (at 322.58 96.52 0))
+    (property "Footprint" "" (id 2) (at 322.58 95.25 0)
       (effects (font (size 1.27 1.27)) hide)
     )
-    (property "Datasheet" "http://www.ti.com/lit/gpn/sn74LS08" (id 3) (at 314.96 353.06 0)
+    (property "Datasheet" "http://www.ti.com/lit/gpn/sn74LS08" (id 3) (at 322.58 95.25 0)
       (effects (font (size 1.27 1.27)) hide)
     )
@@
     (pin "7")
   )
-  (symbol (lib_id "jt74:74LS08") (at 284.48 340.36 0) (unit 1)
+  (symbol (lib_id "jt74:74LS08") (at 292.1 82.55 0) (unit 1)
     (in_bom yes) (on_board yes)
-    (property "Reference" "U1" (id 0) (at 284.48 339.09 0))
-    (property "Value" "74LS08" (id 1) (at 284.48 341.63 0))
-    (property "Footprint" "" (id 2) (at 284.48 340.36 0)
+    (property "Reference" "U1" (id 0) (at 292.1 81.28 0))
+    (property "Value" "74LS08" (id 1) (at 292.1 83.82 0))
+    (property "Footprint" "" (id 2) (at 292.1 82.55 0)
       (effects (font (size 1.27 1.27)) hide)
     )
-    (property "Datasheet" "http://www.ti.com/lit/gpn/sn74LS08" (id 3) (at 284.48 340.36 0)
+    (property "Datasheet" "http://www.ti.com/lit/gpn/sn74LS08" (id 3) (at 292.1 82.55 0)
       (effects (font (size 1.27 1.27)) hide)
     )
@@
     (pin "9")
   )
-  (symbol (lib_id "jt74:74LS08") (at 334.01 354.33 0) (unit 5)
+  (symbol (lib_id "jt74:74LS08") (at 341.63 96.52 0) (unit 5)
     (in_bom yes) (on_board yes)
-    (property "Reference" "U1" (id 0) (at 334.01 353.06 0))
-    (property "Value" "74LS08" (id 1) (at 334.01 355.6 0))
-    (property "Footprint" "" (id 2) (at 334.01 354.33 0)
+    (property "Reference" "U1" (id 0) (at 341.63 95.25 0))
+    (property "Value" "74LS08" (id 1) (at 341.63 97.79 0))
+    (property "Footprint" "" (id 2) (at 341.63 96.52 0)
       (effects (font (size 1.27 1.27)) hide)
     )
-    (property "Datasheet" "http://www.ti.com/lit/gpn/sn74LS08" (id 3) (at 334.01 354.33 0)
+    (property "Datasheet" "http://www.ti.com/lit/gpn/sn74LS08" (id 3) (at 341.63 96.52 0)
       (effects (font (size 1.27 1.27)) hide)
     )

Commit message: uptate_ns
Other:
- note added: "NO SE OBSERVA SALIDA DE SEÑAL FISICA"
Changed lines of the file:
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@@
+    (effects (font (size 1.27 1.27)) (justify left bottom))
+  )
+  (text "NO SE OBSERVA SALIDA DE SEÑAL FISICA\n" (at 201.93 322.58 0)
     (effects (font (size 1.27 1.27)) (justify left bottom))
   )

Commit message: update_cps3
Parts:
- removed unit 5 of U1
Connections:
- net at U1.1: now also G2.29 (AND1)
- net at U1.2: now also G2.28 (AND2)
- net PPU2CCU1: now reaches G2.40 (CCU57)
- net PPU2CCU0: now reaches G2.41 (CCU56)
- net ALE: now reaches G2.78 (ALE)
- net MAIN_D9: now reaches G2.80 (MAIN_D9)
- net MAIN_D10: now reaches G2.81 (MAIN_D10)
- net MAIN_D11: now reaches G2.83 (MAIN_D11)
- net MAIN_D12: now reaches G2.84 (MAIN_D12)
- net CBI_D0 renamed MAIN_D0
- net CBI_D1 renamed MAIN_D1
- net CBI_D2 renamed MAIN_D2
- net CBI_D3 renamed MAIN_D3
- net CBI_D4 renamed MAIN_D4
- net CBI_D5 renamed MAIN_D5
- net CBI_D6 renamed MAIN_D6
- net CBI_D7 renamed MAIN_D7
- net GLL_A0 renamed MAIN_A28
- net GLL_A1 renamed MAIN_A27
- net GLL_A10 renamed MAIN_A5
- net GLL_A11 renamed MAIN_A1
- net GLL_A12 renamed MAIN_A2
- net GLL_A13 renamed MAIN_A3
- net GLL_A14 renamed MAIN_A0
- net GLL_A2 renamed MAIN_A26
- net GLL_A3 renamed MAIN_A25
- net GLL_A4 renamed MAIN_A7
- net GLL_A5 renamed MAIN_A6
- net GLL_A6 renamed MAIN_A4
- net GLL_A7 renamed MAIN_D14
- net GLL_A8 renamed MAIN_D13
- net GLL_A9 renamed MAIN_D8
- net SSU_D0 renamed MAIN_A24
- net SSU_D1 renamed MAIN_A23
- net SSU_D10 renamed MAIN_A14
- net SSU_D11 renamed MAIN_A13
- net SSU_D12 renamed MAIN_A12
- net SSU_D13 renamed MAIN_A11
- net SSU_D14 renamed MAIN_A10
- net SSU_D15 renamed MAIN_A9
- net SSU_D16 renamed MAIN_A8
- net SSU_D2 renamed MAIN_A22
- net SSU_D3 renamed MAIN_A21
- net SSU_D4 renamed MAIN_A20
- net SSU_D5 renamed MAIN_A19
- net SSU_D6 renamed MAIN_A18
- net SSU_D7 renamed MAIN_A17
- net SSU_D8 renamed MAIN_A16
- net SSU_D9 renamed MAIN_A15
- no-connect marks 65 -> 59
Other:
- note added: "MEMORIES FRAME BUFFER?"
- note added: "NO OUTPUT OBSERVED PHYSICAL SIGNAL (UK)"
- note added: "PPU2SSU 16~0"
- note added: "There is no certainty that it is Address Bus"
- note added: "There is no certainty that it is Data Bus"
- note removed: "NO SE OBSERVA SALIDA DE SEÑAL FISICA"
- moved on the sheet: U1A, U1B, U1C, U1D

Commit message: update5
Connections:
- net MAIN_A24 is gone; now on net MAIN_A10: G2.59 (MAIN_A10)
- net MAIN_A25 is gone; now on net MAIN_A9: G2.60 (MAIN_A9)
- net MAIN_A26 is gone; now on net MAIN_A8: G2.61 (MAIN_A8)
- net MAIN_A27 is gone; now on net MAIN_A19: G2.62 (MAIN_A19)
- net MAIN_A28 is gone; now on net MAIN_A20: G2.63 (MAIN_A20)
- net ALE: now also G2.57 (VCC); no longer G2.78 (ALE)
- net MAIN_A0: now also G2.87 (MAIN_A0); no longer G2.23 (MAIN_A0)
- net MAIN_A1: now also G2.86 (MAIN_A1); no longer G2.31 (MAIN_A1)
- net MAIN_A10: no longer G2.44 (MAIN_A10)
- net MAIN_A11: now also G2.37 (MAIN_A11); no longer G2.45 (MAIN_A11)
- net MAIN_A12: now also G2.36 (MAIN_A12); no longer G2.46 (MAIN_A12)
- net MAIN_A13: now also G2.34 (MAIN_A13); no longer G2.47 (MAIN_A13)
- net MAIN_A14: now also G2.35 (MAIN_A14); no longer G2.48 (MAIN_A14)
- net MAIN_A15: now also G2.33 (MAIN_A15); no longer G2.49 (MAIN_A15)
- net MAIN_A16: now also G2.32 (MAIN_A16); no longer G2.50 (MAIN_A16)
- net MAIN_A17: now also G2.31 (MAIN_A17); no longer G2.51 (MAIN_A17)
- net MAIN_A18: now also G2.23 (MAIN_A18); no longer G2.52 (MAIN_A18)
- net MAIN_A19: no longer G2.53 (MAIN_A19)
- net MAIN_A2: now also G2.84 (MAIN_A2); no longer G2.32 (MAIN_A2)
- net MAIN_A20: no longer G2.54 (MAIN_A20)
- net MAIN_A3: now also G2.83 (MAIN_A3); no longer G2.33 (MAIN_A3)
- net MAIN_A4: now also G2.81 (MAIN_A4); no longer G2.34 (MAIN_A4)
- net MAIN_A5: now also G2.80 (MAIN_A5); no longer G2.35 (MAIN_A5)
- net MAIN_A6: now also G2.78 (MAIN_A6); no longer G2.36 (MAIN_A6)
- net MAIN_A7: now also G2.75 (MAIN_A7); no longer G2.37 (MAIN_A7)
- net MAIN_A8: no longer G2.42 (MAIN_A8)
- net MAIN_A9: no longer G2.43 (MAIN_A9)
- net MAIN_D10: now also G2.44 (MAIN_D10); no longer G2.81 (MAIN_D10)
- net MAIN_D11: now also G2.45 (MAIN_D11); no longer G2.83 (MAIN_D11)
- net MAIN_D12: now also G2.46 (MAIN_D12); no longer G2.84 (MAIN_D12)
- net MAIN_D13: now also G2.47 (MAIN_D13); no longer G2.86 (MAIN_D13)
- net MAIN_D14: now also G2.48 (MAIN_D14); no longer G2.87 (MAIN_D14)
- net MAIN_D8: now also G2.42 (MAIN_D8); no longer G2.75 (MAIN_D8)
- net MAIN_D9: now also G2.43 (MAIN_D9); no longer G2.80 (MAIN_D9)
- net PPU2CCU0: now also G2.40 (CCU57); no longer G2.41 (CCU56)
- net PPU2CCU1: now also G2.41 (CCU56); no longer G2.40 (CCU57)
- net MAIN_A21 renamed MAIN_D21
- net MAIN_A22 renamed MAIN_D22
- net MAIN_A23 renamed MAIN_D23
- new net MAIN_D15: G2.49 (MAIN_D15)
- new net MAIN_D16: G2.50 (MAIN_D16)
- new net MAIN_D17: G2.51 (MAIN_D17)
- new net MAIN_D18: G2.52 (MAIN_D18)
- new net MAIN_D19: G2.53 (MAIN_D19)
- new net MAIN_D20: G2.54 (MAIN_D20)
- no-connect marks 59 -> 58
Other:
- moved on the sheet: RN12, RN13, U1A, U1B, U1C, U1D

Commit message: update6_cps
Other:
- note added: "MEMORI MAIN?"
- note added: "PPU2SSU 15~0"
- note removed: "PPU2SSU 16~0"
Changed lines of the file:
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@@
     (stroke (width 0) (type default) (color 0 0 0 0))
   )
+  (bus_entry (at 256.54 360.68) (size 2.54 2.54)
+    (stroke (width 0) (type default) (color 0 0 0 0))
+  )
+  (bus_entry (at 254 360.68) (size 2.54 2.54)
+    (stroke (width 0) (type default) (color 0 0 0 0))
+  )
   (bus_entry (at 283.21 165.1) (size 2.54 -2.54)
     (stroke (width 0) (type default) (color 0 0 0 0))
@@
     (stroke (width 0) (type default) (color 0 0 0 0))
   )
+  (bus (pts (xy 259.08 363.22) (xy 262.89 363.22))
+    (stroke (width 0) (type default) (color 0 0 0 0))
+  )
   (wire (pts (xy 402.59 24.13) (xy 405.13 24.13))
     (stroke (width 0) (type default) (color 0 0 0 0))
@@
     (stroke (width 0) (type default) (color 0 0 0 0))
   )
-  (wire (pts (xy 254 350.52) (xy 254 353.06))
+  (wire (pts (xy 254 350.52) (xy 254 360.68))
     (stroke (width 0) (type default) (color 0 0 0 0))
   )
@@
     (stroke (width 0) (type default) (color 0 0 0 0))
   )
-  (wire (pts (xy 256.54 350.52) (xy 256.54 353.06))
+  (wire (pts (xy 256.54 350.52) (xy 256.54 360.68))
     (stroke (width 0) (type default) (color 0 0 0 0))
   )
@@
     (stroke (width 0) (type default) (color 0 0 0 0))
   )
+  (bus (pts (xy 256.54 363.22) (xy 259.08 363.22))
+    (stroke (width 0) (type default) (color 0 0 0 0))
+  )
   (wire (pts (xy 392.43 163.83) (xy 392.43 165.1))
     (stroke (width 0) (type default) (color 0 0 0 0))
@@
     (effects (font (size 1.27 1.27)) (justify left bottom))
   )
+  (text "NO OUTPUT OBSERVED\nPHYSICAL SIGNAL (UK)" (at 44.45 167.64 0)
+    (effects (font (size 3 3)) (justify left bottom))
+  )
   (text "MEMORIES FRAME BUFFER?\n\n\n" (at 331.47 358.14 0)
     (effects (font (size 1.27 1.27)) (justify left bottom))
@@
     (effects (font (size 1.27 1.27)) (justify left bottom))
   )
-  (text "PPU2SSU 16~0" (at 107.95 191.77 0)
+  (text "PPU2SSU 15~0" (at 107.95 191.77 0)
     (effects (font (size 1.27 1.27)) (justify left bottom))
   )
@@
     (effects (font (size 3 3)) (justify left bottom))
   )
+  (text "MEMORI MAIN?\n" (at 351.79 234.95 0)
+    (effects (font (size 1.27 1.27)) (justify left bottom))
+  )
   (text "42.9545MHz" (at 43.18 149.86 0)
     (effects (font (size 1.27 1.27)) (justify left bottom))
@@
     (effects (font (size 1.27 1.27)) (justify right bottom))
   )
+  (label "PPU2CCU1" (at 256.54 360.68 90)
+    (effects (font (size 1.27 1.27)) (justify left bottom))
+  )
   (label "MAIN_D12" (at 280.67 292.1 180)
     (effects (font (size 1.27 1.27)) (justify right bottom))
@@
     (effects (font (size 1.27 1.27)) (justify right bottom))
   )
+  (label "PPU2CCU0" (at 254 360.68 90)
+    (effects (font (size 1.27 1.27)) (justify left bottom))
+  )
   (label "PPU_A7" (at 328.93 340.36 180)
     (effects (font (size 1.27 1.27)) (justify right bottom))
@@
     (effects (font (size 1.27 1.27)) (justify right))
   )
-  (hierarchical_label "PPU2CCU0" (shape output) (at 254 353.06 270)
-    (effects (font (size 1.27 1.27)) (justify right))
-  )
   (hierarchical_label "BX_SND" (shape output) (at 243.84 100.33 90)
     (effects (font (size 1.27 1.27)) (justify left))
@@
     (effects (font (size 1.27 1.27)) (justify left))
   )
-  (hierarchical_label "PPU2CCU1" (shape output) (at 256.54 353.06 270)
-    (effects (font (size 1.27 1.27)) (justify right))
-  )
   (hierarchical_label "SRITE[15..0]" (shape output) (at 473.71 273.05 0)
     (effects (font (size 1.27 1.27)) (justify left))
@@
     (effects (font (size 1.27 1.27)) (justify left))
   )
+  (hierarchical_label "PPU2CCU[1..0]" (shape bidirectional) (at 262.89 363.22 0)
+    (effects (font (size 1.27 1.27)) (justify left))
+  )
