File: cores/cps3/sch/ppu.kicad_sch (KiCad schematic)
At the start: 22 parts, among them U1 74LS08, X1 7100A OSC 9640, X2 7100A OSC 9640

Commit message: clear_sch_hk_cr
Connections:
- net MAIN_A0 renamed GFX_A0
- net MAIN_A1 renamed GFX_A1
- net MAIN_A10 renamed GFX_A10
- net MAIN_A11 renamed GFX_A11
- net MAIN_A12 renamed GFX_A12
- net MAIN_A13 renamed GFX_A13
- net MAIN_A14 renamed GFX_A14
- net MAIN_A15 renamed GFX_A15
- net MAIN_A16 renamed GFX_A16
- net MAIN_A17 renamed GFX_A17
- net MAIN_A18 renamed GFX_A18
- net MAIN_A19 renamed GFX_A19
- net MAIN_A2 renamed GFX_A2
- net MAIN_A20 renamed GFX_A20
- net MAIN_A3 renamed GFX_A3
- net MAIN_A4 renamed GFX_A4
- net MAIN_A5 renamed GFX_A5
- net MAIN_A6 renamed GFX_A6
- net MAIN_A7 renamed GFX_A7
- net MAIN_A8 renamed GFX_A8
- net MAIN_A9 renamed GFX_A9
Changed lines of the file:
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@@
     (effects (font (size 1.27 1.27)) (justify right bottom))
   )
-  (label "MAIN_A7" (at 198.12 361.95 90)
+  (label "GFX_A7" (at 198.12 361.95 90)
     (effects (font (size 1.27 1.27)) (justify left bottom))
   )
@@
     (effects (font (size 1.27 1.27)) (justify right bottom))
   )
-  (label "MAIN_A11" (at 208.28 361.95 90)
+  (label "GFX_A11" (at 208.28 361.95 90)
     (effects (font (size 1.27 1.27)) (justify left bottom))
   )
@@
     (effects (font (size 1.27 1.27)) (justify right bottom))
   )
-  (label "MAIN_A4" (at 190.5 361.95 90)
+  (label "GFX_A4" (at 190.5 361.95 90)
     (effects (font (size 1.27 1.27)) (justify left bottom))
   )
@@
     (effects (font (size 1.27 1.27)) (justify right bottom))
   )
-  (label "MAIN_A14" (at 215.9 361.95 90)
+  (label "GFX_A14" (at 215.9 361.95 90)
     (effects (font (size 1.27 1.27)) (justify left bottom))
   )
@@
     (effects (font (size 1.27 1.27)) (justify left bottom))
   )
-  (label "MAIN_A19" (at 228.6 361.95 90)
+  (label "GFX_A19" (at 228.6 361.95 90)
     (effects (font (size 1.27 1.27)) (justify left bottom))
   )
@@
     (effects (font (size 1.27 1.27)) (justify right bottom))
   )
-  (label "MAIN_A10" (at 205.74 361.95 90)
+  (label "GFX_A10" (at 205.74 361.95 90)
     (effects (font (size 1.27 1.27)) (justify left bottom))
   )
@@
     (effects (font (size 1.27 1.27)) (justify right bottom))
   )
-  (label "MAIN_A9" (at 203.2 361.95 90)
+  (label "GFX_A9" (at 203.2 361.95 90)
     (effects (font (size 1.27 1.27)) (justify left bottom))
   )
@@
     (effects (font (size 1.27 1.27)) (justify right bottom))
   )
-  (label "MAIN_A6" (at 195.58 361.95 90)
+  (label "GFX_A6" (at 195.58 361.95 90)
     (effects (font (size 1.27 1.27)) (justify left bottom))
   )
@@
     (effects (font (size 1.27 1.27)) (justify left bottom))
   )
-  (label "MAIN_A0" (at 180.34 361.95 90)
+  (label "GFX_A0" (at 180.34 361.95 90)
     (effects (font (size 1.27 1.27)) (justify left bottom))
   )
@@
     (effects (font (size 1.27 1.27)) (justify left bottom))
   )
-  (label "MAIN_A8" (at 200.66 361.95 90)
+  (label "GFX_A8" (at 200.66 361.95 90)
     (effects (font (size 1.27 1.27)) (justify left bottom))
   )
@@
     (effects (font (size 1.27 1.27)) (justify right bottom))
   )
-  (label "MAIN_A3" (at 187.96 361.95 90)
-    (effects (font (size 1.27 1.27)) (justify left bottom))
-  )
-  (label "MAIN_A17" (at 223.52 361.95 90)
+  (label "GFX_A3" (at 187.96 361.95 90)
+    (effects (font (size 1.27 1.27)) (justify left bottom))
+  )
+  (label "GFX_A17" (at 223.52 361.95 90)
     (effects (font (size 1.27 1.27)) (justify left bottom))
   )
@@
     (effects (font (size 1.27 1.27)) (justify left bottom))
   )
-  (label "MAIN_A20" (at 231.14 361.95 90)
+  (label "GFX_A20" (at 231.14 361.95 90)
     (effects (font (size 1.27 1.27)) (justify left bottom))
   )
@@
     (effects (font (size 1.27 1.27)) (justify left bottom))
   )
-  (label "MAIN_A5" (at 193.04 361.95 90)
+  (label "GFX_A5" (at 193.04 361.95 90)
     (effects (font (size 1.27 1.27)) (justify left bottom))
   )
@@
     (effects (font (size 1.27 1.27)) (justify left bottom))
   )
-  (label "MAIN_A13" (at 213.36 361.95 90)
+  (label "GFX_A13" (at 213.36 361.95 90)
     (effects (font (size 1.27 1.27)) (justify left bottom))
   )
@@
     (effects (font (size 1.27 1.27)) (justify left bottom))
   )
-  (label "MAIN_A2" (at 185.42 361.95 90)
+  (label "GFX_A2" (at 185.42 361.95 90)
     (effects (font (size 1.27 1.27)) (justify left bottom))
   )
@@
     (effects (font (size 1.27 1.27)) (justify right bottom))
   )
-  (label "MAIN_A12" (at 210.82 361.95 90)
+  (label "GFX_A12" (at 210.82 361.95 90)
     (effects (font (size 1.27 1.27)) (justify left bottom))
   )
@@
     (effects (font (size 1.27 1.27)) (justify left bottom))
   )
-  (label "MAIN_A18" (at 226.06 361.95 90)
+  (label "GFX_A18" (at 226.06 361.95 90)
     (effects (font (size 1.27 1.27)) (justify left bottom))
   )
@@
     (effects (font (size 1.27 1.27)) (justify right bottom))
   )
-  (label "MAIN_A16" (at 220.98 361.95 90)
+  (label "GFX_A16" (at 220.98 361.95 90)
     (effects (font (size 1.27 1.27)) (justify left bottom))
   )
@@
     (effects (font (size 1.27 1.27)) (justify right bottom))
   )
-  (label "MAIN_A15" (at 218.44 361.95 90)
+  (label "GFX_A15" (at 218.44 361.95 90)
     (effects (font (size 1.27 1.27)) (justify left bottom))
   )
@@
     (effects (font (size 1.27 1.27)) (justify left bottom))
   )
-  (label "MAIN_A1" (at 182.88 361.95 90)
+  (label "GFX_A1" (at 182.88 361.95 90)
     (effects (font (size 1.27 1.27)) (justify left bottom))
   )
@@
     (effects (font (size 1.27 1.27)) (justify right))
   )
-  (hierarchical_label "MAIN_A[20..0]" (shape bidirectional) (at 163.83 364.49 180)
+  (hierarchical_label "GFX_A[20..0]" (shape bidirectional) (at 163.83 364.49 180)
     (effects (font (size 1.27 1.27)) (justify right))
   )
