File: cores/cps3/sch/ppu.kicad_sch (KiCad schematic)
At the start: 27 parts, among them Q1 ZR, U1 74LS08, X1 7100A OSC 9640, X2 7100A OSC 9640

Commit message: wip_cps3_vdac
Parts:
- removed unit 3 of U1
- removed unit 2 of U1
- removed unit 4 of U1
Connections:
- net ALE is gone; now on net VCC: G2.57 (VCC)
- net ~{CS_PAL}H: now reaches G2.171 (UK)
- net ~{CS_PAL}L: now reaches G2.173 (UK)
- net ~{WE_PAL}: now reaches G2.174 (UK)
- net PPU2SSU0: now reaches G2.27 (PPU2SSU0)
- net SNDD: now reaches G2.88 (SND_DATA)
- net WS: now reaches G2.89 (WORD_SELECT)
- net BCK: now reaches G2.90 (BIT_CLK)
- net SYSCLK: now reaches G2.91 (SYSCLK)
- no-connect marks 60 -> 51
Other:
- note added: "NOT CONNECTED"
- note removed: "88 ~ 91 ,27 SI EL 30 NO"
- note removed: "BUS DE DATOS SRAM E9 PIN 6 PIN 171 AL 192"
- note removed: "NO CONECTADO"

Commit message: wip_ssu_cbi_gll
Connections:
- net PPU2CCU1 is gone; now on net PPU_A0: G2.41 (PPU_A0)
- net SYNCB: now reaches G2.29 (SYNCB), U1.1
- net SYNCA: now reaches G2.28 (SYNCA), U1.2
Other:
- removed sheet cbi
- note added: "Processor Data Bus"
- note removed: "RAM DE VIDEO D0?"
- moved on the sheet: Q1, R13, R23, R29, U1A

Commit message: wip_iou_wd
Connections:
- no-connect marks 51 -> 53
Other:
- note added: "Address Bus?"
- note added: "Processor Data Bus?"
Changed lines of the file:
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@@
   (junction (at 127 347.98) (diameter 0) (color 0 0 0 0)
   )
+  (no_connect (at 198.12 351.79))
   (no_connect (at 96.52 140.97))
   (no_connect (at 223.52 109.22))
@@
   (no_connect (at 238.76 67.31))
   (no_connect (at 238.76 52.07))
+  (no_connect (at 283.21 279.4))
   (no_connect (at 213.36 109.22))
   (no_connect (at 238.76 59.69))
@@
     (stroke (width 0) (type default) (color 0 0 0 0))
   )
+  (polyline (pts (xy 176.53 368.3) (xy 176.53 351.79))
+    (stroke (width 0) (type default) (color 0 0 0 0))
+  )
   (wire (pts (xy 104.14 109.22) (xy 106.68 109.22))
     (stroke (width 0) (type default) (color 0 0 0 0))
@@
     (stroke (width 0) (type default) (color 0 0 0 0))
   )
+  (polyline (pts (xy 199.39 361.95) (xy 199.39 370.84))
+    (stroke (width 0) (type default) (color 0 0 0 0))
+  )
   (wire (pts (xy 293.37 363.22) (xy 293.37 369.57))
     (stroke (width 0) (type default) (color 0 0 0 0))
@@
     (stroke (width 0) (type default) (color 0 0 0 0))
   )
+  (polyline (pts (xy 199.39 350.52) (xy 199.39 360.68))
+    (stroke (width 0) (type default) (color 0 0 0 0))
+  )
   (wire (pts (xy 82.55 234.95) (xy 96.52 234.95))
     (stroke (width 0) (type default) (color 0 0 0 0))
@@
     (stroke (width 0) (type default) (color 0 0 0 0))
   )
+  (polyline (pts (xy 231.14 350.52) (xy 199.39 350.52))
+    (stroke (width 0) (type default) (color 0 0 0 0))
+  )
   (wire (pts (xy 77.47 125.73) (xy 95.25 125.73))
     (stroke (width 0) (type default) (color 0 0 0 0))
@@
     (stroke (width 0) (type default) (color 0 0 0 0))
   )
+  (polyline (pts (xy 198.12 354.33) (xy 198.12 368.3))
+    (stroke (width 0) (type default) (color 0 0 0 0))
+  )
   (bus (pts (xy 524.51 298.45) (xy 518.16 298.45))
     (stroke (width 0) (type default) (color 0 0 0 0))
@@
     (stroke (width 0) (type default) (color 0 0 0 0))
   )
+  (polyline (pts (xy 281.94 279.4) (xy 289.56 279.4))
+    (stroke (width 0) (type default) (color 0 0 0 0))
+  )
   (bus (pts (xy 466.09 364.49) (xy 466.09 337.82))
     (stroke (width 0) (type default) (color 0 0 0 0))
@@
     (stroke (width 0) (type default) (color 0 0 0 0))
   )
+  (polyline (pts (xy 284.48 318.77) (xy 289.56 318.77))
+    (stroke (width 0) (type default) (color 0 0 0 0))
+  )
   (wire (pts (xy 392.43 124.46) (xy 392.43 125.73))
     (stroke (width 0) (type default) (color 0 0 0 0))
@@
     (stroke (width 0) (type default) (color 0 0 0 0))
   )
+  (polyline (pts (xy 198.12 368.3) (xy 176.53 368.3))
+    (stroke (width 0) (type default) (color 0 0 0 0))
+  )
   (wire (pts (xy 368.3 246.38) (xy 354.33 246.38))
     (stroke (width 0) (type default) (color 0 0 0 0))
@@
     (stroke (width 0) (type default) (color 0 0 0 0))
   )
+  (polyline (pts (xy 289.56 279.4) (xy 289.56 318.77))
+    (stroke (width 0) (type default) (color 0 0 0 0))
+  )
   (wire (pts (xy 468.63 290.83) (xy 477.52 290.83))
     (stroke (width 0) (type default) (color 0 0 0 0))
@@
     (stroke (width 0) (type default) (color 0 0 0 0))
   )
+  (polyline (pts (xy 231.14 370.84) (xy 231.14 350.52))
+    (stroke (width 0) (type default) (color 0 0 0 0))
+  )
   (wire (pts (xy 419.1 41.91) (xy 419.1 43.18))
     (stroke (width 0) (type default) (color 0 0 0 0))
@@
     (stroke (width 0) (type default) (color 0 0 0 0))
   )
+  (polyline (pts (xy 176.53 351.79) (xy 177.8 351.79))
+    (stroke (width 0) (type default) (color 0 0 0 0))
+  )
   (bus (pts (xy 80.01 247.65) (xy 80.01 250.19))
     (stroke (width 0) (type default) (color 0 0 0 0))
@@
     (stroke (width 0) (type default) (color 0 0 0 0))
   )
+  (polyline (pts (xy 199.39 370.84) (xy 231.14 370.84))
+    (stroke (width 0) (type default) (color 0 0 0 0))
+  )
   (wire (pts (xy 321.31 332.74) (xy 328.93 332.74))
     (stroke (width 0) (type default) (color 0 0 0 0))
@@
     (effects (font (size 1.27 1.27)) (justify left bottom))
   )
+  (text "Address Bus?" (at 209.55 373.38 0)
+    (effects (font (size 1.27 1.27)) (justify left bottom))
+  )
   (text "MEMORIES FRAME BUFFER?\n\n\n" (at 331.47 358.14 0)
     (effects (font (size 1.27 1.27)) (justify left bottom))
@@
     (effects (font (size 3 3)) (justify left bottom))
   )
+  (text "Processor Data Bus?" (at 177.8 372.11 0)
+    (effects (font (size 1.27 1.27)) (justify left bottom))
+  )
   (text "PRIORITY SPRITES" (at 410.21 364.49 0)
     (effects (font (size 1.27 1.27)) (justify left bottom))
@@
     (effects (font (size 1.27 1.27)) (justify left bottom))
   )
+  (text "Address Bus?" (at 290.83 297.18 0)
+    (effects (font (size 1.27 1.27)) (justify left bottom))
+  )

Commit message: wip_ccu
Parts:
- added CP170, CP171, CP172, CP173: 1nF, symbol Device:C_Polarized_US
- added R55, R56, R57, R58, R59: 330Ω, symbol Device:R_US
Connections:
- net VCC: now also G2.16 (VCC), CP170.1, CP171.1, CP172.1, CP173.1
- net VSS: now also CP170.2, CP171.2, CP172.2, CP173.2; no longer G2.16 (VSS), G2.202 (UK)
- net ~{LCAS}: now also R55.1; no longer D1.29 (~{LCAS})
- net ~{RAS}: now also R58.1; no longer D1.14 (~{RAS})
- net ~{UCAS}: now also R56.1; no longer D1.28 (~{UCAS})
- net ~{WE}: now also R59.1; no longer D1.13 (~{WE})
- net at D1.26 (A8): now also R57.2
- new net: D1.29 (~{LCAS}), R55.2
- new net: D1.13 (~{WE}), R59.2
- new net: D1.28 (~{UCAS}), R56.2
- new net: G2.202 (RAMA8), R57.1
- new net: D1.14 (~{RAS}), R58.2
- no-connect marks 53 -> 52
Other:
- sheet memories_fb ports: added ~{RAS_MAIN}; removed ~{RAS}
- moved on the sheet: D1, D7, G2, H1, H2, H3, H4, H5, H6, H9, Q1, R13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

Commit message: wip_ccu_gll2_cassette
Parts:
- R29: value 100Ω -> 100
- R55, R56, R57, R58, R59, RN12, RN13, RN8, RN9: value 330Ω -> 330
- R63, R74, R75: value 110Ω -> 110
- RN10, RN11, RN14: value 620Ω -> 620
Connections:
- net PPU_A0 renamed PPU2CCU1
Changed lines of the file:
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@@
     (effects (font (size 1.27 1.27)) (justify right bottom))
   )
-  (label "PPU_A0" (at 254 358.14 90)
+  (label "PPU2CCU1" (at 254 358.14 90)
     (effects (font (size 1.27 1.27)) (justify left bottom))
   )
@@
     (effects (font (size 1.27 1.27)) (justify right bottom))
   )
-  (label "PPU_A0" (at 328.93 322.58 180)
+  (label "PPU2CCU1" (at 328.93 322.58 180)
     (effects (font (size 1.27 1.27)) (justify right bottom))
   )
@@
     (in_bom yes) (on_board yes)
     (property "Reference" "R75" (id 0) (at 63.5 163.83 90))
-    (property "Value" "110Ω" (id 1) (at 64.77 168.91 90))
+    (property "Value" "110" (id 1) (at 64.77 168.91 90))
     (property "Footprint" "" (id 2) (at 63.754 165.354 90)
       (effects (font (size 1.27 1.27)) hide)
@@
     (in_bom yes) (on_board yes)
     (property "Reference" "R55" (id 0) (at 313.69 270.51 90))
-    (property "Value" "330Ω" (id 1) (at 326.39 270.51 90))
+    (property "Value" "330" (id 1) (at 326.39 270.51 90))
     (property "Footprint" "" (id 2) (at 320.294 270.764 90)
       (effects (font (size 1.27 1.27)) hide)
@@
     (in_bom yes) (on_board yes)
     (property "Reference" "R29" (id 0) (at 273.05 369.57 90))
-    (property "Value" "100Ω" (id 1) (at 273.05 374.65 90))
+    (property "Value" "100" (id 1) (at 273.05 374.65 90))
     (property "Footprint" "" (id 2) (at 273.304 371.094 90)
       (effects (font (size 1.27 1.27)) hide)
@@
     (in_bom yes) (on_board yes)
     (property "Reference" "R63" (id 0) (at 73.66 120.65 90))
-    (property "Value" "110Ω" (id 1) (at 73.66 125.73 90))
+    (property "Value" "110" (id 1) (at 73.66 125.73 90))
     (property "Footprint" "" (id 2) (at 73.914 124.206 90)
       (effects (font (size 1.27 1.27)) hide)
@@
     (in_bom yes) (on_board yes)
     (property "Reference" "RN12" (id 0) (at 316.23 317.5 90))
-    (property "Value" "330Ω" (id 1) (at 316.23 320.04 90))
+    (property "Value" "330" (id 1) (at 316.23 320.04 90))
     (property "Footprint" "" (id 2) (at 316.23 318.135 90)
       (effects (font (size 1.27 1.27)) hide)
@@
     (in_bom yes) (on_board yes)
     (property "Reference" "R59" (id 0) (at 313.69 260.35 90))
-    (property "Value" "330Ω" (id 1) (at 326.39 260.35 90))
+    (property "Value" "330" (id 1) (at 326.39 260.35 90))
     (property "Footprint" "" (id 2) (at 320.294 260.604 90)
       (effects (font (size 1.27 1.27)) hide)
@@
     (in_bom yes) (on_board yes)
     (property "Reference" "R56" (id 0) (at 313.69 267.97 90))
-    (property "Value" "330Ω" (id 1) (at 326.39 267.97 90))
+    (property "Value" "330" (id 1) (at 326.39 267.97 90))
     (property "Footprint" "" (id 2) (at 320.294 268.224 90)
       (effects (font (size 1.27 1.27)) hide)
@@
     (in_bom yes) (on_board yes)
     (property "Reference" "RN13" (id 0) (at 316.23 342.9 90))
-    (property "Value" "330Ω" (id 1) (at 316.23 345.44 90))
+    (property "Value" "330" (id 1) (at 316.23 345.44 90))
     (property "Footprint" "" (id 2) (at 316.23 328.295 90)
       (effects (font (size 1.27 1.27)) hide)
@@
     (in_bom yes) (on_board yes)
     (property "Reference" "RN8" (id 0) (at 312.42 252.73 90))
-    (property "Value" "330Ω" (id 1) (at 312.42 255.27 90))
+    (property "Value" "330" (id 1) (at 312.42 255.27 90))
     (property "Footprint" "" (id 2) (at 304.8 260.985 90)
       (effects (font (size 1.27 1.27)) hide)
@@
     (in_bom yes) (on_board yes)
     (property "Reference" "R57" (id 0) (at 313.69 257.81 90))
-    (property "Value" "330Ω" (id 1) (at 326.39 257.81 90))
+    (property "Value" "330" (id 1) (at 326.39 257.81 90))
     (property "Footprint" "" (id 2) (at 320.294 258.064 90)
       (effects (font (size 1.27 1.27)) hide)
@@
     (in_bom yes) (on_board yes)
     (property "Reference" "RN9" (id 0) (at 312.42 240.03 90))
-    (property "Value" "330Ω" (id 1) (at 312.42 242.57 90))
+    (property "Value" "330" (id 1) (at 312.42 242.57 90))
     (property "Footprint" "" (id 2) (at 304.8 250.825 90)
       (effects (font (size 1.27 1.27)) hide)
@@
     (in_bom yes) (on_board yes)
     (property "Reference" "RN11" (id 0) (at 322.58 218.44 90))
-    (property "Value" "620Ω" (id 1) (at 322.58 220.98 90))
+    (property "Value" "620" (id 1) (at 322.58 220.98 90))
     (property "Footprint" "" (id 2) (at 304.8 230.505 90)
       (effects (font (size 1.27 1.27)) hide)
@@
     (in_bom yes) (on_board yes)
     (property "Reference" "R74" (id 0) (at 67.31 125.73 90))
-    (property "Value" "110Ω" (id 1) (at 67.31 130.81 90))
+    (property "Value" "110" (id 1) (at 67.31 130.81 90))
     (property "Footprint" "" (id 2) (at 67.564 127.254 90)
       (effects (font (size 1.27 1.27)) hide)
@@
     (in_bom yes) (on_board yes)
     (property "Reference" "RN14" (id 0) (at 322.58 210.82 90))
-    (property "Value" "620Ω" (id 1) (at 322.58 213.36 90))
+    (property "Value" "620" (id 1) (at 322.58 213.36 90))
     (property "Footprint" "" (id 2) (at 304.8 220.345 90)
       (effects (font (size 1.27 1.27)) hide)
@@
     (in_bom yes) (on_board yes)
     (property "Reference" "RN10" (id 0) (at 322.58 229.87 90))
-    (property "Value" "620Ω" (id 1) (at 322.58 232.41 90))
+    (property "Value" "620" (id 1) (at 322.58 232.41 90))
     (property "Footprint" "" (id 2) (at 304.8 240.665 90)
       (effects (font (size 1.27 1.27)) hide)
@@
     (in_bom yes) (on_board yes)
     (property "Reference" "R58" (id 0) (at 313.69 262.89 90))
-    (property "Value" "330Ω" (id 1) (at 326.39 262.89 90))
+    (property "Value" "330" (id 1) (at 326.39 262.89 90))
     (property "Footprint" "" (id 2) (at 320.294 263.144 90)
       (effects (font (size 1.27 1.27)) hide)

Commit message: wip_ccu_cassette
Connections:
- net VCC: no longer G2.13 (VCC)
- net CLK_GLL2: now reaches R74.1, R75.1, X2.3 (Out)
- net at R63.2: no longer G2.18 (CLK)
- new net 2GLL2PPU0: G2.13 (2GLL2PPU0)
- no-connect marks 52 -> 51
Changed lines of the file:
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@@
   (junction (at 341.63 233.68) (diameter 0) (color 0 0 0 0)
   )
+  (junction (at 58.42 147.32) (diameter 0) (color 0 0 0 0)
+  )
   (junction (at 392.43 140.97) (diameter 0) (color 0 0 0 0)
   )
@@
   (junction (at 124.46 345.44) (diameter 0) (color 0 0 0 0)
   )
-  (junction (at 96.52 120.65) (diameter 0) (color 0 0 0 0)
-  )
   (junction (at 392.43 148.59) (diameter 0) (color 0 0 0 0)
   )
@@
   (no_connect (at 24.13 166.37))
   (no_connect (at 261.62 57.15))
-  (no_connect (at 215.9 106.68))
   (no_connect (at 96.52 130.81))
   (no_connect (at 261.62 46.99))
@@
     (stroke (width 0) (type default) (color 0 0 0 0))
   )
-  (wire (pts (xy 58.42 128.27) (xy 58.42 166.37))
+  (wire (pts (xy 58.42 128.27) (xy 58.42 147.32))
     (stroke (width 0) (type default) (color 0 0 0 0))
   )
@@
     (stroke (width 0) (type default) (color 0 0 0 0))
   )
+  (wire (pts (xy 58.42 147.32) (xy 63.5 147.32))
+    (stroke (width 0) (type default) (color 0 0 0 0))
+  )
   (bus (pts (xy 378.46 53.34) (xy 378.46 60.96))
     (stroke (width 0) (type default) (color 0 0 0 0))
@@
     (stroke (width 0) (type default) (color 0 0 0 0))
   )
+  (wire (pts (xy 58.42 147.32) (xy 58.42 166.37))
+    (stroke (width 0) (type default) (color 0 0 0 0))
+  )
   (wire (pts (xy 271.78 332.74) (xy 311.15 332.74))
     (stroke (width 0) (type default) (color 0 0 0 0))
@@
     (stroke (width 0) (type default) (color 0 0 0 0))
   )
-  (wire (pts (xy 95.25 125.73) (xy 96.52 125.73))
-    (stroke (width 0) (type default) (color 0 0 0 0))
-  )
   (bus (pts (xy 285.75 193.04) (xy 285.75 195.58))
     (stroke (width 0) (type default) (color 0 0 0 0))
@@
     (stroke (width 0) (type default) (color 0 0 0 0))
   )
-  (polyline (pts (xy 226.06 104.14) (xy 226.06 106.68))
-    (stroke (width 0) (type default) (color 0 0 0 0))
-  )
   (wire (pts (xy 381 38.1) (xy 392.43 38.1))
     (stroke (width 0) (type default) (color 0 0 0 0))
@@
     (stroke (width 0) (type default) (color 0 0 0 0))
   )
-  (wire (pts (xy 85.09 166.37) (xy 96.52 166.37))
-    (stroke (width 0) (type default) (color 0 0 0 0))
-  )
   (bus (pts (xy 80.01 323.85) (xy 80.01 321.31))
     (stroke (width 0) (type default) (color 0 0 0 0))
@@
     (stroke (width 0) (type default) (color 0 0 0 0))
   )
-  (wire (pts (xy 96.52 120.65) (xy 96.52 123.19))
-    (stroke (width 0) (type default) (color 0 0 0 0))
-  )
   (wire (pts (xy 36.83 109.22) (xy 36.83 102.87))
     (stroke (width 0) (type default) (color 0 0 0 0))
@@
     (stroke (width 0) (type default) (color 0 0 0 0))
   )
+  (wire (pts (xy 215.9 97.79) (xy 215.9 104.14))
+    (stroke (width 0) (type default) (color 0 0 0 0))
+  )
   (wire (pts (xy 468.63 327.66) (xy 477.52 327.66))
     (stroke (width 0) (type default) (color 0 0 0 0))
@@
     (stroke (width 0) (type default) (color 0 0 0 0))
   )
-  (polyline (pts (xy 215.9 104.14) (xy 226.06 104.14))
-    (stroke (width 0) (type default) (color 0 0 0 0))
-  )
   (bus (pts (xy 80.01 252.73) (xy 80.01 255.27))
     (stroke (width 0) (type default) (color 0 0 0 0))
@@
     (stroke (width 0) (type default) (color 0 0 0 0))
   )
-  (wire (pts (xy 95.25 123.19) (xy 95.25 125.73))
-    (stroke (width 0) (type default) (color 0 0 0 0))
-  )
   (wire (pts (xy 82.55 245.11) (xy 96.52 245.11))
     (stroke (width 0) (type default) (color 0 0 0 0))
@@
     (effects (font (size 1.27 1.27)) (justify left bottom))
   )
-  (text "NOT \nCONNECTED" (at 215.9 104.14 0)
-    (effects (font (size 1.27 1.27)) (justify left bottom))
-  )
   (label "VCC" (at 403.86 273.05 0)
     (effects (font (size 1.27 1.27)) (justify left bottom))
@@
     (effects (font (size 1.27 1.27)) (justify left bottom))
   )
-  (label "VSS" (at 85.09 166.37 0)
-    (effects (font (size 1.27 1.27)) (justify left bottom))
-  )
   (label "~{WE}" (at 261.62 91.44 270)
     (effects (font (size 1.27 1.27)) (justify right bottom))
@@
     (effects (font (size 1.27 1.27)) (justify left))
   )
+  (hierarchical_label "CLK_GLL2" (shape output) (at 63.5 147.32 0)
+    (effects (font (size 1.27 1.27)) (justify left))
+  )
   (hierarchical_label "SYNC" (shape output) (at 299.72 388.62 0)
     (effects (font (size 1.27 1.27)) (justify left))
@@
     (effects (font (size 1.27 1.27)) (justify left))
   )
+  (hierarchical_label "2GLL2PPU0" (shape bidirectional) (at 215.9 97.79 90)
+    (effects (font (size 1.27 1.27)) (justify left))
+  )
   (hierarchical_label "~{CS_PAL}H" (shape input) (at 213.36 97.79 90)
     (effects (font (size 1.27 1.27)) (justify left))
@@
     (pin "2")
   )
-  (symbol (lib_name "CU383-69K_2") (lib_id "arcade:CU383-69K") (at 488.95 294.64 0) (unit 1)
+  (symbol (lib_id "arcade:CU383-69K") (at 488.95 294.64 0) (unit 1)
     (in_bom yes) (on_board yes)
     (property "Reference" "H4" (id 0) (at 495.3 276.86 0))
@@
     (pin "2")
   )
-  (symbol (lib_name "CU383-69K_1") (lib_id "arcade:CU383-69K") (at 250.19 55.88 0) (unit 1)
+  (symbol (lib_id "arcade:CU383-69K") (at 250.19 55.88 0) (unit 1)
     (in_bom yes) (on_board yes)
     (property "Reference" "D7" (id 0) (at 256.54 38.1 0))
@@
     (pin "2")
   )
-  (symbol (lib_name "CU383-69K_3") (lib_id "arcade:CU383-69K") (at 403.86 294.64 0) (unit 1)
+  (symbol (lib_id "arcade:CU383-69K") (at 403.86 294.64 0) (unit 1)
     (in_bom yes) (on_board yes)
     (property "Reference" "H2" (id 0) (at 410.21 276.86 0))
-    (property "Value" "CU383-69K" (id 1) (at 403.86 306.07 0))
+    (property "Value" "CU383-69K" (id 1) (at 394.97 276.86 0))
     (property "Footprint" "" (id 2) (at 403.86 298.45 90)
       (effects (font (size 1.27 1.27)) hide)
@@
     (in_bom yes) (on_board yes)
     (property "Reference" "H1" (id 0) (at 410.21 320.04 0))
-    (property "Value" "CU383-69K" (id 1) (at 403.86 349.25 0))
+    (property "Value" "CU383-69K" (id 1) (at 394.97 320.04 0))
     (property "Footprint" "" (id 2) (at 403.86 341.63 90)
       (effects (font (size 1.27 1.27)) hide)
@@
     (pin "8")
   )
-  (symbol (lib_name "CU383-69K_1") (lib_id "arcade:CU383-69K") (at 488.95 339.09 0) (unit 1)
+  (symbol (lib_id "arcade:CU383-69K") (at 488.95 339.09 0) (unit 1)
     (in_bom yes) (on_board yes)
     (property "Reference" "H3" (id 0) (at 495.3 321.31 0))
