File: cores/cps3/sch/simms_1-2.kicad_sch (KiCad schematic)
At the start: 8 parts

Commit message: clear_sch_hk_cr
Other:
- note added: "Slot 1"
- note added: "Slot 2"
- note removed: "The pattern table ?"
Changed lines of the file:
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@@
     )
   )
-  (text "The pattern table ?\n" (at 148.59 26.67 0)
-    (effects (font (size 5 5)) (justify left bottom))
+  (text "Slot 1" (at 43.18 163.83 0)
+    (effects (font (size 3 3) bold) (justify left bottom))
+  )
+  (text "Slot 2\n" (at 43.18 76.2 0)
+    (effects (font (size 3 3) bold) (justify left bottom))
   )
   (label "MAIND_D2" (at 360.68 52.07 180)
