File: cores/cps3/sch/capacitors_uu.kicad_sch (KiCad schematic)
At the start: 76 parts, among them U2 74LS08

Commit message: capacitors_snd
Parts:
- added CP100, CP101, CP62, CP63, CP64, CP65, CP66, CP67, CP68, CP69, CP70, CP71, CP72, CP73, CP74, CP75, CP76, CP77, CP78, CP79, CP80, CP81, CP82, CP83, CP84, CP85, CP86, CP87, CP88, CP89, CP90, CP91, CP92, CP93, CP94, CP95, CP96, CP97, CP98, CP99: μ, symbol Device:C_Polarized_US
- added CP117, CP118, CP119, CP120, CP121, CP122: 1016R, symbol Device:C_Polarized_US
- renumbered CP62 to CP102, CP63 to CP103, CP64 to CP104, CP65 to CP105, CP66 to CP106, CP67 to CP107, CP68 to CP108, CP69 to CP109, CP70 to CP110, CP71 to CP111, CP72 to CP112, CP73 to CP113, CP74 to CP114, CP75 to CP115, CP76 to CP116
Connections:
- net VCC: now also CP100.1, CP101.1, CP117.1, CP118.1, CP119.1, CP120.1, CP121.1, CP122.1, CP62.1, CP63.1, CP64.1, CP65.1, CP66.1, CP67.1, CP68.1, CP69.1, CP70.1, CP71.1, CP72.1, CP73.1, CP74.1, CP75.1, CP76.1, CP77.1, CP78.1, CP79.1, CP80.1, CP81.1, CP82.1, CP83.1, CP84.1, CP85.1, CP86.1, CP87.1, CP88.1, CP89.1, CP90.1, CP91.1, CP92.1, CP93.1, CP94.1, CP95.1, CP96.1, CP97.1, CP98.1, CP99.1
- net VSS: now also CP100.2, CP101.2, CP117.2, CP118.2, CP119.2, CP120.2, CP121.2, CP122.2, CP62.2, CP63.2, CP64.2, CP65.2, CP66.2, CP67.2, CP68.2, CP69.2, CP70.2, CP71.2, CP72.2, CP73.2, CP74.2, CP75.2, CP76.2, CP77.2, CP78.2, CP79.2, CP80.2, CP81.2, CP82.2, CP83.2, CP84.2, CP85.2, CP86.2, CP87.2, CP88.2, CP89.2, CP90.2, CP91.2, CP92.2, CP93.2, CP94.2, CP95.2, CP96.2, CP97.2, CP98.2, CP99.2
Other:
- moved on the sheet: CP10, CP102, CP103, CP104, CP105, CP106, CP107, CP108, CP109, CP11, CP110, CP111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
