File: cores/cps3/sch/capacitors_uu.kicad_sch (KiCad schematic)
At the start: 122 parts, among them U2 74LS08

Commit message: wip cps3
Parts:
- added A4, A5: Opamp_Dual, symbol Device:Opamp_Dual
Connections:
- net VCC: now also A4.8 (V+), A5.8 (V+)
- net VSS: now also A4.4 (V-), A5.4 (V-)
Changed lines of the file:
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@@
   (junction (at 88.9 66.04) (diameter 0) (color 0 0 0 0)
   )
+  (junction (at 25.4 149.86) (diameter 0) (color 0 0 0 0)
+  )
   (junction (at 127 73.66) (diameter 0) (color 0 0 0 0)
   )
@@
   (junction (at 114.3 29.21) (diameter 0) (color 0 0 0 0)
   )
+  (junction (at 38.1 165.1) (diameter 0) (color 0 0 0 0)
+  )
+  (junction (at 38.1 149.86) (diameter 0) (color 0 0 0 0)
+  )
   (junction (at 139.7 29.21) (diameter 0) (color 0 0 0 0)
   )
@@
     (stroke (width 0) (type default) (color 0 0 0 0))
   )
-  (wire (pts (xy 25.4 163.83) (xy 25.4 161.29))
+  (wire (pts (xy 25.4 161.29) (xy 25.4 165.1))
     (stroke (width 0) (type default) (color 0 0 0 0))
   )
@@
     (stroke (width 0) (type default) (color 0 0 0 0))
   )
+  (wire (pts (xy 38.1 165.1) (xy 38.1 168.91))
+    (stroke (width 0) (type default) (color 0 0 0 0))
+  )
+  (wire (pts (xy 25.4 165.1) (xy 38.1 165.1))
+    (stroke (width 0) (type default) (color 0 0 0 0))
+  )
   (wire (pts (xy 50.8 52.07) (xy 63.5 52.07))
     (stroke (width 0) (type default) (color 0 0 0 0))
@@
     (stroke (width 0) (type default) (color 0 0 0 0))
   )
+  (wire (pts (xy 25.4 149.86) (xy 38.1 149.86))
+    (stroke (width 0) (type default) (color 0 0 0 0))
+  )
   (wire (pts (xy 50.8 66.04) (xy 63.5 66.04))
     (stroke (width 0) (type default) (color 0 0 0 0))
@@
     (stroke (width 0) (type default) (color 0 0 0 0))
   )
+  (wire (pts (xy 38.1 165.1) (xy 54.61 165.1))
+    (stroke (width 0) (type default) (color 0 0 0 0))
+  )
   (wire (pts (xy 228.6 143.51) (xy 241.3 143.51))
     (stroke (width 0) (type default) (color 0 0 0 0))
@@
     (stroke (width 0) (type default) (color 0 0 0 0))
   )
-  (wire (pts (xy 25.4 151.13) (xy 25.4 153.67))
+  (wire (pts (xy 25.4 147.32) (xy 25.4 149.86))
     (stroke (width 0) (type default) (color 0 0 0 0))
   )
@@
     (stroke (width 0) (type default) (color 0 0 0 0))
   )
+  (wire (pts (xy 25.4 149.86) (xy 25.4 153.67))
+    (stroke (width 0) (type default) (color 0 0 0 0))
+  )
   (wire (pts (xy 38.1 66.04) (xy 50.8 66.04))
     (stroke (width 0) (type default) (color 0 0 0 0))
@@
   )
   (wire (pts (xy 177.8 52.07) (xy 190.5 52.07))
+    (stroke (width 0) (type default) (color 0 0 0 0))
+  )
+  (wire (pts (xy 38.1 149.86) (xy 54.61 149.86))
     (stroke (width 0) (type default) (color 0 0 0 0))
   )
@@
     (effects (font (size 1.27 1.27)) (justify left bottom))
   )
-  (label "VCC" (at 25.4 151.13 0)
+  (label "VCC" (at 25.4 147.32 0)
     (effects (font (size 1.27 1.27)) (justify left bottom))
   )
-  (label "VSS" (at 25.4 163.83 0)
+  (label "VSS" (at 38.1 168.91 0)
     (effects (font (size 1.27 1.27)) (justify left bottom))
   )
@@
     (pin "2")
   )
+  (symbol (lib_id "Device:Opamp_Dual") (at 57.15 157.48 0) (unit 3)
+    (in_bom yes) (on_board yes)
+    (property "Reference" "A5" (id 0) (at 57.15 152.4 0)
+      (effects (font (size 1.27 1.27)) (justify left))
+    )
+    (property "Value" "Opamp_Dual" (id 1) (at 57.15 162.56 0)
+      (effects (font (size 1.27 1.27)) (justify left))
+    )
+    (property "Footprint" "" (id 2) (at 57.15 157.48 0)
+      (effects (font (size 1.27 1.27)) hide)
+    )
+    (property "Datasheet" "~" (id 3) (at 57.15 157.48 0)
+      (effects (font (size 1.27 1.27)) hide)
+    )
+    (pin "1")
+    (pin "2")
+    (pin "3")
+    (pin "5")
+    (pin "6")
+    (pin "7")
+    (pin "4")
+    (pin "8")
+  )
   (symbol (lib_id "Device:C_Polarized_US") (at 139.7 25.4 0) (unit 1)
     (in_bom yes) (on_board yes)
@@
     (pin "2")
   )
+  (symbol (lib_id "Device:Opamp_Dual") (at 40.64 157.48 0) (unit 3)
+    (in_bom yes) (on_board yes)
+    (property "Reference" "A4" (id 0) (at 40.64 152.4 0)
+      (effects (font (size 1.27 1.27)) (justify left))
+    )
+    (property "Value" "Opamp_Dual" (id 1) (at 40.64 162.56 0)
+      (effects (font (size 1.27 1.27)) (justify left))
+    )
+    (property "Footprint" "" (id 2) (at 40.64 157.48 0)
+      (effects (font (size 1.27 1.27)) hide)
+    )
+    (property "Datasheet" "~" (id 3) (at 40.64 157.48 0)
+      (effects (font (size 1.27 1.27)) hide)
+    )
+    (pin "1")
+    (pin "2")
+    (pin "3")
+    (pin "5")
+    (pin "6")
+    (pin "7")
+    (pin "4")
+    (pin "8")
+  )
   (symbol (lib_id "Device:C_Polarized_US") (at 114.3 92.71 0) (unit 1)

Commit message: wip_snd
Parts:
- added CP141, CP142: 220μF, symbol Device:C_Polarized_US
Connections:
- net VCC: now also CP141.1; no longer A4.8 (V+), A5.8 (V+)
- net VSS: now also CP141.2, CP142.2
- new net: A4.8 (V+), A5.8 (V+)
- new net +12V: CP142.1
Other:
- moved on the sheet: A4C, A5C
Changed lines of the file:
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@@
   (junction (at 190.5 52.07) (diameter 0) (color 0 0 0 0)
   )
+  (junction (at 38.1 161.29) (diameter 0) (color 0 0 0 0)
+  )
   (junction (at 101.6 119.38) (diameter 0) (color 0 0 0 0)
   )
@@
   (junction (at 139.7 52.07) (diameter 0) (color 0 0 0 0)
   )
+  (junction (at 25.4 153.67) (diameter 0) (color 0 0 0 0)
+  )
   (junction (at 101.6 96.52) (diameter 0) (color 0 0 0 0)
   )
@@
   (junction (at 177.8 96.52) (diameter 0) (color 0 0 0 0)
   )
+  (junction (at 25.4 161.29) (diameter 0) (color 0 0 0 0)
+  )
   (junction (at 228.6 135.89) (diameter 0) (color 0 0 0 0)
   )
@@
   (junction (at 88.9 66.04) (diameter 0) (color 0 0 0 0)
   )
-  (junction (at 25.4 149.86) (diameter 0) (color 0 0 0 0)
-  )
   (junction (at 127 73.66) (diameter 0) (color 0 0 0 0)
   )
@@
   (junction (at 114.3 29.21) (diameter 0) (color 0 0 0 0)
   )
-  (junction (at 38.1 165.1) (diameter 0) (color 0 0 0 0)
-  )
-  (junction (at 38.1 149.86) (diameter 0) (color 0 0 0 0)
+  (junction (at 53.34 190.5) (diameter 0) (color 0 0 0 0)
+  )
+  (junction (at 53.34 175.26) (diameter 0) (color 0 0 0 0)
   )
   (junction (at 139.7 29.21) (diameter 0) (color 0 0 0 0)
@@
   (junction (at 114.3 73.66) (diameter 0) (color 0 0 0 0)
   )
+  (junction (at 50.8 161.29) (diameter 0) (color 0 0 0 0)
+  )
   (junction (at 139.7 119.38) (diameter 0) (color 0 0 0 0)
   )
@@
     (stroke (width 0) (type default) (color 0 0 0 0))
   )
+  (wire (pts (xy 53.34 175.26) (xy 66.04 175.26))
+    (stroke (width 0) (type default) (color 0 0 0 0))
+  )
   (wire (pts (xy 203.2 66.04) (xy 215.9 66.04))
     (stroke (width 0) (type default) (color 0 0 0 0))
@@
     (stroke (width 0) (type default) (color 0 0 0 0))
   )
+  (wire (pts (xy 38.1 161.29) (xy 50.8 161.29))
+    (stroke (width 0) (type default) (color 0 0 0 0))
+  )
   (wire (pts (xy 50.8 96.52) (xy 63.5 96.52))
     (stroke (width 0) (type default) (color 0 0 0 0))
@@
     (stroke (width 0) (type default) (color 0 0 0 0))
   )
-  (wire (pts (xy 38.1 165.1) (xy 38.1 168.91))
-    (stroke (width 0) (type default) (color 0 0 0 0))
-  )
-  (wire (pts (xy 25.4 165.1) (xy 38.1 165.1))
+  (wire (pts (xy 53.34 190.5) (xy 53.34 194.31))
     (stroke (width 0) (type default) (color 0 0 0 0))
   )
@@
     (stroke (width 0) (type default) (color 0 0 0 0))
   )
-  (wire (pts (xy 25.4 149.86) (xy 38.1 149.86))
-    (stroke (width 0) (type default) (color 0 0 0 0))
-  )
   (wire (pts (xy 50.8 66.04) (xy 63.5 66.04))
     (stroke (width 0) (type default) (color 0 0 0 0))
@@
     (stroke (width 0) (type default) (color 0 0 0 0))
   )
+  (wire (pts (xy 40.64 175.26) (xy 53.34 175.26))
+    (stroke (width 0) (type default) (color 0 0 0 0))
+  )
+  (wire (pts (xy 25.4 153.67) (xy 38.1 153.67))
+    (stroke (width 0) (type default) (color 0 0 0 0))
+  )
   (wire (pts (xy 228.6 66.04) (xy 241.3 66.04))
     (stroke (width 0) (type default) (color 0 0 0 0))
@@
     (stroke (width 0) (type default) (color 0 0 0 0))
   )
+  (wire (pts (xy 50.8 153.67) (xy 50.8 151.13))
+    (stroke (width 0) (type default) (color 0 0 0 0))
+  )
   (wire (pts (xy 101.6 66.04) (xy 114.3 66.04))
     (stroke (width 0) (type default) (color 0 0 0 0))
@@
     (stroke (width 0) (type default) (color 0 0 0 0))
   )
+  (wire (pts (xy 53.34 190.5) (xy 66.04 190.5))
+    (stroke (width 0) (type default) (color 0 0 0 0))
+  )
   (wire (pts (xy 101.6 44.45) (xy 114.3 44.45))
     (stroke (width 0) (type default) (color 0 0 0 0))
@@
     (stroke (width 0) (type default) (color 0 0 0 0))
   )
-  (wire (pts (xy 38.1 165.1) (xy 54.61 165.1))
+  (wire (pts (xy 46.99 151.13) (xy 50.8 151.13))
+    (stroke (width 0) (type default) (color 0 0 0 0))
+  )
+  (wire (pts (xy 40.64 190.5) (xy 53.34 190.5))
     (stroke (width 0) (type default) (color 0 0 0 0))
   )
@@
     (stroke (width 0) (type default) (color 0 0 0 0))
   )
-  (wire (pts (xy 25.4 147.32) (xy 25.4 149.86))
+  (wire (pts (xy 25.4 147.32) (xy 25.4 153.67))
     (stroke (width 0) (type default) (color 0 0 0 0))
   )
@@
     (stroke (width 0) (type default) (color 0 0 0 0))
   )
-  (wire (pts (xy 25.4 149.86) (xy 25.4 153.67))
-    (stroke (width 0) (type default) (color 0 0 0 0))
-  )
   (wire (pts (xy 38.1 66.04) (xy 50.8 66.04))
     (stroke (width 0) (type default) (color 0 0 0 0))
@@
     (stroke (width 0) (type default) (color 0 0 0 0))
   )
+  (wire (pts (xy 50.8 161.29) (xy 76.2 161.29))
+    (stroke (width 0) (type default) (color 0 0 0 0))
+  )
   (wire (pts (xy 25.4 143.51) (xy 38.1 143.51))
     (stroke (width 0) (type default) (color 0 0 0 0))
@@
     (stroke (width 0) (type default) (color 0 0 0 0))
   )
-  (wire (pts (xy 38.1 149.86) (xy 54.61 149.86))
-    (stroke (width 0) (type default) (color 0 0 0 0))
-  )
   (wire (pts (xy 38.1 44.45) (xy 50.8 44.45))
     (stroke (width 0) (type default) (color 0 0 0 0))
@@
   )
   (wire (pts (xy 114.3 119.38) (xy 127 119.38))
+    (stroke (width 0) (type default) (color 0 0 0 0))
+  )
+  (wire (pts (xy 25.4 161.29) (xy 38.1 161.29))
     (stroke (width 0) (type default) (color 0 0 0 0))
   )
@@
     )
   )
+  (label "VSS" (at 25.4 165.1 0)
+    (effects (font (size 1.27 1.27)) (justify left bottom))
+  )
   (label "VCC" (at 139.7 83.82 0)
     (effects (font (size 1.27 1.27)) (justify left bottom))
@@
     (effects (font (size 1.27 1.27)) (justify left bottom))
   )
-  (label "VSS" (at 38.1 168.91 0)
+  (label "VSS" (at 53.34 194.31 0)
     (effects (font (size 1.27 1.27)) (justify left bottom))
   )
@@
     (effects (font (size 1.27 1.27)) (justify left bottom))
   )
+  (hierarchical_label "+12V" (shape passive) (at 46.99 151.13 180)
+    (effects (font (size 1.27 1.27)) (justify right))
+  )
   (symbol (lib_id "Device:C_Polarized_US") (at 228.6 25.4 0) (unit 1)
     (in_bom yes) (on_board yes)
@@
     (pin "2")
   )
+  (symbol (lib_id "Device:C_Polarized_US") (at 50.8 157.48 0) (unit 1)
+    (in_bom yes) (on_board yes)
+    (property "Reference" "CP142" (id 0) (at 51.435 154.94 0)
+      (effects (font (size 1.27 1.27)) (justify left))
+    )
+    (property "Value" "220μF" (id 1) (at 51.435 160.02 0)
+      (effects (font (size 1.27 1.27)) (justify left))
+    )
+    (property "Footprint" "" (id 2) (at 50.8 157.48 0)
+      (effects (font (size 1.27 1.27)) hide)
+    )
+    (property "Datasheet" "~" (id 3) (at 50.8 157.48 0)
+      (effects (font (size 1.27 1.27)) hide)
+    )
+    (pin "1")
+    (pin "2")
+  )
   (symbol (lib_id "Device:C_Polarized_US") (at 50.8 69.85 0) (unit 1)
     (in_bom yes) (on_board yes)
@@
     (pin "2")
   )
-  (symbol (lib_id "Device:Opamp_Dual") (at 57.15 157.48 0) (unit 3)
-    (in_bom yes) (on_board yes)
-    (property "Reference" "A5" (id 0) (at 57.15 152.4 0)
-      (effects (font (size 1.27 1.27)) (justify left))
-    )
-    (property "Value" "Opamp_Dual" (id 1) (at 57.15 162.56 0)
-      (effects (font (size 1.27 1.27)) (justify left))
-    )
-    (property "Footprint" "" (id 2) (at 57.15 157.48 0)
-      (effects (font (size 1.27 1.27)) hide)
-    )
-    (property "Datasheet" "~" (id 3) (at 57.15 157.48 0)
+  (symbol (lib_id "Device:Opamp_Dual") (at 68.58 182.88 0) (unit 3)
+    (in_bom yes) (on_board yes)
+    (property "Reference" "A5" (id 0) (at 67.31 177.8 0)
+      (effects (font (size 1.27 1.27)) (justify left))
+    )
+    (property "Value" "Opamp_Dual" (id 1) (at 62.23 187.96 90)
+      (effects (font (size 1.27 1.27)) (justify left))
+    )
+    (property "Footprint" "" (id 2) (at 68.58 182.88 0)
+      (effects (font (size 1.27 1.27)) hide)
+    )
+    (property "Datasheet" "~" (id 3) (at 68.58 182.88 0)
       (effects (font (size 1.27 1.27)) hide)
     )
@@
     (pin "2")
   )
+  (symbol (lib_id "Device:C_Polarized_US") (at 38.1 157.48 0) (unit 1)
+    (in_bom yes) (on_board yes)
+    (property "Reference" "CP141" (id 0) (at 38.735 154.94 0)
+      (effects (font (size 1.27 1.27)) (justify left))
+    )
+    (property "Value" "220μF" (id 1) (at 38.735 160.02 0)
+      (effects (font (size 1.27 1.27)) (justify left))
+    )
+    (property "Footprint" "" (id 2) (at 38.1 157.48 0)
+      (effects (font (size 1.27 1.27)) hide)
+    )
+    (property "Datasheet" "~" (id 3) (at 38.1 157.48 0)
+      (effects (font (size 1.27 1.27)) hide)
+    )
+    (pin "1")
+    (pin "2")
+  )
   (symbol (lib_id "Device:C_Polarized_US") (at 266.7 92.71 0) (unit 1)
     (in_bom yes) (on_board yes)
@@
     (pin "2")
   )
-  (symbol (lib_id "Device:Opamp_Dual") (at 40.64 157.48 0) (unit 3)
-    (in_bom yes) (on_board yes)
-    (property "Reference" "A4" (id 0) (at 40.64 152.4 0)
-      (effects (font (size 1.27 1.27)) (justify left))
-    )
-    (property "Value" "Opamp_Dual" (id 1) (at 40.64 162.56 0)
-      (effects (font (size 1.27 1.27)) (justify left))
-    )
-    (property "Footprint" "" (id 2) (at 40.64 157.48 0)
-      (effects (font (size 1.27 1.27)) hide)
-    )
-    (property "Datasheet" "~" (id 3) (at 40.64 157.48 0)
-      (effects (font (size 1.27 1.27)) hide)
-    )
+  (symbol (lib_id "Device:Opamp_Dual") (at 55.88 182.88 0) (unit 3)
+    (in_bom yes) (on_board yes)
+    (property "Reference" "A4" (id 0) (at 54.61 177.8 0)
+      (effects (font (size 1.27 1.27)) (justify left))
+    )
+    (property "Value" "Opamp_Dual" (id 1) (at 50.8 187.96 90)
+      (effects (font (size 1.27 1.27)) (justify left))
+    )
+    (property "Footprint" "" (id 2) (at 55.88 182.88 0)
+      (effects (font (size 1.27 1.27)) hide)
+    )
+    (property "Datasheet" "~" (id 3) (at 55.88 182.88 0)
+      (effects (font (size 1.27 1.27)) hide)
+    )

Commit message: wip_video_dac
Parts:
- added CP157: μ, symbol Device:C_Polarized_US
Connections:
- net VCC: now also CP157.1
- net VSS: now also CP157.2
Other:
- moved on the sheet: CP122, CP141, CP142

Commit message: wip_ccu
Parts:
- removed CP118, CP119, CP120, CP121: 1016R, symbol Device:C_Polarized_US
- CP10, CP100, CP101, CP102, CP103, CP104, CP105, CP106, CP107, CP108, CP109, CP11, CP110, CP111, CP112, CP113, CP114, CP115, CP116, CP12, CP13, CP14, CP15, CP157, CP16, CP17, CP18, CP19, CP2, CP20, CP21, CP22, CP23, CP24, CP25, CP26, CP27, CP28, CP29, CP3, CP30, CP31, CP32, CP33, CP34, CP35, CP36, CP37, CP38, CP39, CP4, CP40, CP41, CP42, CP43, CP44, CP45, CP46, CP47, CP48, CP49, CP5, CP50, CP51, CP52, CP53, CP54, CP55, CP56, CP57, CP58, CP59, CP6, CP60, CP61, CP62, CP63, CP64, CP65, CP66, CP67, CP68, CP69, CP7, CP70, CP71, CP72, CP73, CP74, CP75, CP76, CP77, CP78, CP79, CP8, CP80, CP81, CP82, CP83, CP84, CP85, CP86, CP87, CP88, CP89, CP9, CP90, CP91, CP92, CP93, CP94, CP95, CP96, CP97, CP98, CP99: value μ -> 1nF
Connections:
- net VCC: now also A4.8 (V+), A5.8 (V+)

Commit message: wip_ccu_gll2_cassette
Parts:
- removed CP114: 1nF, symbol Device:C_Polarized_US
- added CP118, CP119: 1016R, symbol Device:C_Polarized_US
- CP115, CP116: value 1nF -> 1016R
Connections:
- net VCC: now also CP118.1, CP119.1
- net VSS: now also CP118.2, CP119.2
Other:
- moved on the sheet: CP115, CP116, CP117

Commit message: wip_cassette
Parts:
- added CP180, CP181, CP182, CP183: 1nF, symbol Device:C_Polarized_US
- added CP184: 47μF, symbol Device:C_Polarized_US
- added U1, U4: 7400, symbol jt74:7400
Connections:
- net VCC: now also CP180.1, CP181.1, CP182.1, CP183.1, CP184.1, U1.14 (VCC), U4.14 (VCC)
- net VSS: now also CP180.2, CP181.2, CP182.2, CP183.2, CP184.2, U1.7 (VSS), U4.7 (VSS)
Other:
- moved on the sheet: A4C, A5C, CP122, CP141, CP142, CP157, U2E

Commit message: wip_cassette_sh2
Other:
- moved on the sheet: A4C, A5C, CP10, CP100, CP101, CP102, CP103, CP104, CP105, CP106, CP107, CP108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

Commit message: wip_cre_cps3
Parts:
- renumbered CP157 to CP201
Changed lines of the file:
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@@
   (symbol (lib_id "Device:C_Polarized_US") (at 114.3 195.58 0) (unit 1)
     (in_bom yes) (on_board yes)
-    (property "Reference" "CP157" (id 0) (at 114.935 193.04 0)
+    (property "Reference" "CP201" (id 0) (at 114.935 193.04 0)
       (effects (font (size 1.27 1.27)) (justify left))
     )
