File: cores/cps3/sch/gll1.kicad_sch (KiCad schematic)
At the start: 1 part, among them J11 DL-3429-GLL1

Commit message: iou
Connections:
- net ALE: no longer names the net of J11.42 (ALE)
- net BIC_CLK renamed CBI_CLK
- net CDI_D0 renamed CBI_D0
- net CDI_D1 renamed CBI_D1
- net CDI_D2 renamed CBI_D2
- net CDI_D3 renamed CBI_D3
- net CDI_D4 renamed CBI_D4
- net CDI_D5 renamed CBI_D5
- net CDI_D6 renamed CBI_D6
- net CDI_D7 renamed CBI_D7
Other:
- moved on the sheet: J11

Commit message: uptate_ns
Connections:
- no-connect marks 0 -> 2
Changed lines of the file:
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@@
   (junction (at 109.22 36.83) (diameter 0) (color 0 0 0 0)
   )
+  (no_connect (at 160.02 36.83))
+  (no_connect (at 162.56 36.83))
   (bus_entry (at 62.23 59.69) (size 2.54 -2.54)
     (stroke (width 0) (type default) (color 0 0 0 0))

Commit message: update_cps3
Connections:
- net MAIN_A4: now reaches J11.31 (MAIN_A4)
- net MAIN_D2: now reaches J11.37 (MAIN_D2)
- net MAIN_D3: now reaches J11.38 (MAIN_D3)
- net MAIN_D4: now reaches J11.39 (MAIN_D4)
- net MAIN_D5: now reaches J11.41 (MAIN_D5)
- net ALE: now reaches J11.42 (ALE)
- net MAIN_A5: now reaches J11.57 (MAIN_A5)
- net CBI_D0 renamed MAIN_D14
- net CBI_D1 renamed MAIN_D13
- net CBI_D2 renamed MAIN_D12
- net CBI_D3 renamed MAIN_D11
- net CBI_D4 renamed MAIN_D10
- net CBI_D5 renamed MAIN_D9
- net CBI_D6 renamed MAIN_D8
- net CBI_D7 renamed MAIN_D7
- net GLL_A0 renamed MAIN_A27
- net GLL_A1 renamed MAIN_A28
- net GLL_A10: no longer names the net of J11.67 (A10)
- net GLL_A11 renamed MAIN_A1
- net GLL_A12 renamed MAIN_A2
- net GLL_A13 renamed MAIN_A0
- net GLL_A14 renamed MAIN_A3
- net GLL_A2 renamed MAIN_A26
- net GLL_A3 renamed MAIN_A25
- net GLL_A4 renamed MAIN_A7
- net GLL_A5 renamed MAIN_A6
- net GLL_A6: no longer names the net of J11.32 (A6)
- net GLL_A7 renamed MAIN_D0
- net GLL_A8 renamed MAIN_D1
- net GLL_A9 renamed MAIN_D6
- net SSU_D0 renamed MAIN_A24
- net SSU_D1 renamed MAIN_A23
- net SSU_D10 renamed MAIN_A14
- net SSU_D11 renamed MAIN_A13
- net SSU_D12 renamed MAIN_A12
- net SSU_D13 renamed MAIN_A11
- net SSU_D14 renamed MAIN_A10
- net SSU_D15 renamed MAIN_A9
- net SSU_D16 renamed MAIN_A8
- net SSU_D2 renamed MAIN_A22
- net SSU_D3 renamed MAIN_A21
- net SSU_D4 renamed MAIN_A20
- net SSU_D5 renamed MAIN_A19
- net SSU_D6 renamed MAIN_A18
- net SSU_D7 renamed MAIN_A17
- net SSU_D8 renamed MAIN_A16
- net SSU_D9 renamed MAIN_A15
- no-connect marks 2 -> 0
Other:
- moved on the sheet: J11

Commit message: update5
Connections:
- net ALE is gone; now on net MAIN_A7: J11.42 (MAIN_A7)
- net MAIN_A24 is gone; now on net MAIN_A3: J11.8 (MAIN_A3)
- net MAIN_A25 is gone; now on net MAIN_A4: J11.7 (MAIN_A4)
- net MAIN_A26 is gone; now on net MAIN_A5: J11.6 (MAIN_A5)
- net MAIN_A27 is gone; now on net MAIN_A20: J11.4 (MAIN_A20)
- net MAIN_A28 is gone; now on net MAIN_A19: J11.5 (MAIN_A19)
- net MAIN_A0: now also J11.31 (MAIN_A0); no longer J11.133 (MAIN_A0)
- net MAIN_A1: now also J11.30 (MAIN_A1); no longer J11.131 (MAIN_A1)
- net MAIN_A10: now also J11.38 (MAIN_A10); no longer J11.26 (MAIN_A10)
- net MAIN_A11: now also J11.37 (MAIN_A11); no longer J11.24 (MAIN_A11)
- net MAIN_A12: now also J11.36 (MAIN_A12); no longer J11.23 (MAIN_A12)
- net MAIN_A13: now also J11.35 (MAIN_A13); no longer J11.22 (MAIN_A13)
- net MAIN_A14: now also J11.57 (MAIN_A14); no longer J11.21 (MAIN_A14)
- net MAIN_A15: now also J11.137 (MAIN_A15); no longer J11.20 (MAIN_A15)
- net MAIN_A16: now also J11.132 (MAIN_A16); no longer J11.17 (MAIN_A16)
- net MAIN_A17: now also J11.131 (MAIN_A17); no longer J11.16 (MAIN_A17)
- net MAIN_A18: now also J11.133 (MAIN_A18); no longer J11.15 (MAIN_A18)
- net MAIN_A19: no longer J11.14 (MAIN_A19)
- net MAIN_A2: now also J11.29 (MAIN_A2); no longer J11.132 (MAIN_A2)
- net MAIN_A20: no longer J11.13 (MAIN_A20)
- net MAIN_A3: no longer J11.137 (MAIN_A3)
- net MAIN_A4: no longer J11.31 (MAIN_A4)
- net MAIN_A5: no longer J11.57 (MAIN_A5)
- net MAIN_A6: now also J11.43 (MAIN_A6); no longer J11.30 (MAIN_A6)
- net MAIN_A7: no longer J11.29 (MAIN_A7)
- net MAIN_A8: now also J11.41 (MAIN_A8); no longer J11.28 (MAIN_A8)
- net MAIN_A9: now also J11.39 (MAIN_A9); no longer J11.27 (MAIN_A9)
- net MAIN_D0: now also J11.53 (MAIN_D0); no longer J11.35 (MAIN_D0)
- net MAIN_D1: now also J11.52 (MAIN_D1); no longer J11.36 (MAIN_D1)
- net MAIN_D10: now also J11.26 (MAIN_D10); no longer J11.49 (MAIN_D10)
- net MAIN_D11: now also J11.24 (MAIN_D11); no longer J11.50 (MAIN_D11)
- net MAIN_D12: now also J11.23 (MAIN_D12); no longer J11.51 (MAIN_D12)
- net MAIN_D13: now also J11.22 (MAIN_D13); no longer J11.52 (MAIN_D13)
- net MAIN_D14: now also J11.21 (MAIN_D14); no longer J11.53 (MAIN_D14)
- net MAIN_D2: now also J11.51 (MAIN_D2); no longer J11.37 (MAIN_D2)
- net MAIN_D3: now also J11.50 (MAIN_D3); no longer J11.38 (MAIN_D3)
- net MAIN_D4: now also J11.49 (MAIN_D4); no longer J11.39 (MAIN_D4)
- net MAIN_D5: now also J11.48 (MAIN_D5); no longer J11.41 (MAIN_D5)
- net MAIN_D6: now also J11.46 (MAIN_D6); no longer J11.43 (MAIN_D6)
- net MAIN_D8: now also J11.28 (MAIN_D8); no longer J11.46 (MAIN_D8)
- net MAIN_D9: now also J11.27 (MAIN_D9); no longer J11.48 (MAIN_D9)
- net MAIN_A21 renamed MAIN_D21
- net MAIN_A22 renamed MAIN_D22
- net MAIN_A23 renamed MAIN_D23
- new net MAIN_D15: J11.20 (MAIN_D15)
- new net MAIN_D16: J11.17 (MAIN_D16)
- new net MAIN_D17: J11.16 (MAIN_D17)
- new net MAIN_D18: J11.15 (MAIN_D18)
- new net MAIN_D19: J11.14 (MAIN_D19)
- new net MAIN_D20: J11.13 (MAIN_D20)

Commit message: update6_cps
Connections:
- net GLL2IO0: now reaches J11.123 (GLL2IO0)
- net GLL2IO1: now reaches J11.139 (GLL2IO1)
- net RESET?: now reaches J11.143 (RESET?)
Changed lines of the file:
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@@
+    (stroke (width 0) (type default) (color 0 0 0 0))
+  )
+  (wire (pts (xy 68.58 97.79) (xy 76.2 97.79))
     (stroke (width 0) (type default) (color 0 0 0 0))
   )
@@
     (stroke (width 0) (type default) (color 0 0 0 0))
   )
+  (wire (pts (xy 68.58 102.87) (xy 76.2 102.87))
+    (stroke (width 0) (type default) (color 0 0 0 0))
+  )
   (wire (pts (xy 119.38 143.51) (xy 121.92 143.51))
     (stroke (width 0) (type default) (color 0 0 0 0))
@@
   )
   (bus (pts (xy 121.92 22.86) (xy 124.46 22.86))
+    (stroke (width 0) (type default) (color 0 0 0 0))
+  )
+  (wire (pts (xy 68.58 100.33) (xy 76.2 100.33))
     (stroke (width 0) (type default) (color 0 0 0 0))
   )
@@
     (effects (font (size 1.27 1.27)) (justify left bottom))
   )
+  (label "RESET?" (at 68.58 102.87 0)
+    (effects (font (size 1.27 1.27)) (justify left bottom))
+  )
   (label "MAIN_D18" (at 165.1 34.29 90)
     (effects (font (size 1.27 1.27)) (justify left bottom))
@@
   (label "MAIN_D3" (at 127 25.4 270)
     (effects (font (size 1.27 1.27)) (justify right bottom))
+  )
+  (hierarchical_label "GLL2IO0" (shape input) (at 68.58 97.79 180)
+    (effects (font (size 1.27 1.27)) (justify right))
+  )
+  (hierarchical_label "RESET?" (shape input) (at 68.58 102.87 180)
+    (effects (font (size 1.27 1.27)) (justify right))
   )
   (hierarchical_label "MAIN_A[20..0]" (shape bidirectional) (at 54.61 41.91 180)
@@
     (effects (font (size 1.27 1.27)) (justify left))
   )
+  (hierarchical_label "GLL2IO1" (shape input) (at 68.58 100.33 180)
+    (effects (font (size 1.27 1.27)) (justify right))
+  )
   (hierarchical_label "MAIN_D[23..0]" (shape bidirectional) (at 110.49 22.86 180)

Commit message: clear_sch_hk_cr
Connections:
- net MAIN_A0 renamed GFX_A0
- net MAIN_A1 renamed GFX_A1
- net MAIN_A10 renamed GFX_A10
- net MAIN_A11 renamed GFX_A11
- net MAIN_A12 renamed GFX_A12
- net MAIN_A13 renamed GFX_A13
- net MAIN_A14 renamed GFX_A14
- net MAIN_A15 renamed GFX_A15
- net MAIN_A16 renamed GFX_A16
- net MAIN_A17 renamed GFX_A17
- net MAIN_A18 renamed GFX_A18
- net MAIN_A19 renamed GFX_A19
- net MAIN_A2 renamed GFX_A2
- net MAIN_A20 renamed GFX_A20
- net MAIN_A3 renamed GFX_A3
- net MAIN_A4 renamed GFX_A4
- net MAIN_A5 renamed GFX_A5
- net MAIN_A6 renamed GFX_A6
- net MAIN_A7 renamed GFX_A7
- net MAIN_A8 renamed GFX_A8
- net MAIN_A9 renamed GFX_A9
Changed lines of the file:
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@@
     )
   )
-  (label "MAIN_A1" (at 64.77 46.99 0)
+  (label "GFX_A1" (at 64.77 46.99 0)
     (effects (font (size 1.27 1.27)) (justify left bottom))
   )
@@
     (effects (font (size 1.27 1.27)) (justify right bottom))
   )
-  (label "MAIN_A14" (at 64.77 80.01 0)
+  (label "GFX_A14" (at 64.77 80.01 0)
     (effects (font (size 1.27 1.27)) (justify left bottom))
   )
-  (label "MAIN_A12" (at 64.77 74.93 0)
+  (label "GFX_A12" (at 64.77 74.93 0)
     (effects (font (size 1.27 1.27)) (justify left bottom))
   )
-  (label "MAIN_A19" (at 64.77 92.71 0)
+  (label "GFX_A19" (at 64.77 92.71 0)
     (effects (font (size 1.27 1.27)) (justify left bottom))
   )
@@
     (effects (font (size 1.27 1.27)) (justify left bottom))
   )
-  (label "MAIN_A4" (at 64.77 54.61 0)
+  (label "GFX_A4" (at 64.77 54.61 0)
     (effects (font (size 1.27 1.27)) (justify left bottom))
   )
@@
     (effects (font (size 1.27 1.27)) (justify right bottom))
   )
-  (label "MAIN_A17" (at 64.77 87.63 0)
+  (label "GFX_A17" (at 64.77 87.63 0)
     (effects (font (size 1.27 1.27)) (justify left bottom))
   )
-  (label "MAIN_A6" (at 64.77 59.69 0)
+  (label "GFX_A6" (at 64.77 59.69 0)
     (effects (font (size 1.27 1.27)) (justify left bottom))
   )
-  (label "MAIN_A10" (at 64.77 69.85 0)
+  (label "GFX_A10" (at 64.77 69.85 0)
     (effects (font (size 1.27 1.27)) (justify left bottom))
   )
@@
     (effects (font (size 1.27 1.27)) (justify left bottom))
   )
-  (label "MAIN_A8" (at 64.77 64.77 0)
+  (label "GFX_A8" (at 64.77 64.77 0)
     (effects (font (size 1.27 1.27)) (justify left bottom))
   )
-  (label "MAIN_A13" (at 64.77 77.47 0)
+  (label "GFX_A13" (at 64.77 77.47 0)
     (effects (font (size 1.27 1.27)) (justify left bottom))
   )
@@
     (effects (font (size 1.27 1.27)) (justify right bottom))
   )
-  (label "MAIN_A11" (at 64.77 72.39 0)
+  (label "GFX_A11" (at 64.77 72.39 0)
     (effects (font (size 1.27 1.27)) (justify left bottom))
   )
@@
     (effects (font (size 1.27 1.27)) (justify right bottom))
   )
-  (label "MAIN_A3" (at 64.77 52.07 0)
+  (label "GFX_A3" (at 64.77 52.07 0)
     (effects (font (size 1.27 1.27)) (justify left bottom))
   )
@@
     (effects (font (size 1.27 1.27)) (justify right bottom))
   )
-  (label "MAIN_A20" (at 64.77 95.25 0)
+  (label "GFX_A20" (at 64.77 95.25 0)
     (effects (font (size 1.27 1.27)) (justify left bottom))
   )
-  (label "MAIN_A18" (at 64.77 90.17 0)
+  (label "GFX_A18" (at 64.77 90.17 0)
     (effects (font (size 1.27 1.27)) (justify left bottom))
   )
-  (label "MAIN_A15" (at 64.77 82.55 0)
+  (label "GFX_A15" (at 64.77 82.55 0)
     (effects (font (size 1.27 1.27)) (justify left bottom))
   )
@@
     (effects (font (size 1.27 1.27)) (justify right bottom))
   )
-  (label "MAIN_A7" (at 64.77 62.23 0)
+  (label "GFX_A7" (at 64.77 62.23 0)
     (effects (font (size 1.27 1.27)) (justify left bottom))
   )
-  (label "MAIN_A5" (at 64.77 57.15 0)
+  (label "GFX_A5" (at 64.77 57.15 0)
     (effects (font (size 1.27 1.27)) (justify left bottom))
   )
-  (label "MAIN_A2" (at 64.77 49.53 0)
+  (label "GFX_A2" (at 64.77 49.53 0)
     (effects (font (size 1.27 1.27)) (justify left bottom))
   )
@@
     (effects (font (size 1.27 1.27)) (justify right bottom))
   )
-  (label "MAIN_A0" (at 64.77 44.45 0)
+  (label "GFX_A0" (at 64.77 44.45 0)
     (effects (font (size 1.27 1.27)) (justify left bottom))
   )
@@
     (effects (font (size 1.27 1.27)) (justify right bottom))
   )
-  (label "MAIN_A16" (at 64.77 85.09 0)
+  (label "GFX_A16" (at 64.77 85.09 0)
     (effects (font (size 1.27 1.27)) (justify left bottom))
   )
-  (label "MAIN_A9" (at 64.77 67.31 0)
+  (label "GFX_A9" (at 64.77 67.31 0)
     (effects (font (size 1.27 1.27)) (justify left bottom))
   )
@@
     (effects (font (size 1.27 1.27)) (justify right))
   )
-  (hierarchical_label "MAIN_A[20..0]" (shape bidirectional) (at 54.61 41.91 180)
+  (hierarchical_label "GFX_A[20..0]" (shape bidirectional) (at 54.61 41.91 180)
     (effects (font (size 1.27 1.27)) (justify right))
   )

Commit message: update7
Connections:
- net GFX_A0 renamed MAIN_A0
- net GFX_A1 renamed MAIN_A1
- net GFX_A10 renamed MAIN_A10
- net GFX_A11 renamed MAIN_A11
- net GFX_A12 renamed MAIN_A12
- net GFX_A13 renamed MAIN_A13
- net GFX_A14 renamed MAIN_A14
- net GFX_A15 renamed MAIN_A15
- net GFX_A16 renamed MAIN_A16
- net GFX_A17 renamed MAIN_A17
- net GFX_A18 renamed MAIN_A18
- net GFX_A19 renamed MAIN_A19
- net GFX_A2 renamed MAIN_A2
- net GFX_A20 renamed MAIN_A20
- net GFX_A3 renamed MAIN_A3
- net GFX_A4 renamed MAIN_A4
- net GFX_A5 renamed MAIN_A5
- net GFX_A6 renamed MAIN_A6
- net GFX_A7 renamed MAIN_A7
- net GFX_A8 renamed MAIN_A8
- net GFX_A9 renamed MAIN_A9
Other:
- note added: "NO OUTPUT OBSERVED PHYSICAL SIGNAL. PENDING TO VERIFY PENDING TO CORRECT PIN LENGTH"
- moved on the sheet: J11

Commit message: wip_ssu_cbi_gll
Connections:
- net CBI_CLK renamed CLK_GLL1
Other:
- note added: "8-20MHz square wave clk"
Changed lines of the file:
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@@
-    (stroke (width 0) (type default) (color 0 0 0 0))
-  )
-  (polyline (pts (xy 190.5 50.8) (xy 190.5 78.74))
     (stroke (width 0) (type default) (color 0 0 0 0))
   )
@@
     (stroke (width 0) (type default) (color 0 0 0 0))
   )
-  (wire (pts (xy 185.42 48.26) (xy 193.04 48.26))
+  (wire (pts (xy 187.96 50.8) (xy 195.58 50.8))
     (stroke (width 0) (type default) (color 0 0 0 0))
   )
@@
     (effects (font (size 3 3)) (justify left bottom))
   )
+  (text "8-20MHz square wave clk" (at 207.01 52.07 0)
+    (effects (font (size 1.27 1.27)) (justify left bottom))
+  )
   (label "MAIN_D5" (at 132.08 25.4 270)
     (effects (font (size 1.27 1.27)) (justify right bottom))
@@
     (effects (font (size 1.27 1.27)) (justify right))
   )
-  (hierarchical_label "CBI_CLK" (shape output) (at 193.04 48.26 0)
+  (hierarchical_label "CLK_GLL1" (shape output) (at 195.58 50.8 0)
     (effects (font (size 1.27 1.27)) (justify left))
   )
