File: cores/cps3/sch/gll1.kicad_sch (KiCad schematic)
At the start: 1 part, among them J11 DL-3429-GLL1

Commit message: wip_gfx_gll
Connections:
- net GLL_DRIVER0: now reaches J11.122 (GLL_DRIVER0)
- net GLL_DRIVER2: now reaches J11.138 (GLL_DRIVER2)
- net GLL2IO0 renamed GLL_DRIVER1
- net GLL2IO1 renamed GLL_DRIVER3
Other:
- note added: "PIN78CON53CASSETE"
Changed lines of the file:
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@@
+    (stroke (width 0) (type default) (color 0 0 0 0))
+  )
+  (wire (pts (xy 278.13 45.72) (xy 267.97 45.72))
     (stroke (width 0) (type default) (color 0 0 0 0))
   )
@@
     (stroke (width 0) (type default) (color 0 0 0 0))
   )
-  (wire (pts (xy 68.58 97.79) (xy 76.2 97.79))
-    (stroke (width 0) (type default) (color 0 0 0 0))
-  )
   (wire (pts (xy 175.26 34.29) (xy 175.26 25.4))
     (stroke (width 0) (type default) (color 0 0 0 0))
@@
     (stroke (width 0) (type default) (color 0 0 0 0))
   )
+  (wire (pts (xy 68.58 102.87) (xy 76.2 102.87))
+    (stroke (width 0) (type default) (color 0 0 0 0))
+  )
   (bus (pts (xy 62.23 41.91) (xy 62.23 44.45))
     (stroke (width 0) (type default) (color 0 0 0 0))
@@
     (stroke (width 0) (type default) (color 0 0 0 0))
   )
+  (wire (pts (xy 278.13 38.1) (xy 267.97 38.1))
+    (stroke (width 0) (type default) (color 0 0 0 0))
+  )
   (bus (pts (xy 62.23 49.53) (xy 62.23 52.07))
     (stroke (width 0) (type default) (color 0 0 0 0))
   )
+  (wire (pts (xy 68.58 100.33) (xy 76.2 100.33))
+    (stroke (width 0) (type default) (color 0 0 0 0))
+  )
   (wire (pts (xy 106.68 146.05) (xy 106.68 148.59))
     (stroke (width 0) (type default) (color 0 0 0 0))
@@
     (stroke (width 0) (type default) (color 0 0 0 0))
   )
-  (wire (pts (xy 68.58 102.87) (xy 76.2 102.87))
+  (wire (pts (xy 76.2 97.79) (xy 68.58 97.79))
+    (stroke (width 0) (type default) (color 0 0 0 0))
+  )
+  (wire (pts (xy 68.58 107.95) (xy 76.2 107.95))
     (stroke (width 0) (type default) (color 0 0 0 0))
   )
@@
     (stroke (width 0) (type default) (color 0 0 0 0))
   )
-  (wire (pts (xy 68.58 100.33) (xy 76.2 100.33))
+  (wire (pts (xy 68.58 105.41) (xy 76.2 105.41))
     (stroke (width 0) (type default) (color 0 0 0 0))
   )
@@
     (stroke (width 0) (type default) (color 0 0 0 0))
   )
+  (wire (pts (xy 278.13 50.8) (xy 267.97 50.8))
+    (stroke (width 0) (type default) (color 0 0 0 0))
+  )
   (wire (pts (xy 129.54 34.29) (xy 129.54 25.4))
     (stroke (width 0) (type default) (color 0 0 0 0))
@@
     (stroke (width 0) (type default) (color 0 0 0 0))
   )
+  (wire (pts (xy 278.13 43.18) (xy 267.97 43.18))
+    (stroke (width 0) (type default) (color 0 0 0 0))
+  )
   (wire (pts (xy 154.94 34.29) (xy 154.94 25.4))
     (stroke (width 0) (type default) (color 0 0 0 0))
@@
     (stroke (width 0) (type default) (color 0 0 0 0))
   )
+  (wire (pts (xy 278.13 35.56) (xy 267.97 35.56))
+    (stroke (width 0) (type default) (color 0 0 0 0))
+  )
   (wire (pts (xy 64.77 54.61) (xy 76.2 54.61))
     (stroke (width 0) (type default) (color 0 0 0 0))
@@
     (stroke (width 0) (type default) (color 0 0 0 0))
   )
+  (wire (pts (xy 278.13 57.15) (xy 267.97 57.15))
+    (stroke (width 0) (type default) (color 0 0 0 0))
+  )
   (bus (pts (xy 142.24 22.86) (xy 144.78 22.86))
     (stroke (width 0) (type default) (color 0 0 0 0))
@@
     (stroke (width 0) (type default) (color 0 0 0 0))
   )
+  (wire (pts (xy 278.13 40.64) (xy 267.97 40.64))
+    (stroke (width 0) (type default) (color 0 0 0 0))
+  )
   (wire (pts (xy 64.77 77.47) (xy 76.2 77.47))
     (stroke (width 0) (type default) (color 0 0 0 0))
@@
   )
   (wire (pts (xy 147.32 34.29) (xy 147.32 25.4))
+    (stroke (width 0) (type default) (color 0 0 0 0))
+  )
+  (wire (pts (xy 278.13 48.26) (xy 267.97 48.26))
     (stroke (width 0) (type default) (color 0 0 0 0))
   )
@@
     (effects (font (size 3 3)) (justify left bottom))
   )
+  (text "PIN78CON53CASSETE" (at 212.09 109.22 0)
+    (effects (font (size 1.27 1.27)) (justify left bottom))
+  )
   (text "8-20MHz square wave clk" (at 207.01 52.07 0)
     (effects (font (size 1.27 1.27)) (justify left bottom))
@@
     (effects (font (size 1.27 1.27)) (justify left bottom))
   )
+  (label "GFXC_D6" (at 248.92 39.37 0)
+    (effects (font (size 1.27 1.27)) (justify left bottom))
+  )
+  (label "GFXD_D1" (at 268.1263 50.8 0)
+    (effects (font (size 1.27 1.27)) (justify left bottom))
+  )
   (label "MAIN_D6" (at 134.62 25.4 270)
     (effects (font (size 1.27 1.27)) (justify right bottom))
@@
     (effects (font (size 1.27 1.27)) (justify left bottom))
   )
+  (label "GFXD_D5" (at 267.97 40.64 0)
+    (effects (font (size 1.27 1.27)) (justify left bottom))
+  )
   (label "MAIN_A3" (at 64.77 52.07 0)
     (effects (font (size 1.27 1.27)) (justify left bottom))
   )
+  (label "GFXC_D1" (at 248.92 52.07 0)
+    (effects (font (size 1.27 1.27)) (justify left bottom))
+  )
   (label "MAIN_D19" (at 167.64 34.29 90)
     (effects (font (size 1.27 1.27)) (justify left bottom))
   )
+  (label "GFXD_D2" (at 267.97 48.26 0)
+    (effects (font (size 1.27 1.27)) (justify left bottom))
+  )
   (label "MAIN_A5" (at 64.77 57.15 0)
     (effects (font (size 1.27 1.27)) (justify left bottom))
@@
     (effects (font (size 1.27 1.27)) (justify right bottom))
   )
+  (label "GFXC_D0" (at 248.92 54.61 0)
+    (effects (font (size 1.27 1.27)) (justify left bottom))
+  )
+  (label "GFXD_D4" (at 267.97 43.18 0)
+    (effects (font (size 1.27 1.27)) (justify left bottom))
+  )
+  (label "GFXC_D2" (at 248.92 49.53 0)
+    (effects (font (size 1.27 1.27)) (justify left bottom))
+  )
   (label "MAIN_A8" (at 64.77 64.77 0)
     (effects (font (size 1.27 1.27)) (justify left bottom))
@@
     (effects (font (size 1.27 1.27)) (justify left bottom))
   )
+  (label "GFXD_D0" (at 267.97 57.15 0)
+    (effects (font (size 1.27 1.27)) (justify left bottom))
+  )
   (label "MAIN_D20" (at 170.18 34.29 90)
     (effects (font (size 1.27 1.27)) (justify left bottom))
@@
     (effects (font (size 1.27 1.27)) (justify right bottom))
   )
+  (label "GFXC_D4" (at 248.92 44.45 0)
+    (effects (font (size 1.27 1.27)) (justify left bottom))
+  )
   (label "MAIN_A6" (at 64.77 59.69 0)
     (effects (font (size 1.27 1.27)) (justify left bottom))
@@
     (effects (font (size 1.27 1.27)) (justify left bottom))
   )
+  (label "GFXC_D7" (at 248.92 36.83 0)
+    (effects (font (size 1.27 1.27)) (justify left bottom))
+  )
   (label "MAIN_A13" (at 64.77 77.47 0)
     (effects (font (size 1.27 1.27)) (justify left bottom))
@@
     (effects (font (size 1.27 1.27)) (justify right bottom))
   )
+  (label "GFXC_D3" (at 248.92 46.99 0)
+    (effects (font (size 1.27 1.27)) (justify left bottom))
+  )
+  (label "GFXD_D6" (at 267.97 38.1 0)
+    (effects (font (size 1.27 1.27)) (justify left bottom))
+  )
+  (label "GFXD_D7" (at 267.97 35.56 0)
+    (effects (font (size 1.27 1.27)) (justify left bottom))
+  )
   (label "MAIN_D17" (at 162.56 34.29 90)
     (effects (font (size 1.27 1.27)) (justify left bottom))
@@
     (effects (font (size 1.27 1.27)) (justify right bottom))
   )
+  (label "GFXC_D5" (at 248.92 41.91 0)
+    (effects (font (size 1.27 1.27)) (justify left bottom))
+  )
   (label "MAIN_A12" (at 64.77 74.93 0)
     (effects (font (size 1.27 1.27)) (justify left bottom))
@@
     (effects (font (size 1.27 1.27)) (justify left bottom))
   )
+  (label "GFXD_D3" (at 267.97 45.72 0)
+    (effects (font (size 1.27 1.27)) (justify left bottom))
+  )
   (label "MAIN_D3" (at 127 25.4 270)
     (effects (font (size 1.27 1.27)) (justify right bottom))
   )
-  (hierarchical_label "GLL2IO0" (shape input) (at 68.58 97.79 180)
+  (hierarchical_label "GLL_DRIVER1" (shape input) (at 68.58 100.33 180)
     (effects (font (size 1.27 1.27)) (justify right))
   )
-  (hierarchical_label "RESET?" (shape input) (at 68.58 102.87 180)
+  (hierarchical_label "RESET?" (shape input) (at 68.58 107.95 180)
     (effects (font (size 1.27 1.27)) (justify right))
   )
@@
     (effects (font (size 1.27 1.27)) (justify right))
   )
+  (hierarchical_label "GLL_DRIVER2" (shape input) (at 68.58 102.87 180)
+    (effects (font (size 1.27 1.27)) (justify right))
+  )
+  (hierarchical_label "GLL_DRIVER0" (shape input) (at 68.58 97.79 180)
+    (effects (font (size 1.27 1.27)) (justify right))
+  )
   (hierarchical_label "CLK_GLL1" (shape output) (at 195.58 50.8 0)
     (effects (font (size 1.27 1.27)) (justify left))
   )
-  (hierarchical_label "GLL2IO1" (shape input) (at 68.58 100.33 180)
+  (hierarchical_label "GLL_DRIVER3" (shape input) (at 68.58 105.41 180)
     (effects (font (size 1.27 1.27)) (justify right))
   )

Commit message: wip_gll_cassette
Parts:
- added R88, R90: 101Ω, symbol Device:R_US
- added R93: 472Ω, symbol Device:R_US
Connections:
- net GFXC_D0: now also J11.66 (GFXC_D0)
- net GFXC_D1: now also J11.65 (GFXC_D1)
- net GFXC_D2: now also J11.64 (GFXC_D2)
- net GFXC_D3: now also J11.63 (GFXC_D3)
- net GFXC_D4: now also J11.62 (GFXC_D4)
- net GFXC_D5: now also J11.61 (GFXC_D5)
- net GFXC_D6: now also J11.60 (GFXC_D6)
- net GFXC_D7: now also J11.59 (GFXC_D7)
- net GFXD_D0: now also J11.75 (GFXD_D0)
- net GFXD_D1: now also J11.74 (GFXD_D1)
- net GFXD_D2: now also J11.73 (GFXD_D2)
- net GFXD_D3: now also J11.72 (GFXD_D3)
- net GFXD_D4: now also J11.71 (GFXD_D4)
- net GFXD_D5: now also J11.70 (GFXD_D5)
- net GFXD_D6: now also J11.69 (GFXD_D6)
- net GFXD_D7: now also J11.68 (GFXD_D7)
- net GLL_DRIVER0: now also J11.138 (GLL_DRIVER2); no longer J11.122 (GLL_DRIVER0)
- net GLL_DRIVER1: now also J11.139 (GLL_DRIVER3); no longer J11.123 (GLL_DRIVER1)
- net GLL_DRIVER2: no longer J11.138 (GLL_DRIVER2)
- net GLL_DRIVER3: no longer J11.139 (GLL_DRIVER3)
- net MAIN_A0: now also J11.35 (MAIN_A0); no longer J11.31 (MAIN_A0)
- net MAIN_A1: now also J11.36 (MAIN_A1); no longer J11.30 (MAIN_A1)
- net MAIN_A10: now also J11.8 (MAIN_A10); no longer J11.38 (MAIN_A10)
- net MAIN_A11: now also J11.29 (MAIN_A11); no longer J11.37 (MAIN_A11)
- net MAIN_A12: now also J11.30 (MAIN_A12); no longer J11.36 (MAIN_A12)
- net MAIN_A13: now also J11.32 (MAIN_A13); no longer J11.35 (MAIN_A13)
- net MAIN_A2: now also J11.37 (MAIN_A2); no longer J11.29 (MAIN_A2)
- net MAIN_A3: now also J11.38 (MAIN_A3); no longer J11.8 (MAIN_A3)
- net MAIN_A4: now also J11.39 (MAIN_A4); no longer J11.7 (MAIN_A4)
- net MAIN_A5: now also J11.41 (MAIN_A5); no longer J11.6 (MAIN_A5)
- net MAIN_A6: now also J11.42 (MAIN_A6); no longer J11.43 (MAIN_A6)
- net MAIN_A7: now also J11.43 (MAIN_A7); no longer J11.42 (MAIN_A7)
- net MAIN_A8: now also J11.6 (MAIN_A8); no longer J11.41 (MAIN_A8)
- net MAIN_A9: now also J11.7 (MAIN_A9); no longer J11.39 (MAIN_A9)
- net VCC: now also R93.1
- net VSS: now also J11.67 (VSS)
- net GLL_A17: now reaches J11.100 (GLL_A17)
- net GLL_A18: now reaches J11.101 (GLL_A18)
- net GLL_A19: now reaches J11.102 (GLL_A19)
- net GLL_A20: now reaches J11.103 (GLL_A20)
- net GLL_D0: now reaches J11.104 (GLL_D0)
- net GLL_D1: now reaches J11.105 (GLL_D1)
- net GLL_D2: now reaches J11.106 (GLL_D2)
- net GLL2CCU2: now reaches J11.108 (GLL2CCU2)
- net at J11.109 (GLL2CCU3): now also R88.1
- net GLL_D3: now reaches J11.111 (GLL_D3)
- net GLL_D4: now reaches J11.112 (GLL_D4)
- net GLL_D5: now reaches J11.113 (GLL_D5)
- net GLL_D6: now reaches J11.114 (GLL_D6)
- net GLL_D7: now reaches J11.128 (GLL_D7)
- net GLL2CCU4: now reaches J11.129 (GLL2CCU4)
- net GLL2CCU5: now reaches J11.134 (GLL2CCU5)
- net at J11.135 (PULL_UP): now also J11.140 (PULL_UP), R93.2
- net GLL2CCU1: now reaches J11.56 (GLL2CCU1)
- net GLL2RC0: now reaches J11.78 (GLL2RC0)
- net GLL2CCU0: now reaches J11.79 (GLL2CCU0)
- net GLL_A0: now reaches J11.80 (GLL_A0)
- net GLL_A1: now reaches J11.81 (GLL_A1)
- net GLL_A2: now reaches J11.82 (GLL_A2)
- net GLL_A3: now reaches J11.83 (GLL_A3)
- net GLL_A4: now reaches J11.84 (GLL_A4)
- net GLL_A5: now reaches J11.85 (GLL_A5)
- net GLL_A6: now reaches J11.86 (GLL_A6)
- net GLL_A7: now reaches J11.87 (GLL_A7)
- net GLL_A8: now reaches J11.88 (GLL_A8)
- net GLL_A9: now reaches J11.89 (GLL_A9)
- net GLL_A10: now reaches J11.92 (GLL_A10)
- net GLL_A11: now reaches J11.93 (GLL_A11)
- net GLL_A12: now reaches J11.94 (GLL_A12)
- net GLL_A13: now reaches J11.95 (GLL_A13)
- net GLL_A14: now reaches J11.96 (GLL_A14)
- net GLL_A15: now reaches J11.97 (GLL_A15)
- net GLL_A16: now reaches J11.98 (GLL_A16)
- net RESET? renamed GLL2IOU0
- new net: R88.2, R90.1
- new net GLL2CCU3: R90.2
- new net GLL_DRIVER4: J11.31 (GLL_DRIVER4)
Other:
- note added: "Data bus and addresses. There is no certainty of the order."
- note removed: "NO OUTPUT OBSERVED PHYSICAL SIGNAL. PENDING TO VERIFY PENDING TO CORRECT PIN LENGTH"
- note removed: "PIN78CON53CASSETE"

Commit message: wip_iou_wd
Parts:
- added F12: 16103FPJ, symbol hitachi:16103FPJ
- added R_US: 68KΩ, symbol Device:R_US
Connections:
- net VCC: now also F12.12 (Vcont), F12.13 (VCC), F12.9 (Vout), R_US.1
- net VSS: now also F12.7 (VSS)
- net ~{CS}_GLL1: now reaches J11.116 (~{CS})
- net ~{WE}_GLL1: now reaches J11.117 (~{WE})
- net ~{RE}_GLL1: now reaches J11.118 (~{RE})
- net ~{MR}_GLL1: now reaches J11.121 (~{MR})
- net DRIVER_GLL2: now reaches J11.122 (GLL_DRIVER2)
- net DRIVER_GLL1: now reaches J11.123 (GLL_DRIVER1)
- net GLL2RC0 renamed ~{RST_WD}
- net ~{RST_WD}: now also F12.17 (~{RES})
- net GLL_DRIVER0 renamed DRIVER_GLL0
- net GLL_DRIVER1 renamed DRIVER_GLL3
- net GLL_DRIVER4 renamed DRIVER_GLL4
- new net: F12.15 (VNMIadj), R_US.2
Other:
- note added: "CUT PIN"
- note added: "Square wave clk"
- note removed: "8-20MHz square wave clk"
- moved on the sheet: R88, R90, R93

Commit message: wip_ccu
Parts:
- added CP166, CP167, CP168, CP169: 1nF, symbol Device:C_Polarized_US
- added R68, R82: 184Ω, symbol Device:R_US
- added R72: 153Ω, symbol Device:R_US
Connections:
- net VSS: now also F12.2 (P-RUN), CP166.2, CP167.2, CP168.2, CP169.2, R68.2, R72.2, R82.2
- net at F12.14 (CRES): now also CP169.1
- net at F12.18 (VSYBYadj): now also R72.1
- net ~{STBY_WD}: now reaches F12.19 (~{STBY})
- net at F12.3 (Rf): now also CP166.1, R68.1
- net at F12.4 (Cf): now also CP167.1
- net at F12.5 (Rr): now also R82.1
- net at F12.6 (Cr): now also CP168.1
- no-connect marks 0 -> 2
Other:
- note added: "NOT MOUNTED"
- note added: "WATCHDOG TIMER"
- moved on the sheet: F12, J11, R88, R90, R93, R_US

Commit message: wip_ccu_gll2_cassette
Parts:
- R68, R82: value 184Ω -> 184
- R72: value 153Ω -> 153
- R88, R90: value 101Ω -> 101
Changed lines of the file:
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@@
     (in_bom yes) (on_board yes)
     (property "Reference" "R90" (id 0) (at 69.85 104.14 90))
-    (property "Value" "101Ω" (id 1) (at 68.58 106.68 90))
+    (property "Value" "101" (id 1) (at 68.58 106.68 90))
     (property "Footprint" "" (id 2) (at 73.406 104.394 90)
       (effects (font (size 1.27 1.27)) hide)
@@
     (in_bom yes) (on_board yes)
     (property "Reference" "R68" (id 0) (at 102.87 171.45 0))
-    (property "Value" "184Ω" (id 1) (at 102.87 173.99 0))
+    (property "Value" "184" (id 1) (at 102.87 173.99 0))
     (property "Footprint" "" (id 2) (at 105.664 172.974 90)
       (effects (font (size 1.27 1.27)) hide)
@@
     (in_bom yes) (on_board yes)
     (property "Reference" "R72" (id 0) (at 59.69 186.69 0))
-    (property "Value" "153Ω" (id 1) (at 59.69 189.23 0))
+    (property "Value" "153" (id 1) (at 59.69 189.23 0))
     (property "Footprint" "" (id 2) (at 63.754 188.214 90)
       (effects (font (size 1.27 1.27)) hide)
@@
     (in_bom yes) (on_board yes)
     (property "Reference" "R82" (id 0) (at 90.17 185.42 0))
-    (property "Value" "184Ω" (id 1) (at 90.17 187.96 0))
+    (property "Value" "184" (id 1) (at 90.17 187.96 0))
     (property "Footprint" "" (id 2) (at 91.694 183.134 90)
       (effects (font (size 1.27 1.27)) hide)
@@
     (in_bom yes) (on_board yes)
     (property "Reference" "R88" (id 0) (at 90.17 104.14 90))
-    (property "Value" "101Ω" (id 1) (at 90.17 106.68 90))
+    (property "Value" "101" (id 1) (at 90.17 106.68 90))
     (property "Footprint" "" (id 2) (at 84.836 104.394 90)
       (effects (font (size 1.27 1.27)) hide)

Commit message: wip_cassette
Connections:
- net ~{RST_WD} renamed ~{RST}_WD
Changed lines of the file:
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@@
     (effects (font (size 1.27 1.27)) (justify left bottom))
   )
-  (label "~{RST_WD}" (at 217.17 57.15 180)
+  (label "~{RST}_WD" (at 217.17 57.15 180)
     (effects (font (size 1.27 1.27)) (justify right bottom))
   )
@@
     (effects (font (size 1.27 1.27)) (justify right))
   )
-  (hierarchical_label "~{RST_WD}" (shape output) (at 64.77 176.53 0)
+  (hierarchical_label "~{RST}_WD" (shape output) (at 64.77 176.53 0)
     (effects (font (size 1.27 1.27)) (justify left))
   )
