File: cores/cps3/sch/ssu.kicad_sch (KiCad schematic)
At the start: 1 part

Commit message: ssu_gll
Parts:
- added U?: HD6417604F28_SH2, symbol arcade:HD6417604F28_SH2
- gave numbers to parts that had none: 1
Connections:
- net SSU14: now reaches G6.1 (D14)
- net VSS: now reaches G6.106 (VSS)
- net VSS: now also G6.11 (VSS), G6.19 (VSS), G6.38 (VSS), G6.43 (VSS), G6.44 (VSS), G6.49 (VSS), G6.69 (VSS), G6.91 (VSS)
- net VCC: now reaches G6.113 (VCC)
- net VCC: now also G6.18 (VCC), G6.4 (VCC), G6.54 (VCC), G6.55 (VCC), G6.70 (VCC), G6.75 (VCC), G6.83 (VCC), G6.90 (VCC)
- net CLK_SSU: now reaches G6.128 (CLK)
- net SSU0: now reaches G6.131 (D0)
- net SSU1: now reaches G6.132 (D1)
- net SSU2: now reaches G6.133 (D2)
- net SSU3: now reaches G6.134 (D3)
- net SSU4: now reaches G6.135 (D4)
- net SSU5: now reaches G6.136 (D5)
- net SSU6: now reaches G6.137 (D6)
- net SSU7: now reaches G6.138 (D7)
- net SSU8: now reaches G6.139 (D8)
- net SSU9: now reaches G6.140 (D9)
- net SSU10: now reaches G6.141 (D10)
- net SSU11: now reaches G6.142 (D11)
- net SSU12: now reaches G6.143 (D12)
- net SSU13: now reaches G6.144 (D13)
- net SSU15: now reaches G6.2 (D15)
- net SSU_A16: now reaches G6.20 (A16)
- net SSU_A15: now reaches G6.21 (A15)
- net SSU_A14: now reaches G6.22 (A14)
- net SSU_A13: now reaches G6.23 (A13)
- net SSU_A12: now reaches G6.24 (A12)
- net SSU_A11: now reaches G6.25 (A11)
- net SSU_A10: now reaches G6.26 (A10)
- net SSU_A9: now reaches G6.27 (A9)
- net SSU_A8: now reaches G6.28 (A8)
- net SSU_A7: now reaches G6.29 (A7)
- net SSU16: now reaches G6.3 (D16)
- net SSU_A6: now reaches G6.30 (46)
- net SSU_A5: now reaches G6.31 (A5)
- net SSU_A4: now reaches G6.32 (A4)
- net SSU_A3: now reaches G6.33 (A3)
- net SSU_A2: now reaches G6.34 (A2)
- net SSU_A1: now reaches G6.35 (A1)
- net SSU_A0: now reaches G6.36 (A0)

Commit message: update_symbols_capcom
Parts:
- removed U?: HD6417604F28_SH2, symbol arcade:HD6417604F28_SH2
Connections:
- net SSU0 renamed SSU_D0
- net SSU1 renamed SSU_D1
- net SSU10 renamed SSU_D10
- net SSU11 renamed SSU_D11
- net SSU12 renamed SSU_D12
- net SSU13 renamed SSU_D13
- net SSU14 renamed SSU_D14
- net SSU15 renamed SSU_D15
- net SSU16 renamed SSU_D16
- net SSU2 renamed SSU_D2
- net SSU3 renamed SSU_D3
- net SSU4 renamed SSU_D4
- net SSU5 renamed SSU_D5
- net SSU6 renamed SSU_D6
- net SSU7 renamed SSU_D7
- net SSU8 renamed SSU_D8
- net SSU9 renamed SSU_D9

Commit message: uptate_ns
Connections:
- net CBI_D2: now reaches G6.10 (CBI_D2)
- net CBI_D1: now reaches G6.12 (CBI_D1)
- net CBI_D0: now reaches G6.13 (CBI_D0)
- net CBI_D7: now reaches G6.5 (CBI_D7)
- net CBI_D6: now reaches G6.6 (CBI_D6)
- net CBI_D5: now reaches G6.7 (CBI_D5)
- net CBI_D4: now reaches G6.8 (CBI_D4)
- net CBI_D3: now reaches G6.9 (CBI_D3)

Commit message: update6_cps
Connections:
- net SU2IO0: now reaches G6.121 (SSU2IOU0)
- net MAIN_A1: now reaches G6.122 (MAIN_A1)
- net MAIN_A2: now reaches G6.123 (MAIN_A2)
- net CBI_D0 renamed MAIN_D0
- net CBI_D1 renamed MAIN_D1
- net CBI_D2 renamed MAIN_D2
- net CBI_D3 renamed MAIN_D3
- net CBI_D4 renamed MAIN_D4
- net CBI_D5 renamed MAIN_D5
- net CBI_D6 renamed MAIN_D6
- net CBI_D7 renamed MAIN_D7
- net SSU_D0 renamed MAIN_A3
- net SSU_D1 renamed MAIN_D23
- net SSU_D10 renamed MAIN_D14
- net SSU_D11 renamed MAIN_D13
- net SSU_D12 renamed MAIN_D12
- net SSU_D13 renamed MAIN_D11
- net SSU_D14 renamed MAIN_D10
- net SSU_D15 renamed MAIN_D9
- net SSU_D16 renamed MAIN_D8
- net SSU_D2 renamed MAIN_D22
- net SSU_D3 renamed MAIN_D21
- net SSU_D4 renamed MAIN_D20
- net SSU_D5 renamed MAIN_D19
- net SSU_D6 renamed MAIN_D18
- net SSU_D7 renamed MAIN_D17
- net SSU_D8 renamed MAIN_D16
- net SSU_D9 renamed MAIN_D15

Commit message: clear_sch_hk_cr
Connections:
- net MAIN_A1 renamed GFX_A1
- net MAIN_A2 renamed GFX_A2
- net MAIN_A3 renamed GFX_A3
Changed lines of the file:
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@@
     (effects (font (size 1.27 1.27)) (justify left bottom))
   )
-  (label "MAIN_A1" (at 71.12 109.22 0)
+  (label "GFX_A1" (at 71.12 109.22 0)
     (effects (font (size 1.27 1.27)) (justify left bottom))
   )
@@
     (effects (font (size 1.27 1.27)) (justify left bottom))
   )
-  (label "MAIN_A2" (at 71.12 111.76 0)
+  (label "GFX_A2" (at 71.12 111.76 0)
     (effects (font (size 1.27 1.27)) (justify left bottom))
   )
@@
     (effects (font (size 1.27 1.27)) (justify left bottom))
   )
-  (label "MAIN_A3" (at 71.12 114.3 0)
+  (label "GFX_A3" (at 71.12 114.3 0)
     (effects (font (size 1.27 1.27)) (justify left bottom))
   )

Commit message: update7
Connections:
- net GFX_A1 renamed MAIN_A1
- net GFX_A2 renamed MAIN_A2
- net GFX_A3 renamed MAIN_A3
Other:
- note added: "NO OUTPUT OBSERVED PHYSICAL SIGNAL. PENDING TO VERIFY PENDING TO CORRECT PIN LENGTH"
- moved on the sheet: G6

Commit message: wip_cps3_vdac
Connections:
- net PPU2SSU0: now reaches G6.16 (PPU2SSU0)

Commit message: wip_ssu_cbi_gll
Parts:
- added R85: 472Ω, symbol Device:R_US
Connections:
- net PPU2SSU0: now also G6.17 (PPU2SSU); no longer G6.16 (PPU2SSU0)
- net VCC: now also G6.100 (VCC), G6.127 (VCC), G6.129 (VCC), G6.130 (VCC), G6.60 (VCC), G6.91 (VCC), G6.95 (VCC), R85.2
- net VD_A0: now also G6.59 (RAMVD_A0)
- net VD_A1: now also G6.58 (RAMVD_A1)
- net VD_A10: now also G6.46 (RAMVD_A10)
- net VD_A11: now also G6.45 (RAMVD_A11)
- net VD_A12: now also G6.42 (RAMVD_A12)
- net VD_A13: now also G6.41 (RAMVD_A13)
- net VD_A14: now also G6.40 (RAMVD_A14)
- net VD_A15: now also G6.37 (RAMVD_A16)
- net VD_A16: now also G6.39 (RAMVD_A15)
- net VD_A2: now also G6.57 (RAMVD_A2)
- net VD_A3: now also G6.56 (RAMVD_A3)
- net VD_A4: now also G6.53 (RAMVD_A4)
- net VD_A5: now also G6.52 (RAMVD_A5)
- net VD_A6: now also G6.51 (RAMVD_A6)
- net VD_A7: now also G6.50 (RAMVD_A7)
- net VD_A8: now also G6.48 (RAMVD_A8)
- net VD_A9: now also G6.47 (RAMVD_A9)
- net VSS: now also G6.101 (VSS), G6.112 (VSS), G6.126 (VSS); no longer G6.91 (VSS)
- net at G6.14 (PULL_UP): now also R85.1
- net SYNCB: now reaches G6.15 (SYNCB)
- new net SYNCA: G6.16 (SYNCA)
- no-connect marks 0 -> 24
Other:
- note added: "N34125 PIN1"
- note added: "NOT CONNECTED"
- note removed: "NO OUTPUT OBSERVED PHYSICAL SIGNAL. PENDING TO VERIFY PENDING TO CORRECT PIN LENGTH"
