File: cores/cps3/sch/ssu.kicad_sch (KiCad schematic)
At the start: 2 parts

Commit message: wip_gfx_gll
Parts:
- added F9: N341256SJ_20, symbol arcade:N341256SJ_20
Connections:
- net VCC: now also F9.28 (VCC)
- net VSS: now also F9.14 (VSS), F9.20 (~{CE}), F9.22 (~{OE})
- net A5: now reaches G6.102 (A5)
- net A4: now reaches G6.103 (A4)
- net A3: now reaches G6.104 (A3)
- net A2: now reaches G6.105 (A2)
- net A1: now reaches G6.107 (A1)
- net A0: now reaches G6.108 (A0)
- net ~{WE}: now reaches G6.109 (~{WE})
- net ~{WE}: now also F9.27 (~{WE})
- net D7: now reaches G6.110 (D7)
- net D7: now also F9.19 (D7)
- net D6: now reaches G6.111 (D6)
- net D6: now also F9.18 (D6)
- net D4: now reaches G6.114 (D5)
- net D4: now also F9.16 (D4)
- net D5: now reaches G6.115 (D4)
- net D5: now also F9.17 (D5)
- net D3: now reaches G6.116 (D3)
- net D3: now also F9.15 (D3)
- net D2: now reaches G6.117 (D2)
- net D2: now also F9.13 (D2)
- net D1: now reaches G6.118 (D1)
- net D1: now also F9.12 (D1)
- net D0: now reaches G6.119 (D0)
- net D0: now also F9.11 (D0)
- net GLL_DRIVER1: now reaches G6.120 (GLL_DRIVER0)
- net GLL_DRIVER0: now reaches G6.124 (GLL_DRIVER2)
- net A14: now reaches G6.88 (A14)
- net A13: now reaches G6.89 (A13)
- net A12: now reaches G6.92 (A12)
- net A11: now reaches G6.93 (A11)
- net A10: now reaches G6.94 (A10)
- net A9: now reaches G6.96 (A9)
- net A8: now reaches G6.97 (A8)
- net A7: now reaches G6.98 (A7)
- net A6: now reaches G6.99 (A6)
- new net RAM_A0: F9.10 (A0)
- new net RAM_A1: F9.9 (A1)
- new net RAM_A10: F9.21 (A10)
- new net RAM_A11: F9.23 (A11)
- new net RAM_A12: F9.2 (A12)
- new net RAM_A13: F9.26 (A13)
- new net RAM_A14: F9.1 (A14)
- new net RAM_A2: F9.8 (A2)
- new net RAM_A3: F9.7 (A3)
- new net RAM_A4: F9.6 (A4)
- new net RAM_A5: F9.5 (A5)
- new net RAM_A6: F9.4 (A6)
- new net RAM_A7: F9.3 (A7)
- new net RAM_A8: F9.25 (A8)
- new net RAM_A9: F9.24 (A9)
Other:
- note removed: "N34125 PIN1"
- moved on the sheet: R85

Commit message: wip_iou_wd
Connections:
- net GLL_DRIVER0 renamed DRIVER_GLL0
- net GLL_DRIVER1 renamed DRIVER_GLL2
Changed lines of the file:
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@@
     (effects (font (size 1.27 1.27)) (justify left bottom))
   )
-  (label "GLL_DRIVER0" (at 113.03 29.21 270)
+  (label "DRIVER_GLL0" (at 113.03 29.21 270)
     (effects (font (size 1.27 1.27)) (justify right bottom))
   )
@@
     (effects (font (size 1.27 1.27)) (justify right bottom))
   )
-  (label "GLL_DRIVER1" (at 110.49 29.21 270)
+  (label "DRIVER_GLL2" (at 110.49 29.21 270)
     (effects (font (size 1.27 1.27)) (justify right bottom))
   )
@@
     (effects (font (size 1.27 1.27)) (justify right))
   )
-  (hierarchical_label "GLL_DRIVER[1..0]" (shape input) (at 101.6 26.67 180)
+  (hierarchical_label "DRIVER_GLL[2..0]" (shape input) (at 101.6 26.67 180)
     (effects (font (size 1.27 1.27)) (justify right))
   )

Commit message: wip_ccu
Connections:
- no-connect marks 24 -> 0
Other:
- note removed: "NOT CONNECTED"
Changed lines of the file:
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@@
   (junction (at 87.63 45.72) (diameter 0) (color 0 0 0 0)
   )
-  (no_connect (at 125.73 160.02))
-  (no_connect (at 138.43 160.02))
-  (no_connect (at 120.65 160.02))
-  (no_connect (at 166.37 139.7))
-  (no_connect (at 133.35 160.02))
-  (no_connect (at 153.67 160.02))
-  (no_connect (at 166.37 144.78))
-  (no_connect (at 166.37 142.24))
-  (no_connect (at 130.81 160.02))
-  (no_connect (at 156.21 160.02))
-  (no_connect (at 166.37 137.16))
-  (no_connect (at 166.37 149.86))
-  (no_connect (at 148.59 160.02))
-  (no_connect (at 151.13 160.02))
-  (no_connect (at 140.97 160.02))
-  (no_connect (at 118.11 160.02))
-  (no_connect (at 146.05 160.02))
-  (no_connect (at 166.37 134.62))
-  (no_connect (at 135.89 160.02))
-  (no_connect (at 143.51 160.02))
-  (no_connect (at 166.37 147.32))
-  (no_connect (at 123.19 160.02))
-  (no_connect (at 166.37 132.08))
-  (no_connect (at 128.27 160.02))
   (bus_entry (at 148.59 38.1) (size 2.54 -2.54)
     (stroke (width 0) (type default) (color 0 0 0 0))
@@
     (stroke (width 0) (type default) (color 0 0 0 0))
   )
-  (polyline (pts (xy 118.11 160.02) (xy 118.11 162.56))
-    (stroke (width 0) (type default) (color 0 0 0 0))
-  )
   (wire (pts (xy 184.15 48.26) (xy 195.58 48.26))
     (stroke (width 0) (type default) (color 0 0 0 0))
@@
     (stroke (width 0) (type default) (color 0 0 0 0))
   )
-  (polyline (pts (xy 168.91 162.56) (xy 168.91 132.08))
-    (stroke (width 0) (type default) (color 0 0 0 0))
-  )
   (bus (pts (xy 143.51 35.56) (xy 146.05 35.56))
     (stroke (width 0) (type default) (color 0 0 0 0))
@@
     (stroke (width 0) (type default) (color 0 0 0 0))
   )
-  (polyline (pts (xy 118.11 162.56) (xy 168.91 162.56))
-    (stroke (width 0) (type default) (color 0 0 0 0))
-  )
   (wire (pts (xy 45.72 66.04) (xy 59.69 66.04))
     (stroke (width 0) (type default) (color 0 0 0 0))
@@
   )
   (wire (pts (xy 82.55 45.72) (xy 85.09 45.72))
-    (stroke (width 0) (type default) (color 0 0 0 0))
-  )
-  (polyline (pts (xy 166.37 132.08) (xy 168.91 132.08))
     (stroke (width 0) (type default) (color 0 0 0 0))
   )
@@
     )
   )
-  (text "NOT CONNECTED" (at 135.89 166.37 0)
-    (effects (font (size 1.27 1.27)) (justify left bottom))
-  )
   (label "MAIN_D4" (at 45.72 68.58 0)

Commit message: wip_ccu_gll2_cassette
Parts:
- R85: value 472Ω -> 472
Changed lines of the file:
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@@
     (in_bom yes) (on_board yes)
     (property "Reference" "R85" (id 0) (at 205.74 111.76 0))
-    (property "Value" "472Ω" (id 1) (at 205.74 114.3 0))
+    (property "Value" "472" (id 1) (at 205.74 114.3 0))
     (property "Footprint" "" (id 2) (at 202.946 114.046 90)
       (effects (font (size 1.27 1.27)) hide)

Commit message: wip_cassette
Connections:
- net ~{WE} renamed ~{WE}_SSU
Changed lines of the file:
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@@
     (effects (font (size 1.27 1.27)) (justify right bottom))
   )
-  (label "~{WE}" (at 187.96 76.2 0)
+  (label "~{WE}_SSU" (at 187.96 76.2 0)
     (effects (font (size 1.27 1.27)) (justify left bottom))
   )
@@
     (effects (font (size 1.27 1.27)) (justify right bottom))
   )
-  (label "~{WE}" (at 115.57 29.21 270)
-    (effects (font (size 1.27 1.27)) (justify right bottom))
-  )
+  (label "~{WE}_SSU" (at 115.57 29.21 270)
+    (effects (font (size 1.27 1.27)) (justify right bottom))
+  )

Commit message: wip_cassette_sh2
Parts:
- added Q1: ZR, symbol Device:Q_NPN_BCE
- added R13, R23: 47Ω, symbol Device:R_US
- added R29: 100, symbol Device:R_US
- added U1: 74LS08, symbol jt74:74LS08
Connections:
- net SYNCA: now also U1.2
- net SYNCB: now also U1.1
- net VCC: now also Q1.2 (C)
- net VSS: now also R23.1
- new net: Q1.1 (B), R29.2
- new net: Q1.3 (E), R13.2
- new net: R29.1, U1.3
- new net SYNC: R13.1, R23.2
Other:
- moved on the sheet: F9, G6, R85

Commit message: wip_cre_cps3
Connections:
- net MAIN_A1 is gone; now on net MAIN_D14: G6.122 (MAIN_D14)
- net MAIN_A2 is gone; now on net MAIN_D13: G6.123 (MAIN_D13)
- net MAIN_A3 is gone; now on net MAIN_D12: G6.131 (MAIN_D12)
- net RAM_A0 is gone; now on net A0: F9.10 (A0)
- net RAM_A1 is gone; now on net A1: F9.9 (A1)
- net RAM_A10 is gone; now on net A10: F9.21 (A10)
- net RAM_A11 is gone; now on net A11: F9.23 (A11)
- net RAM_A12 is gone; now on net A12: F9.2 (A12)
- net RAM_A13 is gone; now on net A13: F9.26 (A13)
- net RAM_A14 is gone; now on net A14: F9.1 (A14)
- net RAM_A2 is gone; now on net A2: F9.8 (A2)
- net RAM_A3 is gone; now on net A3: F9.7 (A3)
- net RAM_A4 is gone; now on net A4: F9.6 (A4)
- net RAM_A5 is gone; now on net A5: F9.5 (A5)
- net RAM_A6 is gone; now on net A6: F9.4 (A6)
- net RAM_A7 is gone; now on net A7: F9.3 (A7)
- net RAM_A8 is gone; now on net A8: F9.25 (A8)
- net RAM_A9 is gone; now on net A9: F9.24 (A9)
- net MAIN_D12: no longer G6.143 (MAIN_D12)
- net MAIN_D13: no longer G6.142 (MAIN_D13)
- net MAIN_D14: no longer G6.141 (MAIN_D14)
- net MAIN_D10 renamed MAIN_A10
- net MAIN_D11 renamed MAIN_A11
- net MAIN_D15 renamed MAIN_A15
- net MAIN_D16 renamed MAIN_A16
- net MAIN_D17 renamed MAIN_A17
- net MAIN_D18 renamed MAIN_A18
- net MAIN_D19 renamed MAIN_A19
- net MAIN_D20 renamed MAIN_A20
- net MAIN_D21 renamed MAIN_A21
- net MAIN_D22 renamed MAIN_A22
- net MAIN_D23 renamed MAIN_A23
- net MAIN_D8 renamed MAIN_A8
- net MAIN_D9 renamed MAIN_A9
- new net MAIN_A12: G6.143 (MAIN_A12)
- new net MAIN_A13: G6.142 (MAIN_A13)
- new net MAIN_A14: G6.141 (MAIN_A14)
