File: cores/cps3/sch/sound.kicad_sch (KiCad schematic)
At the start: 64 parts, among them J1 AudioJack2, J2 AudioJack2

Commit message: wip_colmix_snd
Other:
- sheet video_dac ports: added A1-2, B1-2, BLUE, GREEN, RED; removed none
Changed lines of the file:
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@@
-    (stroke (width 0) (type default) (color 0 0 0 0))
-  )
-  (polyline (pts (xy 322.58 123.19) (xy 322.58 227.33))
     (stroke (width 0) (type default) (color 0 0 0 0))
   )
@@
     (stroke (width 0) (type default) (color 0 0 0 0))
   )
+  (wire (pts (xy 266.7 257.81) (xy 278.13 257.81))
+    (stroke (width 0) (type default) (color 0 0 0 0))
+  )
   (wire (pts (xy 231.14 67.31) (xy 231.14 77.47))
     (stroke (width 0) (type default) (color 0 0 0 0))
@@
     (stroke (width 0) (type default) (color 0 0 0 0))
   )
-  (polyline (pts (xy 322.58 227.33) (xy 303.53 227.33))
+  (wire (pts (xy 215.9 255.27) (xy 228.6 255.27))
     (stroke (width 0) (type default) (color 0 0 0 0))
   )
@@
     (stroke (width 0) (type default) (color 0 0 0 0))
   )
+  (wire (pts (xy 266.7 262.89) (xy 278.13 262.89))
+    (stroke (width 0) (type default) (color 0 0 0 0))
+  )
   (wire (pts (xy 231.14 134.62) (xy 231.14 140.97))
     (stroke (width 0) (type default) (color 0 0 0 0))
@@
     (stroke (width 0) (type default) (color 0 0 0 0))
   )
-  (polyline (pts (xy 302.26 123.19) (xy 322.58 123.19))
-    (stroke (width 0) (type default) (color 0 0 0 0))
-  )
   (wire (pts (xy 252.73 220.98) (xy 252.73 217.17))
     (stroke (width 0) (type default) (color 0 0 0 0))
@@
     (stroke (width 0) (type default) (color 0 0 0 0))
   )
+  (wire (pts (xy 266.7 255.27) (xy 278.13 255.27))
+    (stroke (width 0) (type default) (color 0 0 0 0))
+  )
   (wire (pts (xy 311.15 59.69) (xy 311.15 62.23))
     (stroke (width 0) (type default) (color 0 0 0 0))
@@
     (stroke (width 0) (type default) (color 0 0 0 0))
   )
-  (polyline (pts (xy 303.53 121.92) (xy 303.53 227.33))
-    (stroke (width 0) (type default) (color 0 0 0 0))
-  )
   (wire (pts (xy 113.03 91.44) (xy 113.03 113.03))
     (stroke (width 0) (type default) (color 0 0 0 0))
@@
   )
   (wire (pts (xy 288.29 104.14) (xy 288.29 107.95))
+    (stroke (width 0) (type default) (color 0 0 0 0))
+  )
+  (wire (pts (xy 266.7 260.35) (xy 278.13 260.35))
     (stroke (width 0) (type default) (color 0 0 0 0))
   )
@@
     (effects (font (size 1.27 1.27)) (justify left bottom))
   )
+  (hierarchical_label "RED" (shape output) (at 278.13 255.27 0)
+    (effects (font (size 1.27 1.27)) (justify left))
+  )
+  (hierarchical_label "BLUE" (shape output) (at 278.13 260.35 0)
+    (effects (font (size 1.27 1.27)) (justify left))
+  )
   (hierarchical_label "IO_SND32" (shape input) (at 31.75 46.99 180)
     (effects (font (size 1.27 1.27)) (justify right))
   )
+  (hierarchical_label "B1-2" (shape output) (at 278.13 262.89 0)
+    (effects (font (size 1.27 1.27)) (justify left))
+  )
   (hierarchical_label "+12V" (shape passive) (at 234.95 109.22 0)
     (effects (font (size 1.27 1.27)) (justify left))
   )
+  (hierarchical_label "A1-2" (shape input) (at 215.9 255.27 180)
+    (effects (font (size 1.27 1.27)) (justify right))
+  )
   (hierarchical_label "SPEAKER(-)" (shape output) (at 337.82 62.23 0)
+    (effects (font (size 1.27 1.27)) (justify left))
+  )
+  (hierarchical_label "GREEN" (shape output) (at 278.13 257.81 0)
     (effects (font (size 1.27 1.27)) (justify left))
   )
@@
       (effects (font (size 1.27 1.27)) (justify left top))
     )
-  )
+    (pin "RED" output (at 266.7 255.27 0)
+      (effects (font (size 1.27 1.27)) (justify right))
+    )
+    (pin "GREEN" output (at 266.7 257.81 0)
+      (effects (font (size 1.27 1.27)) (justify right))
+    )
+    (pin "BLUE" output (at 266.7 260.35 0)
+      (effects (font (size 1.27 1.27)) (justify right))
+    )
+    (pin "B1-2" output (at 266.7 262.89 0)
+      (effects (font (size 1.27 1.27)) (justify right))
+    )
+    (pin "A1-2" input (at 228.6 255.27 180)
+      (effects (font (size 1.27 1.27)) (justify left))
+    )
+  )

Commit message: pal_snd_ppu
Parts:
- added Q8: ZR, symbol Device:Q_NPN_BCE
- added R42: 472Ω, symbol Device:R_US
- added R43: 101Ω, symbol Device:R_US
- added VD3: BAV99, symbol arcade:BAV99
Connections:
- net BX_SND is gone; now on net VSS: D6.13 (BX)
- net VCC: now also R43.2
- net VSS: now also Q8.3 (E), VD3.
- net at C5.1 (VDDA), C5.8 (CLKS2), CP155.1: now also VD3.
- new net: Q8.2 (C), R43.1
- new net: Q8.1 (B), R42.1
- new net: R42.2, VD3.
Other:
- removed sheet video_dac
- note added: "GIRAR"
- moved on the sheet: 6A, 6B, A4A, A4B, A5A, A5B, B3, C143, C144, C5, CP123, CP130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

Commit message: wip_cps3_vdac
Connections:
- net VD3: now reaches 6B.2 (B), CP137.1, CP147.1, R27.1, R28.1
- net VD3: now also C5.1 (VDDA), C5.10 (VDDD), C5.24 (VDDO), C5.8 (CLKS2), CP153.1, CP154.1, CP155.1, VD3.; no longer A4.3 (+)
- net at A4.5 (+), CP132.1, R27.2: now also A4.3 (+)
- net ~{BE}: now reaches D6.1 (~{BE})
- net ~{BE}: now also Q8.2 (C), R43.1
- net BCK: now reaches D6.3 (A1-1)
- net WS: now reaches D6.4 (A1-2)
- net SNDD: now reaches D6.7 (A2-1)
- net SYSCLK: now reaches D6.8 (A2-2)
- net IO_SND31 renamed APP0
- net IO_SND32 renamed APP1
- net IO_SND41 renamed APP2
- no-connect marks 3 -> 9
Other:
- note removed: "GIRAR"
- moved on the sheet: 6A, 6B, A4A, A4B, A5A, A5B, B3, C143, C144, C5, CP123, CP130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
