File: cores/cps3/sch/trans.kicad_sch (KiCad schematic)
At the start: 17 parts, among them Q16 AHR38, Q18 AHR38

Commit message: wip_ccu_gll2_cassette
Parts:
- removed CP118, CP119, CP120, CP121: 1016R, symbol Device:C_Polarized_US
- removed DA3, Q18: AHR38, symbol Device:Q_NPN_BCE
- removed Q16: AHR38, symbol Device:Q_PNP_EBC
- removed Q16: AHR38, symbol Device:Q_PNP_BCE
- removed R100, R101, R102, R103, R104: 330Ω, symbol Device:R_US
- removed R92: 102Ω, symbol Device:R_US
- removed R94, R97: 103Ω, symbol Device:R_US
- removed R96: 302Ω, symbol Device:R_US
Other:
- note removed: "82N39 3.9V 39 N39"
- note removed: "DETECT VOLATGE"
