File: cores/cps3/sch/cbi.kicad_sch (KiCad schematic)
At the start: 1 part, among them K14 Am33C93A

Commit message: update6_cps
Other:
- company: (none) -> JOTEGO
- title: (none) -> CP SYSTEM III
Changed lines of the file:
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@@
 (kicad_sch (version 20211123) (generator eeschema)
   (paper "A4")
+  (title_block
+    (title "CP SYSTEM III")
+    (date "14/10/22")
+    (rev "José Tejada G.")
+    (company "JOTEGO")
+    (comment 1 "E.Triana")
+  )
   (junction (at 137.16 125.73) (diameter 0) (color 0 0 0 0)
   )

Commit message: snd_colmix
Other:
- moved on the sheet: K14

Commit message: wip_cps3_vdac
Parts:
- added CONN6: Conn_02x25_Odd_Even, symbol Connector_Generic:Conn_02x25_Odd_Even
- added R106: 472Ω, symbol Device:R_US
- added RN22, RN24, RN26, RN28: 221Ω, symbol Device:R_Pack04
- added RN23, RN25, RN27, RN29: 331Ω, symbol Device:R_Pack04
Connections:
- net VCC: now also R106.1, RN22.1 (R1.1), RN22.2 (R2.1), RN22.3 (R3.1), RN22.4 (R4.1), RN24.1 (R1.1), RN24.2 (R2.1), RN24.3 (R3.1), RN24.4 (R4.1), RN26.1 (R1.1), RN26.2 (R2.1), RN26.3 (R3.1), RN26.4 (R4.1), RN28.1 (R1.1), RN28.2 (R2.1), RN28.3 (R3.1), RN28.4 (R4.1)
- net VSS: now also RN23.5 (R4.2), RN23.6 (R3.2), RN23.7 (R2.2), RN23.8 (R1.2), RN25.5 (R4.2), RN25.6 (R3.2), RN25.7 (R2.2), RN25.8 (R1.2), RN27.5 (R4.2), RN27.6 (R3.2), RN27.7 (R2.2), RN27.8 (R1.2), RN29.5 (R4.2), RN29.6 (R3.2), RN29.7 (R2.2), RN29.8 (R1.2)
- net at K14.10 (~{DACK}): now also K14.9 (~{DRQ}), R106.2
- net I/O: now reaches K14.2 (I/O)
- net I/O: now also CONN6.50 (Pin_50), RN24.8 (R1.2), RN25.1 (R1.1)
- net ~{CS}: now reaches K14.24 (~{CS})
- net ~{WE}: now reaches K14.25 (~{WE})
- net ~{RE}: now reaches K14.26 (~{RE})
- net ~{SDP}: now reaches K14.28 (~{SDP})
- net ~{SDP}: now also RN28.5 (R4.2), RN29.4 (R4.1)
- net ~{SD0}: now reaches K14.29 (~{SD0})
- net ~{SD0}: now also RN28.6 (R3.2), RN29.3 (R3.1)
- net ~{MSG}: now reaches K14.3 (~{MSG})
- net ~{MSG}: now also CONN6.42 (Pin_42), RN22.5 (R4.2), RN23.4 (R4.1)
- net ~{SD1}: now reaches K14.30 (~{SD1})
- net ~{SD1}: now also RN28.7 (R2.2), RN29.2 (R2.1)
- net ~{SD2}: now reaches K14.32 (~{SD2})
- net ~{SD2}: now also RN28.8 (R1.2), RN29.1 (R1.1)
- net ~{SD3}: now reaches K14.33 (~{SD3})
- net ~{SD3}: now also RN26.8 (R1.2), RN27.1 (R1.1)
- net ~{SD4}: now reaches K14.34 (~{SD4})
- net ~{SD4}: now also RN26.7 (R2.2), RN27.2 (R2.1)
- net ~{SD5}: now reaches K14.35 (~{SD5})
- net ~{SD5}: now also RN26.6 (R3.2), RN27.3 (R3.1)
- net ~{SD6}: now reaches K14.37 (~{SD6})
- net ~{SD6}: now also RN26.5 (R4.2), RN27.4 (R4.1)
- net ~{MR}: now reaches K14.40 (~{MR})
- net ~{ATN}: now reaches K14.41 (~{ATN})
- net ~{ATN}: now also RN24.5 (R4.2), RN25.4 (R4.1)
- net ~{ACK}: now reaches K14.42 (~{ACK})
- net ~{ACK}: now also RN24.6 (R3.2), RN25.3 (R3.1)
- net ~{REQ}: now reaches K14.43 (~{REQ})
- net ~{REQ}: now also RN24.7 (R2.2), RN25.2 (R2.1)
- net ~{C}/D: now reaches K14.5 (~{C}/D)
- net ~{C}/D: now also CONN6.46 (Pin_46), RN22.6 (R3.2), RN23.3 (R3.1)
- net ~{BSY}: now reaches K14.6 (~{BSY})
- net ~{BSY}: now also CONN6.36 (Pin_36), RN22.7 (R2.2), RN23.2 (R2.1)
- net ~{SEL}: now reaches K14.7 (~{SEL})
- net ~{SEL}: now also CONN6.44 (Pin_44), RN22.8 (R1.2), RN23.1 (R1.1)
- no-connect marks 0 -> 3
Other:
- moved on the sheet: K14

Commit message: wip_ssu_cbi_gll
Parts:
- removed CONN6: Conn_02x25_Odd_Even, symbol Connector_Generic:Conn_02x25_Odd_Even
- added R105: 330Ω, symbol Device:R_US
Connections:
- net PPU_A0: now reaches K14.21 (A0)
- net ~{SD7}: now reaches K14.38 (~{SD7})
- net CBI_CLK: no longer names the net of K14.8 (CLK)
- net CBI_CLK: now also R105.2
- net CBI_D0 renamed MAIN_D0
- net CBI_D1 renamed MAIN_D1
- net CBI_D2 renamed MAIN_D2
- net CBI_D3 renamed MAIN_D3
- net CBI_D4 renamed MAIN_D4
- net CBI_D5 renamed MAIN_D5
- net CBI_D6 renamed MAIN_D6
- net CBI_D7 renamed MAIN_D7
- net ~{CS} renamed ~{CS}_GLL1
- net ~{MR} renamed ~{MR}_GLL1
- net ~{RE} renamed ~{RE}_GLL1
- net ~{WE} renamed ~{WE}_GLL1
- new net CLK_GLL1: R105.1
- no-connect marks 3 -> 5
Other:
- note added: "Processor Data Bus"
- note added: "Small Computer System Interface Data Bus"
- note removed: "8-20MHz square wave clk"
- moved on the sheet: K14, R106, RN22, RN23, RN24, RN25, RN26, RN27, RN28, RN29

Commit message: wip_ccu
Parts:
- added R107: 221Ω, symbol Device:R_US
- added R108: 301Ω, symbol Device:R_US
Connections:
- net VSS: now also R107.1, R108.1
- net ~{SD7}: now also R107.2, R108.2
Changed lines of the file:
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@@
   (junction (at 38.1 76.2) (diameter 0) (color 0 0 0 0)
   )
+  (junction (at 137.16 88.9) (diameter 0) (color 0 0 0 0)
+  )
   (junction (at 38.1 68.58) (diameter 0) (color 0 0 0 0)
   )
   (junction (at 78.74 63.5) (diameter 0) (color 0 0 0 0)
   )
+  (junction (at 140.97 85.09) (diameter 0) (color 0 0 0 0)
+  )
   (junction (at 78.74 48.26) (diameter 0) (color 0 0 0 0)
   )
   (junction (at 38.1 66.04) (diameter 0) (color 0 0 0 0)
+  )
+  (junction (at 153.67 69.85) (diameter 0) (color 0 0 0 0)
   )
   (junction (at 78.74 83.82) (diameter 0) (color 0 0 0 0)
@@
     (stroke (width 0) (type default) (color 0 0 0 0))
   )
+  (wire (pts (xy 153.67 69.85) (xy 160.02 69.85))
+    (stroke (width 0) (type default) (color 0 0 0 0))
+  )
   (bus (pts (xy 162.56 31.75) (xy 162.56 34.29))
     (stroke (width 0) (type default) (color 0 0 0 0))
@@
     (stroke (width 0) (type default) (color 0 0 0 0))
   )
+  (wire (pts (xy 153.67 82.55) (xy 153.67 85.09))
+    (stroke (width 0) (type default) (color 0 0 0 0))
+  )
   (wire (pts (xy 48.26 60.96) (xy 68.58 60.96))
     (stroke (width 0) (type default) (color 0 0 0 0))
@@
     (stroke (width 0) (type default) (color 0 0 0 0))
   )
-  (wire (pts (xy 151.13 69.85) (xy 160.02 69.85))
+  (wire (pts (xy 151.13 69.85) (xy 153.67 69.85))
     (stroke (width 0) (type default) (color 0 0 0 0))
   )
@@
     (stroke (width 0) (type default) (color 0 0 0 0))
   )
-  (wire (pts (xy 137.16 85.09) (xy 137.16 87.63))
+  (wire (pts (xy 137.16 85.09) (xy 137.16 88.9))
     (stroke (width 0) (type default) (color 0 0 0 0))
   )
@@
     (stroke (width 0) (type default) (color 0 0 0 0))
   )
+  (wire (pts (xy 153.67 69.85) (xy 153.67 74.93))
+    (stroke (width 0) (type default) (color 0 0 0 0))
+  )
   (wire (pts (xy 78.74 83.82) (xy 83.82 83.82))
     (stroke (width 0) (type default) (color 0 0 0 0))
@@
     (stroke (width 0) (type default) (color 0 0 0 0))
   )
+  (wire (pts (xy 137.16 88.9) (xy 137.16 90.17))
+    (stroke (width 0) (type default) (color 0 0 0 0))
+  )
   (wire (pts (xy 115.57 54.61) (xy 123.19 54.61))
     (stroke (width 0) (type default) (color 0 0 0 0))
@@
     (stroke (width 0) (type default) (color 0 0 0 0))
   )
+  (wire (pts (xy 160.02 69.85) (xy 160.02 81.28))
+    (stroke (width 0) (type default) (color 0 0 0 0))
+  )
   (wire (pts (xy 115.57 77.47) (xy 123.19 77.47))
     (stroke (width 0) (type default) (color 0 0 0 0))
@@
     (stroke (width 0) (type default) (color 0 0 0 0))
   )
+  (wire (pts (xy 140.97 85.09) (xy 153.67 85.09))
+    (stroke (width 0) (type default) (color 0 0 0 0))
+  )
   (wire (pts (xy 151.13 36.83) (xy 160.02 36.83))
     (stroke (width 0) (type default) (color 0 0 0 0))
@@
   )
   (bus (pts (xy 162.56 62.23) (xy 162.56 59.69))
+    (stroke (width 0) (type default) (color 0 0 0 0))
+  )
+  (wire (pts (xy 137.16 88.9) (xy 160.02 88.9))
     (stroke (width 0) (type default) (color 0 0 0 0))
   )
@@
     (pin "8")
   )
+  (symbol (lib_id "Device:R_US") (at 153.67 78.74 180) (unit 1)
+    (in_bom yes) (on_board yes)
+    (property "Reference" "R108" (id 0) (at 157.48 78.74 0))
+    (property "Value" "301Ω" (id 1) (at 157.48 81.28 0))
+    (property "Footprint" "" (id 2) (at 152.654 78.486 90)
+      (effects (font (size 1.27 1.27)) hide)
+    )
+    (property "Datasheet" "~" (id 3) (at 153.67 78.74 0)
+      (effects (font (size 1.27 1.27)) hide)
+    )
+    (pin "1")
+    (pin "2")
+  )
   (symbol (lib_id "arcade:Am33C93A") (at 137.16 55.88 0) (unit 1)
     (in_bom yes) (on_board yes)
@@
     (pin "8")
   )
+  (symbol (lib_id "Device:R_US") (at 160.02 85.09 180) (unit 1)
+    (in_bom yes) (on_board yes)
+    (property "Reference" "R107" (id 0) (at 163.83 85.09 0))
+    (property "Value" "221Ω" (id 1) (at 163.83 87.63 0))
+    (property "Footprint" "" (id 2) (at 159.004 84.836 90)
+      (effects (font (size 1.27 1.27)) hide)
+    )
+    (property "Datasheet" "~" (id 3) (at 160.02 85.09 0)
+      (effects (font (size 1.27 1.27)) hide)
+    )
+    (pin "1")
+    (pin "2")
+  )
   (symbol (lib_id "Device:R_Pack04") (at 73.66 50.8 270) (unit 1)
     (in_bom yes) (on_board yes)
@@
     (pin "8")
   )
-  (symbol (lib_id "power:VSS") (at 137.16 87.63 180) (unit 1)
-    (in_bom yes) (on_board yes)
-    (property "Reference" "#PWR?" (id 0) (at 137.16 83.82 0)
-      (effects (font (size 1.27 1.27)) hide)
-    )
-    (property "Value" "VSS" (id 1) (at 137.16 91.44 0))
-    (property "Footprint" "" (id 2) (at 137.16 87.63 0)
-      (effects (font (size 1.27 1.27)) hide)
-    )
-    (property "Datasheet" "" (id 3) (at 137.16 87.63 0)
-      (effects (font (size 1.27 1.27)) hide)
-    )
+  (symbol (lib_id "power:VSS") (at 137.16 90.17 180) (unit 1)
+    (in_bom yes) (on_board yes)
+    (property "Reference" "#PWR?" (id 0) (at 137.16 86.36 0)
+      (effects (font (size 1.27 1.27)) hide)
+    )
+    (property "Value" "VSS" (id 1) (at 137.16 93.98 0))
+    (property "Footprint" "" (id 2) (at 137.16 90.17 0)
+      (effects (font (size 1.27 1.27)) hide)
+    )
+    (property "Datasheet" "" (id 3) (at 137.16 90.17 0)
+      (effects (font (size 1.27 1.27)) hide)
+    )

Commit message: wip_ccu_gll2_cassette
Parts:
- R105: value 330Ω -> 330
- R106: value 472Ω -> 472
- R107, RN22, RN24, RN26, RN28: value 221Ω -> 221
- R108: value 301Ω -> 301
- RN23, RN25, RN27, RN29: value 331Ω -> 331
Connections:
- net PPU_A0 renamed PPU2CCU1
Other:
- moved on the sheet: R105
Changed lines of the file:
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@@
     (stroke (width 0) (type default) (color 0 0 0 0))
   )
-  (wire (pts (xy 119.38 36.83) (xy 123.19 36.83))
+  (wire (pts (xy 113.03 36.83) (xy 123.19 36.83))
     (stroke (width 0) (type default) (color 0 0 0 0))
   )
@@
     (stroke (width 0) (type default) (color 0 0 0 0))
   )
-  (wire (pts (xy 115.57 34.29) (xy 123.19 34.29))
+  (wire (pts (xy 100.33 34.29) (xy 123.19 34.29))
     (stroke (width 0) (type default) (color 0 0 0 0))
   )
@@
     (stroke (width 0) (type default) (color 0 0 0 0))
   )
-  (wire (pts (xy 107.95 36.83) (xy 111.76 36.83))
+  (wire (pts (xy 100.33 36.83) (xy 105.41 36.83))
     (stroke (width 0) (type default) (color 0 0 0 0))
   )
@@
     (effects (font (size 1.27 1.27)) (justify right))
   )
-  (hierarchical_label "CLK_GLL1" (shape input) (at 107.95 36.83 180)
-    (effects (font (size 1.27 1.27)) (justify right))
-  )
-  (hierarchical_label "PPU_A0" (shape input) (at 115.57 41.91 180)
+  (hierarchical_label "CLK_GLL1" (shape input) (at 100.33 36.83 180)
+    (effects (font (size 1.27 1.27)) (justify right))
+  )
+  (hierarchical_label "PPU2CCU1" (shape input) (at 115.57 41.91 180)
     (effects (font (size 1.27 1.27)) (justify right))
   )
@@
     (effects (font (size 1.27 1.27)) (justify right))
   )
-  (hierarchical_label "I{slash}O" (shape input) (at 115.57 34.29 180)
+  (hierarchical_label "I{slash}O" (shape input) (at 100.33 34.29 180)
     (effects (font (size 1.27 1.27)) (justify right))
   )
@@
     (effects (font (size 1.27 1.27)) (justify right))
   )
-  (symbol (lib_id "Device:R_US") (at 115.57 36.83 90) (unit 1)
-    (in_bom yes) (on_board yes)
-    (property "Reference" "R105" (id 0) (at 119.38 35.56 90))
-    (property "Value" "330Ω" (id 1) (at 120.65 38.1 90))
-    (property "Footprint" "" (id 2) (at 115.824 35.814 90)
-      (effects (font (size 1.27 1.27)) hide)
-    )
-    (property "Datasheet" "~" (id 3) (at 115.57 36.83 0)
+  (symbol (lib_id "Device:R_US") (at 109.22 36.83 90) (unit 1)
+    (in_bom yes) (on_board yes)
+    (property "Reference" "R105" (id 0) (at 113.03 35.56 90))
+    (property "Value" "330" (id 1) (at 114.3 38.1 90))
+    (property "Footprint" "" (id 2) (at 109.474 35.814 90)
+      (effects (font (size 1.27 1.27)) hide)
+    )
+    (property "Datasheet" "~" (id 3) (at 109.22 36.83 0)
       (effects (font (size 1.27 1.27)) hide)
     )
@@
     (in_bom yes) (on_board yes)
     (property "Reference" "RN29" (id 0) (at 73.66 73.66 90))
-    (property "Value" "331Ω" (id 1) (at 73.66 86.36 90))
+    (property "Value" "331" (id 1) (at 73.66 86.36 90))
     (property "Footprint" "" (id 2) (at 73.66 88.265 90)
       (effects (font (size 1.27 1.27)) hide)
@@
     (in_bom yes) (on_board yes)
     (property "Reference" "RN26" (id 0) (at 43.18 58.42 90))
-    (property "Value" "221Ω" (id 1) (at 43.18 71.12 90))
+    (property "Value" "221" (id 1) (at 43.18 71.12 90))
     (property "Footprint" "" (id 2) (at 43.18 73.025 90)
       (effects (font (size 1.27 1.27)) hide)
@@
     (in_bom yes) (on_board yes)
     (property "Reference" "R108" (id 0) (at 157.48 78.74 0))
-    (property "Value" "301Ω" (id 1) (at 157.48 81.28 0))
+    (property "Value" "301" (id 1) (at 157.48 81.28 0))
     (property "Footprint" "" (id 2) (at 152.654 78.486 90)
       (effects (font (size 1.27 1.27)) hide)
@@
     (in_bom yes) (on_board yes)
     (property "Reference" "RN25" (id 0) (at 73.66 27.94 90))
-    (property "Value" "331Ω" (id 1) (at 73.66 40.64 90))
+    (property "Value" "331" (id 1) (at 73.66 40.64 90))
     (property "Footprint" "" (id 2) (at 73.66 42.545 90)
       (effects (font (size 1.27 1.27)) hide)
@@
     (in_bom yes) (on_board yes)
     (property "Reference" "R107" (id 0) (at 163.83 85.09 0))
-    (property "Value" "221Ω" (id 1) (at 163.83 87.63 0))
+    (property "Value" "221" (id 1) (at 163.83 87.63 0))
     (property "Footprint" "" (id 2) (at 159.004 84.836 90)
       (effects (font (size 1.27 1.27)) hide)
@@
     (in_bom yes) (on_board yes)
     (property "Reference" "RN23" (id 0) (at 73.66 43.18 90))
-    (property "Value" "331Ω" (id 1) (at 73.66 55.88 90))
+    (property "Value" "331" (id 1) (at 73.66 55.88 90))
     (property "Footprint" "" (id 2) (at 73.66 57.785 90)
       (effects (font (size 1.27 1.27)) hide)
@@
     (in_bom yes) (on_board yes)
     (property "Reference" "RN24" (id 0) (at 43.18 27.94 90))
-    (property "Value" "221Ω" (id 1) (at 43.18 40.64 90))
+    (property "Value" "221" (id 1) (at 43.18 40.64 90))
     (property "Footprint" "" (id 2) (at 43.18 42.545 90)
       (effects (font (size 1.27 1.27)) hide)
@@
     (in_bom yes) (on_board yes)
     (property "Reference" "RN28" (id 0) (at 43.18 73.66 90))
-    (property "Value" "221Ω" (id 1) (at 43.18 86.36 90))
+    (property "Value" "221" (id 1) (at 43.18 86.36 90))
     (property "Footprint" "" (id 2) (at 43.18 88.265 90)
       (effects (font (size 1.27 1.27)) hide)
@@
     (in_bom yes) (on_board yes)
     (property "Reference" "RN22" (id 0) (at 43.18 43.18 90))
-    (property "Value" "221Ω" (id 1) (at 43.18 55.88 90))
+    (property "Value" "221" (id 1) (at 43.18 55.88 90))
     (property "Footprint" "" (id 2) (at 43.18 57.785 90)
       (effects (font (size 1.27 1.27)) hide)
@@
     (in_bom yes) (on_board yes)
     (property "Reference" "RN27" (id 0) (at 73.66 58.42 90))
-    (property "Value" "331Ω" (id 1) (at 73.66 71.12 90))
+    (property "Value" "331" (id 1) (at 73.66 71.12 90))
     (property "Footprint" "" (id 2) (at 73.66 73.025 90)
       (effects (font (size 1.27 1.27)) hide)
@@
     (in_bom yes) (on_board yes)
     (property "Reference" "R106" (id 0) (at 99.06 49.53 0))
-    (property "Value" "472Ω" (id 1) (at 99.06 52.07 0))
+    (property "Value" "472" (id 1) (at 99.06 52.07 0))
     (property "Footprint" "" (id 2) (at 103.886 51.054 90)
       (effects (font (size 1.27 1.27)) hide)

Commit message: wip_ccu_cassette
Changed lines of the file:
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@@
     (stroke (width 0) (type default) (color 0 0 0 0))
   )
-  (wire (pts (xy 102.87 41.91) (xy 102.87 46.99))
+  (wire (pts (xy 102.87 44.45) (xy 102.87 46.99))
     (stroke (width 0) (type default) (color 0 0 0 0))
   )
@@
     (effects (font (size 1.27 1.27)) (justify right bottom))
   )
-  (label "VCC" (at 102.87 41.91 0)
-    (effects (font (size 1.27 1.27)) (justify left bottom))
+  (label "VCC" (at 102.87 44.45 180)
+    (effects (font (size 1.27 1.27)) (justify right bottom))
   )
   (label "~{SD4}" (at 160.02 62.23 180)
