File: cores/cps3/sch/gll2.kicad_sch (KiCad schematic)
At the start: 1 part

Commit message: ssu_gll
Changed lines of the file:
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@@
     (comment 1 "E.Triana")
+  )
+  (bus_entry (at 184.15 72.39) (size 2.54 2.54)
+    (stroke (width 0) (type default) (color 0 0 0 0))
+  )
+  (bus_entry (at 184.15 69.85) (size 2.54 2.54)
+    (stroke (width 0) (type default) (color 0 0 0 0))
+  )
+  (bus_entry (at 184.15 67.31) (size 2.54 2.54)
+    (stroke (width 0) (type default) (color 0 0 0 0))
+  )
+  (bus_entry (at 184.15 64.77) (size 2.54 2.54)
+    (stroke (width 0) (type default) (color 0 0 0 0))
+  )
+  (bus_entry (at 184.15 62.23) (size 2.54 2.54)
+    (stroke (width 0) (type default) (color 0 0 0 0))
+  )
+  (bus (pts (xy 186.69 72.39) (xy 186.69 74.93))
+    (stroke (width 0) (type default) (color 0 0 0 0))
+  )
+  (wire (pts (xy 184.15 62.23) (xy 167.64 62.23))
+    (stroke (width 0) (type default) (color 0 0 0 0))
+  )
+  (bus (pts (xy 186.69 69.85) (xy 186.69 72.39))
+    (stroke (width 0) (type default) (color 0 0 0 0))
+  )
+  (wire (pts (xy 184.15 69.85) (xy 167.64 69.85))
+    (stroke (width 0) (type default) (color 0 0 0 0))
+  )
+  (wire (pts (xy 184.15 67.31) (xy 167.64 67.31))
+    (stroke (width 0) (type default) (color 0 0 0 0))
+  )
+  (bus (pts (xy 186.69 67.31) (xy 186.69 69.85))
+    (stroke (width 0) (type default) (color 0 0 0 0))
+  )
+  (bus (pts (xy 186.69 59.69) (xy 186.69 64.77))
+    (stroke (width 0) (type default) (color 0 0 0 0))
+  )
+  (bus (pts (xy 186.69 64.77) (xy 186.69 67.31))
+    (stroke (width 0) (type default) (color 0 0 0 0))
+  )
+  (wire (pts (xy 184.15 64.77) (xy 167.64 64.77))
+    (stroke (width 0) (type default) (color 0 0 0 0))
+  )
+  (wire (pts (xy 184.15 72.39) (xy 167.64 72.39))
+    (stroke (width 0) (type default) (color 0 0 0 0))
   )
   (image (at 274.32 173.99) (scale 0.294008)
@@
     )
   )
+  (label "2GLL0" (at 184.15 62.23 180)
+    (effects (font (size 1.27 1.27)) (justify right bottom))
+  )
+  (label "2GLL5" (at 184.15 74.93 180)
+    (effects (font (size 1.27 1.27)) (justify right bottom))
+  )
+  (label "2GLL3" (at 184.15 69.85 180)
+    (effects (font (size 1.27 1.27)) (justify right bottom))
+  )
+  (label "2GLL4" (at 184.15 72.39 180)
+    (effects (font (size 1.27 1.27)) (justify right bottom))
+  )
+  (label "2GLL1" (at 184.15 64.77 180)
+    (effects (font (size 1.27 1.27)) (justify right bottom))
+  )
+  (label "2GLL2" (at 184.15 67.31 180)
+    (effects (font (size 1.27 1.27)) (justify right bottom))
+  )
   (symbol (lib_id "capcom:DL-3529-GLL2") (at 121.92 87.63 0) (unit 1)

Commit message: iou
Parts:
- gave numbers to parts that had none: 1
Connections:
- net VSS: now reaches G8.1 (VSS)
- net VSS: now also G8.12 (VSS), G8.13 (VSS), G8.18 (VSS), G8.23 (VSS), G8.27 (VSS), G8.33 (VSS), G8.36 (VSS), G8.41 (VSS), G8.46 (VSS), G8.6 (VSS)
- net VCC: now reaches G8.51 (VCC)
- net VCC: now also G8.52 (VCC), G8.58 (VCC), G8.60 (VCC), G8.62 (VCC), G8.65 (VCC), G8.71 (VCC), G8.73 (VCC), G8.76 (VCC)
- net 2GLL_A0: now reaches G8.66 (A0)
- net 2GLL_A1: now reaches G8.67 (A1)
- net 2GLL_A2: now reaches G8.68 (A2)
- net 2GLL_A3: now reaches G8.69 (A3)
- net 2GLL_A4: now reaches G8.70 (A4)
- net 2GLL_A5: now reaches G8.72 (A5)
Changed lines of the file:
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@@
     (comment 1 "E.Triana")
   )
-  (bus_entry (at 184.15 72.39) (size 2.54 2.54)
-    (stroke (width 0) (type default) (color 0 0 0 0))
-  )
-  (bus_entry (at 184.15 69.85) (size 2.54 2.54)
-    (stroke (width 0) (type default) (color 0 0 0 0))
-  )
-  (bus_entry (at 184.15 67.31) (size 2.54 2.54)
-    (stroke (width 0) (type default) (color 0 0 0 0))
-  )
-  (bus_entry (at 184.15 64.77) (size 2.54 2.54)
-    (stroke (width 0) (type default) (color 0 0 0 0))
-  )
-  (bus_entry (at 184.15 62.23) (size 2.54 2.54)
-    (stroke (width 0) (type default) (color 0 0 0 0))
-  )
-  (bus (pts (xy 186.69 72.39) (xy 186.69 74.93))
-    (stroke (width 0) (type default) (color 0 0 0 0))
-  )
-  (wire (pts (xy 184.15 62.23) (xy 167.64 62.23))
-    (stroke (width 0) (type default) (color 0 0 0 0))
-  )
-  (bus (pts (xy 186.69 69.85) (xy 186.69 72.39))
-    (stroke (width 0) (type default) (color 0 0 0 0))
-  )
-  (wire (pts (xy 184.15 69.85) (xy 167.64 69.85))
-    (stroke (width 0) (type default) (color 0 0 0 0))
-  )
-  (wire (pts (xy 184.15 67.31) (xy 167.64 67.31))
-    (stroke (width 0) (type default) (color 0 0 0 0))
-  )
-  (bus (pts (xy 186.69 67.31) (xy 186.69 69.85))
-    (stroke (width 0) (type default) (color 0 0 0 0))
-  )
-  (bus (pts (xy 186.69 59.69) (xy 186.69 64.77))
-    (stroke (width 0) (type default) (color 0 0 0 0))
-  )
-  (bus (pts (xy 186.69 64.77) (xy 186.69 67.31))
-    (stroke (width 0) (type default) (color 0 0 0 0))
-  )
-  (wire (pts (xy 184.15 64.77) (xy 167.64 64.77))
-    (stroke (width 0) (type default) (color 0 0 0 0))
-  )
-  (wire (pts (xy 184.15 72.39) (xy 167.64 72.39))
+  (junction (at 124.46 34.29) (diameter 0) (color 0 0 0 0)
+  )
+  (junction (at 119.38 133.35) (diameter 0) (color 0 0 0 0)
+  )
+  (junction (at 116.84 34.29) (diameter 0) (color 0 0 0 0)
+  )
+  (junction (at 129.54 133.35) (diameter 0) (color 0 0 0 0)
+  )
+  (junction (at 116.84 133.35) (diameter 0) (color 0 0 0 0)
+  )
+  (junction (at 132.08 133.35) (diameter 0) (color 0 0 0 0)
+  )
+  (junction (at 121.92 133.35) (diameter 0) (color 0 0 0 0)
+  )
+  (junction (at 124.46 133.35) (diameter 0) (color 0 0 0 0)
+  )
+  (junction (at 127 34.29) (diameter 0) (color 0 0 0 0)
+  )
+  (junction (at 127 133.35) (diameter 0) (color 0 0 0 0)
+  )
+  (junction (at 121.92 34.29) (diameter 0) (color 0 0 0 0)
+  )
+  (junction (at 111.76 133.35) (diameter 0) (color 0 0 0 0)
+  )
+  (junction (at 119.38 34.29) (diameter 0) (color 0 0 0 0)
+  )
+  (junction (at 129.54 34.29) (diameter 0) (color 0 0 0 0)
+  )
+  (junction (at 114.3 34.29) (diameter 0) (color 0 0 0 0)
+  )
+  (junction (at 114.3 133.35) (diameter 0) (color 0 0 0 0)
+  )
+  (bus_entry (at 80.01 125.73) (size -2.54 2.54)
+    (stroke (width 0) (type default) (color 0 0 0 0))
+  )
+  (bus_entry (at 80.01 123.19) (size -2.54 2.54)
+    (stroke (width 0) (type default) (color 0 0 0 0))
+  )
+  (bus_entry (at 80.01 120.65) (size -2.54 2.54)
+    (stroke (width 0) (type default) (color 0 0 0 0))
+  )
+  (bus_entry (at 80.01 118.11) (size -2.54 2.54)
+    (stroke (width 0) (type default) (color 0 0 0 0))
+  )
+  (bus_entry (at 80.01 115.57) (size -2.54 2.54)
+    (stroke (width 0) (type default) (color 0 0 0 0))
+  )
+  (bus_entry (at 77.47 130.81) (size 2.54 -2.54)
+    (stroke (width 0) (type default) (color 0 0 0 0))
+  )
+  (wire (pts (xy 116.84 34.29) (xy 119.38 34.29))
+    (stroke (width 0) (type default) (color 0 0 0 0))
+  )
+  (wire (pts (xy 80.01 128.27) (xy 96.52 128.27))
+    (stroke (width 0) (type default) (color 0 0 0 0))
+  )
+  (bus (pts (xy 77.47 125.73) (xy 77.47 128.27))
+    (stroke (width 0) (type default) (color 0 0 0 0))
+  )
+  (wire (pts (xy 80.01 115.57) (xy 96.52 115.57))
+    (stroke (width 0) (type default) (color 0 0 0 0))
+  )
+  (wire (pts (xy 114.3 133.35) (xy 116.84 133.35))
+    (stroke (width 0) (type default) (color 0 0 0 0))
+  )
+  (wire (pts (xy 127 34.29) (xy 129.54 34.29))
+    (stroke (width 0) (type default) (color 0 0 0 0))
+  )
+  (bus (pts (xy 77.47 123.19) (xy 77.47 125.73))
+    (stroke (width 0) (type default) (color 0 0 0 0))
+  )
+  (wire (pts (xy 121.92 34.29) (xy 124.46 34.29))
+    (stroke (width 0) (type default) (color 0 0 0 0))
+  )
+  (wire (pts (xy 114.3 34.29) (xy 116.84 34.29))
+    (stroke (width 0) (type default) (color 0 0 0 0))
+  )
+  (wire (pts (xy 121.92 31.75) (xy 121.92 34.29))
+    (stroke (width 0) (type default) (color 0 0 0 0))
+  )
+  (wire (pts (xy 121.92 133.35) (xy 121.92 135.89))
+    (stroke (width 0) (type default) (color 0 0 0 0))
+  )
+  (wire (pts (xy 129.54 133.35) (xy 132.08 133.35))
+    (stroke (width 0) (type default) (color 0 0 0 0))
+  )
+  (wire (pts (xy 80.01 123.19) (xy 96.52 123.19))
+    (stroke (width 0) (type default) (color 0 0 0 0))
+  )
+  (wire (pts (xy 132.08 133.35) (xy 134.62 133.35))
+    (stroke (width 0) (type default) (color 0 0 0 0))
+  )
+  (wire (pts (xy 80.01 120.65) (xy 96.52 120.65))
+    (stroke (width 0) (type default) (color 0 0 0 0))
+  )
+  (wire (pts (xy 119.38 34.29) (xy 121.92 34.29))
+    (stroke (width 0) (type default) (color 0 0 0 0))
+  )
+  (bus (pts (xy 77.47 120.65) (xy 77.47 123.19))
+    (stroke (width 0) (type default) (color 0 0 0 0))
+  )
+  (wire (pts (xy 124.46 34.29) (xy 127 34.29))
+    (stroke (width 0) (type default) (color 0 0 0 0))
+  )
+  (bus (pts (xy 69.85 118.11) (xy 77.47 118.11))
+    (stroke (width 0) (type default) (color 0 0 0 0))
+  )
+  (bus (pts (xy 77.47 118.11) (xy 77.47 120.65))
+    (stroke (width 0) (type default) (color 0 0 0 0))
+  )
+  (wire (pts (xy 124.46 133.35) (xy 127 133.35))
+    (stroke (width 0) (type default) (color 0 0 0 0))
+  )
+  (wire (pts (xy 127 133.35) (xy 129.54 133.35))
+    (stroke (width 0) (type default) (color 0 0 0 0))
+  )
+  (wire (pts (xy 129.54 34.29) (xy 132.08 34.29))
+    (stroke (width 0) (type default) (color 0 0 0 0))
+  )
+  (bus (pts (xy 77.47 128.27) (xy 77.47 130.81))
+    (stroke (width 0) (type default) (color 0 0 0 0))
+  )
+  (wire (pts (xy 109.22 133.35) (xy 111.76 133.35))
+    (stroke (width 0) (type default) (color 0 0 0 0))
+  )
+  (wire (pts (xy 111.76 133.35) (xy 114.3 133.35))
+    (stroke (width 0) (type default) (color 0 0 0 0))
+  )
+  (wire (pts (xy 119.38 133.35) (xy 121.92 133.35))
+    (stroke (width 0) (type default) (color 0 0 0 0))
+  )
+  (wire (pts (xy 80.01 118.11) (xy 96.52 118.11))
+    (stroke (width 0) (type default) (color 0 0 0 0))
+  )
+  (wire (pts (xy 80.01 125.73) (xy 96.52 125.73))
+    (stroke (width 0) (type default) (color 0 0 0 0))
+  )
+  (wire (pts (xy 111.76 34.29) (xy 114.3 34.29))
+    (stroke (width 0) (type default) (color 0 0 0 0))
+  )
+  (wire (pts (xy 116.84 133.35) (xy 119.38 133.35))
+    (stroke (width 0) (type default) (color 0 0 0 0))
+  )
+  (wire (pts (xy 121.92 133.35) (xy 124.46 133.35))
     (stroke (width 0) (type default) (color 0 0 0 0))
   )
@@
     )
   )
-  (label "2GLL0" (at 184.15 62.23 180)
-    (effects (font (size 1.27 1.27)) (justify right bottom))
-  )
-  (label "2GLL5" (at 184.15 74.93 180)
-    (effects (font (size 1.27 1.27)) (justify right bottom))
-  )
-  (label "2GLL3" (at 184.15 69.85 180)
-    (effects (font (size 1.27 1.27)) (justify right bottom))
-  )
-  (label "2GLL4" (at 184.15 72.39 180)
-    (effects (font (size 1.27 1.27)) (justify right bottom))
-  )
-  (label "2GLL1" (at 184.15 64.77 180)
-    (effects (font (size 1.27 1.27)) (justify right bottom))
-  )
-  (label "2GLL2" (at 184.15 67.31 180)
-    (effects (font (size 1.27 1.27)) (justify right bottom))
+  (label "2GLL_A0" (at 80.01 115.57 0)
+    (effects (font (size 1.27 1.27)) (justify left bottom))
+  )
+  (label "2GLL_A5" (at 80.01 128.27 0)
+    (effects (font (size 1.27 1.27)) (justify left bottom))
+  )
+  (label "2GLL_A3" (at 80.01 123.19 0)
+    (effects (font (size 1.27 1.27)) (justify left bottom))
+  )
+  (label "2GLL_A4" (at 80.01 125.73 0)
+    (effects (font (size 1.27 1.27)) (justify left bottom))
+  )
+  (label "2GLL_A1" (at 80.01 118.11 0)
+    (effects (font (size 1.27 1.27)) (justify left bottom))
+  )
+  (label "2GLL_A2" (at 80.01 120.65 0)
+    (effects (font (size 1.27 1.27)) (justify left bottom))
+  )
+  (hierarchical_label "2GLL_A[5..0]" (shape bidirectional) (at 69.85 118.11 180)
+    (effects (font (size 1.27 1.27)) (justify right))
+  )
+  (symbol (lib_id "power:VSS") (at 121.92 135.89 180) (unit 1)
+    (in_bom yes) (on_board yes)
+    (property "Reference" "#PWR?" (id 0) (at 121.92 132.08 0)
+      (effects (font (size 1.27 1.27)) hide)
+    )
+    (property "Value" "VSS" (id 1) (at 121.92 139.7 0))
+    (property "Footprint" "" (id 2) (at 121.92 135.89 0)
+      (effects (font (size 1.27 1.27)) hide)
+    )
+    (property "Datasheet" "" (id 3) (at 121.92 135.89 0)
+      (effects (font (size 1.27 1.27)) hide)
+    )
+    (pin "1")
   )
   (symbol (lib_id "capcom:DL-3529-GLL2") (at 121.92 87.63 0) (unit 1)
     (in_bom yes) (on_board yes)
-    (property "Reference" "U?" (id 0) (at 121.285 84.455 0)
+    (property "Reference" "G8" (id 0) (at 121.285 84.455 0)
       (effects (font (size 1.778 1.778)))
     )
@@
     (pin "9")
   )
+  (symbol (lib_id "power:VCC") (at 121.92 31.75 0) (unit 1)
+    (in_bom yes) (on_board yes)
+    (property "Reference" "#PWR?" (id 0) (at 121.92 35.56 0)
+      (effects (font (size 1.27 1.27)) hide)
+    )
+    (property "Value" "VCC" (id 1) (at 121.92 27.94 0))
+    (property "Footprint" "" (id 2) (at 121.92 31.75 0)
+      (effects (font (size 1.27 1.27)) hide)
+    )
+    (property "Datasheet" "" (id 3) (at 121.92 31.75 0)
+      (effects (font (size 1.27 1.27)) hide)
+    )
+    (pin "1")
+  )
 )

Commit message: wip_gfx_gll
Connections:
- net GLL_DRIVER0: now reaches G8.61 (MA4)
Changed lines of the file:
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@@
+    (stroke (width 0) (type default) (color 0 0 0 0))
+  )
+  (wire (pts (xy 149.86 46.99) (xy 161.29 46.99))
     (stroke (width 0) (type default) (color 0 0 0 0))
   )
@@
     (effects (font (size 1.27 1.27)) (justify left bottom))
   )
+  (hierarchical_label "GLL_DRIVER0" (shape input) (at 161.29 46.99 0)
+    (effects (font (size 1.27 1.27)) (justify left))
+  )
   (hierarchical_label "2GLL_A[5..0]" (shape bidirectional) (at 69.85 118.11 180)

Commit message: wip_iou_wd
Connections:
- net 2GLL2IOU0: now reaches G8.75 (MA20)
- net GLL_DRIVER0 renamed DRIVER_GLL2
Changed lines of the file:
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@@
+    (stroke (width 0) (type default) (color 0 0 0 0))
+  )
+  (wire (pts (xy 149.86 62.23) (xy 163.83 62.23))
     (stroke (width 0) (type default) (color 0 0 0 0))
   )
@@
     (effects (font (size 1.27 1.27)) (justify left bottom))
   )
-  (hierarchical_label "GLL_DRIVER0" (shape input) (at 161.29 46.99 0)
+  (hierarchical_label "2GLL2IOU0" (shape bidirectional) (at 163.83 62.23 0)
     (effects (font (size 1.27 1.27)) (justify left))
   )
+  (hierarchical_label "DRIVER_GLL2" (shape input) (at 161.29 46.99 0)
+    (effects (font (size 1.27 1.27)) (justify left))
+  )

Commit message: wip_ccu_gll2_cassette
Parts:
- added JP1: SolderJumper_2_Open, symbol Jumper:SolderJumper_2_Open
- added R10: 103, symbol Device:R_US
Connections:
- net VCC: now also R10.1
- net VSS: now also JP1.1 (A)
- net at G8.63 (Jumper): now also JP1.2 (B), R10.2

Commit message: wip_ccu_cassette
Connections:
- net ~{WEE}: now reaches G8.10 (~{WEE})
- net ~{OED}: now reaches G8.11 (~{OED})
- net ~{WED}: now reaches G8.14 (~{WED})
- net ~{OEC}: now reaches G8.15 (~{OEC})
- net ~{WEC}: now reaches G8.16 (~{WEC})
- net ~{OEB}: now reaches G8.17 (~{OEB})
- net ~{WEB}: now reaches G8.19 (~{WEB})
- net ~{RESET0}: now reaches G8.2 (~{RESET0})
- net ~{CEP}: now reaches G8.29 (~{CEP})
- net ~{RESET1}: now reaches G8.3 (~{RESET1})
- net ~{CEO}: now reaches G8.30 (~{CEO})
- net ~{CEN}: now reaches G8.31 (~{CEN})
- net ~{CEM}: now reaches G8.32 (~{CEM})
- net ~{CEL}: now reaches G8.34 (~{CEL})
- net ~{CEK}: now reaches G8.35 (~{CEK})
- net ~{CEJ}: now reaches G8.37 (~{CEJ})
- net ~{CEI}: now reaches G8.38 (~{CEI})
- net ~{CEH}: now reaches G8.39 (~{CEH})
- net ~{CEG}: now reaches G8.40 (~{CEG})
- net ~{CEF}: now reaches G8.42 (~{CEF})
- net ~{CEE}: now reaches G8.43 (~{CEE})
- net ~{CED}: now reaches G8.44 (~{CED})
- net ~{CEC}: now reaches G8.45 (~{CEC})
- net ~{CEB}: now reaches G8.47 (~{CEB})
- net ~{CEA}: now reaches G8.48 (~{CEA})
- net BX_SPR: now reaches G8.57 (BX_SPR)
- net CLK_GLL2: now reaches G8.59 (CLK_GLL2)
- net 2GLL2PPU0: now reaches G8.64 (2GLL2PPU0)
- net 2GLL2CCU0: now reaches G8.74 (2GLL2CCU0)
- net ~{RESET4}: now reaches G8.78 (~{RESET4})
- net ~{RESET3}: now reaches G8.79 (~{RESET3})
- net ~{RESET2}: now reaches G8.80 (~{RESET2})
- net ~{OEE}: now reaches G8.9 (~{OEE})
- no-connect marks 0 -> 6
Other:
- note added: "42.9545MHz"
- note added: "CONNECTED TO SLOT 7. THIS SLOT HAS NO SIMM."
- moved on the sheet: JP1, R10
