File: cores/cps3/sch/simms_2~1.kicad_sch (KiCad schematic)
At the start: 8 parts

Commit message: wip_ccu_cassette
Changed lines of the file:
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@@
     (effects (font (size 1.27 1.27)) (justify left bottom))
   )
-  (hierarchical_label "GFXD_D[7..0]" (shape output) (at 368.3 44.45 0)
+  (hierarchical_label "GFXD_D[7..0]" (shape bidirectional) (at 368.3 44.45 0)
     (effects (font (size 1.27 1.27)) (justify left))
   )
-  (hierarchical_label "GFXB_D[7..0]" (shape output) (at 209.55 44.45 0)
+  (hierarchical_label "GFXB_D[7..0]" (shape bidirectional) (at 209.55 44.45 0)
     (effects (font (size 1.27 1.27)) (justify left))
   )
@@
     (effects (font (size 1.27 1.27)) (justify right))
   )
-  (hierarchical_label "GFXA_D[7..0]" (shape output) (at 132.08 44.45 0)
+  (hierarchical_label "GFXA_D[7..0]" (shape bidirectional) (at 132.08 44.45 0)
     (effects (font (size 1.27 1.27)) (justify left))
   )
@@
     (effects (font (size 1.27 1.27)) (justify left))
   )
-  (hierarchical_label "GFXC_D[7..0]" (shape output) (at 288.29 44.45 0)
+  (hierarchical_label "GFXC_D[7..0]" (shape bidirectional) (at 288.29 44.45 0)
     (effects (font (size 1.27 1.27)) (justify left))
   )
