File: cores/cps3/sch/ccu.kicad_sch (KiCad schematic)
At the start: 28 parts, among them J13 DL-2829-CCU, J15 MB814260-70PJ, Q16 AHR38, Q17 AHR38, Q18 AHR38, Q19 AHR38

Commit message: wip_cassette_sh2
Changed lines of the file:
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@@
-    (stroke (width 0) (type default) (color 0 0 0 0))
-  )
-  (wire (pts (xy 344.17 157.48) (xy 349.25 157.48))
     (stroke (width 0) (type default) (color 0 0 0 0))
   )
@@
   )
   (wire (pts (xy 344.17 113.03) (xy 375.92 113.03))
-    (stroke (width 0) (type default) (color 0 0 0 0))
-  )
-  (wire (pts (xy 344.17 99.06) (xy 349.25 99.06))
     (stroke (width 0) (type default) (color 0 0 0 0))
   )
@@
     (effects (font (size 1.27 1.27)) (justify right bottom))
   )
-  (label "?" (at 349.25 99.06 0)
-    (effects (font (size 1.27 1.27)) (justify left bottom))
-  )
   (label "GFXD_D4" (at 308.61 184.15 180)
     (effects (font (size 1.27 1.27)) (justify right bottom))
@@
     (effects (font (size 1.27 1.27)) (justify right bottom))
   )
-  (label "?" (at 349.25 157.48 0)
-    (effects (font (size 1.27 1.27)) (justify left bottom))
-  )
   (label "GFXC_D6" (at 219.71 191.77 180)

Commit message: correction_ppu
Connections:
- net CPUC_A4: now reaches J13.11 (SCU_A22)
- net CPUC_A5: now reaches J13.12 (SCU_A21)
- net CPUC_A6: now reaches J13.13 (SCU_A20)
- net CPUC_A7: now reaches J13.14 (SCU_A19)
- net CPUC_A8: now reaches J13.16 (SCU_A18)
- net CPUC_A9: now reaches J13.17 (SCU_A17)
- net CPUC_A10: now reaches J13.18 (SCU_A16)
- net CPUC_A11: now reaches J13.19 (SCU_A15)
- net CPUC_A12: now reaches J13.20 (SCU_A14)
- net CPUC_A13: now reaches J13.21 (SCU_A13)
- net CPUC_A14: now reaches J13.22 (SCU_A12)
- net CPUC_A15: now reaches J13.23 (SCU_A11)
- net CPUC_A16: now reaches J13.24 (SCU_A10)
- net CPUC_A17: now reaches J13.25 (SCU_A9)
- net CPUC_A18: now reaches J13.27 (SCU_A8)
- net CPUC_A19: now reaches J13.28 (SCU_A7)
- net CPUC_A20: now reaches J13.29 (SCU_A6)
- net CPUC_~{CS2}: now reaches J13.3 (CPU_~{CS2})
- net CPUC_A21: now reaches J13.30 (SCU_A5)
- net CPUC_A22: now reaches J13.31 (SCU_A4)
- net CPUC_A23: now reaches J13.32 (SCU_A3)
- net CPUC_A24: now reaches J13.33 (SCU_A2)
- net CPUC_A25: now reaches J13.34 (SCU_A1)
- net CPUC_A26: now reaches J13.35 (SCU_A0)
- net at J13.36 (PULL_UP): now also J13.45 (PULL_UP), J13.47 (PULL_UP), R87.1
- net CPUC_~{WE3}: now reaches J13.37 (CPUC_~{WE3})
- net CPUC_~{WE2}: now reaches J13.39 (CPUC_~{WE2})
- net CPUC_~{CS1}: now reaches J13.4 (CPU_~{CS1})
- net CPUC_~{WE1}: now reaches J13.40 (CPUC_~{WE1})
- net CPUC_~{WE0}: now reaches J13.41 (CPUC_~{WE0})
- net ~{BS}_CPUC: now reaches J13.42 (~{BS}_CPUC)
- net RD/~{WR}_CPUC: now reaches J13.46 (RD/~{WR}_CPUC)
- net CPUC_~{CS0}: now reaches J13.5 (CPU_~{CS0})
- net WAIT_CPUC: now reaches J13.52 (WAIT_CPUC)
- net CPUC_D31: now reaches J13.58 (SCU_D31)
- net CPUC_D30: now reaches J13.59 (SCU_D30)
- net CPUC_A0: now reaches J13.6 (SCU_A26)
- net CPUC_D29: now reaches J13.62 (SCU_D29)
- net CPUC_D28: now reaches J13.63 (SCU_D28)
- net CPUC_D27: now reaches J13.64 (SCU_D27)
- net CPUC_D26: now reaches J13.65 (SCU_D26)
- net CPUC_D25: now reaches J13.66 (SCU_D25)
- net CPUC_D24: now reaches J13.67 (SCU_D24)
- net CPUC_D23: now reaches J13.68 (SCU_D23)
- net CPUC_D22: now reaches J13.69 (SCU_D22)
- net CPUC_A1: now reaches J13.7 (SCU_A25)
- net CPUC_D21: now reaches J13.70 (SCU_D21)
- net CPUC_D20: now reaches J13.71 (SCU_D20)
- net CPUC_D19: now reaches J13.72 (SCU_D19)
- net CPUC_D18: now reaches J13.73 (SCU_D18)
- net CPUC_D17: now reaches J13.74 (SCU_D17)
- net CPUC_D16: now reaches J13.75 (SCU_D16)
- net CPUC_D15: now reaches J13.77 (SCU_D15)
- net CPUC_D14: now reaches J13.78 (SCU_D14)
- net CPUC_D13: now reaches J13.79 (SCU_D13)
- net CPUC_A2: now reaches J13.8 (SCU_A24)
- net CPUC_D12: now reaches J13.80 (SCU_D12)
- net CPUC_D11: now reaches J13.81 (SCU_D11)
- net CPUC_D10: now reaches J13.82 (SCU_D10)
- net CPUC_D9: now reaches J13.83 (SCU_D9)
- net CPUC_D8: now reaches J13.84 (SCU_D8)
- net CPUC_D7: now reaches J13.85 (SCU_D7)
- net CPUC_D6: now reaches J13.86 (SCU_D6)
- net CPUC_D5: now reaches J13.87 (SCU_D5)
- net CPUC_D4: now reaches J13.88 (SCU_D4)
- net CPUC_D3: now reaches J13.89 (SCU_D3)
- net CPUC_A3: now reaches J13.9 (SCU_A23)
- net CPUC_D2: now reaches J13.90 (SCU_D2)
- net CPUC_D1: now reaches J13.91 (SCU_D1)
- net CPUC_D0: now reaches J13.92 (SCU_D0)
- net ~{CS3} renamed CPUC_~{CS3}
- net ~{RD} renamed ~{RD}_CPUC
- no-connect marks 0 -> 1
Other:
- note added: "ONLY CONNECTED TO PIN52 OF THE FEMALE SLOT"
- moved on the sheet: CP114, R87, R89

Commit message: wip_cre_cps3
Connections:
- net GLL2CCU0: now also J13.49 (GLL2CCU0); no longer J13.57 (PPU2CCU0)
- net GLL2CCU1: now also J13.156 (GLL2CCU1); no longer J13.49 (GLL2CCU0)
- net GLL2CCU2: now also J13.48 (GLL2CCU2); no longer J13.156 (GLL2CCU1)
- net GLL2CCU3: now also J13.199 (GLL2CCU3); no longer J13.48 (GLL2CCU2)
- net GLL2CCU4: now also J13.202 (GLL2CCU4); no longer J13.199 (GLL2CCU3)
- net PPU2CCU0: now also J13.57 (PPU2CCU0); no longer J13.202 (GLL2CCU4)
- net MAIN_A14 renamed MAIN_A5
- net PPU2CCU1 renamed BIC_A0
Other:
- note removed: "COMMUNICATION CONTROL UNIT?"
- moved on the sheet: CP114, CP120, CP121, DA3, DA4, J15, Q16, Q17, Q18, Q19, R100, R101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
