File: cores/cps3/sch/objects.kicad_sch (KiCad schematic)
At the start: 0 parts

Commit message: update7
Other:
- sheet gll1 ports: added MAIN_A[20..0]; removed GFX_A[20..0]
Changed lines of the file:
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@@
 (kicad_sch (version 20211123) (generator eeschema)
-  (paper "A3")
+  (paper "A5")
   (title_block
     (title "CP SYSTEM III")
@@
     (comment 1 "E.Triana")
   )
-  (wire (pts (xy 130.81 91.44) (xy 139.7 91.44))
-    (stroke (width 0) (type default) (color 0 0 0 0))
-  )
-  (wire (pts (xy 130.81 96.52) (xy 139.7 96.52))
-    (stroke (width 0) (type default) (color 0 0 0 0))
-  )
-  (bus (pts (xy 176.53 93.98) (xy 182.88 93.98))
-    (stroke (width 0) (type default) (color 0 0 0 0))
-  )
-  (bus (pts (xy 176.53 91.44) (xy 182.88 91.44))
-    (stroke (width 0) (type default) (color 0 0 0 0))
-  )
-  (bus (pts (xy 247.65 91.44) (xy 254 91.44))
-    (stroke (width 0) (type default) (color 0 0 0 0))
-  )
-  (wire (pts (xy 176.53 96.52) (xy 182.88 96.52))
-    (stroke (width 0) (type default) (color 0 0 0 0))
-  )
-  (wire (pts (xy 130.81 93.98) (xy 139.7 93.98))
-    (stroke (width 0) (type default) (color 0 0 0 0))
-  )
-  (image (at 398.78 261.62) (scale 0.294008)
+  (wire (pts (xy 29.21 38.1) (xy 38.1 38.1))
+    (stroke (width 0) (type default) (color 0 0 0 0))
+  )
+  (wire (pts (xy 29.21 43.18) (xy 38.1 43.18))
+    (stroke (width 0) (type default) (color 0 0 0 0))
+  )
+  (bus (pts (xy 74.93 40.64) (xy 81.28 40.64))
+    (stroke (width 0) (type default) (color 0 0 0 0))
+  )
+  (bus (pts (xy 74.93 38.1) (xy 81.28 38.1))
+    (stroke (width 0) (type default) (color 0 0 0 0))
+  )
+  (bus (pts (xy 125.73 38.1) (xy 132.08 38.1))
+    (stroke (width 0) (type default) (color 0 0 0 0))
+  )
+  (wire (pts (xy 74.93 43.18) (xy 81.28 43.18))
+    (stroke (width 0) (type default) (color 0 0 0 0))
+  )
+  (wire (pts (xy 29.21 40.64) (xy 38.1 40.64))
+    (stroke (width 0) (type default) (color 0 0 0 0))
+  )
+  (image (at 186.69 111.76) (scale 0.294008)
     (data
       iVBORw0KGgoAAAANSUhEUgAAAtEAAAGsCAMAAAAsQwu3AAAAA3NCSVQICAjb4U/gAAADAFBMVEX/
@@
     )
   )
-  (hierarchical_label "MAIN_D[23..0]" (shape bidirectional) (at 182.88 91.44 0)
+  (hierarchical_label "MAIN_D[23..0]" (shape bidirectional) (at 81.28 38.1 0)
     (effects (font (size 1.27 1.27)) (justify left))
   )
-  (hierarchical_label "2GLL_A[5..0]" (shape bidirectional) (at 247.65 91.44 180)
-    (effects (font (size 1.27 1.27)) (justify right))
-  )
-  (hierarchical_label "RESET?" (shape tri_state) (at 130.81 91.44 180)
-    (effects (font (size 1.27 1.27)) (justify right))
-  )
-  (hierarchical_label "GLL2IO1" (shape bidirectional) (at 130.81 96.52 180)
-    (effects (font (size 1.27 1.27)) (justify right))
-  )
-  (hierarchical_label "GFX_A[20..0]" (shape tri_state) (at 182.88 93.98 0)
+  (hierarchical_label "2GLL_A[5..0]" (shape bidirectional) (at 125.73 38.1 180)
+    (effects (font (size 1.27 1.27)) (justify right))
+  )
+  (hierarchical_label "RESET?" (shape tri_state) (at 29.21 38.1 180)
+    (effects (font (size 1.27 1.27)) (justify right))
+  )
+  (hierarchical_label "GLL2IO1" (shape bidirectional) (at 29.21 43.18 180)
+    (effects (font (size 1.27 1.27)) (justify right))
+  )
+  (hierarchical_label "MAIN_A[20..0]" (shape tri_state) (at 81.28 40.64 0)
     (effects (font (size 1.27 1.27)) (justify left))
   )
-  (hierarchical_label "CBI_CLK" (shape output) (at 182.88 96.52 0)
+  (hierarchical_label "CBI_CLK" (shape output) (at 81.28 43.18 0)
     (effects (font (size 1.27 1.27)) (justify left))
   )
-  (hierarchical_label "GLL2IO0" (shape tri_state) (at 130.81 93.98 180)
-    (effects (font (size 1.27 1.27)) (justify right))
-  )
-  (sheet (at 254 88.9) (size 36.83 44.45) (fields_autoplaced)
+  (hierarchical_label "GLL2IO0" (shape tri_state) (at 29.21 40.64 180)
+    (effects (font (size 1.27 1.27)) (justify right))
+  )
+  (sheet (at 132.08 35.56) (size 36.83 44.45) (fields_autoplaced)
     (stroke (width 0.1524) (type solid) (color 0 0 0 0))
     (fill (color 0 0 0 0.0000))
-    (property "Sheet name" "gll2" (id 0) (at 254 88.1884 0)
+    (property "Sheet name" "gll2" (id 0) (at 132.08 34.8484 0)
       (effects (font (size 1.27 1.27)) (justify left bottom))
     )
-    (property "Sheet file" "gll2.kicad_sch" (id 1) (at 254 133.9346 0)
+    (property "Sheet file" "gll2.kicad_sch" (id 1) (at 132.08 80.5946 0)
       (effects (font (size 1.27 1.27)) (justify left top))
     )
-    (pin "2GLL_A[5..0]" bidirectional (at 254 91.44 180)
-      (effects (font (size 1.27 1.27)) (justify left))
-    )
-  )
-  (sheet (at 139.7 88.9) (size 36.83 44.45) (fields_autoplaced)
+    (pin "2GLL_A[5..0]" bidirectional (at 132.08 38.1 180)
+      (effects (font (size 1.27 1.27)) (justify left))
+    )
+  )
+  (sheet (at 38.1 35.56) (size 36.83 44.45) (fields_autoplaced)
     (stroke (width 0.1524) (type solid) (color 0 0 0 0))
     (fill (color 0 0 0 0.0000))
-    (property "Sheet name" "gll1" (id 0) (at 139.7 88.1884 0)
+    (property "Sheet name" "gll1" (id 0) (at 38.1 34.8484 0)
       (effects (font (size 1.27 1.27)) (justify left bottom))
     )
-    (property "Sheet file" "gll1.kicad_sch" (id 1) (at 139.7 133.9346 0)
+    (property "Sheet file" "gll1.kicad_sch" (id 1) (at 38.1 80.5946 0)
       (effects (font (size 1.27 1.27)) (justify left top))
     )
-    (pin "CBI_CLK" output (at 176.53 96.52 0)
+    (pin "CBI_CLK" output (at 74.93 43.18 0)
       (effects (font (size 1.27 1.27)) (justify right))
     )
-    (pin "MAIN_D[23..0]" bidirectional (at 176.53 91.44 0)
+    (pin "MAIN_D[23..0]" bidirectional (at 74.93 38.1 0)
       (effects (font (size 1.27 1.27)) (justify right))
     )
-    (pin "GFX_A[20..0]" bidirectional (at 176.53 93.98 0)
+    (pin "RESET?" input (at 38.1 38.1 180)
+      (effects (font (size 1.27 1.27)) (justify left))
+    )
+    (pin "GLL2IO0" input (at 38.1 40.64 180)
+      (effects (font (size 1.27 1.27)) (justify left))
+    )
+    (pin "GLL2IO1" input (at 38.1 43.18 180)
+      (effects (font (size 1.27 1.27)) (justify left))
+    )
+    (pin "MAIN_A[20..0]" bidirectional (at 74.93 40.64 0)
       (effects (font (size 1.27 1.27)) (justify right))
     )
-    (pin "RESET?" input (at 139.7 91.44 180)
-      (effects (font (size 1.27 1.27)) (justify left))
-    )
-    (pin "GLL2IO0" input (at 139.7 93.98 180)
-      (effects (font (size 1.27 1.27)) (justify left))
-    )
-    (pin "GLL2IO1" input (at 139.7 96.52 180)
-      (effects (font (size 1.27 1.27)) (justify left))
-    )
-  )
+  )

Commit message: wip_ssu_cbi_gll
Other:
- sheet gll1 ports: added CLK_GLL1; removed CBI_CLK
Changed lines of the file:
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@@
     (effects (font (size 1.27 1.27)) (justify left))
   )
-  (hierarchical_label "CBI_CLK" (shape output) (at 81.28 43.18 0)
+  (hierarchical_label "CLK_GLL1" (shape output) (at 81.28 43.18 0)
     (effects (font (size 1.27 1.27)) (justify left))
   )
@@
       (effects (font (size 1.27 1.27)) (justify left top))
     )
-    (pin "CBI_CLK" output (at 74.93 43.18 0)
+    (pin "CLK_GLL1" output (at 74.93 43.18 0)
       (effects (font (size 1.27 1.27)) (justify right))
     )

Commit message: wip_gfx_gll
Other:
- sheet gll1 ports: added GLL_DRIVER1, GLL_DRIVER3; removed GLL2IO0, GLL2IO1
Changed lines of the file:
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@@
     (effects (font (size 1.27 1.27)) (justify right))
   )
-  (hierarchical_label "GLL2IO1" (shape bidirectional) (at 29.21 43.18 180)
+  (hierarchical_label "GLL_DRIVER3" (shape bidirectional) (at 29.21 43.18 180)
     (effects (font (size 1.27 1.27)) (justify right))
   )
@@
     (effects (font (size 1.27 1.27)) (justify left))
   )
-  (hierarchical_label "GLL2IO0" (shape tri_state) (at 29.21 40.64 180)
+  (hierarchical_label "GLL_DRIVER1" (shape tri_state) (at 29.21 40.64 180)
     (effects (font (size 1.27 1.27)) (justify right))
   )
@@
       (effects (font (size 1.27 1.27)) (justify left))
     )
-    (pin "GLL2IO0" input (at 38.1 40.64 180)
+    (pin "GLL_DRIVER1" input (at 38.1 40.64 180)
       (effects (font (size 1.27 1.27)) (justify left))
     )
-    (pin "GLL2IO1" input (at 38.1 43.18 180)
+    (pin "GLL_DRIVER3" input (at 38.1 43.18 180)
       (effects (font (size 1.27 1.27)) (justify left))
     )

Commit message: wip_gll_cassette
Other:
- added sheet ram_cassette (ram_cassette.kicad_sch)
- sheet gll1 ports: added GFXC_D[7..0], GFXD_D[7..0], GLL2IOU0, GLL2RC0, GLL_A[20..0], GLL_DRIVER0, GLL_DRIVER2, GLL_DRIVER4, GLL_D[7..0]; removed RESET?
- sheet gll2 ports: added GLL_DRIVER0; removed none
Changed lines of the file:
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@@
+    (stroke (width 0) (type default) (color 0 0 0 0))
+  )
+  (wire (pts (xy 29.21 50.8) (xy 38.1 50.8))
+    (stroke (width 0) (type default) (color 0 0 0 0))
+  )
+  (wire (pts (xy 29.21 48.26) (xy 38.1 48.26))
     (stroke (width 0) (type default) (color 0 0 0 0))
   )
@@
     (stroke (width 0) (type default) (color 0 0 0 0))
   )
+  (bus (pts (xy 74.93 55.88) (xy 81.28 55.88))
+    (stroke (width 0) (type default) (color 0 0 0 0))
+  )
+  (bus (pts (xy 74.93 50.8) (xy 81.28 50.8))
+    (stroke (width 0) (type default) (color 0 0 0 0))
+  )
+  (wire (pts (xy 74.93 45.72) (xy 81.28 45.72))
+    (stroke (width 0) (type default) (color 0 0 0 0))
+  )
+  (bus (pts (xy 74.93 48.26) (xy 81.28 48.26))
+    (stroke (width 0) (type default) (color 0 0 0 0))
+  )
   (bus (pts (xy 74.93 38.1) (xy 81.28 38.1))
     (stroke (width 0) (type default) (color 0 0 0 0))
   )
+  (wire (pts (xy 26.67 96.52) (xy 38.1 96.52))
+    (stroke (width 0) (type default) (color 0 0 0 0))
+  )
   (bus (pts (xy 125.73 38.1) (xy 132.08 38.1))
     (stroke (width 0) (type default) (color 0 0 0 0))
   )
+  (wire (pts (xy 111.76 40.64) (xy 132.08 40.64))
+    (stroke (width 0) (type default) (color 0 0 0 0))
+  )
+  (wire (pts (xy 74.93 96.52) (xy 81.28 96.52))
+    (stroke (width 0) (type default) (color 0 0 0 0))
+  )
   (wire (pts (xy 74.93 43.18) (xy 81.28 43.18))
     (stroke (width 0) (type default) (color 0 0 0 0))
   )
-  (wire (pts (xy 29.21 40.64) (xy 38.1 40.64))
+  (wire (pts (xy 29.21 45.72) (xy 38.1 45.72))
+    (stroke (width 0) (type default) (color 0 0 0 0))
+  )
+  (bus (pts (xy 74.93 53.34) (xy 81.28 53.34))
+    (stroke (width 0) (type default) (color 0 0 0 0))
+  )
+  (wire (pts (xy 16.51 40.64) (xy 38.1 40.64))
     (stroke (width 0) (type default) (color 0 0 0 0))
   )
@@
     )
   )
+  (label "GLL_DRIVER0" (at 16.51 40.64 0)
+    (effects (font (size 1.27 1.27)) (justify left bottom))
+  )
+  (label "GLL_DRIVER0" (at 111.76 40.64 0)
+    (effects (font (size 1.27 1.27)) (justify left bottom))
+  )
+  (label "GLL2RC0" (at 26.67 96.52 0)
+    (effects (font (size 1.27 1.27)) (justify left bottom))
+  )
+  (hierarchical_label "PULL_UP1" (shape passive) (at 81.28 96.52 0)
+    (effects (font (size 1.27 1.27)) (justify left))
+  )
   (hierarchical_label "MAIN_D[23..0]" (shape bidirectional) (at 81.28 38.1 0)
     (effects (font (size 1.27 1.27)) (justify left))
@@
     (effects (font (size 1.27 1.27)) (justify right))
   )
-  (hierarchical_label "RESET?" (shape tri_state) (at 29.21 38.1 180)
-    (effects (font (size 1.27 1.27)) (justify right))
-  )
-  (hierarchical_label "GLL_DRIVER3" (shape bidirectional) (at 29.21 43.18 180)
-    (effects (font (size 1.27 1.27)) (justify right))
+  (hierarchical_label "GFXD_D[7..0]" (shape output) (at 81.28 48.26 0)
+    (effects (font (size 1.27 1.27)) (justify left))
+  )
+  (hierarchical_label "GLL2IOU0" (shape tri_state) (at 29.21 38.1 180)
+    (effects (font (size 1.27 1.27)) (justify right))
+  )
+  (hierarchical_label "GLL2RC0" (shape output) (at 81.28 45.72 0)
+    (effects (font (size 1.27 1.27)) (justify left))
+  )
+  (hierarchical_label "GLL_A[20..0]" (shape output) (at 81.28 53.34 0)
+    (effects (font (size 1.27 1.27)) (justify left))
+  )
+  (hierarchical_label "GLL_DRIVER4" (shape bidirectional) (at 29.21 50.8 180)
+    (effects (font (size 1.27 1.27)) (justify right))
+  )
+  (hierarchical_label "GLL_DRIVER2" (shape bidirectional) (at 29.21 45.72 180)
+    (effects (font (size 1.27 1.27)) (justify right))
+  )
+  (hierarchical_label "GFXC_D[7..0]" (shape output) (at 81.28 50.8 0)
+    (effects (font (size 1.27 1.27)) (justify left))
+  )
+  (hierarchical_label "GLL_DRIVER3" (shape bidirectional) (at 29.21 48.26 180)
+    (effects (font (size 1.27 1.27)) (justify right))
+  )
+  (hierarchical_label "GLL_D[7..0]" (shape output) (at 81.28 55.88 0)
+    (effects (font (size 1.27 1.27)) (justify left))
   )
   (hierarchical_label "MAIN_A[20..0]" (shape tri_state) (at 81.28 40.64 0)
@@
     (effects (font (size 1.27 1.27)) (justify left))
   )
-  (hierarchical_label "GLL_DRIVER1" (shape tri_state) (at 29.21 40.64 180)
+  (hierarchical_label "GLL_DRIVER1" (shape tri_state) (at 29.21 43.18 180)
     (effects (font (size 1.27 1.27)) (justify right))
   )
@@
       (effects (font (size 1.27 1.27)) (justify left))
     )
-  )
-  (sheet (at 38.1 35.56) (size 36.83 44.45) (fields_autoplaced)
+    (pin "GLL_DRIVER0" input (at 132.08 40.64 180)
+      (effects (font (size 1.27 1.27)) (justify left))
+    )
+  )
+  (sheet (at 38.1 93.98) (size 36.83 24.13) (fields_autoplaced)
+    (stroke (width 0.1524) (type solid) (color 0 0 0 0))
+    (fill (color 0 0 0 0.0000))
+    (property "Sheet name" "ram_cassette" (id 0) (at 38.1 93.2684 0)
+      (effects (font (size 1.27 1.27)) (justify left bottom))
+    )
+    (property "Sheet file" "ram_cassette.kicad_sch" (id 1) (at 38.1 118.6946 0)
+      (effects (font (size 1.27 1.27)) (justify left top))
+    )
+    (pin "PULL_UP1" passive (at 74.93 96.52 0)
+      (effects (font (size 1.27 1.27)) (justify right))
+    )
+    (pin "GLL2RC0" input (at 38.1 96.52 180)
+      (effects (font (size 1.27 1.27)) (justify left))
+    )
+  )
+  (sheet (at 38.1 35.56) (size 36.83 22.86) (fields_autoplaced)
     (stroke (width 0.1524) (type solid) (color 0 0 0 0))
     (fill (color 0 0 0 0.0000))
@@
       (effects (font (size 1.27 1.27)) (justify left bottom))
     )
-    (property "Sheet file" "gll1.kicad_sch" (id 1) (at 38.1 80.5946 0)
+    (property "Sheet file" "gll1.kicad_sch" (id 1) (at 38.1 59.0046 0)
       (effects (font (size 1.27 1.27)) (justify left top))
     )
@@
       (effects (font (size 1.27 1.27)) (justify right))
     )
-    (pin "RESET?" input (at 38.1 38.1 180)
-      (effects (font (size 1.27 1.27)) (justify left))
-    )
-    (pin "GLL_DRIVER1" input (at 38.1 40.64 180)
-      (effects (font (size 1.27 1.27)) (justify left))
-    )
-    (pin "GLL_DRIVER3" input (at 38.1 43.18 180)
-      (effects (font (size 1.27 1.27)) (justify left))
-    )
     (pin "MAIN_A[20..0]" bidirectional (at 74.93 40.64 0)
       (effects (font (size 1.27 1.27)) (justify right))
     )
+    (pin "GLL_DRIVER0" input (at 38.1 40.64 180)
+      (effects (font (size 1.27 1.27)) (justify left))
+    )
+    (pin "GLL_DRIVER2" input (at 38.1 45.72 180)
+      (effects (font (size 1.27 1.27)) (justify left))
+    )
+    (pin "GLL_DRIVER1" input (at 38.1 43.18 180)
+      (effects (font (size 1.27 1.27)) (justify left))
+    )
+    (pin "GLL_DRIVER3" input (at 38.1 48.26 180)
+      (effects (font (size 1.27 1.27)) (justify left))
+    )
+    (pin "GLL_DRIVER4" input (at 38.1 50.8 180)
+      (effects (font (size 1.27 1.27)) (justify left))
+    )
+    (pin "GLL2IOU0" bidirectional (at 38.1 38.1 180)
+      (effects (font (size 1.27 1.27)) (justify left))
+    )
+    (pin "GLL2RC0" output (at 74.93 45.72 0)
+      (effects (font (size 1.27 1.27)) (justify right))
+    )
+    (pin "GFXD_D[7..0]" output (at 74.93 48.26 0)
+      (effects (font (size 1.27 1.27)) (justify right))
+    )
+    (pin "GFXC_D[7..0]" output (at 74.93 50.8 0)
+      (effects (font (size 1.27 1.27)) (justify right))
+    )
+    (pin "GLL_A[20..0]" output (at 74.93 53.34 0)
+      (effects (font (size 1.27 1.27)) (justify right))
+    )
+    (pin "GLL_D[7..0]" output (at 74.93 55.88 0)
+      (effects (font (size 1.27 1.27)) (justify right))
+    )
