File: cores/cps3/sch/objects.kicad_sch (KiCad schematic)
At the start: 0 parts

Commit message: wip_iou_wd
Other:
- sheet gll1 ports: added DRIVER_GLL[4..0], GLL2CCU[5..0], ~{CS}_GLL1, ~{MR}_GLL1, ~{RE}_GLL1, ~{RST_WD}, ~{WE}_GLL1; removed GLL2RC0, GLL_DRIVER0, GLL_DRIVER1, GLL_DRIVER2, GLL_DRIVER3, GLL_DRIVER4
- sheet gll2 ports: added DRIVER_GLL2; removed GLL_DRIVER0
- sheet ram_cassette ports: added ~{RST_WD}; removed GLL2RC0
Changed lines of the file:
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@@
     (stroke (width 0) (type default) (color 0 0 0 0))
   )
-  (wire (pts (xy 29.21 50.8) (xy 38.1 50.8))
-    (stroke (width 0) (type default) (color 0 0 0 0))
-  )
-  (wire (pts (xy 29.21 48.26) (xy 38.1 48.26))
-    (stroke (width 0) (type default) (color 0 0 0 0))
-  )
-  (wire (pts (xy 29.21 43.18) (xy 38.1 43.18))
+  (wire (pts (xy 74.93 63.5) (xy 81.28 63.5))
+    (stroke (width 0) (type default) (color 0 0 0 0))
+  )
+  (wire (pts (xy 74.93 66.04) (xy 81.28 66.04))
+    (stroke (width 0) (type default) (color 0 0 0 0))
+  )
+  (bus (pts (xy 74.93 58.42) (xy 81.28 58.42))
     (stroke (width 0) (type default) (color 0 0 0 0))
   )
@@
     (stroke (width 0) (type default) (color 0 0 0 0))
   )
+  (bus (pts (xy 29.21 40.64) (xy 38.1 40.64))
+    (stroke (width 0) (type default) (color 0 0 0 0))
+  )
   (bus (pts (xy 74.93 38.1) (xy 81.28 38.1))
     (stroke (width 0) (type default) (color 0 0 0 0))
   )
+  (wire (pts (xy 74.93 60.96) (xy 81.28 60.96))
+    (stroke (width 0) (type default) (color 0 0 0 0))
+  )
   (wire (pts (xy 26.67 96.52) (xy 38.1 96.52))
     (stroke (width 0) (type default) (color 0 0 0 0))
@@
     (stroke (width 0) (type default) (color 0 0 0 0))
   )
-  (wire (pts (xy 29.21 45.72) (xy 38.1 45.72))
+  (wire (pts (xy 74.93 68.58) (xy 81.28 68.58))
     (stroke (width 0) (type default) (color 0 0 0 0))
   )
   (bus (pts (xy 74.93 53.34) (xy 81.28 53.34))
-    (stroke (width 0) (type default) (color 0 0 0 0))
-  )
-  (wire (pts (xy 16.51 40.64) (xy 38.1 40.64))
     (stroke (width 0) (type default) (color 0 0 0 0))
   )
@@
     )
   )
-  (label "GLL_DRIVER0" (at 16.51 40.64 0)
+  (label "DRIVER_GLL2" (at 111.76 40.64 0)
     (effects (font (size 1.27 1.27)) (justify left bottom))
   )
-  (label "GLL_DRIVER0" (at 111.76 40.64 0)
+  (label "~{RST_WD}" (at 26.67 96.52 0)
     (effects (font (size 1.27 1.27)) (justify left bottom))
   )
-  (label "GLL2RC0" (at 26.67 96.52 0)
-    (effects (font (size 1.27 1.27)) (justify left bottom))
-  )
   (hierarchical_label "PULL_UP1" (shape passive) (at 81.28 96.52 0)
     (effects (font (size 1.27 1.27)) (justify left))
@@
   (hierarchical_label "MAIN_D[23..0]" (shape bidirectional) (at 81.28 38.1 0)
     (effects (font (size 1.27 1.27)) (justify left))
+  )
+  (hierarchical_label "GLL2CCU[5..0]" (shape bidirectional) (at 29.21 40.64 180)
+    (effects (font (size 1.27 1.27)) (justify right))
   )
   (hierarchical_label "2GLL_A[5..0]" (shape bidirectional) (at 125.73 38.1 180)
@@
     (effects (font (size 1.27 1.27)) (justify right))
   )
-  (hierarchical_label "GLL2RC0" (shape output) (at 81.28 45.72 0)
+  (hierarchical_label "~{RST_WD}" (shape output) (at 81.28 45.72 0)
+    (effects (font (size 1.27 1.27)) (justify left))
+  )
+  (hierarchical_label "~{MR}_GLL1" (shape output) (at 81.28 60.96 0)
     (effects (font (size 1.27 1.27)) (justify left))
   )
@@
     (effects (font (size 1.27 1.27)) (justify left))
   )
-  (hierarchical_label "GLL_DRIVER4" (shape bidirectional) (at 29.21 50.8 180)
-    (effects (font (size 1.27 1.27)) (justify right))
-  )
-  (hierarchical_label "GLL_DRIVER2" (shape bidirectional) (at 29.21 45.72 180)
-    (effects (font (size 1.27 1.27)) (justify right))
+  (hierarchical_label "~{RE}_GLL1" (shape output) (at 81.28 63.5 0)
+    (effects (font (size 1.27 1.27)) (justify left))
+  )
+  (hierarchical_label "~{CS}_GLL1" (shape output) (at 81.28 68.58 0)
+    (effects (font (size 1.27 1.27)) (justify left))
+  )
+  (hierarchical_label "DRIVER_GLL[4..0]" (shape bidirectional) (at 81.28 58.42 0)
+    (effects (font (size 1.27 1.27)) (justify left))
+  )
+  (hierarchical_label "~{WE}_GLL1" (shape output) (at 81.28 66.04 0)
+    (effects (font (size 1.27 1.27)) (justify left))
   )
   (hierarchical_label "GFXC_D[7..0]" (shape output) (at 81.28 50.8 0)
     (effects (font (size 1.27 1.27)) (justify left))
   )
-  (hierarchical_label "GLL_DRIVER3" (shape bidirectional) (at 29.21 48.26 180)
-    (effects (font (size 1.27 1.27)) (justify right))
-  )
   (hierarchical_label "GLL_D[7..0]" (shape output) (at 81.28 55.88 0)
     (effects (font (size 1.27 1.27)) (justify left))
@@
   (hierarchical_label "CLK_GLL1" (shape output) (at 81.28 43.18 0)
     (effects (font (size 1.27 1.27)) (justify left))
-  )
-  (hierarchical_label "GLL_DRIVER1" (shape tri_state) (at 29.21 43.18 180)
-    (effects (font (size 1.27 1.27)) (justify right))
   )
   (sheet (at 132.08 35.56) (size 36.83 44.45) (fields_autoplaced)
@@
       (effects (font (size 1.27 1.27)) (justify left))
     )
-    (pin "GLL_DRIVER0" input (at 132.08 40.64 180)
+    (pin "DRIVER_GLL2" input (at 132.08 40.64 180)
       (effects (font (size 1.27 1.27)) (justify left))
     )
@@
       (effects (font (size 1.27 1.27)) (justify right))
     )
-    (pin "GLL2RC0" input (at 38.1 96.52 180)
+    (pin "~{RST_WD}" input (at 38.1 96.52 180)
       (effects (font (size 1.27 1.27)) (justify left))
     )
   )
-  (sheet (at 38.1 35.56) (size 36.83 22.86) (fields_autoplaced)
+  (sheet (at 38.1 35.56) (size 36.83 35.56) (fields_autoplaced)
     (stroke (width 0.1524) (type solid) (color 0 0 0 0))
     (fill (color 0 0 0 0.0000))
@@
       (effects (font (size 1.27 1.27)) (justify left bottom))
     )
-    (property "Sheet file" "gll1.kicad_sch" (id 1) (at 38.1 59.0046 0)
+    (property "Sheet file" "gll1.kicad_sch" (id 1) (at 38.1 71.7046 0)
       (effects (font (size 1.27 1.27)) (justify left top))
     )
@@
     (pin "MAIN_A[20..0]" bidirectional (at 74.93 40.64 0)
       (effects (font (size 1.27 1.27)) (justify right))
-    )
-    (pin "GLL_DRIVER0" input (at 38.1 40.64 180)
-      (effects (font (size 1.27 1.27)) (justify left))
-    )
-    (pin "GLL_DRIVER2" input (at 38.1 45.72 180)
-      (effects (font (size 1.27 1.27)) (justify left))
-    )
-    (pin "GLL_DRIVER1" input (at 38.1 43.18 180)
-      (effects (font (size 1.27 1.27)) (justify left))
-    )
-    (pin "GLL_DRIVER3" input (at 38.1 48.26 180)
-      (effects (font (size 1.27 1.27)) (justify left))
-    )
-    (pin "GLL_DRIVER4" input (at 38.1 50.8 180)
-      (effects (font (size 1.27 1.27)) (justify left))
     )
     (pin "GLL2IOU0" bidirectional (at 38.1 38.1 180)
       (effects (font (size 1.27 1.27)) (justify left))
     )
-    (pin "GLL2RC0" output (at 74.93 45.72 0)
+    (pin "~{RST_WD}" output (at 74.93 45.72 0)
       (effects (font (size 1.27 1.27)) (justify right))
     )
@@
       (effects (font (size 1.27 1.27)) (justify right))
     )
+    (pin "GLL2CCU[5..0]" bidirectional (at 38.1 40.64 180)
+      (effects (font (size 1.27 1.27)) (justify left))
+    )
+    (pin "DRIVER_GLL[4..0]" output (at 74.93 58.42 0)
+      (effects (font (size 1.27 1.27)) (justify right))
+    )
+    (pin "~{MR}_GLL1" output (at 74.93 60.96 0)
+      (effects (font (size 1.27 1.27)) (justify right))
+    )
+    (pin "~{RE}_GLL1" output (at 74.93 63.5 0)
+      (effects (font (size 1.27 1.27)) (justify right))
+    )
+    (pin "~{WE}_GLL1" output (at 74.93 66.04 0)
+      (effects (font (size 1.27 1.27)) (justify right))
+    )
+    (pin "~{CS}_GLL1" output (at 74.93 68.58 0)
+      (effects (font (size 1.27 1.27)) (justify right))
+    )

Commit message: wip_ccu_gll2_cassette
Other:
- sheet gll1 ports: added ~{STBY_WD}; removed none
- sheet gll2 ports: added 2GLL2IOU0; removed none
Changed lines of the file:
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@@
+    (stroke (width 0) (type default) (color 0 0 0 0))
+  )
+  (wire (pts (xy 74.93 71.12) (xy 81.28 71.12))
     (stroke (width 0) (type default) (color 0 0 0 0))
   )
@@
   )
   (bus (pts (xy 29.21 40.64) (xy 38.1 40.64))
+    (stroke (width 0) (type default) (color 0 0 0 0))
+  )
+  (wire (pts (xy 125.73 43.18) (xy 132.08 43.18))
     (stroke (width 0) (type default) (color 0 0 0 0))
   )
@@
     (effects (font (size 1.27 1.27)) (justify right))
   )
+  (hierarchical_label "2GLL2IOU0" (shape bidirectional) (at 125.73 43.18 180)
+    (effects (font (size 1.27 1.27)) (justify right))
+  )
+  (hierarchical_label "~{STBY_WD}" (shape output) (at 81.28 71.12 0)
+    (effects (font (size 1.27 1.27)) (justify left))
+  )
   (hierarchical_label "GFXD_D[7..0]" (shape output) (at 81.28 48.26 0)
     (effects (font (size 1.27 1.27)) (justify left))
@@
       (effects (font (size 1.27 1.27)) (justify left))
     )
+    (pin "2GLL2IOU0" bidirectional (at 132.08 43.18 180)
+      (effects (font (size 1.27 1.27)) (justify left))
+    )
   )
   (sheet (at 38.1 93.98) (size 36.83 24.13) (fields_autoplaced)
@@
     )
   )
-  (sheet (at 38.1 35.56) (size 36.83 35.56) (fields_autoplaced)
+  (sheet (at 38.1 35.56) (size 36.83 38.1) (fields_autoplaced)
     (stroke (width 0.1524) (type solid) (color 0 0 0 0))
     (fill (color 0 0 0 0.0000))
@@
       (effects (font (size 1.27 1.27)) (justify left bottom))
     )
-    (property "Sheet file" "gll1.kicad_sch" (id 1) (at 38.1 71.7046 0)
+    (property "Sheet file" "gll1.kicad_sch" (id 1) (at 38.1 74.2446 0)
       (effects (font (size 1.27 1.27)) (justify left top))
     )
@@
       (effects (font (size 1.27 1.27)) (justify right))
     )
+    (pin "~{STBY_WD}" output (at 74.93 71.12 0)
+      (effects (font (size 1.27 1.27)) (justify right))
+    )

Commit message: wip_ccu_cassette
Other:
- sheet gll2 ports: added 2GLL2CCU0, 2GLL2PPU0, BX_SPR, CLK_GLL2, ~{CEA}, ~{CEB}, ~{CEC}, ~{CED}, ~{CEE}, ~{CEF}, ~{CEG}, ~{CEH}, ~{CEI}, ~{CEJ}, ~{CEK}, ~{CEL}, ~{CEM}, ~{CEN}, ~{CEO}, ~{CEP}, ~{OEB}, ~{OEC}, ~{OED}, ~{OEE}, ~{RESET[4..0]}, ~{WEB}, ~{WEC}, ~{WED}, ~{WEE}; removed none

Commit message: wip_cassette
Other:
- sheet gll1 ports: added ~{RST}_WD; removed ~{RST_WD}
- sheet ram_cassette ports: added ~{RST}_WD; removed ~{RST_WD}
Changed lines of the file:
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@@
     (effects (font (size 1.27 1.27)) (justify left bottom))
   )
-  (label "~{RST_WD}" (at 26.67 96.52 0)
+  (label "~{RST}_WD" (at 26.67 96.52 0)
     (effects (font (size 1.27 1.27)) (justify left bottom))
   )
@@
     (effects (font (size 1.27 1.27)) (justify left))
   )
-  (hierarchical_label "~{RST_WD}" (shape output) (at 81.28 45.72 0)
+  (hierarchical_label "~{RST}_WD" (shape output) (at 81.28 45.72 0)
     (effects (font (size 1.27 1.27)) (justify left))
   )
@@
       (effects (font (size 1.27 1.27)) (justify right))
     )
-    (pin "~{RST_WD}" input (at 38.1 96.52 180)
+    (pin "~{RST}_WD" input (at 38.1 96.52 180)
       (effects (font (size 1.27 1.27)) (justify left))
     )
@@
       (effects (font (size 1.27 1.27)) (justify left))
     )
-    (pin "~{RST_WD}" output (at 74.93 45.72 0)
-      (effects (font (size 1.27 1.27)) (justify right))
-    )
+    (pin "~{RST}_WD" output (at 74.93 45.72 0)
+      (effects (font (size 1.27 1.27)) (justify right))
+    )
