File: cores/cps3/sch/objects.kicad_sch (KiCad schematic)
At the start: 0 parts

Commit message: wip_cassette_rg
Other:
- note added: "OK"
Changed lines of the file:
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@@
     )
+  )
+  (text "OK" (at 48.26 60.96 0)
+    (effects (font (size 1.27 1.27)) (justify left bottom))
+  )
+  (text "OK" (at 147.32 68.58 0)
+    (effects (font (size 1.27 1.27)) (justify left bottom))
   )
   (label "DRIVER_GLL[4..0]" (at 111.76 40.64 0)

Commit message: wip_cassette_scu
Other:
- removed sheet ram_cassette
Changed lines of the file:
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@@
-    (stroke (width 0) (type default) (color 0 0 0 0))
-  )
-  (wire (pts (xy 26.67 96.52) (xy 38.1 96.52))
     (stroke (width 0) (type default) (color 0 0 0 0))
   )
@@
   )
   (bus (pts (xy 125.73 38.1) (xy 132.08 38.1))
-    (stroke (width 0) (type default) (color 0 0 0 0))
-  )
-  (wire (pts (xy 74.93 96.52) (xy 81.28 96.52))
     (stroke (width 0) (type default) (color 0 0 0 0))
   )
@@
     (effects (font (size 1.27 1.27)) (justify left bottom))
   )
-  (label "~{RST}_WD" (at 26.67 96.52 0)
-    (effects (font (size 1.27 1.27)) (justify left bottom))
-  )
-  (hierarchical_label "PULL_UP1" (shape passive) (at 81.28 96.52 0)
-    (effects (font (size 1.27 1.27)) (justify left))
-  )
   (hierarchical_label "MAIN_D[23..0]" (shape bidirectional) (at 81.28 38.1 0)
     (effects (font (size 1.27 1.27)) (justify left))
@@
     )
   )
-  (sheet (at 38.1 93.98) (size 36.83 24.13) (fields_autoplaced)
-    (stroke (width 0.1524) (type solid) (color 0 0 0 0))
-    (fill (color 0 0 0 0.0000))
-    (property "Sheet name" "ram_cassette" (id 0) (at 38.1 93.2684 0)
-      (effects (font (size 1.27 1.27)) (justify left bottom))
-    )
-    (property "Sheet file" "ram_cassette.kicad_sch" (id 1) (at 38.1 118.6946 0)
-      (effects (font (size 1.27 1.27)) (justify left top))
-    )
-    (pin "PULL_UP1" passive (at 74.93 96.52 0)
-      (effects (font (size 1.27 1.27)) (justify right))
-    )
-    (pin "~{RST}_WD" input (at 38.1 96.52 180)
-      (effects (font (size 1.27 1.27)) (justify left))
-    )
-  )

Commit message: wip_cassette_sh2
Parts:
- added CP166, CP167, CP168, CP169: 1nF, symbol Device:C_Polarized_US
- added F12: 16103FPJ, symbol hitachi:16103FPJ
- added G8: DL-3529-GLL2, symbol capcom:DL-3529-GLL2
- added J11: DL-3429-GLL1, symbol capcom:DL-3429-GLL1
- added JP1: SolderJumper_2_Open, symbol Jumper:SolderJumper_2_Open
- added R10: 103, symbol Device:R_US
- added R68, R82: 184, symbol Device:R_US
- added R72: 153, symbol Device:R_US
- added R88, R90: 101, symbol Device:R_US
- added R93: 472Ω, symbol Device:R_US
- added R_US: 68KΩ, symbol Device:R_US
Connections:
- net 2GLL2CCU0: now also G8.74 (2GLL2CCU0)
- net 2GLL2IOU0: now also G8.75 (2GLL2IOU0)
- net 2GLL2PPU0: now also G8.64 (2GLL2PPU0)
- net BX_SPR: now also G8.57 (BX_SPR)
- net CLK_GLL1: now also J11.142 (CLK)
- net CLK_GLL2: now also G8.59 (CLK_GLL2)
- net GLL2IOU0: now also J11.143 (GLL2IOU0)
- net ~{CEA}: now also G8.48 (~{CEA})
- net ~{CEB}: now also G8.47 (~{CEB})
- net ~{CEC}: now also G8.45 (~{CEC})
- net ~{CED}: now also G8.44 (~{CED})
- net ~{CEE}: now also G8.43 (~{CEE})
- net ~{CEF}: now also G8.42 (~{CEF})
- net ~{CEG}: now also G8.40 (~{CEG})
- net ~{CEH}: now also G8.39 (~{CEH})
- net ~{CEI}: now also G8.38 (~{CEI})
- net ~{CEJ}: now also G8.37 (~{CEJ})
- net ~{CEK}: now also G8.35 (~{CEK})
- net ~{CEL}: now also G8.34 (~{CEL})
- net ~{CEM}: now also G8.32 (~{CEM})
- net ~{CEN}: now also G8.31 (~{CEN})
- net ~{CEO}: now also G8.30 (~{CEO})
- net ~{CEP}: now also G8.29 (~{CEP})
- net ~{CS}_GLL1: now also J11.116 (~{CS})
- net ~{MR}_GLL1: now also J11.121 (~{MR})
- net ~{OEB}: now also G8.17 (~{OEB})
- net ~{OEC}: now also G8.15 (~{OEC})
- net ~{OED}: now also G8.11 (~{OED})
- net ~{OEE}: now also G8.9 (~{OEE})
- net ~{RE}_GLL1: now also J11.118 (~{RE})
- net ~{RST}_WD: now also F12.17 (~{RES}), J11.78 (~{RESET})
- net ~{STBY_WD}: now also F12.19 (~{STBY})
- net ~{WEB}: now also G8.19 (~{WEB})
- net ~{WEC}: now also G8.16 (~{WEC})
- net ~{WED}: now also G8.14 (~{WED})
- net ~{WEE}: now also G8.10 (~{WEE})
- net ~{WE}_GLL1: now also J11.117 (~{WE})
- new net: F12.15 (VNMIadj), R_US.2
- new net: F12.5 (Rr), R82.1
- new net: F12.18 (VSYBYadj), R72.1
- new net: CP166.1, F12.3 (Rf), R68.1
- new net: J11.109 (GLL2CCU3), R88.1
- new net: R88.2, R90.1
- new net: CP169.1, F12.14 (CRES)
- new net: CP167.1, F12.4 (Cf)
- new net: CP168.1, F12.6 (Cr)
- new net: G8.63 (Jumper), JP1.2 (B), R10.2
- new net: J11.135 (PULL_UP), J11.140 (PULL_UP), R93.2
- new net 2GLL_A0: G8.66 (A0)
- new net 2GLL_A1: G8.67 (A1)
- new net 2GLL_A2: G8.68 (A2)
- new net 2GLL_A3: G8.69 (A3)
- new net 2GLL_A4: G8.70 (A4)
- new net 2GLL_A5: G8.72 (A5)
- new net DRIVER_GLL0: J11.138 (GLL_DRIVER0)
- new net DRIVER_GLL1: J11.123 (GLL_DRIVER1)
- new net DRIVER_GLL2: G8.61 (DRIVER_GLL2), J11.122 (GLL_DRIVER2)
- new net DRIVER_GLL3: J11.139 (GLL_DRIVER3)
- new net DRIVER_GLL4: J11.31 (GLL_DRIVER4)
- new net GFXC_D0: J11.66 (GFXC_D0)
- new net GFXC_D1: J11.65 (GFXC_D1)
- new net GFXC_D2: J11.64 (GFXC_D2)
- new net GFXC_D3: J11.63 (GFXC_D3)
- new net GFXC_D4: J11.62 (GFXC_D4)
- new net GFXC_D5: J11.61 (GFXC_D5)
- new net GFXC_D6: J11.60 (GFXC_D6)
- new net GFXC_D7: J11.59 (GFXC_D7)
- new net GFXD_D0: J11.75 (GFXD_D0)
- new net GFXD_D1: J11.74 (GFXD_D1)
- new net GFXD_D2: J11.73 (GFXD_D2)
- new net GFXD_D3: J11.72 (GFXD_D3)
- new net GFXD_D4: J11.71 (GFXD_D4)
- new net GFXD_D5: J11.70 (GFXD_D5)
- new net GFXD_D6: J11.69 (GFXD_D6)
- new net GFXD_D7: J11.68 (GFXD_D7)
- new net GLL2CCU0: J11.79 (GLL2CCU0)
- new net GLL2CCU1: J11.56 (GLL2CCU1)
- new net GLL2CCU2: J11.108 (GLL2CCU2)
- new net GLL2CCU3: R90.2
- new net GLL2CCU4: J11.129 (GLL2CCU4)
- new net GLL2CCU5: J11.134 (GLL2CCU5)
- new net GLL_A0: J11.80 (GLL_A0)
- new net GLL_A1: J11.81 (GLL_A1)
- new net GLL_A10: J11.92 (GLL_A10)
- new net GLL_A11: J11.93 (GLL_A11)
- new net GLL_A12: J11.94 (GLL_A12)
- new net GLL_A13: J11.95 (GLL_A13)
- new net GLL_A14: J11.96 (GLL_A14)
- new net GLL_A15: J11.97 (GLL_A15)
- new net GLL_A16: J11.98 (GLL_A16)
- new net GLL_A17: J11.100 (GLL_A17)
- new net GLL_A18: J11.101 (GLL_A18)
- new net GLL_A19: J11.102 (GLL_A19)
- new net GLL_A2: J11.82 (GLL_A2)
- new net GLL_A20: J11.103 (GLL_A20)
- new net GLL_A3: J11.83 (GLL_A3)
- new net GLL_A4: J11.84 (GLL_A4)
- new net GLL_A5: J11.85 (GLL_A5)
- new net GLL_A6: J11.86 (GLL_A6)
- new net GLL_A7: J11.87 (GLL_A7)
- new net GLL_A8: J11.88 (GLL_A8)
- new net GLL_A9: J11.89 (GLL_A9)
- new net GLL_D0: J11.104 (GLL_D0)
- new net GLL_D1: J11.105 (GLL_D1)
- new net GLL_D2: J11.106 (GLL_D2)
- new net GLL_D3: J11.111 (GLL_D3)
- new net GLL_D4: J11.112 (GLL_D4)
- new net GLL_D5: J11.113 (GLL_D5)
- new net GLL_D6: J11.114 (GLL_D6)
- new net GLL_D7: J11.128 (GLL_D7)
- new net MAIN_A0: J11.35 (MAIN_A0)
- new net MAIN_A1: J11.36 (MAIN_A1)
- new net MAIN_A10: J11.8 (MAIN_A10)
- new net MAIN_A11: J11.29 (MAIN_A11)
- new net MAIN_A12: J11.30 (MAIN_A12)
- new net MAIN_A13: J11.32 (MAIN_A13)
- new net MAIN_A14: J11.57 (MAIN_A14)
- new net MAIN_A15: J11.137 (MAIN_A15)
- new net MAIN_A16: J11.132 (MAIN_A16)
- new net MAIN_A17: J11.131 (MAIN_A17)
- new net MAIN_A18: J11.133 (MAIN_A18)
- new net MAIN_A19: J11.5 (MAIN_A19)
- new net MAIN_A2: J11.37 (MAIN_A2)
- new net MAIN_A20: J11.4 (MAIN_A20)
- new net MAIN_A3: J11.38 (MAIN_A3)
- new net MAIN_A4: J11.39 (MAIN_A4)
- new net MAIN_A5: J11.41 (MAIN_A5)
- new net MAIN_A6: J11.42 (MAIN_A6)
- new net MAIN_A7: J11.43 (MAIN_A7)
- new net MAIN_A8: J11.6 (MAIN_A8)
- new net MAIN_A9: J11.7 (MAIN_A9)
- new net MAIN_D0: J11.53 (MAIN_D0)
- new net MAIN_D1: J11.52 (MAIN_D1)
- new net MAIN_D10: J11.26 (MAIN_D10)
- new net MAIN_D11: J11.24 (MAIN_D11)
- new net MAIN_D12: J11.23 (MAIN_D12)
- new net MAIN_D13: J11.22 (MAIN_D13)
- new net MAIN_D14: J11.21 (MAIN_D14)
- new net MAIN_D15: J11.20 (MAIN_D15)
- new net MAIN_D16: J11.17 (MAIN_D16)
- new net MAIN_D17: J11.16 (MAIN_D17)
- new net MAIN_D18: J11.15 (MAIN_D18)
- new net MAIN_D19: J11.14 (MAIN_D19)
- new net MAIN_D2: J11.51 (MAIN_D2)
- new net MAIN_D20: J11.13 (MAIN_D20)
- new net MAIN_D21: J11.12 (MAIN_D21)
- new net MAIN_D22: J11.11 (MAIN_D22)
- new net MAIN_D23: J11.10 (MAIN_D23)
- new net MAIN_D3: J11.50 (MAIN_D3)
- new net MAIN_D4: J11.49 (MAIN_D4)
- new net MAIN_D5: J11.48 (MAIN_D5)
- new net MAIN_D6: J11.46 (MAIN_D6)
- new net MAIN_D7: J11.45 (MAIN_D7)
- new net MAIN_D8: J11.28 (MAIN_D8)
- new net MAIN_D9: J11.27 (MAIN_D9)
- new net VCC: F12.12 (Vcont), F12.13 (VCC), F12.9 (Vout), G8.51 (VCC), G8.52 (VCC), G8.58 (VCC), G8.60 (VCC), G8.62 (VCC), G8.65 (VCC), G8.71 (VCC), G8.73 (VCC), G8.76 (VCC), J11.18 (VCC), J11.19 (VCC), J11.25 (VCC), J11.34 (VCC), J11.40 (VCC), J11.44 (VCC), J11.47 (VCC), J11.54 (VCC), J11.55 (VCC), J11.58 (VCC), J11.76 (VCC), J11.77 (VCC), J11.9 (VCC), R10.1, R93.1, R_US.1
- new net VSS: CP166.2, CP167.2, CP168.2, CP169.2, F12.2 (P-RUN), F12.7 (VSS), G8.1 (VSS), G8.12 (VSS), G8.13 (VSS), G8.18 (VSS), G8.23 (VSS), G8.27 (VSS), G8.33 (VSS), G8.36 (VSS), G8.41 (VSS), G8.46 (VSS), G8.6 (VSS), J11.1 (VSS), J11.107 (VSS), J11.110 (VSS), J11.115 (VSS), J11.120 (VSS), J11.126 (VSS), J11.127 (VSS), J11.130 (VSS), J11.136 (VSS), J11.141 (VSS), J11.144 (VSS), J11.33 (VSS), J11.67 (VSS), J11.90 (VSS), J11.91 (VSS), J11.99 (VSS), JP1.1 (A), R68.2, R72.2, R82.2
- new net ~{RESET0}: G8.2 (~{RESET0})
- new net ~{RESET1}: G8.3 (~{RESET1})
- new net ~{RESET2}: G8.80 (~{RESET2})
- new net ~{RESET3}: G8.79 (~{RESET3})
- new net ~{RESET4}: G8.78 (~{RESET4})
- no-connect marks 0 -> 8
Other:
- removed sheet gll1
- removed sheet gll2
- note added: "42.9545MHz"
- note added: "CONNECTED TO SLOT 7. THIS SLOT HAS NO SIMM."
- note added: "CUT PIN"
- note added: "Data bus and addresses. There is no certainty of the order."
- note added: "GRAPHIC LAYER LAYOUT 1"
- note added: "GRAPHIC LAYER LAYOUT 2"
- note added: "NOT MOUNTED"
- note added: "Square wave clk"
- note added: "WATCHDOG TIMER"
- note removed: "OK"

Commit message: wip_cst_ccu
Other:
- moved on the sheet: CP166, CP167, CP168, CP169, R68, R82

Commit message: correction_ppu
Connections:
- net ~{RESET1}: now also G8.1 (~{RESET1}); no longer G8.3 (~{RESET1})
- net GLL_A0 renamed RD/~{WR}_CPUC
- net GLL_A1 renamed CPUC_A23
- net GLL_A10 renamed CPUC_A14
- net GLL_A11 renamed CPUC_A13
- net GLL_A12 renamed CPUC_A12
- net GLL_A13 renamed CPUC_A11
- net GLL_A14 renamed CPUC_A10
- net GLL_A15 renamed CPUC_A9
- net GLL_A16 renamed CPUC_A8
- net GLL_A17 renamed CPUC_A7
- net GLL_A18 renamed CPUC_A6
- net GLL_A19 renamed CPUC_A5
- net GLL_A2 renamed CPUC_A22
- net GLL_A20 renamed CPUC_A4
- net GLL_A3 renamed CPUC_A21
- net GLL_A4 renamed CPUC_A20
- net GLL_A5 renamed CPUC_A19
- net GLL_A6 renamed CPUC_A18
- net GLL_A7 renamed CPUC_A17
- net GLL_A8 renamed CPUC_A16
- net GLL_A9 renamed CPUC_A15
- net GLL_D0 renamed CPUC_A3
- net GLL_D1 renamed CPUC_A2
- net GLL_D2 renamed CPUC_A1
- net GLL_D3 renamed ~{IRL3}_CPUC
- net GLL_D4 renamed ~{IRL2}_CPUC
- net GLL_D5 renamed ~{IRL1}_CPUC
- net GLL_D6 renamed ~{IRL0}_CPUC
- net GLL_D7 renamed ~{RST}_CPUC
- removed net ~{RESET0}: G8.2 (~{RESET0})
- no-connect marks 8 -> 9
Other:
- note added: "SIMM 7 NOT MOUNTED"
- note removed: "42.9545MHz"
- note removed: "Data bus and addresses. There is no certainty of the order."

Commit message: wip_cre_cps3
Connections:
- net MAIN_D16 is gone; now on net MAIN_A16: J11.17 (MAIN_A16)
- net MAIN_D17 is gone; now on net MAIN_A17: J11.16 (MAIN_A17)
- net MAIN_D18 is gone; now on net MAIN_A18: J11.15 (MAIN_A18)
- net MAIN_D19 is gone; now on net MAIN_A19: J11.14 (MAIN_A19)
- net MAIN_D20 is gone; now on net MAIN_A20: J11.13 (MAIN_A20)
- net MAIN_A0: now also J11.133 (MAIN_A0); no longer J11.35 (MAIN_A0)
- net MAIN_A1: now also J11.131 (MAIN_A1); no longer J11.36 (MAIN_A1)
- net MAIN_A10: now also J11.26 (MAIN_A10); no longer J11.8 (MAIN_A10)
- net MAIN_A11: now also J11.24 (MAIN_A11); no longer J11.29 (MAIN_A11)
- net MAIN_A12: now also J11.23 (MAIN_A12); no longer J11.30 (MAIN_A12)
- net MAIN_A13: now also J11.22 (MAIN_A13); no longer J11.32 (MAIN_A13)
- net MAIN_A14: now also J11.21 (MAIN_A14); no longer J11.57 (MAIN_A14)
- net MAIN_A15: now also J11.20 (MAIN_A15); no longer J11.137 (MAIN_A15)
- net MAIN_A16: no longer J11.132 (MAIN_A16)
- net MAIN_A17: no longer J11.131 (MAIN_A17)
- net MAIN_A18: no longer J11.133 (MAIN_A18)
- net MAIN_A19: no longer J11.5 (MAIN_A19)
- net MAIN_A2: now also J11.132 (MAIN_A2); no longer J11.37 (MAIN_A2)
- net MAIN_A20: no longer J11.4 (MAIN_A20)
- net MAIN_A3: now also J11.137 (MAIN_A3); no longer J11.38 (MAIN_A3)
- net MAIN_A4: now also J11.57 (MAIN_A5); no longer J11.39 (MAIN_A4)
- net MAIN_A5: now also J11.32 (MAIN_A4); no longer J11.41 (MAIN_A5)
- net MAIN_A6: now also J11.30 (MAIN_A6); no longer J11.42 (MAIN_A6)
- net MAIN_A7: now also J11.29 (MAIN_A7); no longer J11.43 (MAIN_A7)
- net MAIN_A8: now also J11.28 (MAIN_A8); no longer J11.6 (MAIN_A8)
- net MAIN_A9: now also J11.27 (MAIN_A9); no longer J11.7 (MAIN_A9)
- net MAIN_D10: now also J11.41 (MAIN_D10); no longer J11.26 (MAIN_D10)
- net MAIN_D11: now also J11.39 (MAIN_D11); no longer J11.24 (MAIN_D11)
- net MAIN_D12: now also J11.38 (MAIN_D12); no longer J11.23 (MAIN_D12)
- net MAIN_D13: now also J11.37 (MAIN_D13); no longer J11.22 (MAIN_D13)
- net MAIN_D14: now also J11.36 (MAIN_D14); no longer J11.21 (MAIN_D14)
- net MAIN_D15: now also J11.35 (MAIN_D15); no longer J11.20 (MAIN_D15)
- net MAIN_D8: now also J11.43 (MAIN_D8); no longer J11.28 (MAIN_D8)
- net MAIN_D9: now also J11.42 (MAIN_D9); no longer J11.27 (MAIN_D9)
- net ~{RST}_WD: no longer F12.17 (~{RES})
- net MAIN_D21 renamed MAIN_A21
- net MAIN_D22 renamed MAIN_A22
- net MAIN_D23 renamed MAIN_A23
- new net MAIN_A24: J11.8 (MAIN_A24)
- new net MAIN_A25: J11.7 (MAIN_A25)
- new net MAIN_A26: J11.6 (MAIN_A26)
- new net MAIN_A27: J11.5 (MAIN_A27)
- new net MAIN_A28: J11.4 (MAIN_A28)
- no-connect marks 9 -> 10
Other:
- note added: "~{RST}_WD"

Commit message: cps3_finished
Parts:
- renumbered R_US to R203
Changed lines of the file:
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@@
     (company "JOTEGO")
     (comment 1 "E.Triana")
+    (comment 2 "14/10/22-30/01/23")
   )
   (junction (at 97.79 62.23) (diameter 0) (color 0 0 0 0)
@@
     (stroke (width 0) (type default) (color 0 0 0 0))
   )
-  (bus_entry (at 214.63 135.89) (size 2.54 -2.54)
-    (stroke (width 0) (type default) (color 0 0 0 0))
-  )
   (bus_entry (at 364.49 77.47) (size 2.54 2.54)
     (stroke (width 0) (type default) (color 0 0 0 0))
@@
     (stroke (width 0) (type default) (color 0 0 0 0))
   )
-  (bus_entry (at 214.63 133.35) (size 2.54 -2.54)
-    (stroke (width 0) (type default) (color 0 0 0 0))
-  )
   (bus_entry (at 115.57 50.8) (size -2.54 2.54)
     (stroke (width 0) (type default) (color 0 0 0 0))
@@
     (stroke (width 0) (type default) (color 0 0 0 0))
   )
-  (bus_entry (at 214.63 140.97) (size 2.54 -2.54)
-    (stroke (width 0) (type default) (color 0 0 0 0))
-  )
-  (bus_entry (at 214.63 143.51) (size 2.54 -2.54)
-    (stroke (width 0) (type default) (color 0 0 0 0))
-  )
   (bus_entry (at 71.12 87.63) (size 2.54 2.54)
     (stroke (width 0) (type default) (color 0 0 0 0))
@@
     (stroke (width 0) (type default) (color 0 0 0 0))
   )
-  (bus_entry (at 214.63 138.43) (size 2.54 -2.54)
-    (stroke (width 0) (type default) (color 0 0 0 0))
-  )
   (bus_entry (at 214.63 102.87) (size 2.54 -2.54)
     (stroke (width 0) (type default) (color 0 0 0 0))
@@
     (stroke (width 0) (type default) (color 0 0 0 0))
   )
-  (bus (pts (xy 217.17 138.43) (xy 217.17 135.89))
-    (stroke (width 0) (type default) (color 0 0 0 0))
-  )
-  (wire (pts (xy 196.85 140.97) (xy 214.63 140.97))
-    (stroke (width 0) (type default) (color 0 0 0 0))
-  )
   (bus (pts (xy 176.53 50.8) (xy 179.07 50.8))
     (stroke (width 0) (type default) (color 0 0 0 0))
@@
     (stroke (width 0) (type default) (color 0 0 0 0))
   )
-  (bus (pts (xy 217.17 130.81) (xy 222.25 130.81))
-    (stroke (width 0) (type default) (color 0 0 0 0))
-  )
   (bus (pts (xy 71.12 102.87) (xy 71.12 105.41))
     (stroke (width 0) (type default) (color 0 0 0 0))
@@
     (stroke (width 0) (type default) (color 0 0 0 0))
   )
-  (bus (pts (xy 217.17 133.35) (xy 217.17 130.81))
-    (stroke (width 0) (type default) (color 0 0 0 0))
-  )
-  (wire (pts (xy 196.85 135.89) (xy 214.63 135.89))
-    (stroke (width 0) (type default) (color 0 0 0 0))
-  )
   (wire (pts (xy 146.05 53.34) (xy 146.05 62.23))
     (stroke (width 0) (type default) (color 0 0 0 0))
@@
     (stroke (width 0) (type default) (color 0 0 0 0))
   )
-  (bus (pts (xy 217.17 140.97) (xy 217.17 138.43))
-    (stroke (width 0) (type default) (color 0 0 0 0))
-  )
   (wire (pts (xy 307.34 158.75) (xy 309.88 158.75))
     (stroke (width 0) (type default) (color 0 0 0 0))
@@
     (stroke (width 0) (type default) (color 0 0 0 0))
   )
+  (wire (pts (xy 196.85 133.35) (xy 204.47 133.35))
+    (stroke (width 0) (type default) (color 0 0 0 0))
+  )
   (wire (pts (xy 158.75 168.91) (xy 158.75 171.45))
     (stroke (width 0) (type default) (color 0 0 0 0))
@@
     (stroke (width 0) (type default) (color 0 0 0 0))
   )
-  (wire (pts (xy 196.85 133.35) (xy 214.63 133.35))
-    (stroke (width 0) (type default) (color 0 0 0 0))
-  )
   (bus (pts (xy 63.5 82.55) (xy 71.12 82.55))
     (stroke (width 0) (type default) (color 0 0 0 0))
@@
     (stroke (width 0) (type default) (color 0 0 0 0))
   )
+  (wire (pts (xy 196.85 138.43) (xy 204.47 138.43))
+    (stroke (width 0) (type default) (color 0 0 0 0))
+  )
   (wire (pts (xy 85.09 74.93) (xy 85.09 72.39))
     (stroke (width 0) (type default) (color 0 0 0 0))
@@
     (stroke (width 0) (type default) (color 0 0 0 0))
   )
+  (wire (pts (xy 196.85 140.97) (xy 204.47 140.97))
+    (stroke (width 0) (type default) (color 0 0 0 0))
+  )
   (wire (pts (xy 345.44 146.05) (xy 356.87 146.05))
     (stroke (width 0) (type default) (color 0 0 0 0))
@@
     (stroke (width 0) (type default) (color 0 0 0 0))
   )
-  (bus (pts (xy 217.17 135.89) (xy 217.17 133.35))
-    (stroke (width 0) (type default) (color 0 0 0 0))
-  )
   (wire (pts (xy 345.44 140.97) (xy 356.87 140.97))
     (stroke (width 0) (type default) (color 0 0 0 0))
@@
     (stroke (width 0) (type default) (color 0 0 0 0))
   )
-  (wire (pts (xy 196.85 143.51) (xy 214.63 143.51))
-    (stroke (width 0) (type default) (color 0 0 0 0))
-  )
   (wire (pts (xy 85.09 59.69) (xy 85.09 62.23))
     (stroke (width 0) (type default) (color 0 0 0 0))
@@
     (stroke (width 0) (type default) (color 0 0 0 0))
   )
+  (wire (pts (xy 196.85 135.89) (xy 204.47 135.89))
+    (stroke (width 0) (type default) (color 0 0 0 0))
+  )
   (wire (pts (xy 196.85 120.65) (xy 214.63 120.65))
     (stroke (width 0) (type default) (color 0 0 0 0))
@@
     (stroke (width 0) (type default) (color 0 0 0 0))
   )
-  (wire (pts (xy 196.85 138.43) (xy 214.63 138.43))
-    (stroke (width 0) (type default) (color 0 0 0 0))
-  )
   (wire (pts (xy 73.66 105.41) (xy 85.09 105.41))
     (stroke (width 0) (type default) (color 0 0 0 0))
@@
   )
   (wire (pts (xy 135.89 184.15) (xy 135.89 168.91))
+    (stroke (width 0) (type default) (color 0 0 0 0))
+  )
+  (wire (pts (xy 196.85 143.51) (xy 204.47 143.51))
     (stroke (width 0) (type default) (color 0 0 0 0))
   )
@@
     (effects (font (size 1.27 1.27)) (justify left bottom))
   )
-  (label "DRIVER_GLL1" (at 214.63 135.89 180)
-    (effects (font (size 1.27 1.27)) (justify right bottom))
-  )
   (label "VSS" (at 162.56 262.89 0)
     (effects (font (size 1.27 1.27)) (justify left bottom))
@@
     (effects (font (size 1.27 1.27)) (justify left bottom))
   )
-  (label "DRIVER_GLL4" (at 214.63 143.51 180)
-    (effects (font (size 1.27 1.27)) (justify right bottom))
-  )
   (label "GFXD_D0" (at 204.47 113.03 0)
     (effects (font (size 1.27 1.27)) (justify left bottom))
@@
     (effects (font (size 1.27 1.27)) (justify left bottom))
   )
-  (label "DRIVER_GLL3" (at 214.63 140.97 180)
-    (effects (font (size 1.27 1.27)) (justify right bottom))
-  )
   (label "MAIN_D15" (at 73.66 123.19 0)
     (effects (font (size 1.27 1.27)) (justify left bottom))
@@
     (effects (font (size 1.27 1.27)) (justify right bottom))
   )
-  (label "DRIVER_GLL0" (at 214.63 133.35 180)
-    (effects (font (size 1.27 1.27)) (justify right bottom))
-  )
   (label "MAIN_A22" (at 163.83 62.23 90)
     (effects (font (size 1.27 1.27)) (justify left bottom))
@@
     (effects (font (size 1.27 1.27)) (justify left bottom))
   )
-  (label "DRIVER_GLL2" (at 214.63 138.43 180)
-    (effects (font (size 1.27 1.27)) (justify right bottom))
-  )
   (label "CPUC_A12" (at 123.19 179.07 90)
     (effects (font (size 1.27 1.27)) (justify left bottom))
@@
   (label "CPUC_A7" (at 110.49 179.07 90)
     (effects (font (size 1.27 1.27)) (justify left bottom))
+  )
+  (hierarchical_label "DRIVER_GLL0" (shape output) (at 204.47 133.35 0)
+    (effects (font (size 1.27 1.27)) (justify left))
   )
   (hierarchical_label "MAIN_D[15..0]" (shape bidirectional) (at 63.5 82.55 180)
@@
     (effects (font (size 1.27 1.27)) (justify left))
   )
+  (hierarchical_label "DRIVER_GLL3" (shape output) (at 204.47 140.97 0)
+    (effects (font (size 1.27 1.27)) (justify left))
+  )
   (hierarchical_label "~{IRL2}_CPUC" (shape input) (at 158.75 171.45 270)
     (effects (font (size 1.27 1.27)) (justify right))
   )
+  (hierarchical_label "DRIVER_GLL4" (shape output) (at 204.47 143.51 0)
+    (effects (font (size 1.27 1.27)) (justify left))
+  )
   (hierarchical_label "~{WED}" (shape output) (at 356.87 140.97 0)
     (effects (font (size 1.27 1.27)) (justify left))
@@
     (effects (font (size 1.27 1.27)) (justify left))
   )
-  (hierarchical_label "DRIVER_GLL[4..0]" (shape output) (at 222.25 130.81 0)
-    (effects (font (size 1.27 1.27)) (justify left))
-  )
   (hierarchical_label "~{WEC}" (shape output) (at 356.87 135.89 0)
     (effects (font (size 1.27 1.27)) (justify left))
   )
   (hierarchical_label "~{OEE}" (shape output) (at 356.87 148.59 0)
+    (effects (font (size 1.27 1.27)) (justify left))
+  )
+  (hierarchical_label "DRIVER_GLL1" (shape output) (at 204.47 135.89 0)
     (effects (font (size 1.27 1.27)) (justify left))
   )
@@
     (effects (font (size 1.27 1.27)) (justify left))
   )
+  (hierarchical_label "DRIVER_GLL2" (shape output) (at 204.47 138.43 0)
+    (effects (font (size 1.27 1.27)) (justify left))
+  )
   (hierarchical_label "CLK_GLL1" (shape output) (at 204.47 72.39 0)
     (effects (font (size 1.27 1.27)) (justify left))
@@
   (symbol (lib_id "Device:R_US") (at 82.55 229.87 0) (mirror y) (unit 1)
     (in_bom yes) (on_board yes)
-    (property "Reference" "R_US" (id 0) (at 77.47 228.6 0))
+    (property "Reference" "R203" (id 0) (at 77.47 228.6 0))
     (property "Value" "68KΩ" (id 1) (at 77.47 231.14 0))
     (property "Footprint" "" (id 2) (at 81.534 230.124 90)
@@
       (effects (font (size 3.81 3.81)))
     )
-    (property "Footprint" "" (id 2) (at 142.24 116.84 0)
+    (property "Footprint" "" (id 2) (at 142.24 125.73 0)
       (effects (font (size 1.27 1.27)) hide)
     )
-    (property "Datasheet" "" (id 3) (at 142.24 116.84 0)
+    (property "Datasheet" "" (id 3) (at 142.24 125.73 0)
       (effects (font (size 1.27 1.27)) hide)
     )
