File: cores/cps3/sch/ram_cassette.kicad_sch (KiCad schematic)
At the start: 1 part

Commit message: wip_iou_wd
Connections:
- net GLL2RC0 renamed ~{RST_WD}
Other:
- company: (none) -> JOTEGO
- title: (none) -> CP SYSTEM III
Changed lines of the file:
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@@
 (kicad_sch (version 20211123) (generator eeschema)
   (paper "A4")
+  (title_block
+    (title "CP SYSTEM III")
+    (date "14/10/22")
+    (rev "José Tejada G.")
+    (company "JOTEGO")
+    (comment 1 "E.Triana")
+  )
   (junction (at 30.48 173.99) (diameter 0) (color 0 0 0 0)
   )
@@
     (effects (font (size 1.27 1.27)) (justify left))
   )
-  (hierarchical_label "GLL2RC0" (shape input) (at 49.53 92.71 0)
+  (hierarchical_label "~{RST_WD}" (shape input) (at 49.53 92.71 0)
     (effects (font (size 1.27 1.27)) (justify left))
   )

Commit message: wip_ccu_gll2_cassette
Parts:
- added U? (x10): 7400, symbol jt74:7400
- added U?: 29F400TA-90PF, symbol arcade:29F400TA-90PF
- added Y?: Crystal, symbol Device:Crystal
Connections:
- net VCC: now also U?.14 (VCC), U?.14 (VCC)
- net VSS: now also U?.7 (VSS), U?.7 (VSS)
Other:
- note added: "6.25SC6L"

Commit message: wip_cassette
Parts:
- added CP174, CP175, CP176: 10μF, symbol Device:C_Polarized_US
- added R2: 105, symbol Device:R_US
- added R20: 103, symbol Device:R_US
- added U3-SCU: HD6417604F28_SH2, symbol arcade:HD6417604F28_SH2
- gave numbers to parts that had none: 3
Connections:
- net VCC: now also U?.10 (Pin_10), U?.108 (Pin_108), U?.118 (Pin_118), U?.120 (Pin_120), U?.16 (Pin_16), U?.2, U?.26 (Pin_26), U?.36 (Pin_36), U?.46 (Pin_46), U?.54 (Pin_54), U?.6, U?.60 (Pin_60), U?.68 (Pin_68), U?.74 (Pin_74), U?.78 (Pin_78), U?.80 (Pin_80), U?.88 (Pin_88), U?.98 (Pin_98), CP176.1, U3-SCU.104 (VCC), U3-SCU.112 (~{CKPREQ}/CKM), U3-SCU.113 (VCC), U3-SCU.12 (VCC), U3-SCU.123 (VCC), U3-SCU.132 (VCC), U3-SCU.139 (VCC), U3-SCU.18 (VCC), U3-SCU.24 (VCC), U3-SCU.4 (VCC), U3-SCU.40 (VCC), U3-SCU.48 (VCC), U3-SCU.54 (VCC), U3-SCU.60 (VCC), U3-SCU.67 (VCC), U3-SCU.84 (VCC), U3-SCU.96 (VCC); no longer U?.107 (Pin_107), U?.117 (Pin_117), U?.119 (Pin_119), U?.15 (Pin_15), U?.25 (Pin_25), U?.35 (Pin_35), U?.45 (Pin_45), U?.5 (Pin_5), U?.51 (Pin_51), U?.55 (Pin_55), U?.57 (Pin_57), U?.61 (Pin_61), U?.69 (Pin_69), U?.75 (Pin_75), U?.79 (Pin_79), U?.87 (Pin_87), U?.97 (Pin_97)
- net VSS: now also U?.107 (Pin_107), U?.117 (Pin_117), U?.119 (Pin_119), U?.15 (Pin_15), U?.25 (Pin_25), U?.35 (Pin_35), U?.45 (Pin_45), U?.5 (Pin_5), U?.51 (Pin_51), U?.55 (Pin_55), U?.57 (Pin_57), U?.61 (Pin_61), U?.69 (Pin_69), U?.75 (Pin_75), U?.79 (Pin_79), U?.87 (Pin_87), U?.97 (Pin_97), CP174.2, CP175.2, U3-SCU.106 (VSS), U3-SCU.115 (VSS), U3-SCU.121 (VSS), U3-SCU.134 (VSS), U3-SCU.14 (VSS), U3-SCU.141 (VSS), U3-SCU.20 (VSS), U3-SCU.26 (VSS), U3-SCU.33 (VSS), U3-SCU.42 (VSS), U3-SCU.50 (VSS), U3-SCU.56 (VSS), U3-SCU.6 (VSS), U3-SCU.62 (VSS), U3-SCU.69 (VSS), U3-SCU.78 (VSS), U3-SCU.86 (VSS), U3-SCU.91 (VSS), U3-SCU.98 (VSS); no longer U?.10 (Pin_10), U?.108 (Pin_108), U?.118 (Pin_118), U?.120 (Pin_120), U?.2, U?.26 (Pin_26), U?.36 (Pin_36), U?.46 (Pin_46), U?.54 (Pin_54), U?.6, U?.60 (Pin_60), U?.68 (Pin_68), U?.74 (Pin_74), U?.78 (Pin_78), U?.80 (Pin_80), U?.88 (Pin_88), U?.98 (Pin_98)
- net at U1.6: now also U3-SCU.89 (~{WAIT})
- net at X1.1: now also CP175.1, R2.1, U3-SCU.116 (XTAL)
- net at X1.2: now also CP174.1, R2.2, U3-SCU.114 (EXTAL)
- net at U4.8: now also U3-SCU.122 (~{RESET})
- net ~{CE}R_CST: now reaches U?.26 (~{CE})
- new net: CP176.2, R20.2
- new net: R20.1, U3-SCU.125 (NMI)
- new net CAP1: U3-SCU.108 (CAP1)
- new net CAP2: U3-SCU.109 (CAP2)
- new net CKE: U3-SCU.88 (CKE)
- new net CKIO_SCU: U3-SCU.118 (CKIO)
- new net DACK0: U3-SCU.66 (DACK0)
- new net DACK1: U3-SCU.68 (DACK1)
- new net DREQ0: U3-SCU.70 (DREQ0)
- new net DREQ1: U3-SCU.71 (DREQ1)
- new net FTCI: U3-SCU.100 (FTCI)
- new net FTI: U3-SCU.99 (FTI)
- new net FTOA: U3-SCU.97 (FTOA)
- new net FTOB: U3-SCU.95 (FTOB)
- new net MD0: U3-SCU.105 (MD0)
- new net MD1: U3-SCU.107 (MD1)
- new net MD2: U3-SCU.110 (MD2)
- new net MD3: U3-SCU.117 (MD3)
- new net MD4: U3-SCU.119 (MD4)
- new net MD5: U3-SCU.120 (MD5)
- new net RxD: U3-SCU.101 (RxD)
- new net SCK: U3-SCU.103 (SCK)
- new net SCU_A0: U3-SCU.30 (A0)
- new net SCU_A1: U3-SCU.31 (A1)
- new net SCU_A10: U3-SCU.43 (A10)
- new net SCU_A11: U3-SCU.44 (A11)
- new net SCU_A12: U3-SCU.45 (A12)
- new net SCU_A13: U3-SCU.46 (A13)
- new net SCU_A14: U3-SCU.47 (A14)
- new net SCU_A15: U3-SCU.49 (A15)
- new net SCU_A16: U3-SCU.51 (A16)
- new net SCU_A17: U3-SCU.52 (A17)
- new net SCU_A18: U3-SCU.53 (A18)
- new net SCU_A19: U3-SCU.55 (A19)
- new net SCU_A2: U3-SCU.32 (A2)
- new net SCU_A20: U3-SCU.57 (A20)
- new net SCU_A21: U3-SCU.58 (A21)
- new net SCU_A22: U3-SCU.59 (A22)
- new net SCU_A23: U3-SCU.61 (A23)
- new net SCU_A24: U3-SCU.63 (A24)
- new net SCU_A25: U3-SCU.64 (A25)
- new net SCU_A26: U3-SCU.65 (A26)
- new net SCU_A3: U3-SCU.34 (A3)
- new net SCU_A4: U3-SCU.35 (A4)
- new net SCU_A5: U3-SCU.36 (A5)
- new net SCU_A6: U3-SCU.37 (A6)
- new net SCU_A7: U3-SCU.38 (A7)
- new net SCU_A8: U3-SCU.39 (A8)
- new net SCU_A9: U3-SCU.41 (A9)
- new net SCU_D0: U3-SCU.130 (D0)
- new net SCU_D1: U3-SCU.131 (D1)
- new net SCU_D10: U3-SCU.144 (D10)
- new net SCU_D11: U3-SCU.1 (D11)
- new net SCU_D12: U3-SCU.2 (D12)
- new net SCU_D13: U3-SCU.3 (D13)
- new net SCU_D14: U3-SCU.5 (D14)
- new net SCU_D15: U3-SCU.7 (D15)
- new net SCU_D16: U3-SCU.8 (D16)
- new net SCU_D17: U3-SCU.9 (D17)
- new net SCU_D18: U3-SCU.10 (D18)
- new net SCU_D19: U3-SCU.11 (D19)
- new net SCU_D2: U3-SCU.133 (D2)
- new net SCU_D20: U3-SCU.13 (D20)
- new net SCU_D21: U3-SCU.15 (D21)
- new net SCU_D22: U3-SCU.16 (D22)
- new net SCU_D23: U3-SCU.17 (D23)
- new net SCU_D24: U3-SCU.19 (D24)
- new net SCU_D25: U3-SCU.21 (D25)
- new net SCU_D26: U3-SCU.22 (D26)
- new net SCU_D27: U3-SCU.23 (D27)
- new net SCU_D28: U3-SCU.25 (D28)
- new net SCU_D29: U3-SCU.27 (D29)
- new net SCU_D3: U3-SCU.135 (D3)
- new net SCU_D30: U3-SCU.28 (D30)
- new net SCU_D31: U3-SCU.29 (D31)
- new net SCU_D4: U3-SCU.136 (D4)
- new net SCU_D5: U3-SCU.137 (D5)
- new net SCU_D6: U3-SCU.138 (D6)
- new net SCU_D7: U3-SCU.140 (D7)
- new net SCU_D8: U3-SCU.142 (D8)
- new net SCU_D9: U3-SCU.143 (D9)
- new net TxD: U3-SCU.102 (TxD)
- new net ~{BACK}/~{BRLS}: U3-SCU.92 (~{BACK}/~{BRLS})
- new net ~{BREQ}/~{BGR}: U3-SCU.93 (~{BREQ}/~{BGR})
- new net ~{BS}: U3-SCU.76 (~{BS})
- new net ~{CASLL}/DQMLL/~{WE0}: U3-SCU.85 (~{CASLL}/DQMLL/~{WE0})
- new net ~{CASLL}/DQMLL/~{WE1}: U3-SCU.83 (~{CASHH}/DQMUU/~{WE1})
- new net ~{CASLL}/DQMLL/~{WE2}: U3-SCU.82 (~{CASHH}/DQMUU/~{WE2})
- new net ~{CASLL}/DQMLL/~{WE3}: U3-SCU.81 (~{CASHH}/DQMUU/~{WE3})
- new net ~{CAS}/~{OE}: U3-SCU.80 (~{CAS}/~{OE})
- new net ~{CKPACK}: U3-SCU.111 (~{CKPACK})
- new net ~{CS0}: U3-SCU.72 (~{CS0})
- new net ~{CS1}: U3-SCU.73 (~{CS1})
- new net ~{CS2}: U3-SCU.74 (~{CS2})
- new net ~{CS3}: U3-SCU.75 (~{CS3})
- new net ~{IRL0}: U3-SCU.129 (~{IRL0})
- new net ~{IRL1}: U3-SCU.128 (~{IRL1})
- new net ~{IRL2}: U3-SCU.127 (~{IRL2})
- new net ~{IRL3}: U3-SCU.126 (~{IRL3})
- new net ~{IVECF}: U3-SCU.124 (~{IVECF})
- new net ~{RAS}/~{CE}: U3-SCU.79 (~{RAS}/~{CE})
- new net ~{RD}: U3-SCU.87 (~{RD})
- new net ~{RD}/~{WR}: U3-SCU.77 (RD/~{WR})
- new net ~{WDTOVF}: U3-SCU.94 (~{WDTOVF})
Other:
- moved on the sheet: U1A, U1C, U1D, U1E, U4A, U4B, U4D, U4E, U?, X1

Commit message: wip_cassette
Parts:
- removed unit 5 of U1
- removed unit 1 of U4
- removed unit 5 of U4
- added BT1: Battery-95682B-3, symbol Device:Battery
- added CP177, CP178, CP179, CP180: 10μF, symbol Device:C_Polarized_US
- added CP185, CP187, CP189: 47μF, symbol Device:C_Polarized_US
- added CP186: 101, symbol Device:C
- added CP186, CP188: 1nF, symbol Device:C_Polarized_US
- added RR19, RR3, RR4: 103, symbol Device:R_US
- added U6: FM1208S-250SC, symbol arcade:FM1208S-250SC
- added VD1, VDD2: VD-ESDAxxSCx, symbol arcade:VD-ESDAxxSCx
- gave numbers to parts that had none: 1
- renumbered R2 to RR2, R20 to RR20
Connections:
- net MD3 is gone; now on an unnamed net: U3-SCU.117 (MD3)
- net ~{RST_WD} is gone; now on net ~{RST}_WD: U?.53 (Pin_53)
- net MD4: now also U4.5, U?.58 (Pin_58), CP178.1, RR4.2; no longer U3-SCU.119 (MD4)
- net SCU_A24: now also U1.9, U?.86 (Pin_86)
- net VCC: now also U4.9, U?.117 (Pin_117), U?.119 (Pin_119), CP180.1, U6.24 (VCC)
- net VSS: now also U2.27 (VSS), U2.46 (VSS), BT1.2 (-), CP177.2, CP178.2, CP179.2, CP180.2, CP185.2, CP186.2, CP187.2, CP188.2, CP189.2, RR4.1, U6.12 (VSS), VD1.3 (K); no longer U?.117 (Pin_117), U?.119 (Pin_119)
- net ~{CE}R_CST: now also U1.12, U?.3, CP186.2, VD1.1 (K)
- net ~{CS1}: now also U1.13, U?.82 (Pin_82)
- net ~{WAIT}: now reaches U1.4
- net ~{WAIT}: now also U1.3
- net ~{CE}_SCU: now reaches U1.5
- net ~{CE}_SCU: now also U1.8, U6.18 (~{CE})
- net at U4.11: now also U4.10
- net ~{RST}_WD: now reaches U4.12
- net ~{RST}_WD: now also RR19.1
- net at U4.13: now also CP177.1, RR3.2
- net at CP176.2, RR20.2: now also RR19.2
- net at U1.10: now also U1.11
- net ~{RST}_SCU: now reaches U?.56 (Pin_56)
- net ~{RST}_SCU: now also RR3.1
- net P66: now reaches U?.66 (Pin_66)
- net P66: now also U1.2
- net at U1.1: now also U2.37 (VCC), CP179.1
- net at U4.6: now also U3-SCU.119 (MD4)
- new net: CP185.1, CP186.1, CP186.1
- new net: BT1.1 (+), CP189.1
- new net: CP187.1, VD1.2 (A)
- new net ?: CP188.1, VD1.5 (K)
- no-connect marks 0 -> 2
Other:
- note added: "Monolithic Voltage Suppressors"
- note added: "NOT MOUNTED"
- note added: "RES"
- moved on the sheet: CP174, CP176, U2, U4C

Commit message: wip_cassette_rg
Parts:
- removed BT1: Battery-95682B-3, symbol Device:Battery
- removed VD1, VDD2: VD-ESDAxxSCx, symbol arcade:VD-ESDAxxSCx
- added BT1: Battery, symbol Device:Battery_Cell
- added CP190: 1nF, symbol Device:C_Polarized_US
- added CP191, CP192: 10μF, symbol Device:C_Polarized_US
- added RR16, RR17: 302, symbol Device:R_US
- added V.D1, V.D2: VD-BD5xExx, symbol arcade:VD-BD5xExx
- CP187: value 47μF -> 10nF
Connections:
- net MD2 is gone; now on net VSS: U3-SCU.110 (MD2)
- net CAP1: no longer U3-SCU.108 (CAP1)
- net CAP2: no longer U3-SCU.109 (CAP2)
- net CKIO_SCU: now also U?.59 (Pin_59)
- net VCC: now also CP185.1, CP186.1, CP187.1, CP189.1, U?.5 (Pin_5), BT1.1 (+), V.D1.2 (VCC), V.D2.2 (VCC); no longer U?.10 (Pin_10), U?.108 (Pin_108), U?.16 (Pin_16), U?.2, U?.26 (Pin_26), U?.36 (Pin_36), U?.46 (Pin_46), U?.54 (Pin_54), U?.6, U?.60 (Pin_60), U?.68 (Pin_68), U?.74 (Pin_74), U?.78 (Pin_78), U?.80 (Pin_80), U?.88 (Pin_88), U?.98 (Pin_98)
- net VSS: now also U?.108 (Pin_108), U?.16 (Pin_16), U?.2, U?.26 (Pin_26), U?.36 (Pin_36), U?.46 (Pin_46), U?.54 (Pin_54), U?.6, U?.60 (Pin_60), U?.68 (Pin_68), U?.74 (Pin_74), U?.78 (Pin_78), U?.88 (Pin_88), U?.98 (Pin_98), BT1.2 (-), CP190.2, CP191.2, CP192.2, V.D1.3 (VSS), V.D2.3 (VSS); no longer CP186.2, U?.5 (Pin_5)
- net ~{CE}R_CST: no longer CP186.2
- net ~{IRL0}: now also U?.48 (Pin_48)
- net ~{IRL1}: now also U?.47 (Pin_47)
- net ~{IRL2}: now also U?.50 (Pin_50)
- net ~{IRL3}: now also U?.49 (Pin_49)
- net ~{RST}_WD: now also CP186.1, V.D1.1 (VOUT)
- net ?: no longer names the net of CP188.1
- net ?: now also V.D1.5 (CT)
- new net: CP186.2, CP186.2
- new net: CP190.1, V.D2.5 (CT)
- new net: RR17.2, U3-SCU.108 (CAP1)
- new net: RR16.2, U3-SCU.109 (CAP2)
- new net: CP192.1, RR17.1
- new net: CP191.1, RR16.1
- no-connect marks 2 -> 7
Other:
- note added: "Capacitor connection terminal for output delay time"
- note added: "STANDBY"
- note removed: "Monolithic Voltage Suppressors"
- note removed: "RES"
- moved on the sheet: CP174, CP175, CP176, CP177, CP178, CP179, CP180, CP185, CP186, CP187, CP188, RR19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
