File: cores/cps3/sch/cassette.kicad_sch (KiCad schematic)
At the start: 55 parts, among them U1 7400, U2 29F400TA-90PF, U3-SCU HD6417604F28_SH2, U4 7400, U6 FM1208S-250SC, X1 Crystal

Commit message: wip_cassette_scu
Parts:
- added CP196: 10μF, symbol Device:C_Polarized_US
Connections:
- net CAP1: now also RR17.2, U3-SCU.108 (CAP1)
- net CAP2: now also RR16.2, U3-SCU.109 (CAP2)
- net VCC: no longer U3-SCU.112 (~{CKPREQ}/CKM), U3-SCU.113 (VCC)
- net VSS: now also CP196.2
- net MD: now reaches U3-SCU.117 (MD3), U3-SCU.119 (MD4), U4.6
- new net ~{CKPREQ}/CKM: CP196.1, U3-SCU.112 (~{CKPREQ}/CKM), U3-SCU.113 (VCC)
Other:
- moved on the sheet: CP174, CP175, CP193, CP195, RR2, X1
