File: cores/cps3/sch/cassette.kicad_sch (KiCad schematic)
At the start: 56 parts, among them U1 7400, U2 29F400TA-90PF, U3-SCU HD6417604F28_SH2, U4 7400, U6 FM1208S-250SC, X1 Crystal

Commit message: wip_cassette_sh2
Parts:
- QQ1: value BR39? -> BR39
- QQ2: value AEY? -> AEY
Connections:
- net MD0 is gone; now on net VSS: U3-SCU.105 (MD0)
- net MD5 is gone; now on net VSS: U3-SCU.120 (MD5)
- net DREQ: now also QQ2.1 (B)
- net RxD: now also U?.63 (Pin_63)
- net SCU_A0: now also U2.45 (D15/A-1), U?.116 (Pin_116)
- net SCU_A1: now also U2.25 (A0), U?.115 (Pin_115)
- net SCU_A10: now also U2.7 (A9), U?.104 (Pin_104)
- net SCU_A11: now also U2.6 (A10), U?.103 (Pin_103)
- net SCU_A12: now also U2.5 (A11), U?.102 (Pin_102)
- net SCU_A13: now also U2.4 (A12), U?.101 (Pin_101)
- net SCU_A14: now also U2.3 (A13), U?.100 (Pin_100)
- net SCU_A15: now also U2.2 (A14), U?.99 (Pin_99)
- net SCU_A16: now also U2.1 (A15), U?.96 (Pin_96)
- net SCU_A17: now also U2.48 (A16), U?.95 (Pin_95)
- net SCU_A18: now also U2.17 (A17), U?.94 (Pin_94)
- net SCU_A2: now also U2.24 (A1), U?.114 (Pin_114)
- net SCU_A3: now also U2.23 (A2), U?.113 (Pin_113)
- net SCU_A4: now also U2.22 (A3), U?.112 (Pin_112)
- net SCU_A5: now also U2.21 (A4), U?.111 (Pin_111)
- net SCU_A6: now also U2.20 (A5), U?.110 (Pin_110)
- net SCU_A7: now also U2.19 (A6), U?.109 (Pin_109)
- net SCU_A8: now also U2.18 (A7), U?.106 (Pin_106)
- net SCU_A9: now also U2.8 (A8), U?.105 (Pin_105)
- net ~{CASLL}/DQMLL/~{WE0}: now also U6.21 (~{WE}), U?.70 (Pin_70)
- net ~{CASLL}/DQMLL/~{WE1}: now also U?.71 (Pin_71)
- net ~{CASLL}/DQMLL/~{WE2}: now also U?.72 (Pin_72)
- net ~{CASLL}/DQMLL/~{WE3}: now also U?.73 (Pin_73)
- net ~{CS0}: now also U?.83 (Pin_83)
- net ~{CS2}: now also U?.81 (Pin_81)
- net ~{CS3}: now also U?.80 (Pin_80)
- net ~{RD}: now also U?.67 (Pin_67)
- net CKE: no longer names the net of U3-SCU.88 (CKE)
- net DACK0: no longer names the net of U3-SCU.66 (DACK0)
- net DACK1: no longer names the net of U3-SCU.68 (DACK1)
- net FTOA: no longer names the net of U3-SCU.97 (FTOA)
- net FTOB: no longer names the net of U3-SCU.95 (FTOB)
- net TxD: no longer names the net of U3-SCU.102 (TxD)
- net TxD: no longer U?.63 (Pin_63)
- net ~{BREQ}/~{BGR}: no longer names the net of U3-SCU.93 (~{BREQ}/~{BGR})
- net ~{CAS}/~{OE}: no longer names the net of U3-SCU.80 (~{CAS}/~{OE})
- net ~{CKPACK}: no longer names the net of CP195.1, U3-SCU.111 (~{CKPACK})
- net ~{RAS}/~{CE}: no longer names the net of U3-SCU.79 (~{RAS}/~{CE})
- net ~{WDTOVF}: no longer names the net of U3-SCU.94 (~{WDTOVF})
- no-connect marks 4 -> 12
Other:
- note removed: "BAT?"
- note removed: "VCC"
- moved on the sheet: CP178, CP193, QQ1, QQ2, RR4, RR5, RR7, RR8, U1C, U1D, U4B, U6

Commit message: wip_cst_ccu
Parts:
- removed CP179, CP180: 10μF, symbol Device:C_Polarized_US
- removed unit 3 of U1
- removed unit 4 of U1
- removed unit 1 of U1
- removed U2: 29F400TA-90PF, symbol arcade:29F400TA-90PF
- removed U6: FM1208S-250SC, symbol arcade:FM1208S-250SC
- gave numbers to parts that had none: 1
Connections:
- net SCU_A5 is gone; now on net SCU_A4: CNN5.111 (Pin_111), U3-SCU.36 (A5)
- net SCU_A19: now also CNN5.93 (Pin_93)
- net SCU_A20: now also CNN5.92 (Pin_92)
- net SCU_A21: now also CNN5.91 (Pin_91)
- net SCU_A22: now also CNN5.90 (Pin_90)
- net SCU_A23: now also CNN5.89 (Pin_89)
- net SCU_A25: now also CNN5.85 (Pin_85)
- net SCU_A26: now also CNN5.84 (Pin_84)
- net SCU_D0: now also CNN5.43 (Pin_43)
- net SCU_D1: now also CNN5.44 (Pin_44)
- net SCU_D10: now also CNN5.31 (Pin_31)
- net SCU_D11: now also CNN5.32 (Pin_32)
- net SCU_D12: now also CNN5.29 (Pin_29)
- net SCU_D13: now also CNN5.30 (Pin_30)
- net SCU_D14: now also CNN5.27 (Pin_27)
- net SCU_D15: now also CNN5.28 (Pin_28)
- net SCU_D16: now also CNN5.23 (Pin_23)
- net SCU_D17: now also CNN5.24 (Pin_24)
- net SCU_D18: now also CNN5.21 (Pin_21)
- net SCU_D19: now also CNN5.22 (Pin_22)
- net SCU_D2: now also CNN5.41 (Pin_41)
- net SCU_D20: now also CNN5.19 (Pin_19)
- net SCU_D21: now also CNN5.20 (Pin_20)
- net SCU_D22: now also CNN5.17 (Pin_17)
- net SCU_D23: now also CNN5.18 (Pin_18)
- net SCU_D24: now also CNN5.13 (Pin_13)
- net SCU_D25: now also CNN5.14 (Pin_14)
- net SCU_D26: now also CNN5.11 (Pin_11)
- net SCU_D27: now also CNN5.12 (Pin_12)
- net SCU_D28: now also CNN5.9 (Pin_9)
- net SCU_D29: now also CNN5.10 (Pin_10)
- net SCU_D3: now also CNN5.42 (Pin_42)
- net SCU_D30: now also CNN5.7 (Pin_7)
- net SCU_D31: now also CNN5.8
- net SCU_D4: now also CNN5.39 (Pin_39)
- net SCU_D5: now also CNN5.40 (Pin_40)
- net SCU_D6: now also CNN5.37 (Pin_37)
- net SCU_D7: now also CNN5.38 (Pin_38)
- net SCU_D8: now also CNN5.33 (Pin_33)
- net SCU_D9: now also CNN5.34 (Pin_34)
- net VCC: no longer CNN5.5 (Pin_5)
- net VSS: no longer CNN5.2, CNN5.6
- net Vpp: now reaches CNN5.4
- net MD4 renamed ~{CE}_FRAM
- net P66 renamed WAIT
- net PULL_UP1 renamed ~{WE}_CMOS
- net ~{CASLL}/DQMLL/~{WE0} renamed ~{WE0}_CST
- net ~{CE}_SCU renamed ~{CE}_FR
- new net ~{BYTE}: CNN5.6
- new net ~{OE}_CMOS: CNN5.2
- new net ~{RST}_CMOS: CNN5.5 (Pin_5)
- no-connect marks 12 -> 13
Other:
- added sheet memories_scu (memories_scu.kicad_sch)
- note added: "OK"
- moved on the sheet: BT1, CNN5, CP174, CP175, CP176, CP177, CP178, CP185, CP186, CP187, CP188, CP189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

Commit message: correction_ppu
Connections:
- net CAP1: no longer names the net of RR17.2, U3-SCU.108 (CAP1)
- net CAP2: no longer names the net of RR16.2, U3-SCU.109 (CAP2)
- net CKIO_SCU renamed CKIO_CPUC
- net FTCI renamed FTCI_CPUC
- net FTI renamed FTI_CPUC
- net RD/~{WR} renamed RD/~{WR}_CPUC
- net RxD renamed RxD_CPUC
- net SCK renamed SCK_CPUC
- net SCU_A0 renamed CPUC_A0
- net SCU_A1 renamed CPUC_A1
- net SCU_A10 renamed CPUC_A10
- net SCU_A11 renamed CPUC_A11
- net SCU_A12 renamed CPUC_A12
- net SCU_A13 renamed CPUC_A13
- net SCU_A14 renamed CPUC_A14
- net SCU_A15 renamed CPUC_A15
- net SCU_A16 renamed CPUC_A16
- net SCU_A17 renamed CPUC_A17
- net SCU_A18 renamed CPUC_A18
- net SCU_A19 renamed CPUC_A19
- net SCU_A2 renamed CPUC_A2
- net SCU_A20 renamed CPUC_A20
- net SCU_A21 renamed CPUC_A21
- net SCU_A22 renamed CPUC_A22
- net SCU_A23 renamed CPUC_A23
- net SCU_A24 renamed CPUC_A24
- net SCU_A25 renamed CPUC_A25
- net SCU_A26 renamed CPUC_A26
- net SCU_A3 renamed CPUC_A3
- net SCU_A4 renamed CPUC_A4
- net SCU_A6 renamed CPUC_A6
- net SCU_A7 renamed CPUC_A7
- net SCU_A8 renamed CPUC_A8
- net SCU_A9 renamed CPUC_A9
- net SCU_D0 renamed CPUC_D0
- net SCU_D1 renamed CPUC_D1
- net SCU_D10 renamed CPUC_D10
- net SCU_D11 renamed CPUC_D11
- net SCU_D12 renamed CPUC_D12
- net SCU_D13 renamed CPUC_D13
- net SCU_D14 renamed CPUC_D14
- net SCU_D15 renamed CPUC_D15
- net SCU_D16 renamed CPUC_D16
- net SCU_D17 renamed CPUC_D17
- net SCU_D18 renamed CPUC_D18
- net SCU_D19 renamed CPUC_D19
- net SCU_D2 renamed CPUC_D2
- net SCU_D20 renamed CPUC_D20
- net SCU_D21 renamed CPUC_D21
- net SCU_D22 renamed CPUC_D22
- net SCU_D23 renamed CPUC_D23
- net SCU_D24 renamed CPUC_D24
- net SCU_D25 renamed CPUC_D25
- net SCU_D26 renamed CPUC_D26
- net SCU_D27 renamed CPUC_D27
- net SCU_D28 renamed CPUC_D28
- net SCU_D29 renamed CPUC_D29
- net SCU_D3 renamed CPUC_D3
- net SCU_D30 renamed CPUC_D30
- net SCU_D31 renamed CPUC_D31
- net SCU_D4 renamed CPUC_D4
- net SCU_D5 renamed CPUC_D5
- net SCU_D6 renamed CPUC_D6
- net SCU_D7 renamed CPUC_D7
- net SCU_D8 renamed CPUC_D8
- net SCU_D9 renamed CPUC_D9
- net WAIT renamed WAIT_CPUC
- net ~{BS} renamed ~{BS}_CPUC
- net ~{CASLL}/DQMLL/~{WE1} renamed CPUC_~{WE1}
- net ~{CASLL}/DQMLL/~{WE2} renamed CPUC_~{WE2}
- net ~{CASLL}/DQMLL/~{WE3} renamed CPUC_~{WE3}
- net ~{CE}_FRAM renamed ~{STBY_WD}
- net ~{CS0} renamed CPUC_~{CS0}
- net ~{CS1} renamed CPUC_~{CS1}
- net ~{CS2} renamed CPUC_~{CS2}
- net ~{CS3} renamed CPUC_~{CS3}
- net ~{IRL0} renamed ~{IRL0}_CPUC
- net ~{IRL1} renamed ~{IRL1}_CPUC
- net ~{IRL2} renamed ~{IRL2}_CPUC
- net ~{IRL3} renamed ~{IRL3}_CPUC
- net ~{IVECF}: no longer names the net of U3-SCU.124 (~{IVECF})
- net ~{RD} renamed ~{RD}_CPUC
- net ~{RST}_SCU renamed ~{RST}_CPUC
- net ~{WAIT} renamed ~{WAIT_CPUC}
- net ~{WE0}_CST renamed CPUC_~{WE0}
- no-connect marks 13 -> 14
Other:
- sheet memories_scu ports: added CPUC_A[26..0], CPUC_D[31..0], CPUC_~{CS1}, CPUC_~{WE0}, WAIT_CPUC, ~{STBY_WD}, ~{WAIT_CPUC}; removed SCU_A[24..0], SCU_D[31..0], WAIT, ~{CE}_FRAM, ~{CS1}, ~{WAIT}, ~{WE0}_CST
- note added: "CASSETTE MALE CONNECTOR"
- note added: "REDUCED INSTRUCTION SET COMPUTER"
- moved on the sheet: BT1, CP174, CP176, CP177, CP185, CP186, CP187, CP188, CP189, CP190, CP191, CP192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

Commit message: cps3_finished
Parts:
- renumbered CP186 to CP205, U3-SCU to SCU3, U1 to T1, U4 to T4
Connections:
- net Vpp is gone; now on net ~{WE}_CMOS: CNN5.4
- net CPUC_A4: no longer CNN5.111 (Pin_111)
- net DREQ: no longer SCU3.104 (VCC), SCU3.12 (VCC), SCU3.18 (VCC), SCU3.24 (VCC), SCU3.4 (VCC), SCU3.40 (VCC), SCU3.48 (VCC), SCU3.54 (VCC), SCU3.60 (VCC)
- net VCC: now also SCU3.104 (VCC), SCU3.113 (VCC), SCU3.12 (VCC), SCU3.18 (VCC), SCU3.24 (VCC), SCU3.4 (VCC), SCU3.40 (VCC), SCU3.48 (VCC), SCU3.54 (VCC), SCU3.60 (VCC)
- net ~{CKPREQ}/CKM: no longer SCU3.113 (VCC)
- net ~{CE}_FR renamed ~{CE}_FRAM
- new net CPUC_A5: CNN5.111 (Pin_111)
Other:
- sheet memories_scu ports: added ~{CE}_FRAM; removed Vpp, ~{STBY_WD}
- note added: "CPUC_A5"
- note added: "DREQ"
- note added: "Vpp"
- note added: "~{CKPREQ}/CKM"

Commit message: cassette_wip_rv
Connections:
- net ~{BACK}/~{BRLS}? is gone; now on net DREQ: CP194.1, DA1.2 (OUT), SCU3.92 (~{BACK}/~{BRLS})
- net DREQ: now also RR18.1, SCU3.12 (VCC), SCU3.18 (VCC), SCU3.24 (VCC), SCU3.4 (VCC), SCU3.40 (VCC), SCU3.48 (VCC), SCU3.54 (VCC), SCU3.60 (VCC), SCU3.71 (DREQ1); no longer CP193.1, RR18.2
- net VCC: no longer SCU3.104 (VCC), SCU3.113 (VCC), SCU3.12 (VCC), SCU3.18 (VCC), SCU3.24 (VCC), SCU3.4 (VCC), SCU3.40 (VCC), SCU3.48 (VCC), SCU3.54 (VCC), SCU3.60 (VCC)
- net ~{CKPREQ}/CKM: now also CP176.2, RR19.2, RR20.2, SCU3.113 (VCC)
- new net VCC-PLL: CP193.1, RR18.2, SCU3.104 (VCC)
Other:
- note added: "(SCU) System Control Unit? SLAVE?"
- note added: "regulador de voltaje?"
- note removed: "DREQ"
- note removed: "~{CKPREQ}/CKM"
- moved on the sheet: CP193, CP194, DA1, QQ1, RR18, RR6

Commit message: wip_sh2_cps3
Parts:
- removed CP189: 47μF, symbol Device:C_Polarized_US
- added CP189: x, symbol Device:C
- added DA1: B3 61t, symbol Device:D_Zener
- CP174, CP175, CP176, CP178, CP191, CP192, CP193, CP194, CP195, CP196: value 10μF -> 1µF
- CP177: value 10μF -> -
- CP186, CP188: value 1nF -> 1µF
- CP187: value 10nF -> 1µF
- CP190: value 1nF -> -
- RR19: value 103 -> -
Connections:
- net VCC: now also CP189.2; no longer CP176.1, RR6.2
- net VSS: now also CP176.2
- net at DA1.3 (VBAT): no longer RR6.1
- net ?: now reaches QQ1.2 (C), RR8.1
- net ~{BACK}/~{BRLS}: now reaches T4.4
- net ~{BACK}/~{BRLS}: now also CP176.1, CP194.1, CP196.1, QQ2.1 (B), RR18.1, RR19.2, RR20.2, SCU3.112 (~{CKPREQ}/CKM), SCU3.113 (VCC), SCU3.12 (VCC), SCU3.18 (VCC), SCU3.24 (VCC), SCU3.4 (VCC), SCU3.40 (VCC), SCU3.48 (VCC), SCU3.54 (VCC), SCU3.60 (VCC), SCU3.70 (DREQ0), SCU3.71 (DREQ1), SCU3.92 (~{BACK}/~{BRLS}), DA1.1 (K)
- removed net DREQ: CP194.1, DA1.2 (OUT), QQ2.1 (B), RR18.1, SCU3.12 (VCC), SCU3.18 (VCC), SCU3.24 (VCC), SCU3.4 (VCC), SCU3.40 (VCC), SCU3.48 (VCC), SCU3.54 (VCC), SCU3.60 (VCC), SCU3.70 (DREQ0), SCU3.71 (DREQ1), SCU3.92 (~{BACK}/~{BRLS})
- removed net ~{CKPREQ}/CKM: CP176.2, CP196.1, RR19.2, RR20.2, SCU3.112 (~{CKPREQ}/CKM), SCU3.113 (VCC)
- new net: DA1.2 (A), RR6.1
- new net: CP189.1, RR6.2
- no-connect marks 14 -> 13
Other:
- note added: "No device mounted there is only the footprint"
- note added: "Small Signal Zener Diode"
- moved on the sheet: BT1, CNN5, CP176, CP178, CP187, CP194, DA1, RR4, RR5, RR6, RR7, T4B
