File: cores/cps3/sch/cassette.kicad_sch (KiCad schematic)
At the start: 53 parts, among them T1 7400, T4 7400, X1 Crystal

Commit message: latest_update_cps3
Parts:
- removed DA1: VMON_XXN, symbol arcade:VMON_XXN
- added CP206: 1µF, symbol Device:C_Polarized_US
- CP177, CP190, RR19: value - -> X
- CP189: value x -> X
Connections:
- net CKIO_CPUC: now also CNN5.60 (Pin_60); no longer CNN5.59 (Pin_59)
- net CPUC_A0: now also CNN5.115 (Pin_115); no longer CNN5.116 (Pin_116)
- net CPUC_A1: now also CNN5.116 (Pin_116); no longer CNN5.115 (Pin_115)
- net CPUC_A10: now also CNN5.103 (Pin_103); no longer CNN5.104 (Pin_104)
- net CPUC_A11: now also CNN5.104 (Pin_104); no longer CNN5.103 (Pin_103)
- net CPUC_A12: now also CNN5.101 (Pin_101); no longer CNN5.102 (Pin_102)
- net CPUC_A13: now also CNN5.102 (Pin_102); no longer CNN5.101 (Pin_101)
- net CPUC_A14: now also CNN5.99 (Pin_99); no longer CNN5.100 (Pin_100)
- net CPUC_A15: now also CNN5.100 (Pin_100); no longer CNN5.99 (Pin_99)
- net CPUC_A16: now also CNN5.95 (Pin_95); no longer CNN5.96 (Pin_96)
- net CPUC_A17: now also CNN5.96 (Pin_96); no longer CNN5.95 (Pin_95)
- net CPUC_A18: now also CNN5.93 (Pin_93); no longer CNN5.94 (Pin_94)
- net CPUC_A19: now also CNN5.94 (Pin_94); no longer CNN5.93 (Pin_93)
- net CPUC_A2: now also CNN5.113 (Pin_113); no longer CNN5.114 (Pin_114)
- net CPUC_A20: now also CNN5.91 (Pin_91); no longer CNN5.92 (Pin_92)
- net CPUC_A21: now also CNN5.92 (Pin_92); no longer CNN5.91 (Pin_91)
- net CPUC_A22: now also CNN5.89 (Pin_89); no longer CNN5.90 (Pin_90)
- net CPUC_A23: now also CNN5.90 (Pin_90); no longer CNN5.89 (Pin_89)
- net CPUC_A24: now also CNN5.85 (Pin_85); no longer CNN5.86 (Pin_86)
- net CPUC_A25: now also CNN5.86 (Pin_86); no longer CNN5.85 (Pin_85)
- net CPUC_A26: now also CNN5.83 (Pin_83); no longer CNN5.84 (Pin_84)
- net CPUC_A3: now also CNN5.114 (Pin_114); no longer CNN5.113 (Pin_113)
- net CPUC_A4: now also CNN5.111 (Pin_111); no longer CNN5.112 (Pin_112)
- net CPUC_A5: now also CNN5.112 (Pin_112); no longer CNN5.111 (Pin_111)
- net CPUC_A6: now also CNN5.109 (Pin_109); no longer CNN5.110 (Pin_110)
- net CPUC_A7: now also CNN5.110 (Pin_110); no longer CNN5.109 (Pin_109)
- net CPUC_A8: now also CNN5.105 (Pin_105); no longer CNN5.106 (Pin_106)
- net CPUC_A9: now also CNN5.106 (Pin_106); no longer CNN5.105 (Pin_105)
- net CPUC_D0: now also CNN5.44 (Pin_44); no longer CNN5.43 (Pin_43)
- net CPUC_D1: now also CNN5.43 (Pin_43); no longer CNN5.44 (Pin_44)
- net CPUC_D10: now also CNN5.32 (Pin_32); no longer CNN5.31 (Pin_31)
- net CPUC_D11: now also CNN5.31 (Pin_31); no longer CNN5.32 (Pin_32)
- net CPUC_D12: now also CNN5.30 (Pin_30); no longer CNN5.29 (Pin_29)
- net CPUC_D13: now also CNN5.29 (Pin_29); no longer CNN5.30 (Pin_30)
- net CPUC_D14: now also CNN5.28 (Pin_28); no longer CNN5.27 (Pin_27)
- net CPUC_D15: now also CNN5.27 (Pin_27); no longer CNN5.28 (Pin_28)
- net CPUC_D16: now also CNN5.24 (Pin_24); no longer CNN5.23 (Pin_23)
- net CPUC_D17: now also CNN5.23 (Pin_23); no longer CNN5.24 (Pin_24)
- net CPUC_D18: now also CNN5.22 (Pin_22); no longer CNN5.21 (Pin_21)
- net CPUC_D19: now also CNN5.21 (Pin_21); no longer CNN5.22 (Pin_22)
- net CPUC_D2: now also CNN5.42 (Pin_42); no longer CNN5.41 (Pin_41)
- net CPUC_D20: now also CNN5.20 (Pin_20); no longer CNN5.19 (Pin_19)
- net CPUC_D21: now also CNN5.19 (Pin_19); no longer CNN5.20 (Pin_20)
- net CPUC_D22: now also CNN5.18 (Pin_18); no longer CNN5.17 (Pin_17)
- net CPUC_D23: now also CNN5.17 (Pin_17); no longer CNN5.18 (Pin_18)
- net CPUC_D24: now also CNN5.14 (Pin_14); no longer CNN5.13 (Pin_13)
- net CPUC_D25: now also CNN5.13 (Pin_13); no longer CNN5.14 (Pin_14)
- net CPUC_D26: now also CNN5.12 (Pin_12); no longer CNN5.11 (Pin_11)
- net CPUC_D27: now also CNN5.11 (Pin_11); no longer CNN5.12 (Pin_12)
- net CPUC_D28: now also CNN5.10 (Pin_10); no longer CNN5.9 (Pin_9)
- net CPUC_D29: now also CNN5.9 (Pin_9); no longer CNN5.10 (Pin_10)
- net CPUC_D3: now also CNN5.41 (Pin_41); no longer CNN5.42 (Pin_42)
- net CPUC_D30: now also CNN5.8; no longer CNN5.7 (Pin_7)
- net CPUC_D31: now also CNN5.7 (Pin_7); no longer CNN5.8
- net CPUC_D4: now also CNN5.40 (Pin_40); no longer CNN5.39 (Pin_39)
- net CPUC_D5: now also CNN5.39 (Pin_39); no longer CNN5.40 (Pin_40)
- net CPUC_D6: now also CNN5.38 (Pin_38); no longer CNN5.37 (Pin_37)
- net CPUC_D7: now also CNN5.37 (Pin_37); no longer CNN5.38 (Pin_38)
- net CPUC_D8: now also CNN5.34 (Pin_34); no longer CNN5.33 (Pin_33)
- net CPUC_D9: now also CNN5.33 (Pin_33); no longer CNN5.34 (Pin_34)
- net CPUC_~{CS0}: now also CNN5.84 (Pin_84); no longer CNN5.83 (Pin_83)
- net CPUC_~{CS1}: now also CNN5.81 (Pin_81); no longer CNN5.82 (Pin_82)
- net CPUC_~{CS2}: now also CNN5.82 (Pin_82); no longer CNN5.81 (Pin_81)
- net CPUC_~{CS3}: now also CNN5.79 (Pin_79); no longer CNN5.80 (Pin_80)
- net CPUC_~{WE0}: now also CNN5.69 (Pin_69); no longer CNN5.70 (Pin_70)
- net CPUC_~{WE1}: now also CNN5.72 (Pin_72); no longer CNN5.71 (Pin_71)
- net CPUC_~{WE2}: now also CNN5.71 (Pin_71); no longer CNN5.72 (Pin_72)
- net CPUC_~{WE3}: now also CNN5.74 (Pin_74); no longer CNN5.73 (Pin_73)
- net FTCI_CPUC: now also CNN5.63 (Pin_63); no longer CNN5.64 (Pin_64)
- net FTI_CPUC: now also CNN5.66 (Pin_66); no longer CNN5.65 (Pin_65)
- net RD/~{WR}_CPUC: now also CNN5.75 (Pin_75); no longer CNN5.76 (Pin_76)
- net RxD_CPUC: now also CNN5.64 (Pin_64); no longer CNN5.63 (Pin_63)
- net SCK_CPUC: now also CNN5.61 (Pin_61); no longer CNN5.62 (Pin_62)
- net VSS: now also CNN5.52 (Pin_52), CNN5.53 (Pin_53), CNN5.56 (Pin_56), CNN5.58 (Pin_58), CNN5.59 (Pin_59), CNN5.62 (Pin_62), CNN5.67 (Pin_67), CNN5.70 (Pin_70), CNN5.73 (Pin_73), CNN5.76 (Pin_76), CNN5.77 (Pin_77), CNN5.80 (Pin_80), CP206.2; no longer CNN5.51 (Pin_51), CNN5.54 (Pin_54), CNN5.55 (Pin_55), CNN5.57 (Pin_57), CNN5.60 (Pin_60), CNN5.61 (Pin_61), CNN5.68 (Pin_68), CNN5.69 (Pin_69), CNN5.74 (Pin_74), CNN5.75 (Pin_75), CNN5.78 (Pin_78), CNN5.79 (Pin_79)
- net WAIT_CPUC: now also CNN5.65 (Pin_65); no longer CNN5.66 (Pin_66)
- net ~{BS}_CPUC: now also CNN5.78 (Pin_78); no longer CNN5.77 (Pin_77)
- net ~{BYTE}: now also CNN5.5 (Pin_5); no longer CNN5.6
- net ~{CE}R_CST: now also CNN5.4; no longer CNN5.3
- net ~{IRL0}_CPUC: now also CNN5.47 (Pin_47); no longer CNN5.48 (Pin_48)
- net ~{IRL1}_CPUC: now also CNN5.48 (Pin_48); no longer CNN5.47 (Pin_47)
- net ~{IRL2}_CPUC: now also CNN5.49 (Pin_49); no longer CNN5.50 (Pin_50)
- net ~{IRL3}_CPUC: now also CNN5.50 (Pin_50); no longer CNN5.49 (Pin_49)
- net ~{OE}_CMOS: now also CNN5.1; no longer CNN5.2
- net ~{RD}_CPUC: now also CNN5.68 (Pin_68); no longer CNN5.67 (Pin_67)
- net ~{RST}_CMOS: now also CNN5.6; no longer CNN5.5 (Pin_5)
- net ~{RST}_CPUC: now also CNN5.55 (Pin_55); no longer CNN5.56 (Pin_56)
- net ~{RST}_WD: now also CNN5.54 (Pin_54), RR19.2; no longer CNN5.53 (Pin_53), RR19.1
- net ~{STBY_WD}: now also CNN5.57 (Pin_57); no longer CNN5.58 (Pin_58)
- net ~{WE}_CMOS: now also CNN5.2, CNN5.3; no longer CNN5.1, CNN5.4
- net ~{WAIT}: now reaches RR15.2, SCU3.89 (~{WAIT}), T1.6
- net VCC-PLL renamed VCC(PLL)
- net ~{BACK}/~{BRLS} renamed +5V
- net +5V: now also RR19.1, CP206.1; no longer RR19.2
Other:
- note added: "BREAKDOWN?"
- note added: "Revisar aquí"
- note added: "Small Signal Zener Diode?"
- note removed: "BREAKDOWN"
- note removed: "OK"
- note removed: "Small Signal Zener Diode"
- moved on the sheet: BT1, CP174, CP175, CP176, CP177, CP178, CP185, CP186, CP187, CP188, CP189, CP190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
