File: cores/cps3/sch/video_dac.kicad_sch (KiCad schematic)
At the start: 58 parts, among them Q2 Q_NPN_ECB, Q3 Q_NPN_ECB, Q4 Q_NPN_ECB, Q5 Q_PNP_ECB, Q6 Q_PNP_ECB, Q7 Q_PNP_ECB, Q9 ZR

Commit message: wip_ccu
Connections:
- net PAL7: no longer names the net of E9.27 (D7)
Changed lines of the file:
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@@
   (no_connect (at 152.4 118.11))
   (no_connect (at 152.4 113.03))
-  (no_connect (at 114.3 80.01))
   (no_connect (at 170.18 129.54))
   (no_connect (at 152.4 107.95))
@@
   (no_connect (at 152.4 59.69))
   (no_connect (at 180.34 129.54))
+  (no_connect (at 106.68 80.01))
   (no_connect (at 152.4 64.77))
   (no_connect (at 152.4 168.91))
@@
   )
   (bus (pts (xy 116.84 147.32) (xy 116.84 149.86))
-    (stroke (width 0) (type default) (color 0 0 0 0))
-  )
-  (wire (pts (xy 106.68 80.01) (xy 114.3 80.01))
     (stroke (width 0) (type default) (color 0 0 0 0))
   )
@@
     (effects (font (size 1.27 1.27)) (justify left bottom))
   )
-  (label "PAL7" (at 114.3 80.01 180)
-    (effects (font (size 1.27 1.27)) (justify right bottom))
-  )
   (label "~{BLK}" (at 120.65 189.23 0)

Commit message: wip_ccu_gll2_cassette
Parts:
- R14, R15: value 101Ω -> 101
- R24, R25, R26: value 301Ω -> 301
- R30: value 240Ω -> 240
- R31: value 640Ω -> 640
- R36: value 241Ω -> 241
- R39: value 561Ω -> 561
- R46: value 472Ω -> 472
- R47: value 103Ω -> 103
- RN15, RN16, RN17, RN18, RN19, RN4, RN5, RN6, RN7: value 620Ω -> 620
Changed lines of the file:
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@@
     (in_bom yes) (on_board yes)
     (property "Reference" "R31" (id 0) (at 397.51 114.3 0))
-    (property "Value" "640Ω" (id 1) (at 397.51 116.84 0))
+    (property "Value" "640" (id 1) (at 397.51 116.84 0))
     (property "Footprint" "" (id 2) (at 392.684 116.586 90)
       (effects (font (size 1.27 1.27)) hide)
@@
   (symbol (lib_id "Device:R_US") (at 379.73 78.74 0) (unit 1)
     (in_bom yes) (on_board yes)
-    (property "Reference" "R47" (id 0) (at 375.92 77.47 0))
-    (property "Value" "103Ω" (id 1) (at 367.03 80.01 0))
+    (property "Reference" "R47" (id 0) (at 383.54 77.47 0))
+    (property "Value" "103" (id 1) (at 383.54 80.01 0))
     (property "Footprint" "" (id 2) (at 380.746 78.994 90)
       (effects (font (size 1.27 1.27)) hide)
@@
     (in_bom yes) (on_board yes)
     (property "Reference" "RN17" (id 0) (at 50.8 90.17 90))
-    (property "Value" "620Ω" (id 1) (at 50.8 102.87 90))
+    (property "Value" "620" (id 1) (at 50.8 102.87 90))
     (property "Footprint" "" (id 2) (at 50.8 104.775 90)
       (effects (font (size 1.27 1.27)) hide)
@@
     (in_bom yes) (on_board yes)
     (property "Reference" "RN5" (id 0) (at 175.26 102.87 90))
-    (property "Value" "620Ω" (id 1) (at 175.26 115.57 90))
+    (property "Value" "620" (id 1) (at 175.26 115.57 90))
     (property "Footprint" "" (id 2) (at 175.26 117.475 90)
       (effects (font (size 1.27 1.27)) hide)
@@
     (in_bom yes) (on_board yes)
     (property "Reference" "R14" (id 0) (at 304.8 209.55 0))
-    (property "Value" "101Ω" (id 1) (at 304.8 212.09 0))
+    (property "Value" "101" (id 1) (at 304.8 212.09 0))
     (property "Footprint" "" (id 2) (at 302.006 210.566 90)
       (effects (font (size 1.27 1.27)) hide)
@@
     (in_bom yes) (on_board yes)
     (property "Reference" "R46" (id 0) (at 367.03 96.52 90))
-    (property "Value" "472Ω" (id 1) (at 367.03 101.6 90))
+    (property "Value" "472" (id 1) (at 367.03 101.6 90))
     (property "Footprint" "" (id 2) (at 366.776 100.076 90)
       (effects (font (size 1.27 1.27)) hide)
@@
   (symbol (lib_id "Device:R_Pack04") (at 50.8 110.49 270) (mirror x) (unit 1)
     (in_bom yes) (on_board yes)
-    (property "Reference" "RN19" (id 0) (at 50.8 118.11 90))
-    (property "Value" "620Ω" (id 1) (at 50.8 105.41 90))
+    (property "Reference" "RN19" (id 0) (at 50.8 105.41 90))
+    (property "Value" "620" (id 1) (at 50.8 118.11 90))
     (property "Footprint" "" (id 2) (at 50.8 103.505 90)
       (effects (font (size 1.27 1.27)) hide)
@@
     (in_bom yes) (on_board yes)
     (property "Reference" "R24" (id 0) (at 292.1 148.59 0))
-    (property "Value" "301Ω" (id 1) (at 292.1 151.13 0))
+    (property "Value" "301" (id 1) (at 292.1 151.13 0))
     (property "Footprint" "" (id 2) (at 289.306 149.606 90)
       (effects (font (size 1.27 1.27)) hide)
@@
     (in_bom yes) (on_board yes)
     (property "Reference" "R30" (id 0) (at 360.68 68.58 0))
-    (property "Value" "240Ω" (id 1) (at 360.68 71.12 0))
+    (property "Value" "240" (id 1) (at 360.68 71.12 0))
     (property "Footprint" "" (id 2) (at 355.854 69.596 90)
       (effects (font (size 1.27 1.27)) hide)
@@
   (symbol (lib_id "Device:R_US") (at 378.46 207.01 0) (mirror x) (unit 1)
     (in_bom yes) (on_board yes)
-    (property "Reference" "R14" (id 0) (at 382.27 200.66 0))
-    (property "Value" "101Ω" (id 1) (at 382.27 203.2 0))
+    (property "Reference" "R14" (id 0) (at 382.27 205.74 0))
+    (property "Value" "101" (id 1) (at 382.27 208.28 0))
     (property "Footprint" "" (id 2) (at 379.476 206.756 90)
       (effects (font (size 1.27 1.27)) hide)
@@
     (in_bom yes) (on_board yes)
     (property "Reference" "R39" (id 0) (at 342.9 66.04 0))
-    (property "Value" "561Ω" (id 1) (at 342.9 68.58 0))
+    (property "Value" "561" (id 1) (at 342.9 68.58 0))
     (property "Footprint" "" (id 2) (at 338.836 67.056 90)
       (effects (font (size 1.27 1.27)) hide)
@@
   (symbol (lib_id "Device:R_Pack04") (at 50.8 125.73 270) (mirror x) (unit 1)
     (in_bom yes) (on_board yes)
-    (property "Reference" "RN18" (id 0) (at 50.8 133.35 90))
-    (property "Value" "620Ω" (id 1) (at 50.8 120.65 90))
+    (property "Reference" "RN18" (id 0) (at 50.8 120.65 90))
+    (property "Value" "620" (id 1) (at 50.8 133.35 90))
     (property "Footprint" "" (id 2) (at 50.8 118.745 90)
       (effects (font (size 1.27 1.27)) hide)
@@
     (in_bom yes) (on_board yes)
     (property "Reference" "RN15" (id 0) (at 50.8 74.93 90))
-    (property "Value" "620Ω" (id 1) (at 50.8 87.63 90))
+    (property "Value" "620" (id 1) (at 50.8 87.63 90))
     (property "Footprint" "" (id 2) (at 50.8 89.535 90)
       (effects (font (size 1.27 1.27)) hide)
@@
     (in_bom yes) (on_board yes)
     (property "Reference" "RN16" (id 0) (at 50.8 59.69 90))
-    (property "Value" "620Ω" (id 1) (at 50.8 72.39 90))
+    (property "Value" "620" (id 1) (at 50.8 72.39 90))
     (property "Footprint" "" (id 2) (at 50.8 74.295 90)
       (effects (font (size 1.27 1.27)) hide)
@@
     (in_bom yes) (on_board yes)
     (property "Reference" "RN7" (id 0) (at 175.26 67.31 90))
-    (property "Value" "620Ω" (id 1) (at 175.26 80.01 90))
+    (property "Value" "620" (id 1) (at 175.26 80.01 90))
     (property "Footprint" "" (id 2) (at 175.26 81.915 90)
       (effects (font (size 1.27 1.27)) hide)
@@
     (in_bom yes) (on_board yes)
     (property "Reference" "R25" (id 0) (at 328.93 148.59 0))
-    (property "Value" "301Ω" (id 1) (at 328.93 151.13 0))
+    (property "Value" "301" (id 1) (at 328.93 151.13 0))
     (property "Footprint" "" (id 2) (at 326.136 149.606 90)
       (effects (font (size 1.27 1.27)) hide)
@@
     (in_bom yes) (on_board yes)
     (property "Reference" "R36" (id 0) (at 248.92 129.54 90))
-    (property "Value" "241Ω" (id 1) (at 248.92 132.08 90))
+    (property "Value" "241" (id 1) (at 248.92 132.08 90))
     (property "Footprint" "" (id 2) (at 255.016 129.794 90)
       (effects (font (size 1.27 1.27)) hide)
@@
     (in_bom yes) (on_board yes)
     (property "Reference" "RN6" (id 0) (at 175.26 85.09 90))
-    (property "Value" "620Ω" (id 1) (at 175.26 97.79 90))
+    (property "Value" "620" (id 1) (at 175.26 97.79 90))
     (property "Footprint" "" (id 2) (at 175.26 99.695 90)
       (effects (font (size 1.27 1.27)) hide)
@@
     (in_bom yes) (on_board yes)
     (property "Reference" "RN4" (id 0) (at 175.26 119.38 90))
-    (property "Value" "620Ω" (id 1) (at 175.26 132.08 90))
+    (property "Value" "620" (id 1) (at 175.26 132.08 90))
     (property "Footprint" "" (id 2) (at 175.26 133.985 90)
       (effects (font (size 1.27 1.27)) hide)
@@
     (in_bom yes) (on_board yes)
     (property "Reference" "R26" (id 0) (at 370.84 147.32 0))
-    (property "Value" "301Ω" (id 1) (at 370.84 149.86 0))
+    (property "Value" "301" (id 1) (at 370.84 149.86 0))
     (property "Footprint" "" (id 2) (at 368.046 148.336 90)
       (effects (font (size 1.27 1.27)) hide)
@@
     (in_bom yes) (on_board yes)
     (property "Reference" "R15" (id 0) (at 346.71 205.74 0))
-    (property "Value" "101Ω" (id 1) (at 346.71 208.28 0))
+    (property "Value" "101" (id 1) (at 346.71 208.28 0))
     (property "Footprint" "" (id 2) (at 343.916 206.756 90)
       (effects (font (size 1.27 1.27)) hide)

Commit message: wip_cassette
Connections:
- net ~{WE} renamed ~{WE}_VD
Changed lines of the file:
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@@
     (effects (font (size 1.27 1.27)) (justify left bottom))
   )
-  (label "~{WE}" (at 60.96 100.33 180)
+  (label "~{WE}_VD" (at 60.96 100.33 180)
     (effects (font (size 1.27 1.27)) (justify right bottom))
   )
@@
     (effects (font (size 1.27 1.27)) (justify left bottom))
   )
-  (label "~{WE}" (at 73.66 185.42 0)
+  (label "~{WE}_VD" (at 73.66 185.42 0)
     (effects (font (size 1.27 1.27)) (justify left bottom))
   )
@@
     (effects (font (size 1.27 1.27)) (justify left bottom))
   )
-  (label "~{WE}" (at 73.66 107.95 0)
-    (effects (font (size 1.27 1.27)) (justify left bottom))
-  )
+  (label "~{WE}_VD" (at 73.66 107.95 0)
+    (effects (font (size 1.27 1.27)) (justify left bottom))
+  )

Commit message: wip_cassette
Parts:
- removed VD2: BAV99, symbol arcade:BAV99
- added VD2: VD-BAV99, symbol arcade:VD-BAV99
Connections:
- net VSS: now also VD2.
- net at 7B.2 (B), C9.7 (CX1), CP126.1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: now also VD2.
- net at R46.2: now also VD2.
Changed lines of the file:
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@@
     (pin "3")
+  )
+  (symbol (lib_id "arcade:VD-BAV99") (at 337.82 92.71 0) (mirror y) (unit 1)
+    (in_bom yes) (on_board yes)
+    (property "Reference" "VD2" (id 0) (at 331.47 86.36 0))
+    (property "Value" "VD-BAV99" (id 1) (at 337.82 88.9 0))
+    (property "Footprint" "" (id 2) (at 337.82 91.44 0)
+      (effects (font (size 1.27 1.27)) hide)
+    )
+    (property "Datasheet" "https://assets.nexperia.com/documents/data-sheet/BAV99_SER.pdf" (id 3) (at 337.82 106.68 0)
+      (effects (font (size 1.27 1.27)) hide)
+    )
+    (pin "")
+    (pin "")
+    (pin "")
   )
   (symbol (lib_id "Device:R_US") (at 300.99 210.82 0) (mirror x) (unit 1)
@@
     (pin "8")
   )
-  (symbol (lib_id "arcade:BAV99") (at 337.82 92.71 0) (mirror y) (unit 1)
-    (in_bom yes) (on_board yes)
-    (property "Reference" "VD2" (id 0) (at 335.28 88.9 0))
-    (property "Value" "BAV99" (id 1) (at 341.63 88.9 0))
-    (property "Footprint" "" (id 2) (at 337.82 91.44 0)
-      (effects (font (size 1.27 1.27)) hide)
-    )
-    (property "Datasheet" "https://assets.nexperia.com/documents/data-sheet/BAV99_SER.pdf" (id 3) (at 337.82 106.68 0)
-      (effects (font (size 1.27 1.27)) hide)
-    )
-    (pin "")
-    (pin "")
-    (pin "")
-  )
   (symbol (lib_id "arcade:CU383-69K") (at 140.97 71.12 0) (unit 1)
