File: cores/cps3/sch/simm4.kicad_sch (KiCad schematic)
At the start: 8 parts

Commit message: wip_cassette_sh2
Parts:
- removed JE1, JE2, JE3, JE4, JE5, JE6, JE7, JE8: 29F016-90PFTN, symbol arcade:29F016-90PFTN
- added JD1, JD2, JD3, JD4, JD5, JD6, JD7, JD8: 29F016-90PFTN, symbol arcade:29F016-90PFTN
Connections:
- net OAM_A0: now also JD1.30 (A0), JD2.30 (A0), JD3.30 (A0), JD4.30 (A0), JD5.30 (A0), JD6.30 (A0), JD7.30 (A0), JD8.30 (A0)
- net OAM_A1: now also JD1.29 (A1), JD2.29 (A1), JD3.29 (A1), JD4.29 (A1), JD5.29 (A1), JD6.29 (A1), JD7.29 (A1), JD8.29 (A1)
- net OAM_A10: now also JD1.16 (A10), JD2.16 (A10), JD3.16 (A10), JD4.16 (A10), JD5.16 (A10), JD6.16 (A10), JD7.16 (A10), JD8.16 (A10)
- net OAM_A11: now also JD1.15 (A11), JD2.15 (A11), JD3.15 (A11), JD4.15 (A11), JD5.15 (A11), JD6.15 (A11), JD7.15 (A11), JD8.15 (A11)
- net OAM_A12: now also JD1.10 (A12), JD2.10 (A12), JD3.10 (A12), JD4.10 (A12), JD5.10 (A12), JD6.10 (A12), JD7.10 (A12), JD8.10 (A12)
- net OAM_A13: now also JD1.9 (A13), JD2.9 (A13), JD3.9 (A13), JD4.9 (A13), JD5.9 (A13), JD6.9 (A13), JD7.9 (A13), JD8.9 (A13)
- net OAM_A14: now also JD1.8 (A14), JD2.8 (A14), JD3.8 (A14), JD4.8 (A14), JD5.8 (A14), JD6.8 (A14), JD7.8 (A14), JD8.8 (A14)
- net OAM_A15: now also JD1.7 (A15), JD2.7 (A15), JD3.7 (A15), JD4.7 (A15), JD5.7 (A15), JD6.7 (A15), JD7.7 (A15), JD8.7 (A15)
- net OAM_A16: now also JD1.6 (A16), JD2.6 (A16), JD3.6 (A16), JD4.6 (A16), JD5.6 (A16), JD6.6 (A16), JD7.6 (A16), JD8.6 (A16)
- net OAM_A17: now also JD1.5 (A17), JD2.5 (A17), JD3.5 (A17), JD4.5 (A17), JD5.5 (A17), JD6.5 (A17), JD7.5 (A17), JD8.5 (A17)
- net OAM_A18: now also JD1.4 (A18), JD2.4 (A18), JD3.4 (A18), JD4.4 (A18), JD5.4 (A18), JD6.4 (A18), JD7.4 (A18), JD8.4 (A18)
- net OAM_A19: now also JD1.3 (A19), JD2.3 (A19), JD3.3 (A19), JD4.3 (A19), JD5.3 (A19), JD6.3 (A19), JD7.3 (A19), JD8.3 (A19)
- net OAM_A2: now also JD1.28 (A2), JD2.28 (A2), JD3.28 (A2), JD4.28 (A2), JD5.28 (A2), JD6.28 (A2), JD7.28 (A2), JD8.28 (A2)
- net OAM_A20: now also JD1.46 (A20), JD2.46 (A20), JD3.46 (A20), JD4.46 (A20), JD5.46 (A20), JD6.46 (A20), JD7.46 (A20), JD8.46 (A20)
- net OAM_A3: now also JD1.27 (A3), JD2.27 (A3), JD3.27 (A3), JD4.27 (A3), JD5.27 (A3), JD6.27 (A3), JD7.27 (A3), JD8.27 (A3)
- net OAM_A4: now also JD1.22 (A4), JD2.22 (A4), JD3.22 (A4), JD4.22 (A4), JD5.22 (A4), JD6.22 (A4), JD7.22 (A4), JD8.22 (A4)
- net OAM_A5: now also JD1.21 (A5), JD2.21 (A5), JD3.21 (A5), JD4.21 (A5), JD5.21 (A5), JD6.21 (A5), JD7.21 (A5), JD8.21 (A5)
- net OAM_A6: now also JD1.20 (A6), JD2.20 (A6), JD3.20 (A6), JD4.20 (A6), JD5.20 (A6), JD6.20 (A6), JD7.20 (A6), JD8.20 (A6)
- net OAM_A7: now also JD1.19 (A7), JD2.19 (A7), JD3.19 (A7), JD4.19 (A7), JD5.19 (A7), JD6.19 (A7), JD7.19 (A7), JD8.19 (A7)
- net OAM_A8: now also JD1.18 (A8), JD2.18 (A8), JD3.18 (A8), JD4.18 (A8), JD5.18 (A8), JD6.18 (A8), JD7.18 (A8), JD8.18 (A8)
- net OAM_A9: now also JD1.17 (A9), JD2.17 (A9), JD3.17 (A9), JD4.17 (A9), JD5.17 (A9), JD6.17 (A9), JD7.17 (A9), JD8.17 (A9)
- net SPRITEB_D0: now also JD1.31 (D0), JD3.31 (D0), JD5.31 (D0), JD7.31 (D0)
- net SPRITEB_D1: now also JD1.32 (D1), JD3.32 (D1), JD5.32 (D1), JD7.32 (D1)
- net SPRITEB_D2: now also JD1.33 (D2), JD3.33 (D2), JD5.33 (D2), JD7.33 (D2)
- net SPRITEB_D3: now also JD1.34 (D3), JD3.34 (D3), JD5.34 (D3), JD7.34 (D3)
- net SPRITEB_D4: now also JD1.38 (D4), JD3.38 (D4), JD5.38 (D4), JD7.38 (D4)
- net SPRITEB_D5: now also JD1.39 (D5), JD3.39 (D5), JD5.39 (D5), JD7.39 (D5)
- net SPRITEB_D6: now also JD1.40 (D6), JD3.40 (D6), JD5.40 (D6), JD7.40 (D6)
- net SPRITEB_D7: now also JD1.41 (D7), JD3.41 (D7), JD5.41 (D7), JD7.41 (D7)
- net SPRITED_D0: now also JD2.31 (D0), JD4.31 (D0), JD6.31 (D0), JD8.31 (D0)
- net SPRITED_D1: now also JD2.32 (D1), JD4.32 (D1), JD6.32 (D1), JD8.32 (D1)
- net SPRITED_D2: now also JD2.33 (D2), JD4.33 (D2), JD6.33 (D2), JD8.33 (D2)
- net SPRITED_D3: now also JD2.34 (D3), JD4.34 (D3), JD6.34 (D3), JD8.34 (D3)
- net SPRITED_D4: now also JD2.38 (D4), JD4.38 (D4), JD6.38 (D4), JD8.38 (D4)
- net SPRITED_D5: now also JD2.39 (D5), JD4.39 (D5), JD6.39 (D5), JD8.39 (D5)
- net SPRITED_D6: now also JD2.40 (D6), JD4.40 (D6), JD6.40 (D6), JD8.40 (D6)
- net SPRITED_D7: now also JD2.41 (D7), JD4.41 (D7), JD6.41 (D7), JD8.41 (D7)
- net VCC: now also JD1.12 (VCC), JD1.37 (VCC), JD2.12 (VCC), JD2.37 (VCC), JD3.12 (VCC), JD3.37 (VCC), JD4.12 (VCC), JD4.37 (VCC), JD5.12 (VCC), JD5.37 (VCC), JD6.12 (VCC), JD6.37 (VCC), JD7.12 (VCC), JD7.37 (VCC), JD8.12 (VCC), JD8.37 (VCC)
- net VSS: now also JD1.35 (VSS), JD1.36 (VSS), JD1.42 (RY/~{BY}), JD2.35 (VSS), JD2.36 (VSS), JD2.42 (RY/~{BY}), JD3.35 (VSS), JD3.36 (VSS), JD3.42 (RY/~{BY}), JD4.35 (VSS), JD4.36 (VSS), JD4.42 (RY/~{BY}), JD5.35 (VSS), JD5.36 (VSS), JD5.42 (RY/~{BY}), JD6.35 (VSS), JD6.36 (VSS), JD6.42 (RY/~{BY}), JD7.35 (VSS), JD7.36 (VSS), JD7.42 (RY/~{BY}), JD8.35 (VSS), JD8.36 (VSS), JD8.42 (RY/~{BY})
- new net ~{CEI}: JD1.11 (~{CE}), JD4.11 (~{CE})
- new net ~{CEJ}: JD2.11 (~{CE}), JD3.11 (~{CE})
- new net ~{CEK}: JD5.11 (~{CE}), JD8.11 (~{CE})
- new net ~{CEL}: JD6.11 (~{CE}), JD7.11 (~{CE})
- new net ~{OEC}: JD4.43 (~{OE}), JD6.43 (~{OE}), JD8.43 (~{OE})
- new net ~{OED}: JD1.43 (~{OE}), JD2.43 (~{OE}), JD3.43 (~{OE}), JD5.43 (~{OE}), JD7.43 (~{OE})
- new net ~{RESET3}: JD1.14 (~{RESET}), JD2.14 (~{RESET}), JD3.14 (~{RESET}), JD4.14 (~{RESET}), JD5.14 (~{RESET}), JD6.14 (~{RESET}), JD7.14 (~{RESET}), JD8.14 (~{RESET})
- new net ~{WEC}: JD4.44 (~{WE}), JD6.44 (~{WE}), JD8.44 (~{WE})
- new net ~{WED}: JD1.44 (~{WE}), JD2.44 (~{WE}), JD3.44 (~{WE}), JD5.44 (~{WE}), JD7.44 (~{WE})
Other:
- note added: "Simm 4"
- note removed: "Simm 3"
