File: cores/cps3/sch/simm4.kicad_sch (KiCad schematic)
At the start: 8 parts

Commit message: wip_cre_cps3
Connections:
- net VSS: no longer JD1.42 (RY/~{BY}), JD2.42 (RY/~{BY}), JD3.42 (RY/~{BY}), JD4.42 (RY/~{BY}), JD5.42 (RY/~{BY}), JD6.42 (RY/~{BY}), JD7.42 (RY/~{BY}), JD8.42 (RY/~{BY})
- net OAM_A0 renamed SPRITE_AB0
- net OAM_A1 renamed SPRITE_AB1
- net OAM_A10 renamed SPRITE_AB10
- net OAM_A11 renamed SPRITE_AB11
- net OAM_A12 renamed SPRITE_AB12
- net OAM_A13 renamed SPRITE_AB13
- net OAM_A14 renamed SPRITE_AB14
- net OAM_A15 renamed SPRITE_AB15
- net OAM_A16 renamed SPRITE_AB16
- net OAM_A17 renamed SPRITE_AB17
- net OAM_A18 renamed SPRITE_AB18
- net OAM_A19 renamed SPRITE_AB19
- net OAM_A2 renamed SPRITE_AB2
- net OAM_A20 renamed SPRITE_AB20
- net OAM_A3 renamed SPRITE_AB3
- net OAM_A4 renamed SPRITE_AB4
- net OAM_A5 renamed SPRITE_AB5
- net OAM_A6 renamed SPRITE_AB6
- net OAM_A7 renamed SPRITE_AB7
- net OAM_A8 renamed SPRITE_AB8
- net OAM_A9 renamed SPRITE_AB9
- no-connect marks 0 -> 8
Other:
- note added: "VSS"
