File: cores/cps3/sch/simm4.kicad_sch (KiCad schematic)
At the start: 8 parts

Commit message: cps3_finished
Connections:
- net ~{OEC} is gone; now on net ~{OED}: JD4.43 (~{OE}), JD6.43 (~{OE}), JD8.43 (~{OE})
- net ~{WEC} is gone; now on net ~{WED}: JD4.44 (~{WE}), JD6.44 (~{WE}), JD8.44 (~{WE})
Changed lines of the file:
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@@
     (company "JOTEGO")
     (comment 1 "E.Triana")
+    (comment 2 "14/10/22-30/01/23")
   )
   (junction (at 300.99 226.06) (diameter 0) (color 0 0 0 0)
@@
     (effects (font (size 1.27 1.27)) (justify left bottom))
   )
-  (label "~{WEC}" (at 132.08 215.9 0)
-    (effects (font (size 1.27 1.27)) (justify left bottom))
-  )
   (label "SPRITE_AB10" (at 200.66 185.42 0)
     (effects (font (size 1.27 1.27)) (justify left bottom))
@@
     (effects (font (size 1.27 1.27)) (justify left bottom))
   )
+  (label "~{WED}" (at 132.08 215.9 0)
+    (effects (font (size 1.27 1.27)) (justify left bottom))
+  )
   (label "~{RESET3}" (at 132.08 123.19 0)
     (effects (font (size 1.27 1.27)) (justify left bottom))
@@
     (effects (font (size 1.27 1.27)) (justify right bottom))
   )
-  (label "~{OEC}" (at 132.08 213.36 0)
+  (label "~{OED}" (at 132.08 213.36 0)
     (effects (font (size 1.27 1.27)) (justify left bottom))
   )
@@
     (effects (font (size 1.27 1.27)) (justify right bottom))
   )
-  (label "~{WEC}" (at 200.66 215.9 0)
+  (label "~{WED}" (at 200.66 215.9 0)
     (effects (font (size 1.27 1.27)) (justify left bottom))
   )
@@
     (effects (font (size 1.27 1.27)) (justify left bottom))
   )
-  (label "~{OEC}" (at 269.24 213.36 0)
+  (label "~{OED}" (at 269.24 213.36 0)
     (effects (font (size 1.27 1.27)) (justify left bottom))
   )
@@
     (effects (font (size 1.27 1.27)) (justify left bottom))
   )
-  (label "~{OEC}" (at 200.66 213.36 0)
+  (label "~{OED}" (at 200.66 213.36 0)
     (effects (font (size 1.27 1.27)) (justify left bottom))
   )
@@
     (effects (font (size 1.27 1.27)) (justify left bottom))
   )
-  (label "~{WEC}" (at 269.24 215.9 0)
+  (label "~{WED}" (at 269.24 215.9 0)
     (effects (font (size 1.27 1.27)) (justify left bottom))
   )
