File: cores/cps3/sch/simm5.kicad_sch (KiCad schematic)
At the start: 8 parts

Commit message: wip_cassette_sh2
Parts:
- removed JE1, JE2, JE3, JE4, JE5, JE6, JE7, JE8: 29F016-90PFTN, symbol arcade:29F016-90PFTN
- added JC1, JC2, JC3, JC4, JC5, JC6, JC7, JC8: 29F016-90PFTN, symbol arcade:29F016-90PFTN
Connections:
- net OAM_A0: now also JC1.30 (A0), JC2.30 (A0), JC3.30 (A0), JC4.30 (A0), JC5.30 (A0), JC6.30 (A0), JC7.30 (A0), JC8.30 (A0)
- net OAM_A1: now also JC1.29 (A1), JC2.29 (A1), JC3.29 (A1), JC4.29 (A1), JC5.29 (A1), JC6.29 (A1), JC7.29 (A1), JC8.29 (A1)
- net OAM_A10: now also JC1.16 (A10), JC2.16 (A10), JC3.16 (A10), JC4.16 (A10), JC5.16 (A10), JC6.16 (A10), JC7.16 (A10), JC8.16 (A10)
- net OAM_A11: now also JC1.15 (A11), JC2.15 (A11), JC3.15 (A11), JC4.15 (A11), JC5.15 (A11), JC6.15 (A11), JC7.15 (A11), JC8.15 (A11)
- net OAM_A12: now also JC1.10 (A12), JC2.10 (A12), JC3.10 (A12), JC4.10 (A12), JC5.10 (A12), JC6.10 (A12), JC7.10 (A12), JC8.10 (A12)
- net OAM_A13: now also JC1.9 (A13), JC2.9 (A13), JC3.9 (A13), JC4.9 (A13), JC5.9 (A13), JC6.9 (A13), JC7.9 (A13), JC8.9 (A13)
- net OAM_A14: now also JC1.8 (A14), JC2.8 (A14), JC3.8 (A14), JC4.8 (A14), JC5.8 (A14), JC6.8 (A14), JC7.8 (A14), JC8.8 (A14)
- net OAM_A15: now also JC1.7 (A15), JC2.7 (A15), JC3.7 (A15), JC4.7 (A15), JC5.7 (A15), JC6.7 (A15), JC7.7 (A15), JC8.7 (A15)
- net OAM_A16: now also JC1.6 (A16), JC2.6 (A16), JC3.6 (A16), JC4.6 (A16), JC5.6 (A16), JC6.6 (A16), JC7.6 (A16), JC8.6 (A16)
- net OAM_A17: now also JC1.5 (A17), JC2.5 (A17), JC3.5 (A17), JC4.5 (A17), JC5.5 (A17), JC6.5 (A17), JC7.5 (A17), JC8.5 (A17)
- net OAM_A18: now also JC1.4 (A18), JC2.4 (A18), JC3.4 (A18), JC4.4 (A18), JC5.4 (A18), JC6.4 (A18), JC7.4 (A18), JC8.4 (A18)
- net OAM_A19: now also JC1.3 (A19), JC2.3 (A19), JC3.3 (A19), JC4.3 (A19), JC5.3 (A19), JC6.3 (A19), JC7.3 (A19), JC8.3 (A19)
- net OAM_A2: now also JC1.28 (A2), JC2.28 (A2), JC3.28 (A2), JC4.28 (A2), JC5.28 (A2), JC6.28 (A2), JC7.28 (A2), JC8.28 (A2)
- net OAM_A20: now also JC1.46 (A20), JC2.46 (A20), JC3.46 (A20), JC4.46 (A20), JC5.46 (A20), JC6.46 (A20), JC7.46 (A20), JC8.46 (A20)
- net OAM_A3: now also JC1.27 (A3), JC2.27 (A3), JC3.27 (A3), JC4.27 (A3), JC5.27 (A3), JC6.27 (A3), JC7.27 (A3), JC8.27 (A3)
- net OAM_A4: now also JC1.22 (A4), JC2.22 (A4), JC3.22 (A4), JC4.22 (A4), JC5.22 (A4), JC6.22 (A4), JC7.22 (A4), JC8.22 (A4)
- net OAM_A5: now also JC1.21 (A5), JC2.21 (A5), JC3.21 (A5), JC4.21 (A5), JC5.21 (A5), JC6.21 (A5), JC7.21 (A5), JC8.21 (A5)
- net OAM_A6: now also JC1.20 (A6), JC2.20 (A6), JC3.20 (A6), JC4.20 (A6), JC5.20 (A6), JC6.20 (A6), JC7.20 (A6), JC8.20 (A6)
- net OAM_A7: now also JC1.19 (A7), JC2.19 (A7), JC3.19 (A7), JC4.19 (A7), JC5.19 (A7), JC6.19 (A7), JC7.19 (A7), JC8.19 (A7)
- net OAM_A8: now also JC1.18 (A8), JC2.18 (A8), JC3.18 (A8), JC4.18 (A8), JC5.18 (A8), JC6.18 (A8), JC7.18 (A8), JC8.18 (A8)
- net OAM_A9: now also JC1.17 (A9), JC2.17 (A9), JC3.17 (A9), JC4.17 (A9), JC5.17 (A9), JC6.17 (A9), JC7.17 (A9), JC8.17 (A9)
- net SPRITEB_D0: now also JC1.31 (D0), JC3.31 (D0), JC5.31 (D0), JC7.31 (D0)
- net SPRITEB_D1: now also JC1.32 (D1), JC3.32 (D1), JC5.32 (D1), JC7.32 (D1)
- net SPRITEB_D2: now also JC1.33 (D2), JC3.33 (D2), JC5.33 (D2), JC7.33 (D2)
- net SPRITEB_D3: now also JC1.34 (D3), JC3.34 (D3), JC5.34 (D3), JC7.34 (D3)
- net SPRITEB_D4: now also JC1.38 (D4), JC3.38 (D4), JC5.38 (D4), JC7.38 (D4)
- net SPRITEB_D5: now also JC1.39 (D5), JC3.39 (D5), JC5.39 (D5), JC7.39 (D5)
- net SPRITEB_D6: now also JC1.40 (D6), JC3.40 (D6), JC5.40 (D6), JC7.40 (D6)
- net SPRITEB_D7: now also JC1.41 (D7), JC3.41 (D7), JC5.41 (D7), JC7.41 (D7)
- net SPRITED_D0: now also JC2.31 (D0), JC4.31 (D0), JC6.31 (D0), JC8.31 (D0)
- net SPRITED_D1: now also JC2.32 (D1), JC4.32 (D1), JC6.32 (D1), JC8.32 (D1)
- net SPRITED_D2: now also JC2.33 (D2), JC4.33 (D2), JC6.33 (D2), JC8.33 (D2)
- net SPRITED_D3: now also JC2.34 (D3), JC4.34 (D3), JC6.34 (D3), JC8.34 (D3)
- net SPRITED_D4: now also JC2.38 (D4), JC4.38 (D4), JC6.38 (D4), JC8.38 (D4)
- net SPRITED_D5: now also JC2.39 (D5), JC4.39 (D5), JC6.39 (D5), JC8.39 (D5)
- net SPRITED_D6: now also JC2.40 (D6), JC4.40 (D6), JC6.40 (D6), JC8.40 (D6)
- net SPRITED_D7: now also JC2.41 (D7), JC4.41 (D7), JC6.41 (D7), JC8.41 (D7)
- net VCC: now also JC1.12 (VCC), JC1.37 (VCC), JC2.12 (VCC), JC2.37 (VCC), JC3.12 (VCC), JC3.37 (VCC), JC4.12 (VCC), JC4.37 (VCC), JC5.12 (VCC), JC5.37 (VCC), JC6.12 (VCC), JC6.37 (VCC), JC7.12 (VCC), JC7.37 (VCC), JC8.12 (VCC), JC8.37 (VCC)
- net VSS: now also JC1.35 (VSS), JC1.36 (VSS), JC1.42 (RY/~{BY}), JC2.35 (VSS), JC2.36 (VSS), JC2.42 (RY/~{BY}), JC3.35 (VSS), JC3.36 (VSS), JC3.42 (RY/~{BY}), JC4.35 (VSS), JC4.36 (VSS), JC4.42 (RY/~{BY}), JC5.35 (VSS), JC5.36 (VSS), JC5.42 (RY/~{BY}), JC6.35 (VSS), JC6.36 (VSS), JC6.42 (RY/~{BY}), JC7.35 (VSS), JC7.36 (VSS), JC7.42 (RY/~{BY}), JC8.35 (VSS), JC8.36 (VSS), JC8.42 (RY/~{BY})
- new net ~{CEE}: JC1.11 (~{CE}), JC4.11 (~{CE})
- new net ~{CEF}: JC2.11 (~{CE}), JC3.11 (~{CE})
- new net ~{CEG}: JC5.11 (~{CE}), JC8.11 (~{CE})
- new net ~{CEH}: JC6.11 (~{CE}), JC7.11 (~{CE})
- new net ~{OEC}: JC1.43 (~{OE}), JC2.43 (~{OE}), JC3.43 (~{OE}), JC4.43 (~{OE}), JC5.43 (~{OE}), JC6.43 (~{OE}), JC7.43 (~{OE}), JC8.43 (~{OE})
- new net ~{RESET2}: JC1.14 (~{RESET}), JC2.14 (~{RESET}), JC3.14 (~{RESET}), JC4.14 (~{RESET}), JC5.14 (~{RESET}), JC6.14 (~{RESET}), JC7.14 (~{RESET}), JC8.14 (~{RESET})
- new net ~{WEC}: JC1.44 (~{WE}), JC2.44 (~{WE}), JC3.44 (~{WE}), JC4.44 (~{WE}), JC5.44 (~{WE}), JC6.44 (~{WE}), JC7.44 (~{WE}), JC8.44 (~{WE})
Other:
- note added: "Simm 5"
- note removed: "Simm 3"
