File: cores/cps3/sch/simm5.kicad_sch (KiCad schematic)
At the start: 8 parts

Commit message: cps3_finished
Connections:
- no-connect marks 7 -> 8
Changed lines of the file:
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@@
     (company "JOTEGO")
     (comment 1 "E.Triana")
+    (comment 2 "14/10/22-30/01/23")
   )
   (junction (at 195.58 238.76) (diameter 0) (color 0 0 0 0)
@@
   )
   (no_connect (at 176.53 185.42))
+  (no_connect (at 245.11 185.42))
   (no_connect (at 107.95 185.42))
   (no_connect (at 313.69 82.55))
