File: cores/cps3/sch/simm6.kicad_sch (KiCad schematic)
At the start: 8 parts

Commit message: wip_cassette_sh2
Parts:
- removed JE1, JE2, JE3, JE4, JE5, JE6, JE7, JE8: 29F016-90PFTN, symbol arcade:29F016-90PFTN
- added JB1, JB2, JB3, JB4, JB5, JB6, JB7, JB8: 29F016-90PFTN, symbol arcade:29F016-90PFTN
Connections:
- net VCC: now also JB1.12 (VCC), JB1.37 (VCC), JB2.12 (VCC), JB2.37 (VCC), JB3.12 (VCC), JB3.37 (VCC), JB4.12 (VCC), JB4.37 (VCC), JB5.12 (VCC), JB5.37 (VCC), JB6.12 (VCC), JB6.37 (VCC), JB7.12 (VCC), JB7.37 (VCC), JB8.12 (VCC), JB8.37 (VCC)
- net VSS: now also JB1.35 (VSS), JB1.36 (VSS), JB1.42 (RY/~{BY}), JB2.35 (VSS), JB2.36 (VSS), JB2.42 (RY/~{BY}), JB3.35 (VSS), JB3.36 (VSS), JB3.42 (RY/~{BY}), JB4.35 (VSS), JB4.36 (VSS), JB4.42 (RY/~{BY}), JB5.35 (VSS), JB5.36 (VSS), JB5.42 (RY/~{BY}), JB6.35 (VSS), JB6.36 (VSS), JB6.42 (RY/~{BY}), JB7.35 (VSS), JB7.36 (VSS), JB7.42 (RY/~{BY}), JB8.35 (VSS), JB8.36 (VSS), JB8.42 (RY/~{BY})
- new net OAMB_A0: JB1.30 (A0), JB2.30 (A0), JB3.30 (A0), JB4.30 (A0), JB5.30 (A0), JB6.30 (A0), JB7.30 (A0), JB8.30 (A0)
- new net OAMB_A1: JB1.29 (A1), JB2.29 (A1), JB3.29 (A1), JB4.29 (A1), JB5.29 (A1), JB6.29 (A1), JB7.29 (A1), JB8.29 (A1)
- new net OAMB_A10: JB1.16 (A10), JB2.16 (A10), JB3.16 (A10), JB4.16 (A10), JB5.16 (A10), JB6.16 (A10), JB7.16 (A10), JB8.16 (A10)
- new net OAMB_A11: JB1.15 (A11), JB2.15 (A11), JB3.15 (A11), JB4.15 (A11), JB5.15 (A11), JB6.15 (A11), JB7.15 (A11), JB8.15 (A11)
- new net OAMB_A12: JB1.10 (A12), JB2.10 (A12), JB3.10 (A12), JB4.10 (A12), JB5.10 (A12), JB6.10 (A12), JB7.10 (A12), JB8.10 (A12)
- new net OAMB_A13: JB1.9 (A13), JB2.9 (A13), JB3.9 (A13), JB4.9 (A13), JB5.9 (A13), JB6.9 (A13), JB7.9 (A13), JB8.9 (A13)
- new net OAMB_A14: JB1.8 (A14), JB2.8 (A14), JB3.8 (A14), JB4.8 (A14), JB5.8 (A14), JB6.8 (A14), JB7.8 (A14), JB8.8 (A14)
- new net OAMB_A15: JB1.7 (A15), JB2.7 (A15), JB3.7 (A15), JB4.7 (A15), JB5.7 (A15), JB6.7 (A15), JB7.7 (A15), JB8.7 (A15)
- new net OAMB_A16: JB1.6 (A16), JB2.6 (A16), JB3.6 (A16), JB4.6 (A16), JB5.6 (A16), JB6.6 (A16), JB7.6 (A16), JB8.6 (A16)
- new net OAMB_A17: JB1.5 (A17), JB2.5 (A17), JB3.5 (A17), JB4.5 (A17), JB5.5 (A17), JB6.5 (A17), JB7.5 (A17), JB8.5 (A17)
- new net OAMB_A18: JB1.4 (A18), JB2.4 (A18), JB3.4 (A18), JB4.4 (A18), JB5.4 (A18), JB6.4 (A18), JB7.4 (A18), JB8.4 (A18)
- new net OAMB_A19: JB1.3 (A19), JB2.3 (A19), JB3.3 (A19), JB4.3 (A19), JB5.3 (A19), JB6.3 (A19), JB7.3 (A19), JB8.3 (A19)
- new net OAMB_A2: JB1.28 (A2), JB2.28 (A2), JB3.28 (A2), JB4.28 (A2), JB5.28 (A2), JB6.28 (A2), JB7.28 (A2), JB8.28 (A2)
- new net OAMB_A20: JB1.46 (A20), JB2.46 (A20), JB3.46 (A20), JB4.46 (A20), JB5.46 (A20), JB6.46 (A20), JB7.46 (A20), JB8.46 (A20)
- new net OAMB_A3: JB1.27 (A3), JB2.27 (A3), JB3.27 (A3), JB4.27 (A3), JB5.27 (A3), JB6.27 (A3), JB7.27 (A3), JB8.27 (A3)
- new net OAMB_A4: JB1.22 (A4), JB2.22 (A4), JB3.22 (A4), JB4.22 (A4), JB5.22 (A4), JB6.22 (A4), JB7.22 (A4), JB8.22 (A4)
- new net OAMB_A5: JB1.21 (A5), JB2.21 (A5), JB3.21 (A5), JB4.21 (A5), JB5.21 (A5), JB6.21 (A5), JB7.21 (A5), JB8.21 (A5)
- new net OAMB_A6: JB1.20 (A6), JB2.20 (A6), JB3.20 (A6), JB4.20 (A6), JB5.20 (A6), JB6.20 (A6), JB7.20 (A6), JB8.20 (A6)
- new net OAMB_A7: JB1.19 (A7), JB2.19 (A7), JB3.19 (A7), JB4.19 (A7), JB5.19 (A7), JB6.19 (A7), JB7.19 (A7), JB8.19 (A7)
- new net OAMB_A8: JB1.18 (A8), JB2.18 (A8), JB3.18 (A8), JB4.18 (A8), JB5.18 (A8), JB6.18 (A8), JB7.18 (A8), JB8.18 (A8)
- new net OAMB_A9: JB1.17 (A9), JB2.17 (A9), JB3.17 (A9), JB4.17 (A9), JB5.17 (A9), JB6.17 (A9), JB7.17 (A9), JB8.17 (A9)
- new net SPRITEA_D0: JB1.31 (D0), JB3.31 (D0), JB5.31 (D0), JB7.31 (D0)
- new net SPRITEA_D1: JB1.32 (D1), JB3.32 (D1), JB5.32 (D1), JB7.32 (D1)
- new net SPRITEA_D2: JB1.33 (D2), JB3.33 (D2), JB5.33 (D2), JB7.33 (D2)
- new net SPRITEA_D3: JB1.34 (D3), JB3.34 (D3), JB5.34 (D3), JB7.34 (D3)
- new net SPRITEA_D4: JB1.38 (D4), JB3.38 (D4), JB5.38 (D4), JB7.38 (D4)
- new net SPRITEA_D5: JB1.39 (D5), JB3.39 (D5), JB5.39 (D5), JB7.39 (D5)
- new net SPRITEA_D6: JB1.40 (D6), JB3.40 (D6), JB5.40 (D6), JB7.40 (D6)
- new net SPRITEA_D7: JB1.41 (D7), JB3.41 (D7), JB5.41 (D7), JB7.41 (D7)
- new net SPRITEC_D0: JB2.31 (D0), JB4.31 (D0), JB6.31 (D0), JB8.31 (D0)
- new net SPRITEC_D1: JB2.32 (D1), JB4.32 (D1), JB6.32 (D1), JB8.32 (D1)
- new net SPRITEC_D2: JB2.33 (D2), JB4.33 (D2), JB6.33 (D2), JB8.33 (D2)
- new net SPRITEC_D3: JB2.34 (D3), JB4.34 (D3), JB6.34 (D3), JB8.34 (D3)
- new net SPRITEC_D4: JB2.38 (D4), JB4.38 (D4), JB6.38 (D4), JB8.38 (D4)
- new net SPRITEC_D5: JB2.39 (D5), JB4.39 (D5), JB6.39 (D5), JB8.39 (D5)
- new net SPRITEC_D6: JB2.40 (D6), JB4.40 (D6), JB6.40 (D6), JB8.40 (D6)
- new net SPRITEC_D7: JB2.41 (D7), JB4.41 (D7), JB6.41 (D7), JB8.41 (D7)
- new net ~{CEA}: JB1.11 (~{CE}), JB4.11 (~{CE})
- new net ~{CEB}: JB2.11 (~{CE}), JB3.11 (~{CE})
- new net ~{CEC}: JB5.11 (~{CE}), JB8.11 (~{CE})
- new net ~{CED}: JB6.11 (~{CE}), JB7.11 (~{CE})
- new net ~{OEB}: JB1.43 (~{OE}), JB2.43 (~{OE}), JB3.43 (~{OE}), JB4.43 (~{OE}), JB5.43 (~{OE}), JB6.43 (~{OE}), JB7.43 (~{OE}), JB8.43 (~{OE})
- new net ~{RESET1}: JB1.14 (~{RESET}), JB2.14 (~{RESET}), JB3.14 (~{RESET}), JB4.14 (~{RESET}), JB5.14 (~{RESET}), JB6.14 (~{RESET}), JB7.14 (~{RESET}), JB8.14 (~{RESET})
- new net ~{WEB}: JB1.44 (~{WE}), JB2.44 (~{WE}), JB3.44 (~{WE}), JB4.44 (~{WE}), JB5.44 (~{WE}), JB6.44 (~{WE}), JB7.44 (~{WE}), JB8.44 (~{WE})
Other:
- note added: "Simm 6"
- note removed: "Simm 3"
