File: cores/cps3/sch/simm6.kicad_sch (KiCad schematic)
At the start: 8 parts

Commit message: wip_cre_cps3
Connections:
- net VSS: no longer JB1.42 (RY/~{BY}), JB2.42 (RY/~{BY}), JB3.42 (RY/~{BY}), JB4.42 (RY/~{BY}), JB5.42 (RY/~{BY}), JB6.42 (RY/~{BY}), JB7.42 (RY/~{BY}), JB8.42 (RY/~{BY})
- net OAMB_A0 renamed 2SPRITE_AB0
- net OAMB_A1 renamed 2SPRITE_AB1
- net OAMB_A10 renamed 2SPRITE_AB10
- net OAMB_A11 renamed 2SPRITE_AB11
- net OAMB_A12 renamed 2SPRITE_AB12
- net OAMB_A13 renamed 2SPRITE_AB13
- net OAMB_A14 renamed 2SPRITE_AB14
- net OAMB_A15 renamed 2SPRITE_AB15
- net OAMB_A16 renamed 2SPRITE_AB16
- net OAMB_A17 renamed 2SPRITE_AB17
- net OAMB_A18 renamed 2SPRITE_AB18
- net OAMB_A19 renamed 2SPRITE_AB19
- net OAMB_A2 renamed 2SPRITE_AB2
- net OAMB_A20 renamed 2SPRITE_AB20
- net OAMB_A3 renamed 2SPRITE_AB3
- net OAMB_A4 renamed 2SPRITE_AB4
- net OAMB_A5 renamed 2SPRITE_AB5
- net OAMB_A6 renamed 2SPRITE_AB6
- net OAMB_A7 renamed 2SPRITE_AB7
- net OAMB_A8 renamed 2SPRITE_AB8
- net OAMB_A9 renamed 2SPRITE_AB9
- no-connect marks 0 -> 8
Other:
- note added: "VSS"
