File: cores/cps3/sch/h_description.kicad_sch (KiCad schematic)
At the start: 0 parts

Commit message: clear_sch_hk_cr
Other:
- removed sheet gll1
- removed sheet gll2
- note added: "1. JoJo no Kimyouna Bouken / JoJo's Venture 2. JoJo no Kimyouna Bouken Miraie no Isan / JoJo's Bizarre Adventure. 3. Street Fighter III 2nd Impact: Giant Attack. 4. Street Fighter III 3rd Strike: Fight for the Future. 5. Street Fighter III : New Generation. 6. Warzard / Red Earth"
- note added: "Font: The Museum Arcade System 16"
- note added: "HARDWARE DESCRIPTION"
- note added: "KNOWN CP SYSTEM III (CPS3) GAME LIST"
- note added: "Main CPU : Hitachi SH2 @ 25 MHz Storage : SCSI CD Rom, RAM and Flash ROM. RAM : SIMMs on the left will physically hold 16M of data each (each has 8x 16M Flash ROMs, there's 4 SIMMs plugged in on this board). The SIMMs on the right will physically hold 8M each (there's 4 Flash ROMs on each board and there are 2 SIMMs plugged in) OSC : 60MHz. 42.9545MHz, XTAL :3.6864MHz"
Changed lines of the file:
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@@
 (kicad_sch (version 20211123) (generator eeschema)
-  (paper "A3")
+  (paper "A5")
   (title_block
     (title "CP SYSTEM III")
@@
     (comment 1 "E.Triana")
   )
-  (wire (pts (xy 130.81 91.44) (xy 139.7 91.44))
-    (stroke (width 0) (type default) (color 0 0 0 0))
-  )
-  (wire (pts (xy 130.81 96.52) (xy 139.7 96.52))
-    (stroke (width 0) (type default) (color 0 0 0 0))
-  )
-  (bus (pts (xy 176.53 93.98) (xy 182.88 93.98))
-    (stroke (width 0) (type default) (color 0 0 0 0))
-  )
-  (bus (pts (xy 176.53 91.44) (xy 182.88 91.44))
-    (stroke (width 0) (type default) (color 0 0 0 0))
-  )
-  (bus (pts (xy 247.65 91.44) (xy 254 91.44))
-    (stroke (width 0) (type default) (color 0 0 0 0))
-  )
-  (wire (pts (xy 176.53 96.52) (xy 182.88 96.52))
-    (stroke (width 0) (type default) (color 0 0 0 0))
-  )
-  (wire (pts (xy 130.81 93.98) (xy 139.7 93.98))
-    (stroke (width 0) (type default) (color 0 0 0 0))
-  )
-  (image (at 398.78 261.62) (scale 0.294008)
+  (image (at 187.96 111.76) (scale 0.294008)
     (data
       iVBORw0KGgoAAAANSUhEUgAAAtEAAAGsCAMAAAAsQwu3AAAAA3NCSVQICAjb4U/gAAADAFBMVEX/
@@
     )
   )
-  (hierarchical_label "MAIN_D[23..0]" (shape bidirectional) (at 182.88 91.44 0)
-    (effects (font (size 1.27 1.27)) (justify left))
-  )
-  (hierarchical_label "2GLL_A[5..0]" (shape bidirectional) (at 247.65 91.44 180)
-    (effects (font (size 1.27 1.27)) (justify right))
-  )
-  (hierarchical_label "RESET?" (shape tri_state) (at 130.81 91.44 180)
-    (effects (font (size 1.27 1.27)) (justify right))
-  )
-  (hierarchical_label "GLL2IO1" (shape bidirectional) (at 130.81 96.52 180)
-    (effects (font (size 1.27 1.27)) (justify right))
-  )
-  (hierarchical_label "GFX_A[20..0]" (shape tri_state) (at 182.88 93.98 0)
-    (effects (font (size 1.27 1.27)) (justify left))
-  )
-  (hierarchical_label "CBI_CLK" (shape output) (at 182.88 96.52 0)
-    (effects (font (size 1.27 1.27)) (justify left))
-  )
-  (hierarchical_label "GLL2IO0" (shape tri_state) (at 130.81 93.98 180)
-    (effects (font (size 1.27 1.27)) (justify right))
-  )
-  (sheet (at 254 88.9) (size 36.83 44.45) (fields_autoplaced)
-    (stroke (width 0.1524) (type solid) (color 0 0 0 0))
-    (fill (color 0 0 0 0.0000))
-    (property "Sheet name" "gll2" (id 0) (at 254 88.1884 0)
-      (effects (font (size 1.27 1.27)) (justify left bottom))
-    )
-    (property "Sheet file" "gll2.kicad_sch" (id 1) (at 254 133.9346 0)
-      (effects (font (size 1.27 1.27)) (justify left top))
-    )
-    (pin "2GLL_A[5..0]" bidirectional (at 254 91.44 180)
-      (effects (font (size 1.27 1.27)) (justify left))
-    )
-  )
-  (sheet (at 139.7 88.9) (size 36.83 44.45) (fields_autoplaced)
-    (stroke (width 0.1524) (type solid) (color 0 0 0 0))
-    (fill (color 0 0 0 0.0000))
-    (property "Sheet name" "gll1" (id 0) (at 139.7 88.1884 0)
-      (effects (font (size 1.27 1.27)) (justify left bottom))
-    )
-    (property "Sheet file" "gll1.kicad_sch" (id 1) (at 139.7 133.9346 0)
-      (effects (font (size 1.27 1.27)) (justify left top))
-    )
-    (pin "CBI_CLK" output (at 176.53 96.52 0)
-      (effects (font (size 1.27 1.27)) (justify right))
-    )
-    (pin "MAIN_D[23..0]" bidirectional (at 176.53 91.44 0)
-      (effects (font (size 1.27 1.27)) (justify right))
-    )
-    (pin "GFX_A[20..0]" bidirectional (at 176.53 93.98 0)
-      (effects (font (size 1.27 1.27)) (justify right))
-    )
-    (pin "RESET?" input (at 139.7 91.44 180)
-      (effects (font (size 1.27 1.27)) (justify left))
-    )
-    (pin "GLL2IO0" input (at 139.7 93.98 180)
-      (effects (font (size 1.27 1.27)) (justify left))
-    )
-    (pin "GLL2IO1" input (at 139.7 96.52 180)
-      (effects (font (size 1.27 1.27)) (justify left))
-    )
+  (text "HARDWARE DESCRIPTION" (at 26.035 31.115 0)
+    (effects (font (size 3 3) (thickness 0.6) bold) (justify left bottom))
+  )
+  (text "1. JoJo no Kimyouna Bouken / JoJo's Venture\n2. JoJo no Kimyouna Bouken Miraie no Isan /\n   JoJo's Bizarre Adventure.\n3. Street Fighter III 2nd Impact: Giant Attack.\n4. Street Fighter III 3rd Strike: Fight for the Future.\n5. Street Fighter III : New Generation.\n6. Warzard / Red Earth "
+    (at 110.49 62.23 0)
+    (effects (font (size 2 2) italic) (justify left bottom))
+  )
+  (text "Font:\nThe Museum Arcade System 16\n\n" (at 101.6 86.36 0)
+    (effects (font (size 2 2) bold) (justify left bottom))
+  )
+  (text "Main CPU : Hitachi SH2 @ 25 MHz\nStorage : SCSI CD Rom, RAM and Flash ROM.\nRAM : SIMMs on the left will physically \nhold 16M of data each (each has 8x 16M\nFlash ROMs, there's 4 SIMMs plugged in on \nthis board). The SIMMs on the right will\nphysically hold 8M each (there's 4 Flash \nROMs on each board and there are 2 SIMMs \nplugged in)\nOSC : 60MHz. 42.9545MHz, XTAL :3.6864MHz"
+    (at 18.415 71.755 0)
+    (effects (font (size 2 2) italic) (justify left bottom))
+  )
+  (text "KNOWN CP SYSTEM III (CPS3) GAME LIST" (at 101.6 30.48 0)
+    (effects (font (size 3 3) bold) (justify left bottom))
   )
 )

Commit message: wip_cassette_sh2
Changed lines of the file:
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@@
 (kicad_sch (version 20211123) (generator eeschema)
-  (paper "A5")
+  (paper "A3")
   (title_block
     (title "CP SYSTEM III")
@@
     (comment 1 "E.Triana")
   )
-  (image (at 187.96 111.76) (scale 0.294008)
+  (image (at 397.51 261.62) (scale 0.294008)
     (data
       iVBORw0KGgoAAAANSUhEUgAAAtEAAAGsCAMAAAAsQwu3AAAAA3NCSVQICAjb4U/gAAADAFBMVEX/
@@
     )
   )
-  (text "HARDWARE DESCRIPTION" (at 26.035 31.115 0)
+  (text "HARDWARE DESCRIPTION" (at 114.3 110.49 0)
     (effects (font (size 3 3) (thickness 0.6) bold) (justify left bottom))
   )
   (text "1. JoJo no Kimyouna Bouken / JoJo's Venture\n2. JoJo no Kimyouna Bouken Miraie no Isan /\n   JoJo's Bizarre Adventure.\n3. Street Fighter III 2nd Impact: Giant Attack.\n4. Street Fighter III 3rd Strike: Fight for the Future.\n5. Street Fighter III : New Generation.\n6. Warzard / Red Earth "
-    (at 110.49 62.23 0)
+    (at 229.87 140.97 0)
     (effects (font (size 2 2) italic) (justify left bottom))
   )
-  (text "Font:\nThe Museum Arcade System 16\n\n" (at 101.6 86.36 0)
+  (text "Font:\nThe Museum Arcade System 16\n\n" (at 220.98 165.1 0)
     (effects (font (size 2 2) bold) (justify left bottom))
   )
   (text "Main CPU : Hitachi SH2 @ 25 MHz\nStorage : SCSI CD Rom, RAM and Flash ROM.\nRAM : SIMMs on the left will physically \nhold 16M of data each (each has 8x 16M\nFlash ROMs, there's 4 SIMMs plugged in on \nthis board). The SIMMs on the right will\nphysically hold 8M each (there's 4 Flash \nROMs on each board and there are 2 SIMMs \nplugged in)\nOSC : 60MHz. 42.9545MHz, XTAL :3.6864MHz"
-    (at 18.415 71.755 0)
+    (at 106.68 151.13 0)
     (effects (font (size 2 2) italic) (justify left bottom))
   )
-  (text "KNOWN CP SYSTEM III (CPS3) GAME LIST" (at 101.6 30.48 0)
+  (text "KNOWN CP SYSTEM III (CPS3) GAME LIST" (at 220.98 109.22 0)
     (effects (font (size 3 3) bold) (justify left bottom))
   )

Commit message: correction_ppu
Other:
- note added: "All six games are developed by Capcom and are all head-to-head fighting games in a list of games that appears to be as small as the CP System Dash library."
- note added: "Main CPU : Main CPU: Hitachi HD6417099 (SH-2) at 25 MHz Storage : SCSI CD Rom, RAM and Flash ROM. RAM : SIMMs on the left will physically hold 16M of data each (each has 8x 16M Flash ROMs, there's 4 SIMMs plugged in on this board). The SIMMs on the right will physically hold 8M each (there's 4 Flash ROMs on each board and there are 2 SIMMs plugged in) OSC : 60MHz. 42.9545MHz, XTAL :3.6864MHz *Sou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"
- note removed: "1. JoJo no Kimyouna Bouken / JoJo's Venture 2. JoJo no Kimyouna Bouken Miraie no Isan / JoJo's Bizarre Adventure. 3. Street Fighter III 2nd Impact: Giant Attack. 4. Street Fighter III 3rd Strike: Fight for the Future. 5. Street Fighter III : New Generation. 6. Warzard / Red Earth"
- note removed: "Main CPU : Hitachi SH2 @ 25 MHz Storage : SCSI CD Rom, RAM and Flash ROM. RAM : SIMMs on the left will physically hold 16M of data each (each has 8x 16M Flash ROMs, there's 4 SIMMs plugged in on this board). The SIMMs on the right will physically hold 8M each (there's 4 Flash ROMs on each board and there are 2 SIMMs plugged in) OSC : 60MHz. 42.9545MHz, XTAL :3.6864MHz"
