File: cores/cps3/sch/buffer_line_driver.kicad_sch (KiCad schematic)
At the start: 3 parts

Commit message: wip_cre_cps3
Connections:
- net OAMB_A0 renamed 2SPRITE_AB0
- net OAMB_A1 renamed 2SPRITE_AB1
- net OAMB_A10 renamed 2SPRITE_AB10
- net OAMB_A11 renamed 2SPRITE_AB11
- net OAMB_A12 renamed 2SPRITE_AB12
- net OAMB_A13 renamed 2SPRITE_AB13
- net OAMB_A14 renamed 2SPRITE_AB14
- net OAMB_A15 renamed 2SPRITE_AB15
- net OAMB_A16 renamed 2SPRITE_AB16
- net OAMB_A17 renamed 2SPRITE_AB17
- net OAMB_A18 renamed 2SPRITE_AB18
- net OAMB_A19 renamed 2SPRITE_AB19
- net OAMB_A2 renamed 2SPRITE_AB2
- net OAMB_A20 renamed 2SPRITE_AB20
- net OAMB_A3 renamed 2SPRITE_AB3
- net OAMB_A4 renamed 2SPRITE_AB4
- net OAMB_A5 renamed 2SPRITE_AB5
- net OAMB_A6 renamed 2SPRITE_AB6
- net OAMB_A7 renamed 2SPRITE_AB7
- net OAMB_A8 renamed 2SPRITE_AB8
- net OAMB_A9 renamed 2SPRITE_AB9
- net OAM_A0 renamed SPRITE_AB0
- net OAM_A1 renamed SPRITE_AB1
- net OAM_A10 renamed SPRITE_AB10
- net OAM_A11 renamed SPRITE_AB11
- net OAM_A12 renamed SPRITE_AB12
- net OAM_A13 renamed SPRITE_AB13
- net OAM_A14 renamed SPRITE_AB14
- net OAM_A15 renamed SPRITE_AB15
- net OAM_A16 renamed SPRITE_AB16
- net OAM_A17 renamed SPRITE_AB17
- net OAM_A18 renamed SPRITE_AB18
- net OAM_A19 renamed SPRITE_AB19
- net OAM_A2 renamed SPRITE_AB2
- net OAM_A20 renamed SPRITE_AB20
- net OAM_A3 renamed SPRITE_AB3
- net OAM_A4 renamed SPRITE_AB4
- net OAM_A5 renamed SPRITE_AB5
- net OAM_A6 renamed SPRITE_AB6
- net OAM_A7 renamed SPRITE_AB7
- net OAM_A8 renamed SPRITE_AB8
- net OAM_A9 renamed SPRITE_AB9
- net PPU0 renamed SPRITE_A0
- net PPU1 renamed SPRITE_A1
- net PPU10 renamed SPRITE_A10
- net PPU11 renamed SPRITE_A11
- net PPU12 renamed SPRITE_A12
- net PPU13 renamed SPRITE_A13
- net PPU14 renamed SPRITE_A14
- net PPU15 renamed SPRITE_A15
- net PPU16 renamed SPRITE_A16
- net PPU17 renamed SPRITE_A17
- net PPU18 renamed SPRITE_A18
- net PPU19 renamed SPRITE_A19
- net PPU2 renamed SPRITE_A2
- net PPU20 renamed SPRITE_A20
- net PPU3 renamed SPRITE_A3
- net PPU4 renamed SPRITE_A4
- net PPU5 renamed SPRITE_A5
- net PPU6 renamed SPRITE_A6
- net PPU7 renamed SPRITE_A7
- net PPU8 renamed SPRITE_A8
- net PPU9 renamed SPRITE_A9
Other:
- note removed: "Object Attribute Memory?"
