File: cores/cps3/sch/buffer_line_driver.kicad_sch (KiCad schematic)
At the start: 3 parts

Commit message: cps3_finished
Changed lines of the file:
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@@
     (company "JOTEGO")
     (comment 1 "E.Triana")
+    (comment 2 "14/10/22-30/01/23")
   )
   (junction (at 185.42 69.85) (diameter 0) (color 0 0 0 0)
@@
     (effects (font (size 1.27 1.27)) (justify left bottom))
   )
-  (label "VCC" (at 199.39 24.13 0)
-    (effects (font (size 1.27 1.27)) (justify left bottom))
-  )
   (label "VSS" (at 168.91 53.34 0)
     (effects (font (size 1.27 1.27)) (justify left bottom))
@@
   )
   (label "SPRITE_AB4" (at 224.79 68.58 0)
-    (effects (font (size 1.27 1.27)) (justify left bottom))
-  )
-  (label "VSS" (at 199.39 275.59 0)
     (effects (font (size 1.27 1.27)) (justify left bottom))
   )
@@
     (pin "9")
   )
+  (symbol (lib_id "power:VSS") (at 199.39 275.59 180) (unit 1)
+    (in_bom yes) (on_board yes)
+    (property "Reference" "#PWR0159" (id 0) (at 199.39 271.78 0)
+      (effects (font (size 1.27 1.27)) hide)
+    )
+    (property "Value" "VSS" (id 1) (at 199.39 279.4 0))
+    (property "Footprint" "" (id 2) (at 199.39 275.59 0)
+      (effects (font (size 1.27 1.27)) hide)
+    )
+    (property "Datasheet" "" (id 3) (at 199.39 275.59 0)
+      (effects (font (size 1.27 1.27)) hide)
+    )
+    (pin "1")
+  )
   (symbol (lib_name "74FCT-16244ATPV_2") (lib_id "arcade:74FCT-16244ATPV") (at 199.39 149.86 0) (unit 1)
     (in_bom yes) (on_board yes)
@@
     (pin "9")
   )
+  (symbol (lib_id "power:VCC") (at 199.39 24.13 0) (unit 1)
+    (in_bom yes) (on_board yes)
+    (property "Reference" "#PWR0158" (id 0) (at 199.39 27.94 0)
+      (effects (font (size 1.27 1.27)) hide)
+    )
+    (property "Value" "VCC" (id 1) (at 199.39 20.32 0))
+    (property "Footprint" "" (id 2) (at 199.39 24.13 0)
+      (effects (font (size 1.27 1.27)) hide)
+    )
+    (property "Datasheet" "" (id 3) (at 199.39 24.13 0)
+      (effects (font (size 1.27 1.27)) hide)
+    )
+    (pin "1")
+  )
   (symbol (lib_name "74FCT-16244ATPV_1") (lib_id "arcade:74FCT-16244ATPV") (at 199.39 234.95 0) (unit 1)
