File: cores/cps3/sch/memories_fb.kicad_sch (KiCad schematic)
At the start: 4 parts

Commit message: wip_ccu
Parts:
- added R60, R61, R62: 330Ω, symbol Device:R_US
Connections:
- net PPU_A8: now also R61.1; no longer D2.27 (A8)
- net PPU_A9: now also R62.1; no longer D2.28 (A9)
- net ~{RAS} renamed ~{RAS_MAIN}
- net ~{RAS_MAIN}: now also R60.1; no longer D2.14 (~{RAS})
- new net: D2.28 (A9), R62.2
- new net: D2.14 (~{RAS}), R60.2
- new net: D2.27 (A8), R61.2
Other:
- moved on the sheet: D2, D3, D4, D5

Commit message: wip_ccu_gll2_cassette
Parts:
- R60, R61, R62: value 330Ω -> 330
Connections:
- net PPU_A0 renamed PPU2CCU1
Changed lines of the file:
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@@
     (effects (font (size 1.27 1.27)) (justify left bottom))
   )
-  (label "PPU_A0" (at 83.82 38.1 0)
+  (label "PPU2CCU1" (at 83.82 38.1 0)
     (effects (font (size 1.27 1.27)) (justify left bottom))
   )
@@
     (effects (font (size 1.27 1.27)) (justify right bottom))
   )
-  (label "PPU_A0" (at 166.37 105.41 0)
+  (label "PPU2CCU1" (at 166.37 105.41 0)
     (effects (font (size 1.27 1.27)) (justify left bottom))
   )
@@
     (effects (font (size 1.27 1.27)) (justify right bottom))
   )
-  (label "PPU_A0" (at 166.37 38.1 0)
+  (label "PPU2CCU1" (at 166.37 38.1 0)
     (effects (font (size 1.27 1.27)) (justify left bottom))
   )
@@
     (effects (font (size 1.27 1.27)) (justify left bottom))
   )
-  (label "PPU_A0" (at 83.82 102.87 0)
+  (label "PPU2CCU1" (at 83.82 102.87 0)
     (effects (font (size 1.27 1.27)) (justify left bottom))
   )
@@
     (in_bom yes) (on_board yes)
     (property "Reference" "R62" (id 0) (at 78.74 59.69 90))
-    (property "Value" "330Ω" (id 1) (at 91.44 59.69 90))
+    (property "Value" "330" (id 1) (at 91.44 59.69 90))
     (property "Footprint" "" (id 2) (at 85.344 59.944 90)
       (effects (font (size 1.27 1.27)) hide)
@@
     (in_bom yes) (on_board yes)
     (property "Reference" "R60" (id 0) (at 78.74 64.77 90))
-    (property "Value" "330Ω" (id 1) (at 91.44 64.77 90))
+    (property "Value" "330" (id 1) (at 91.44 64.77 90))
     (property "Footprint" "" (id 2) (at 85.344 65.024 90)
       (effects (font (size 1.27 1.27)) hide)
@@
     (in_bom yes) (on_board yes)
     (property "Reference" "R61" (id 0) (at 78.74 57.15 90))
-    (property "Value" "330Ω" (id 1) (at 91.44 57.15 90))
+    (property "Value" "330" (id 1) (at 91.44 57.15 90))
     (property "Footprint" "" (id 2) (at 85.344 57.404 90)
       (effects (font (size 1.27 1.27)) hide)

Commit message: wip_cassette
Connections:
- net ~{WE}_B: no longer D5.13 (~{WE})
- net ~{WE}_A renamed ~{WE}_PPU_A
- new net ~{WE}_PPU_B: D5.13 (~{WE})

Commit message: wip_cassette_sh2
Other:
- note added: "MEMORIES FRAME BUFFER"
- note removed: "MEMORIES FRAME BUFFER?"
- moved on the sheet: D2, D3, D4, D5, R60, R61, R62

Commit message: wip_cre_cps3
Connections:
- net ~{WE}_B is gone; now on net ~{WE}_PPU_B: D3.13 (~{WE})
- net PPU2CCU1 renamed FB_A0
- net PPU_A1 renamed FB_A1
- net PPU_A2 renamed FB_A2
- net PPU_A3 renamed FB_A3
- net PPU_A4 renamed FB_A4
- net PPU_A5 renamed FB_A5
- net PPU_A6 renamed FB_A6
- net PPU_A7 renamed FB_A7
- net PPU_A8 renamed FB_A8
- net PPU_A9 renamed FB_A9
- net PPU_D0 renamed FB_D0
- net PPU_D1 renamed FB_D1
- net PPU_D10 renamed FB_D10
- net PPU_D11 renamed FB_D11
- net PPU_D12 renamed FB_D12
- net PPU_D13 renamed FB_D13
- net PPU_D14 renamed FB_D14
- net PPU_D15 renamed FB_D15
- net PPU_D16 renamed FB_D16
- net PPU_D17 renamed FB_D17
- net PPU_D18 renamed FB_D18
- net PPU_D19 renamed FB_D19
- net PPU_D2 renamed FB_D2
- net PPU_D20 renamed FB_D20
- net PPU_D21 renamed FB_D21
- net PPU_D22 renamed FB_D22
- net PPU_D23 renamed FB_D23
- net PPU_D24 renamed FB_D24
- net PPU_D25 renamed FB_D25
- net PPU_D26 renamed FB_D26
- net PPU_D27 renamed FB_D27
- net PPU_D28 renamed FB_D28
- net PPU_D29 renamed FB_D29
- net PPU_D3 renamed FB_D3
- net PPU_D30 renamed FB_D30
- net PPU_D31 renamed FB_D31
- net PPU_D4 renamed FB_D4
- net PPU_D5 renamed FB_D5
- net PPU_D6 renamed FB_D6
- net PPU_D7 renamed FB_D7
- net PPU_D8 renamed FB_D8
- net PPU_D9 renamed FB_D9
