File: cores/cps3/sch/simm_connector.kicad_sch (KiCad schematic)
At the start: 12 parts

Commit message: cps3_finished
Parts:
- renumbered SIMM1E to SM1, SIMM2D to SM2, SIMM3E to SM3, SIMM4D to SM4, SIMM5C to SM5, SIMM6B to SM6, SIMM1E to SMM1, SIMM2D to SMM2, SIMM3EE to SMM3, SIMM4DD to SMM4, SIMM5CC to SMM5, SIMM6BB to SMM6
Changed lines of the file:
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@@
     (company "JOTEGO")
     (comment 1 "E.Triana")
+    (comment 2 "14/10/22-30/01/23")
   )
   (junction (at 250.19 40.64) (diameter 0) (color 0 0 0 0)
   )
-  (junction (at 288.29 234.95) (diameter 0) (color 0 0 0 0)
-  )
   (junction (at 247.65 234.95) (diameter 0) (color 0 0 0 0)
   )
@@
     (stroke (width 0) (type default) (color 0 0 0 0))
   )
-  (bus (pts (xy 332.74 198.12) (xy 332.74 234.95))
-    (stroke (width 0) (type default) (color 0 0 0 0))
-  )
   (wire (pts (xy 101.6 53.34) (xy 111.76 53.34))
     (stroke (width 0) (type default) (color 0 0 0 0))
@@
     (stroke (width 0) (type default) (color 0 0 0 0))
   )
-  (bus (pts (xy 288.29 234.95) (xy 332.74 234.95))
-    (stroke (width 0) (type default) (color 0 0 0 0))
-  )
   (wire (pts (xy 101.6 199.39) (xy 110.49 199.39))
     (stroke (width 0) (type default) (color 0 0 0 0))
@@
   (symbol (lib_id "Connector:Conn_01x36_Male") (at 266.7 88.9 0) (unit 1)
     (in_bom yes) (on_board yes)
-    (property "Reference" "SIMM5C" (id 0) (at 266.7 43.18 0))
+    (property "Reference" "SM5" (id 0) (at 266.7 43.18 0))
     (property "Value" "Conn_01x36_Male" (id 1) (at 265.43 86.36 90))
     (property "Footprint" "" (id 2) (at 266.7 88.9 0)
@@
   (symbol (lib_id "Connector:Conn_01x36_Male") (at 157.48 88.9 0) (mirror y) (unit 1)
     (in_bom yes) (on_board yes)
-    (property "Reference" "SIMM2D" (id 0) (at 157.48 43.18 0))
+    (property "Reference" "SM2" (id 0) (at 157.48 43.18 0))
     (property "Value" "Conn_01x36_Male" (id 1) (at 160.02 86.36 90))
     (property "Footprint" "" (id 2) (at 157.48 88.9 0)
@@
   (symbol (lib_id "Connector:Conn_01x36_Male") (at 187.96 185.42 0) (unit 1)
     (in_bom yes) (on_board yes)
-    (property "Reference" "SIMM3EE" (id 0) (at 187.96 139.7 0))
+    (property "Reference" "SMM3" (id 0) (at 187.96 139.7 0))
     (property "Value" "Conn_01x36_Male" (id 1) (at 187.96 233.68 0))
     (property "Footprint" "" (id 2) (at 187.96 185.42 0)
@@
   (symbol (lib_id "Connector:Conn_01x36_Male") (at 187.96 88.9 0) (unit 1)
     (in_bom yes) (on_board yes)
-    (property "Reference" "SIMM3E" (id 0) (at 187.96 43.18 0))
+    (property "Reference" "SM3" (id 0) (at 187.96 43.18 0))
     (property "Value" "Conn_01x36_Male" (id 1) (at 186.69 86.36 90))
     (property "Footprint" "" (id 2) (at 187.96 88.9 0)
@@
   (symbol (lib_id "Connector:Conn_01x36_Male") (at 306.07 185.42 0) (unit 1)
     (in_bom yes) (on_board yes)
-    (property "Reference" "SIMM6BB" (id 0) (at 307.34 139.7 0))
+    (property "Reference" "SMM6" (id 0) (at 307.34 139.7 0))
     (property "Value" "Conn_01x36_Male" (id 1) (at 306.07 233.68 0))
     (property "Footprint" "" (id 2) (at 306.07 185.42 0)
@@
   (symbol (lib_id "Connector:Conn_01x36_Male") (at 267.97 185.42 0) (unit 1)
     (in_bom yes) (on_board yes)
-    (property "Reference" "SIMM5CC" (id 0) (at 267.97 139.7 0))
+    (property "Reference" "SMM5" (id 0) (at 267.97 139.7 0))
     (property "Value" "Conn_01x36_Male" (id 1) (at 268.605 233.68 0))
     (property "Footprint" "" (id 2) (at 267.97 185.42 0)
@@
   (symbol (lib_id "Connector:Conn_01x36_Male") (at 96.52 184.15 0) (unit 1)
     (in_bom yes) (on_board yes)
-    (property "Reference" "SIMM1E" (id 0) (at 96.52 138.43 0))
+    (property "Reference" "SMM1" (id 0) (at 96.52 138.43 0))
     (property "Value" "Conn_01x36_Male" (id 1) (at 96.52 232.41 0))
     (property "Footprint" "" (id 2) (at 96.52 184.15 0)
@@
   (symbol (lib_id "Connector:Conn_01x36_Male") (at 96.52 88.9 0) (unit 1)
     (in_bom yes) (on_board yes)
-    (property "Reference" "SIMM1E" (id 0) (at 96.52 43.18 0))
+    (property "Reference" "SM1" (id 0) (at 96.52 43.18 0))
     (property "Value" "Conn_01x36_Male" (id 1) (at 93.98 86.36 90))
     (property "Footprint" "" (id 2) (at 96.52 88.9 0)
@@
   (symbol (lib_id "Connector:Conn_01x36_Male") (at 158.75 184.15 0) (mirror y) (unit 1)
     (in_bom yes) (on_board yes)
-    (property "Reference" "SIMM2D" (id 0) (at 158.75 138.43 0))
+    (property "Reference" "SMM2" (id 0) (at 158.75 138.43 0))
     (property "Value" "Conn_01x36_Male" (id 1) (at 143.51 232.41 0))
     (property "Footprint" "" (id 2) (at 158.75 184.15 0)
@@
   (symbol (lib_id "Connector:Conn_01x36_Male") (at 228.6 88.9 0) (unit 1)
     (in_bom yes) (on_board yes)
-    (property "Reference" "SIMM4D" (id 0) (at 228.6 43.18 0))
+    (property "Reference" "SM4" (id 0) (at 228.6 43.18 0))
     (property "Value" "Conn_01x36_Male" (id 1) (at 227.33 86.36 90))
     (property "Footprint" "" (id 2) (at 228.6 88.9 0)
@@
   (symbol (lib_id "Connector:Conn_01x36_Male") (at 304.8 88.9 0) (unit 1)
     (in_bom yes) (on_board yes)
-    (property "Reference" "SIMM6B" (id 0) (at 314.96 43.18 0))
+    (property "Reference" "SM6" (id 0) (at 314.96 43.18 0))
     (property "Value" "Conn_01x36_Male" (id 1) (at 303.53 86.36 90))
     (property "Footprint" "" (id 2) (at 304.8 88.9 0)
@@
   (symbol (lib_id "Connector:Conn_01x36_Male") (at 227.33 185.42 0) (unit 1)
     (in_bom yes) (on_board yes)
-    (property "Reference" "SIMM4DD" (id 0) (at 227.33 139.7 0))
+    (property "Reference" "SMM4" (id 0) (at 227.33 139.7 0))
     (property "Value" "Conn_01x36_Male" (id 1) (at 227.965 233.68 0))
     (property "Footprint" "" (id 2) (at 227.33 185.42 0)
