File: cores/cps3/sch/slots_females.kicad_sch (KiCad schematic)
At the start: 12 parts

Commit message: wip_ccu_gll2_cassette
Connections:
- net VBAT_S1-2: now reaches JSIMM3EE.36 (Pin_36)
- net VBAT_S1-2: now also JSIMM4DD.36 (Pin_36), JSIMM5CC.36 (Pin_36), JSIMM6BB.36 (Pin_36)
- net VBAT_S6~3: now reaches JSIMM1EE.36 (Pin_36)
- net VBAT_S6~3: now also JSIMM2DD.36 (Pin_36)
- no-connect marks 82 -> 76

Commit message: wip_ccu_cassette
Connections:
- net VBAT_S1-2: now also JSIMM1EE.36 (Pin_36), JSIMM2DD.36 (Pin_36); no longer JSIMM3EE.36 (Pin_36), JSIMM4DD.36 (Pin_36), JSIMM5CC.36 (Pin_36), JSIMM6BB.36 (Pin_36)
- net VBAT_S6~3: now also JSIMM3EE.36 (Pin_36), JSIMM4DD.36 (Pin_36), JSIMM5CC.36 (Pin_36), JSIMM6BB.36 (Pin_36); no longer JSIMM1EE.36 (Pin_36), JSIMM2DD.36 (Pin_36)

Commit message: wip_cassette
Connections:
- net GFX_A21: now reaches JSIMM1EE.2 (Pin_2)
- net UK renamed UK_CCU
- net ~{CE} renamed ~{CE_}S1
- net ~{CE_}S1: no longer JSIMM2DD.31 (Pin_31)
- net ~{OE} renamed ~{OE}_CCU
- net ~{WE} renamed ~{WE}_CCU
- new net ~{CE}_S2: JSIMM2DD.31 (Pin_31)
- no-connect marks 76 -> 75
Other:
- note added: "GFX_A21"

Commit message: wip_cre_cps3
Connections:
- net OAMB_A0 renamed 2SPRITE_AB0
- net OAMB_A1 renamed 2SPRITE_AB1
- net OAMB_A10 renamed 2SPRITE_AB10
- net OAMB_A11 renamed 2SPRITE_AB11
- net OAMB_A12 renamed 2SPRITE_AB12
- net OAMB_A13 renamed 2SPRITE_AB13
- net OAMB_A14 renamed 2SPRITE_AB14
- net OAMB_A15 renamed 2SPRITE_AB15
- net OAMB_A16 renamed 2SPRITE_AB16
- net OAMB_A17 renamed 2SPRITE_AB17
- net OAMB_A18 renamed 2SPRITE_AB18
- net OAMB_A19 renamed 2SPRITE_AB19
- net OAMB_A2 renamed 2SPRITE_AB2
- net OAMB_A20 renamed 2SPRITE_AB20
- net OAMB_A3 renamed 2SPRITE_AB3
- net OAMB_A4 renamed 2SPRITE_AB4
- net OAMB_A5 renamed 2SPRITE_AB5
- net OAMB_A6 renamed 2SPRITE_AB6
- net OAMB_A7 renamed 2SPRITE_AB7
- net OAMB_A8 renamed 2SPRITE_AB8
- net OAMB_A9 renamed 2SPRITE_AB9
- net OAM_A0 renamed SPRITE_AB0
- net OAM_A1 renamed SPRITE_AB1
- net OAM_A10 renamed SPRITE_AB10
- net OAM_A11 renamed SPRITE_AB11
- net OAM_A12 renamed SPRITE_AB12
- net OAM_A13 renamed SPRITE_AB13
- net OAM_A14 renamed SPRITE_AB14
- net OAM_A15 renamed SPRITE_AB15
- net OAM_A16 renamed SPRITE_AB16
- net OAM_A17 renamed SPRITE_AB17
- net OAM_A18 renamed SPRITE_AB18
- net OAM_A19 renamed SPRITE_AB19
- net OAM_A2 renamed SPRITE_AB2
- net OAM_A20 renamed SPRITE_AB20
- net OAM_A3 renamed SPRITE_AB3
- net OAM_A4 renamed SPRITE_AB4
- net OAM_A5 renamed SPRITE_AB5
- net OAM_A6 renamed SPRITE_AB6
- net OAM_A7 renamed SPRITE_AB7
- net OAM_A8 renamed SPRITE_AB8
- net OAM_A9 renamed SPRITE_AB9
- no-connect marks 75 -> 79
