File: cores/cps3/sch/slots_females.kicad_sch (KiCad schematic)
At the start: 12 parts

Commit message: cps3_finished
Parts:
- renumbered JSIMM1E to S1, JSIMM2D to S2, JSIMM3E to S3, JSIMM4D to S4, JSIMM5C to S5, JSIMM6B to S6, JSIMM1EE to SS1, JSIMM2DD to SS2, JSIMM3EE to SS3, JSIMM4DD to SS4, JSIMM5CC to SS5, JSIMM6BB to SS6
Connections:
- no-connect marks 79 -> 80
