File: cores/cps3/sch/memories_scu.kicad_sch (KiCad schematic)
At the start: 6 parts, among them U1 7400, U2 29F400TA-90PF, U5 28F400-200BX/BL, U6 FM1208S-250SC

Commit message: correction_ppu
Connections:
- net SCU_A0 renamed CPUC_A0
- net SCU_A1 renamed CPUC_A1
- net SCU_A10 renamed CPUC_A10
- net SCU_A11 renamed CPUC_A11
- net SCU_A12 renamed CPUC_A12
- net SCU_A13 renamed CPUC_A13
- net SCU_A14 renamed CPUC_A14
- net SCU_A15 renamed CPUC_A15
- net SCU_A16 renamed CPUC_A16
- net SCU_A17 renamed CPUC_A17
- net SCU_A18 renamed CPUC_A18
- net SCU_A2 renamed CPUC_A2
- net SCU_A24 renamed CPUC_A24
- net SCU_A3 renamed CPUC_A3
- net SCU_A4 renamed CPUC_A4
- net SCU_A6 renamed CPUC_A6
- net SCU_A7 renamed CPUC_A7
- net SCU_A8 renamed CPUC_A8
- net SCU_A9 renamed CPUC_A9
- net SCU_D0 renamed CPUC_D0
- net SCU_D1 renamed CPUC_D1
- net SCU_D10 renamed CPUC_D10
- net SCU_D11 renamed CPUC_D11
- net SCU_D12 renamed CPUC_D12
- net SCU_D13 renamed CPUC_D13
- net SCU_D14 renamed CPUC_D14
- net SCU_D2 renamed CPUC_D2
- net SCU_D3 renamed CPUC_D3
- net SCU_D4 renamed CPUC_D4
- net SCU_D5 renamed CPUC_D5
- net SCU_D6 renamed CPUC_D6
- net SCU_D7 renamed CPUC_D7
- net SCU_D8 renamed CPUC_D8
- net SCU_D9 renamed CPUC_D9
- net WAIT renamed WAIT_CPUC
- net ~{CE}_FRAM renamed ~{STBY_WD}
- net ~{CS1} renamed CPUC_~{CS1}
- net ~{WAIT} renamed ~{WAIT_CPUC}
- net ~{WE0}_CST renamed CPUC_~{WE0}

Commit message: cps3_finished
Parts:
- renumbered CP180 to CCP180, U1 to T1, U2 to Z2, U5 to Z5, U6 to Z6
Connections:
- net CPUC_A0: no longer Z5.31 (D15/A-1)
- net CPUC_D0: no longer Z5.15 (D0)
- net CPUC_D1: no longer Z5.17 (D1)
- net CPUC_D10: no longer Z5.20 (D10)
- net CPUC_D11: no longer Z5.22 (D11)
- net CPUC_D12: no longer Z5.25 (D12)
- net CPUC_D13: no longer Z5.27 (D13)
- net CPUC_D14: no longer Z5.29 (D14)
- net CPUC_D2: no longer Z5.19 (D2)
- net CPUC_D3: no longer Z5.21 (D3)
- net CPUC_D4: no longer Z5.24 (D4)
- net CPUC_D5: no longer Z5.26 (D5)
- net CPUC_D6: no longer Z5.28 (D6)
- net CPUC_D7: no longer Z5.30 (D7)
- net CPUC_D8: no longer Z5.16 (D8)
- net CPUC_D9: no longer Z5.18 (D9)
- net VCC: now also CP179.1, T1.1, Z2.37 (VCC)
- net Vpp: no longer names the net of Z5.1 (Vpp)
- net ~{STBY_WD} renamed ~{CE}_FRAM
- no-connect marks 2 -> 20
Other:
- note added: "CPUC_A0"
- note added: "CPUC_A5"
- note added: "CPUC_D0"
- note added: "CPUC_D1"
- note added: "CPUC_D10"
- note added: "CPUC_D11"
- note added: "CPUC_D12"
- note added: "CPUC_D13"
- note added: "CPUC_D14"
- note added: "CPUC_D2"
- note added: "CPUC_D3"
- note added: "CPUC_D4"
- note added: "CPUC_D5"
- note added: "CPUC_D6"
- note added: "CPUC_D7"
- note added: "CPUC_D8"
- note added: "CPUC_D9"
- note added: "Vpp"
