File: cores/cps3/sch/memories_scu.kicad_sch (KiCad schematic)
At the start: 6 parts, among them T1 7400

Commit message: wip_sh2_cps3
Parts:
- CCP180: value 10μF -> 1µF
Changed lines of the file:
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@@
       (effects (font (size 1.27 1.27)) (justify left))
     )
-    (property "Value" "10μF" (id 1) (at 204.47 214.63 0)
+    (property "Value" "1µF" (id 1) (at 204.47 214.63 0)
       (effects (font (size 1.27 1.27)) (justify left))
     )
