File: cores/cps3/colmix.kicad_sch (KiCad schematic)
At the start: 0 parts

Commit message: moved sch folder
Other:
- company: (none) -> JOTEGO
- title: (none) -> CP SYSTEM III
Changed lines of the file:
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@@
 (kicad_sch (version 20211123) (generator eeschema)
-  (paper "A2")
+  (paper "A3")
   (title_block
+    (title "CP SYSTEM III")
     (date "14/10/22")
+    (rev "José Tejada G.")
+    (company "JOTEGO")
+    (comment 1 "E.Triana")
   )
-  (image (at 572.77 383.54) (scale 0.294008)
+  (image (at 398.78 261.62) (scale 0.294008)
     (data
       iVBORw0KGgoAAAANSUhEUgAAAtEAAAGsCAMAAAAsQwu3AAAAA3NCSVQICAjb4U/gAAADAFBMVEX/
