File: cores/cps3/memories_gfx.kicad_sch (KiCad schematic)
At the start: 8 parts

Commit message: moved sch folder
Other:
- company: (none) -> JOTEGO
- title: (none) -> CP SYSTEM III
Changed lines of the file:
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@@
   (paper "A3")
   (title_block
+    (title "CP SYSTEM III")
     (date "14/10/22")
+    (rev "José Tejada G.")
+    (company "JOTEGO")
+    (comment 1 "E.Triana")
   )
   (junction (at 217.17 214.63) (diameter 0) (color 0 0 0 0)
